Commit message: robot parameter parsing update

File: interactive_marker_test/urdf/prr_simple.xacro (robot description, xacro)
@@ -34,5 +34,5 @@
   <sensor name="my_test_sensor" update_rate="20">
     <parent link="right_leg"/>
-    <origin xyz="0 0 0" rpy="0 0 0"/>
+    <origin xyz="5 0 0" rpy="0 0 0"/>
     <camera>
       <image width="640" height="480" hfov="1.5708" format="RGB8" near="0.01" far="50.0"/>
