Commit message: update1

File: interactive_marker_test/urdf/prr.xacro (robot description, xacro)
@@ -142,79 +142,94 @@
     </visual>
   </link>
-  <!--<joint name="left_gripper_joint" type="fixed">-->
-    <!--<origin rpy="0 0 0" xyz="0.2 0.01 0"/>-->
-    <!--<parent link="gripper_pole"/>-->
-    <!--<child link="left_gripper"/>-->
-  <!--</joint>-->
-  <!--<link name="left_gripper">-->
-    <!--<visual>-->
-      <!--<origin rpy="0.0 0 0" xyz="0 0 0"/>-->
-      <!--<geometry>-->
-        <!--<mesh filename="package://interactive_marker_test/meshes/l_finger.dae"/>-->
-      <!--</geometry>-->
-    <!--</visual>-->
-  <!--</link>-->
-  <!--<joint name="left_tip_joint" type="fixed">-->
-    <!--<parent link="left_gripper"/>-->
-    <!--<child link="left_tip"/>-->
-  <!--</joint>-->
-  <!--<link name="left_tip">-->
-    <!--<visual>-->
-      <!--<origin rpy="0.0 0 0" xyz="0.09137 0.00495 0"/>-->
-      <!--<geometry>-->
-        <!--<mesh filename="package://interactive_marker_test/meshes/l_finger_tip.dae"/>-->
-      <!--</geometry>-->
-    <!--</visual>-->
-  <!--</link>-->
-  <!--<joint name="right_gripper_joint" type="fixed">-->
-    <!--<origin rpy="0 0 0" xyz="0.2 -0.01 0"/>-->
-    <!--<parent link="gripper_pole"/>-->
-    <!--<child link="right_gripper"/>-->
-  <!--</joint>-->
-  <!--<link name="right_gripper">-->
-    <!--<visual>-->
-      <!--<origin rpy="-3.1415 0 0" xyz="0 0 0"/>-->
-      <!--<geometry>-->
-        <!--<mesh filename="package://interactive_marker_test/meshes/l_finger.dae"/>-->
-      <!--</geometry>-->
-    <!--</visual>-->
-  <!--</link>-->
-  <!--<joint name="right_tip_joint" type="fixed">-->
-    <!--<parent link="right_gripper"/>-->
-    <!--<child link="right_tip"/>-->
-  <!--</joint>-->
-  <!--<link name="right_tip">-->
-    <!--<visual>-->
-      <!--<origin rpy="-3.1415 0 0" xyz="0.09137 0.00495 0"/>-->
-      <!--<geometry>-->
-        <!--<mesh filename="package://interactive_marker_test/meshes/l_finger_tip.dae"/>-->
-      <!--</geometry>-->
-    <!--</visual>-->
-  <!--</link>-->
-  <!--<link name="head">-->
-    <!--<visual>-->
-      <!--<geometry>-->
-        <!--<sphere radius="0.2"/>-->
-      <!--</geometry>-->
-      <!--<material name="white"/>-->
-    <!--</visual>-->
-  <!--</link>-->
-  <!--<joint name="head_swivel" type="fixed">-->
-    <!--<parent link="base_link"/>-->
-    <!--<child link="head"/>-->
-    <!--<origin xyz="0 0 0.3"/>-->
-  <!--</joint>-->
-  <!--<link name="box">-->
-    <!--<visual>-->
-      <!--<geometry>-->
-        <!--<box size="0.08 0.08 0.08"/>-->
-      <!--</geometry>-->
-      <!--<material name="blue"/>-->
-    <!--</visual>-->
-  <!--</link>-->
-  <!--<joint name="tobox" type="fixed">-->
-    <!--<parent link="head"/>-->
-    <!--<child link="box"/>-->
-    <!--<origin xyz="0.1814 0 0.1414"/>-->
-  <!--</joint>-->
+  <link name="head">
+    <visual>
+      <geometry>
+        <sphere radius="0.2"/>
+      </geometry>
+      <material name="white"/>
+    </visual>
+  </link>
+  <joint name="head_swivel" type="fixed">
+    <parent link="base_link"/>
+    <child link="head"/>
+    <origin xyz="0 0 0.3"/>
+  </joint>
+  <link name="box">
+    <visual>
+      <geometry>
+        <box size="0.08 0.08 0.08"/>
+      </geometry>
+      <material name="blue"/>
+    </visual>
+  </link>
+  <joint name="tobox" type="fixed">
+    <parent link="head"/>
+    <child link="box"/>
+    <origin xyz="0.1814 0 0.1414"/>
+  </joint>
+  <link name="marker1">
+    <visual>
+      <geometry>
+        <cylinder length="0.1" radius="0.05"/>
+      </geometry>
+      <origin rpy="0.7853981634 0 0 " xyz="0.15 0 0"/>
+    </visual>
+  </link>
+  <joint name="right_marker" type="fixed">
+    <parent link="base_link"/>
+    <child link="marker1"/>
+    <origin rpy="0 0 0" xyz="0 -0.22 0.2"/>
+  </joint>
+  <link name="marker2">
+    <visual>
+      <geometry>
+        <cylinder length="0.1" radius="0.05"/>
+      </geometry>
+      <origin rpy="-0.7853981634 0 0 " xyz="0.15 0 0"/>
+    </visual>
+  </link>
+  <joint name="left_marker" type="fixed">
+    <parent link="base_link"/>
+    <child link="marker2"/>
+    <origin rpy="0 0 0" xyz="0 0.22 0.2"/>
+  </joint>
+  <link name="marker3">
+    <visual>
+      <geometry>
+        <cylinder length="0.1" radius="0.05"/>
+      </geometry>
+      <origin rpy="0 0 0 " xyz="0 0 0"/>
+    </visual>
+  </link>
+  <joint name="central_marker" type="fixed">
+    <parent link="base_link"/>
+    <child link="marker3"/>
+    <origin rpy="0 0 0" xyz="0.4 0 0.2"/>
+  </joint>
+    <link name="marker4">
+    <visual>
+      <geometry>
+        <cylinder length="0.1" radius="0.05"/>
+      </geometry>
+      <origin rpy="1.5707963268 0 0 " xyz="0 0 0"/>
+    </visual>
+  </link>
+  <joint name="left_side_marker" type="fixed">
+    <parent link="base_link"/>
+    <child link="marker4"/>
+    <origin rpy="0 0 0" xyz="0 0.32 -0.25"/>
+  </joint>
+      <link name="marker5">
+    <visual>
+      <geometry>
+        <cylinder length="0.1" radius="0.05"/>
+      </geometry>
+      <origin rpy="1.5707963268 0 0 " xyz="0 0 0"/>
+    </visual>
+  </link>
+  <joint name="right_side_marker" type="fixed">
+    <parent link="base_link"/>
+    <child link="marker5"/>
+    <origin rpy="0 0 0" xyz="0 -0.32 -0.25"/>
+  </joint>
 </robot>

Commit message: #4 urdf_domparser.py seems to work but not for sensors

File: interactive_marker_test/urdf/prr.xacro (robot description, xacro)
@@ -233,3 +233,10 @@
     <origin rpy="0 0 0" xyz="0 -0.32 -0.25"/>
   </joint>
+  <sensor name="my_test_sensor" update_rate="20">
+    <parent link="marker5"/>
+    <origin xyz="0 0 0" rpy="0 0 0"/>
+    <camera>
+      <image width="640" height="480" hfov="1.5708" format="RGB8" near="0.01" far="50.0"/>
+    </camera>
+  </sensor>
 </robot>

Commit message: update to sensors

File: interactive_marker_test/urdf/prr.xacro (robot description, xacro)
@@ -168,72 +168,35 @@
     <origin xyz="0.1814 0 0.1414"/>
   </joint>
-  <link name="marker1">
-    <visual>
-      <geometry>
-        <cylinder length="0.1" radius="0.05"/>
-      </geometry>
-      <origin rpy="0.7853981634 0 0 " xyz="0.15 0 0"/>
-    </visual>
-  </link>
-  <joint name="right_marker" type="fixed">
-    <parent link="base_link"/>
-    <child link="marker1"/>
-    <origin rpy="0 0 0" xyz="0 -0.22 0.2"/>
-  </joint>
-  <link name="marker2">
-    <visual>
-      <geometry>
-        <cylinder length="0.1" radius="0.05"/>
-      </geometry>
-      <origin rpy="-0.7853981634 0 0 " xyz="0.15 0 0"/>
-    </visual>
-  </link>
-  <joint name="left_marker" type="fixed">
-    <parent link="base_link"/>
-    <child link="marker2"/>
-    <origin rpy="0 0 0" xyz="0 0.22 0.2"/>
-  </joint>
-  <link name="marker3">
-    <visual>
-      <geometry>
-        <cylinder length="0.1" radius="0.05"/>
-      </geometry>
-      <origin rpy="0 0 0 " xyz="0 0 0"/>
-    </visual>
-  </link>
-  <joint name="central_marker" type="fixed">
-    <parent link="base_link"/>
-    <child link="marker3"/>
-    <origin rpy="0 0 0" xyz="0.4 0 0.2"/>
-  </joint>
-    <link name="marker4">
-    <visual>
-      <geometry>
-        <cylinder length="0.1" radius="0.05"/>
-      </geometry>
-      <origin rpy="1.5707963268 0 0 " xyz="0 0 0"/>
-    </visual>
-  </link>
-  <joint name="left_side_marker" type="fixed">
-    <parent link="base_link"/>
-    <child link="marker4"/>
-    <origin rpy="0 0 0" xyz="0 0.32 -0.25"/>
-  </joint>
-      <link name="marker5">
-    <visual>
-      <geometry>
-        <cylinder length="0.1" radius="0.05"/>
-      </geometry>
-      <origin rpy="1.5707963268 0 0 " xyz="0 0 0"/>
-    </visual>
-  </link>
-  <joint name="right_side_marker" type="fixed">
-    <parent link="base_link"/>
-    <child link="marker5"/>
-    <origin rpy="0 0 0" xyz="0 -0.32 -0.25"/>
-  </joint>
-  <sensor name="my_test_sensor" update_rate="20">
-    <parent link="marker5"/>
-    <origin xyz="0 0 0" rpy="0 0 0"/>
+  <sensor name="sensor1" update_rate="20">
+    <parent link="base_link"/>
+    <origin xyz="0.15 -0.22 0.2" rpy="0.7853981634 0 0"/>
+    <camera>
+      <image width="640" height="480" hfov="1.5708" format="RGB8" near="0.01" far="50.0"/>
+    </camera>
+  </sensor>
+  <sensor name="sensor2" update_rate="20">
+    <parent link="base_link"/>
+    <origin xyz="0.15 0.22 0.2" rpy="-0.7853981634 0 0"/>
+    <camera>
+      <image width="640" height="480" hfov="1.5708" format="RGB8" near="0.01" far="50.0"/>
+    </camera>
+  </sensor>
+  <sensor name="sensor3" update_rate="20">
+    <parent link="base_link"/>
+    <origin xyz="0 0 0.55" rpy="0 0 0"/>
+    <camera>
+      <image width="640" height="480" hfov="1.5708" format="RGB8" near="0.01" far="50.0"/>
+    </camera>
+  </sensor>
+  <sensor name="sensor4" update_rate="20">
+    <parent link="base_link"/>
+    <origin xyz="0 0.32 -0.25" rpy="1.5707963268 0 0"/>
+    <camera>
+      <image width="640" height="480" hfov="1.5708" format="RGB8" near="0.01" far="50.0"/>
+    </camera>
+  </sensor>
+  <sensor name="sensor5" update_rate="20">
+    <parent link="base_link"/>
+    <origin xyz="0 -0.32 -0.25" rpy="1.5707963268 0 0"/>
     <camera>
       <image width="640" height="480" hfov="1.5708" format="RGB8" near="0.01" far="50.0"/>

Commit message: publishing and listening sensors and marker positions

File: interactive_marker_test/urdf/prr.xacro (robot description, xacro)
@@ -10,4 +10,7 @@
     <color rgba="1 1 1 1"/>
   </material>
+  <material name="Kinect2Grey">
+      <color rgba="0.15 0.15 0.15 1.0"/>
+  </material>
   <link name="base_link">
     <visual>
@@ -170,36 +173,111 @@
   <sensor name="sensor1" update_rate="20">
     <parent link="base_link"/>
-    <origin xyz="0.15 -0.22 0.2" rpy="0.7853981634 0 0"/>
-    <camera>
-      <image width="640" height="480" hfov="1.5708" format="RGB8" near="0.01" far="50.0"/>
-    </camera>
-  </sensor>
+    <origin xyz="0 0 0" rpy="0 0 0"/>
+    <camera>
+      <image width="640" height="480" hfov="1.5708" format="RGB8" near="0.01" far="50.0"/>
+    </camera>
+  </sensor>
+  <link name="sensor1">
+      <visual>
+        <origin rpy="0 0 0" xyz="0 0 0"/>
+        <geometry>
+          <!-- these meshes were exported in mm, so scale back to m -->
+          <mesh filename="package://interactive_marker_test/meshes/kinect2_origin_on_rgb_optical_frame.stl" scale="0.001 0.001 0.001"/>
+        </geometry>
+        <material name="Kinect2Grey"/>
+      </visual>
+  </link>
+  <joint name="base_to_sensor1" type="fixed">
+    <parent link="base_link"/>
+    <child link="sensor1"/>
+    <origin rpy="0.7853981634 0 0" xyz="0.15 -0.22 0.2"/>
+  </joint>
   <sensor name="sensor2" update_rate="20">
     <parent link="base_link"/>
-    <origin xyz="0.15 0.22 0.2" rpy="-0.7853981634 0 0"/>
-    <camera>
-      <image width="640" height="480" hfov="1.5708" format="RGB8" near="0.01" far="50.0"/>
-    </camera>
-  </sensor>
+    <origin xyz="0 0 0" rpy="0 0 0"/>
+    <camera>
+      <image width="640" height="480" hfov="1.5708" format="RGB8" near="0.01" far="50.0"/>
+    </camera>
+  </sensor>
+  <link name="sensor2">
+      <visual>
+        <origin rpy="0 0 0" xyz="0 0 0"/>
+        <geometry>
+          <!-- these meshes were exported in mm, so scale back to m -->
+          <mesh filename="package://interactive_marker_test/meshes/kinect2_origin_on_rgb_optical_frame.stl" scale="0.001 0.001 0.001"/>
+        </geometry>
+        <material name="Kinect2Grey"/>
+      </visual>
+  </link>
+  <joint name="base_to_sensor2" type="fixed">
+    <parent link="base_link"/>
+    <child link="sensor2"/>
+    <origin rpy="-0.7853981634 0 0" xyz="0.15 0.22 0.2"/>
+  </joint>
   <sensor name="sensor3" update_rate="20">
     <parent link="base_link"/>
-    <origin xyz="0 0 0.55" rpy="0 0 0"/>
-    <camera>
-      <image width="640" height="480" hfov="1.5708" format="RGB8" near="0.01" far="50.0"/>
-    </camera>
-  </sensor>
+    <origin xyz="0 0 0" rpy="0 0 0"/>
+    <camera>
+      <image width="640" height="480" hfov="1.5708" format="RGB8" near="0.01" far="50.0"/>
+    </camera>
+  </sensor>
+  <link name="sensor3">
+      <visual>
+        <origin rpy="0 0 0" xyz="0 0 0"/>
+        <geometry>
+          <!-- these meshes were exported in mm, so scale back to m -->
+          <mesh filename="package://interactive_marker_test/meshes/kinect2_origin_on_rgb_optical_frame.stl" scale="0.001 0.001 0.001"/>
+        </geometry>
+        <material name="Kinect2Grey"/>
+      </visual>
+  </link>
+  <joint name="base_to_sensor3" type="fixed">
+    <parent link="base_link"/>
+    <child link="sensor3"/>
+    <origin rpy="0 0 0" xyz="0 0 0.55"/>
+  </joint>
   <sensor name="sensor4" update_rate="20">
     <parent link="base_link"/>
-    <origin xyz="0 0.32 -0.25" rpy="1.5707963268 0 0"/>
-    <camera>
-      <image width="640" height="480" hfov="1.5708" format="RGB8" near="0.01" far="50.0"/>
-    </camera>
-  </sensor>
+    <origin xyz="0 0 0" rpy="0 0 0"/>
+    <camera>
+      <image width="640" height="480" hfov="1.5708" format="RGB8" near="0.01" far="50.0"/>
+    </camera>
+  </sensor>
+  <link name="sensor4">
+      <visual>
+        <origin rpy="0 0 0" xyz="0 0 0"/>
+        <geometry>
+          <!-- these meshes were exported in mm, so scale back to m -->
+          <mesh filename="package://interactive_marker_test/meshes/kinect2_origin_on_rgb_optical_frame.stl" scale="0.001 0.001 0.001"/>
+        </geometry>
+        <material name="Kinect2Grey"/>
+      </visual>
+  </link>
+  <joint name="base_to_sensor4" type="fixed">
+    <parent link="base_link"/>
+    <child link="sensor4"/>
+    <origin rpy="1.5707963268 0 0" xyz="0 0.32 -0.25"/>
+  </joint>
   <sensor name="sensor5" update_rate="20">
     <parent link="base_link"/>
-    <origin xyz="0 -0.32 -0.25" rpy="1.5707963268 0 0"/>
-    <camera>
-      <image width="640" height="480" hfov="1.5708" format="RGB8" near="0.01" far="50.0"/>
-    </camera>
-  </sensor>
+    <origin xyz="0 0 0" rpy="0 0 0"/>
+    <camera>
+      <image width="640" height="480" hfov="1.5708" format="RGB8" near="0.01" far="50.0"/>
+    </camera>
+  </sensor>
+  <link name="sensor5">
+      <visual>
+        <origin rpy="0 0 0" xyz="0 0 0"/>
+        <geometry>
+          <!-- these meshes were exported in mm, so scale back to m -->
+          <mesh filename="package://interactive_marker_test/meshes/kinect2_origin_on_rgb_optical_frame.stl" scale="0.001 0.001 0.001"/>
+        </geometry>
+        <material name="Kinect2Grey"/>
+      </visual>
+  </link>
+  <joint name="base_to_sensor5" type="fixed">
+    <parent link="base_link"/>
+    <child link="sensor5"/>
+    <origin rpy="1.5707963268 0 0" xyz="0 -0.32 -0.25"/>
+  </joint>
 </robot>

File: interactive_marker_test/urdf/prr_simple.xacro (robot description, xacro)
@@ -1,5 +1,5 @@
 <?xml version="1.0"?>
 <robot name="visual">
-<material name="blue">
+  <material name="blue">
     <color rgba="0 0 0.8 1"/>
   </material>
@@ -9,4 +9,7 @@
   <material name="white">
     <color rgba="1 1 1 1"/>
+  </material>
+  <material name="Kinect2Grey">
+      <color rgba="0.15 0.15 0.15 1.0"/>
   </material>
   <link name="base_link">
@@ -30,9 +33,46 @@
     <parent link="base_link"/>
     <child link="right_leg"/>
-    <origin xyz="0 -0.22 0.25"/>
+    <origin xyz="-5 -0.22 0.25"/>
   </joint>
+  <joint name="base_to_sensor" type="fixed">
+    <parent link="base_link"/>
+    <child link="my_test_sensor"/>
+    <origin rpy="0 1.57075 0" xyz="1 0 0"/>
+  </joint>
+  <link name="my_test_sensor">
+      <visual>
+        <origin rpy="0 0 0" xyz="0 0 0"/>
+        <geometry>
+          <!-- these meshes were exported in mm, so scale back to m -->
+          <mesh filename="package://interactive_marker_test/meshes/kinect2_origin_on_rgb_optical_frame.stl" scale="0.001 0.001 0.001"/>
+        </geometry>
+        <material name="Kinect2Grey"/>
+      </visual>
+    </link>
   <sensor name="my_test_sensor" update_rate="20">
-    <parent link="right_leg"/>
-    <origin xyz="5 0 0" rpy="0 0 0"/>
+    <parent link="my_test_sensor"/>
+    <origin xyz="0 0 0" rpy="0 0 0"/>
+    <camera>
+      <image width="640" height="480" hfov="1.5708" format="RGB8" near="0.01" far="50.0"/>
+    </camera>
+  </sensor>
+  <joint name="base_to_sensor2" type="fixed">
+    <parent link="base_link"/>
+    <child link="my_test_sensor2"/>
+    <origin rpy="0 1.57075 0" xyz="1 4 0"/>
+  </joint>
+  <link name="my_test_sensor2">
+      <visual>
+        <origin rpy="0 0 0" xyz="0 0 0"/>
+        <geometry>
+          <!-- these meshes were exported in mm, so scale back to m -->
+          <mesh filename="package://interactive_marker_test/meshes/kinect2_origin_on_rgb_optical_frame.stl" scale="0.001 0.001 0.001"/>
+        </geometry>
+        <material name="Kinect2Grey"/>
+      </visual>
+    </link>
+  <sensor name="my_test_sensor2" update_rate="20">
+    <parent link="my_test_sensor2"/>
+    <origin xyz="0 0 0" rpy="0 0 0"/>
     <camera>
       <image width="640" height="480" hfov="1.5708" format="RGB8" near="0.01" far="50.0"/>
