Commit message: now for atlascar xacro

File: interactive_marker_test/urdf/atlas_macro.urdf.xacro (robot description, xacro)
@@ -20,4 +20,8 @@
         </joint>
         <xacro:sick_lms1xx frame="${prefix}frontal_laser_left" />
+         <sensor name="${prefix}frontal_laser_left" update_rate="20">
+             <parent link="${prefix}frontal_laser_left"/>
+             <origin xyz="0 0 0" rpy="0 0 0"/>
+         </sensor>
         <joint name="${prefix}base_link_to_${prefix}frontal_laser_left" type="fixed">
             <origin xyz="0.6 0 0" rpy="0 0 ${-pi/3}" />

File: interactive_marker_test/urdf/prr.xacro (robot description, xacro)
@@ -171,6 +171,7 @@
     <origin xyz="0.1814 0 0.1414"/>
   </joint>
-  <sensor name="sensor1" update_rate="20">
-    <parent link="base_link"/>
+  <sensor name="sensor1_aaa" update_rate="20">
+    <!--<parent link="base_link"/>-->
+    <parent link="sensor1"/>
     <origin xyz="0 0 0" rpy="0 0 0"/>
     <camera>

File: interactive_marker_test/urdf/prr_simple.xacro (robot description, xacro)
@@ -35,10 +35,10 @@
     <origin xyz="-5 -0.22 0.25"/>
   </joint>
-  <joint name="base_to_sensor" type="fixed">
+  <joint name="base_to_sensor_joint" type="fixed">
     <parent link="base_link"/>
-    <child link="my_test_sensor"/>
+    <child link="my_test_sensor_link"/>
     <origin rpy="0 1.57075 0" xyz="1 0 0"/>
   </joint>
-  <link name="my_test_sensor">
+  <link name="my_test_sensor_link">
       <visual>
         <origin rpy="0 0 0" xyz="0 0 0"/>
@@ -50,6 +50,6 @@
       </visual>
     </link>
-  <sensor name="my_test_sensor" update_rate="20">
-    <parent link="my_test_sensor"/>
+  <sensor name="my_test_sensor_sensor" update_rate="20">
+    <parent link="my_test_sensor_link"/>
     <origin xyz="0 0 0" rpy="0 0 0"/>
     <camera>
@@ -57,25 +57,25 @@
     </camera>
   </sensor>
-  <joint name="base_to_sensor2" type="fixed">
-    <parent link="base_link"/>
-    <child link="my_test_sensor2"/>
-    <origin rpy="0 1.57075 0" xyz="1 4 0"/>
-  </joint>
-  <link name="my_test_sensor2">
-      <visual>
-        <origin rpy="0 0 0" xyz="0 0 0"/>
-        <geometry>
-          <!-- these meshes were exported in mm, so scale back to m -->
-          <mesh filename="package://interactive_marker_test/meshes/kinect2_origin_on_rgb_optical_frame.stl" scale="0.001 0.001 0.001"/>
-        </geometry>
-        <material name="Kinect2Grey"/>
-      </visual>
-    </link>
-  <sensor name="my_test_sensor2" update_rate="20">
-    <parent link="my_test_sensor2"/>
-    <origin xyz="0 0 0" rpy="0 0 0"/>
-    <camera>
-      <image width="640" height="480" hfov="1.5708" format="RGB8" near="0.01" far="50.0"/>
-    </camera>
-  </sensor>
+  <!--<joint name="base_to_sensor2" type="fixed">-->
+    <!--<parent link="base_link"/>-->
+    <!--<child link="my_test_sensor2"/>-->
+    <!--<origin rpy="0 1.57075 0" xyz="1 4 0"/>-->
+  <!--</joint>-->
+  <!--<link name="my_test_sensor2">-->
+      <!--<visual>-->
+        <!--<origin rpy="0 0 0" xyz="0 0 0"/>-->
+        <!--<geometry>-->
+          <!--&lt;!&ndash; these meshes were exported in mm, so scale back to m &ndash;&gt;-->
+          <!--<mesh filename="package://interactive_marker_test/meshes/kinect2_origin_on_rgb_optical_frame.stl" scale="0.001 0.001 0.001"/>-->
+        <!--</geometry>-->
+        <!--<material name="Kinect2Grey"/>-->
+      <!--</visual>-->
+    <!--</link>-->
+  <!--<sensor name="my_test_sensor2" update_rate="20">-->
+    <!--<parent link="my_test_sensor2"/>-->
+    <!--<origin xyz="0 0 0" rpy="0 0 0"/>-->
+    <!--<camera>-->
+      <!--<image width="640" height="480" hfov="1.5708" format="RGB8" near="0.01" far="50.0"/>-->
+    <!--</camera>-->
+  <!--</sensor>-->
 </robot>
