Commit message: sensors elements added

File: interactive_marker_test/urdf/atlas2_model_macro.urdf.xacro (robot description, xacro)
@@ -1,9 +1,8 @@
 <?xml version="1.0"?>
-<robot
-    xmlns:xacro="http://www.ros.org/wiki/xacro">
-    <xacro:macro name="car" params="prefix">
-        <link name="${prefix}base_link">
+<robot xmlns:xacro="http://www.ros.org/wiki/xacro">
+    <xacro:macro name="atlas2_model" params="prefix">
+        <link name="${prefix}model">
             <visual>
-                <origin xyz="-0.9 0 -0.5" rpy="0 0 0" />
+                <origin xyz="-0.9 0 0" rpy="0 0 0" />
                 <geometry>
                     <mesh filename="package://interactive_marker_test/meshes/mitsubishi_miev.dae" />
