Commit message: Changing the package name from interactive_marker_test to interactive_calibration

File: interactive_calibration/calibrations/pr2/pr2_no_arms.xacro (robot description, xacro)
@@ -23,5 +23,5 @@
   <xacro:include filename="$(find pr2_description)/urdf/materials.urdf.xacro" />
   <!--#TODO Added by Miguel-->
-  <xacro:include filename="$(find interactive_marker_test)/calibrations/pr2/pr2_calibration.xacro" />
+  <xacro:include filename="$(find interactive_calibration)/calibrations/pr2/pr2_calibration.xacro" />
    <xacro:pr2_calibration name="sensors"/>
   <!-- Now we can start using the macros included above to define the actual PR2 -->

File: interactive_calibration/urdf/prr_simple.xacro (robot description, xacro)
@@ -67,5 +67,5 @@
         <!--<geometry>-->
           <!--&lt;!&ndash; these meshes were exported in mm, so scale back to m &ndash;&gt;-->
-          <!--<mesh filename="package://interactive_marker_test/meshes/kinect2_origin_on_rgb_optical_frame.stl" scale="0.001 0.001 0.001"/>-->
+          <!--<mesh filename="package://interactive_calibration/meshes/kinect2_origin_on_rgb_optical_frame.stl" scale="0.001 0.001 0.001"/>-->
         <!--</geometry>-->
         <!--<material name="Kinect2Grey"/>-->
