Commit message: #35

File: interactive_calibration/calibrations/atlascar2/atlascar2.urdf.xacro (robot description, xacro)
@@ -1,5 +1,6 @@
 <?xml version="1.0"?>
 <robot xmlns:xacro="http://www.ros.org/wiki/xacro" name="atlas">
-    <xacro:include filename="$(find atlas2_description)/urdf/atlas2_macro.urdf.xacro"/>
+<!--    <xacro:include filename="$(find atlas2_description)/urdf/atlas2_macro.urdf.xacro"/>-->
+    <xacro:include filename="$(find interactive_calibration)/calibrations/atlascar2/atlas2_macro.urdf.xacro"/>
     <xacro:atlas2 prefix=""/>
     <!--#TODO Added by Miguel-->

File: interactive_calibration/calibrations/atlascar2/atlascar2_calibration.xacro (robot description, xacro)
@@ -23,11 +23,11 @@
             <topic topic="/top_right_camera/image_color"/>
         </sensor>
-        <sensor name="${prefix}frontal_laser" update_rate="20">
-            <parent link="${prefix}frontal_laser"/>
-            <origin xyz="0 0 0" rpy="0 0 0"/>
-            <calibration_parent link="${prefix}car_center"/>
-            <calibration_child link="${prefix}frontal_laser_mount_link"/>
-            <topic topic="/frontal_laser/cloud"/>
-        </sensor>
+<!--        <sensor name="${prefix}frontal_laser" update_rate="20">-->
+<!--            <parent link="${prefix}frontal_laser"/>-->
+<!--            <origin xyz="0 0 0" rpy="0 0 0"/>-->
+<!--            <calibration_parent link="${prefix}car_center"/>-->
+<!--            <calibration_child link="${prefix}frontal_laser_mount_link"/>-->
+<!--            <topic topic="/frontal_laser/cloud"/>-->
+<!--        </sensor>-->
         <sensor name="${prefix}left_laser" update_rate="20">
             <parent link="${prefix}left_laser"/>

Commit message: Changing xacro

File: interactive_calibration/calibrations/atlascar2/atlascar2.urdf.xacro (robot description, xacro)
@@ -2,5 +2,5 @@
 <robot xmlns:xacro="http://www.ros.org/wiki/xacro" name="atlas">
 <!--    <xacro:include filename="$(find atlas2_description)/urdf/atlas2_macro.urdf.xacro"/>-->
-    <xacro:include filename="$(find interactive_calibration)/calibrations/atlascar2/atlas2_macro.urdf.xacro"/>
+    <xacro:include filename="$(find atlas2_description)/urdf/atlas2_macro.urdf.xacro"/>
     <xacro:atlas2 prefix=""/>
     <!--#TODO Added by Miguel-->

File: interactive_calibration/calibrations/atlascar2/atlascar2_calibration.xacro (robot description, xacro)
@@ -2,23 +2,16 @@
 <robot xmlns:xacro="http://www.ros.org/wiki/xacro">
     <xacro:macro name="atlascar2_calibration" params="prefix">
-        <!--<sensor name="wide_stereo_left" update_rate="20.0">-->
-            <!--<parent link="car_center"/>-->
-            <!--<origin xyz="0.0 0.0 0.0" rpy="0.0 0.0 0.0"/>-->
-            <!--<calibration_parent link="double_stereo_link"/>-->
-            <!--<calibration_child link="wide_stereo_link"/>-->
-            <!--<topic topic="/wide_stereo/left/image_rect"/>-->
-        <!--</sensor>-->
-        <sensor name="${prefix}frontal_camera" update_rate="20">
-            <parent link="${prefix}frontal_camera_optical"/>
-            <origin xyz="0 0 0" rpy="0 0 0"/>
-            <calibration_parent link="${prefix}car_center"/>
-            <calibration_child link="${prefix}frontal_camera"/>
-            <topic topic="/frontal_camera/image_color"/>
-        </sensor>
         <sensor name="${prefix}top_right_camera" update_rate="20">
             <parent link="${prefix}top_right_camera_optical"/>
             <origin xyz="0 0 0" rpy="0 0 0"/>
-            <calibration_parent link="${prefix}car_center"/>
+            <calibration_parent link="${prefix}base_link"/>
             <calibration_child link="${prefix}top_right_camera"/>
+            <topic topic="/top_right_camera/image_color"/>
+        </sensor>
+        <sensor name="${prefix}top_left_camera" update_rate="20">
+            <parent link="${prefix}top_left_camera_optical"/>
+            <origin xyz="0 0 0" rpy="0 0 0"/>
+            <calibration_parent link="${prefix}base_link"/>
+            <calibration_child link="${prefix}top_left_camera"/>
             <topic topic="/top_right_camera/image_color"/>
         </sensor>
@@ -26,5 +19,5 @@
 <!--            <parent link="${prefix}frontal_laser"/>-->
 <!--            <origin xyz="0 0 0" rpy="0 0 0"/>-->
-<!--            <calibration_parent link="${prefix}car_center"/>-->
+<!--            <calibration_parent link="${prefix}base_link"/>-->
 <!--            <calibration_child link="${prefix}frontal_laser_mount_link"/>-->
 <!--            <topic topic="/frontal_laser/cloud"/>-->
@@ -33,5 +26,5 @@
             <parent link="${prefix}left_laser"/>
             <origin xyz="0 0 0" rpy="0 0 0"/>
-            <calibration_parent link="${prefix}car_center"/>
+            <calibration_parent link="${prefix}base_link"/>
             <calibration_child link="${prefix}left_laser"/>
             <topic topic="/left_laser/laserscan"/>
@@ -40,5 +33,5 @@
             <parent link="${prefix}right_laser"/>
             <origin xyz="0 0 0" rpy="0 0 0"/>
-            <calibration_parent link="${prefix}car_center"/>
+            <calibration_parent link="${prefix}base_link"/>
             <calibration_child link="${prefix}right_laser"/>
             <topic topic="/right_laser/laserscan"/>
