Commit message: Revising xacro for atlascar2

File: interactive_calibration/calibrations/atlascar2/atlascar2_calibration.xacro (robot description, xacro)
@@ -14,16 +14,19 @@
             <calibration_parent link="${prefix}car_center"/>
             <calibration_child link="${prefix}frontal_camera"/>
+            <topic topic="/frontal_camera/image_color"/>
         </sensor>
-        <!--<sensor name="${prefix}top_camera" update_rate="20">-->
-            <!--<parent link="${prefix}top_camera_optical"/>-->
-            <!--<origin xyz="0 0 0" rpy="0 0 0"/>-->
-            <!--<calibration_parent link="${prefix}car_center"/>-->
-            <!--<calibration_child link="${prefix}top_camera"/>-->
-        <!--</sensor>-->
-        <sensor name="${prefix}front_laser" update_rate="20">
-            <parent link="${prefix}front_laser"/>
+        <sensor name="${prefix}top_right_camera" update_rate="20">
+            <parent link="${prefix}top_right_camera"/>
             <origin xyz="0 0 0" rpy="0 0 0"/>
             <calibration_parent link="${prefix}car_center"/>
-            <calibration_child link="${prefix}front_laser_mount_link"/>
+            <calibration_child link="${prefix}top_right_camera"/>
+            <topic topic="/top_right_camera/image_color"/>
+        </sensor>
+        <sensor name="${prefix}frontal_laser" update_rate="20">
+            <parent link="${prefix}frontal_laser"/>
+            <origin xyz="0 0 0" rpy="0 0 0"/>
+            <calibration_parent link="${prefix}car_center"/>
+            <calibration_child link="${prefix}frontal_laser_mount_link"/>
+            <topic topic="/frontal_laser/cloud"/>
         </sensor>
         <sensor name="${prefix}left_laser" update_rate="20">
@@ -32,4 +35,5 @@
             <calibration_parent link="${prefix}car_center"/>
             <calibration_child link="${prefix}left_laser"/>
+            <topic topic="/left_laser/laserscan"/>
         </sensor>
         <sensor name="${prefix}right_laser" update_rate="20">
@@ -38,4 +42,5 @@
             <calibration_parent link="${prefix}car_center"/>
             <calibration_child link="${prefix}right_laser"/>
+            <topic topic="/right_laser/laserscan"/>
         </sensor>
     </xacro:macro>

Commit message: #35 reding json

File: interactive_calibration/calibrations/atlascar2/atlascar2_calibration.xacro (robot description, xacro)
@@ -10,5 +10,5 @@
         <!--</sensor>-->
         <sensor name="${prefix}frontal_camera" update_rate="20">
-            <parent link="${prefix}frontal_camera"/>
+            <parent link="${prefix}frontal_camera_optical"/>
             <origin xyz="0 0 0" rpy="0 0 0"/>
             <calibration_parent link="${prefix}car_center"/>
@@ -17,5 +17,5 @@
         </sensor>
         <sensor name="${prefix}top_right_camera" update_rate="20">
-            <parent link="${prefix}top_right_camera"/>
+            <parent link="${prefix}top_right_camera_optical"/>
             <origin xyz="0 0 0" rpy="0 0 0"/>
             <calibration_parent link="${prefix}car_center"/>

Commit message: Changed the loading of the calibration setup from a xacro to a json. Also fixes #41.

File: interactive_calibration/calibrations/atlascar2/atlascar2_calibration.xacro (robot description, xacro)
@@ -14,5 +14,5 @@
             <calibration_parent link="${prefix}base_link"/>
             <calibration_child link="${prefix}top_left_camera"/>
-            <topic topic="/top_right_camera/image_color"/>
+            <topic topic="/top_left_camera/image_color"/>
         </sensor>
 <!--        <sensor name="${prefix}frontal_laser" update_rate="20">-->

File: interactive_calibration/calibrations/atlascar2/first_guess.urdf.xacro (robot description, xacro)
@@ -46,7 +46,43 @@
     <child link="top_right_camera_optical"/>
   </joint>
-  <gazebo reference="top_right_camera_optical"/>
+  <gazebo reference="top_right_camera_optical"><material>Gazebo/Grey</material>
+    <sensor name="top_right_camera" type="camera">
+      <update_rate>120</update_rate>
+      <camera name="top_right_camera">
+        <pose>0 0 0 0 -1.5707 1.5707</pose>
+        <horizontal_fov>1.0471975512</horizontal_fov>
+        <image>
+          <width>1272</width>
+          <height>1016</height>
+          <format>R8G8B8</format>
+        </image>
+        <clip>
+          <near>0.5</near>
+          <far>300</far>
+        </clip>
+        <noise>
+          <type>gaussian</type>
+          <mean>0.0</mean>
+          <stddev>0.007</stddev>
+        </noise>
+      </camera>
+      <plugin filename="libgazebo_ros_camera.so" name="camera_controller">
+        <alwaysOn>true</alwaysOn>
+        <updateRate>120</updateRate>
+        <cameraName>top_right_camera</cameraName>
+        <imageTopicName>image_raw</imageTopicName>
+        <cameraInfoTopicName>camera_info</cameraInfoTopicName>
+        <frameName>top_right_camera_optical</frameName>
+        <hackBaseline>0.07</hackBaseline>
+        <distortionK1>0.0</distortionK1>
+        <distortionK2>0.0</distortionK2>
+        <distortionK3>0.0</distortionK3>
+        <distortionT1>0.0</distortionT1>
+        <distortionT2>0.0</distortionT2>
+      </plugin>
+    </sensor>
+  </gazebo>
   <joint name="base_link_to_top_right_camera" type="fixed">
-    <origin xyz="-1.77280187607 -0.233933746815 1.25" rpy="-6.41765959721e-08 0.236651372034 -0.0570543483677"/>
+    <origin xyz="-1.5 -0.12 1.25" rpy="0.0 0.4 0.0"/>
     <parent link="base_link"/>
     <child link="top_right_camera"/>
@@ -77,7 +113,43 @@
     <child link="top_left_camera_optical"/>
   </joint>
-  <gazebo reference="top_left_camera_optical"/>
+  <gazebo reference="top_left_camera_optical"><material>Gazebo/Grey</material>
+    <sensor name="top_left_camera" type="camera">
+      <update_rate>120</update_rate>
+      <camera name="top_left_camera">
+        <pose>0 0 0 0 -1.5707 1.5707</pose>
+        <horizontal_fov>1.0471975512</horizontal_fov>
+        <image>
+          <width>1272</width>
+          <height>1016</height>
+          <format>R8G8B8</format>
+        </image>
+        <clip>
+          <near>0.5</near>
+          <far>300</far>
+        </clip>
+        <noise>
+          <type>gaussian</type>
+          <mean>0.0</mean>
+          <stddev>0.007</stddev>
+        </noise>
+      </camera>
+      <plugin filename="libgazebo_ros_camera.so" name="camera_controller">
+        <alwaysOn>true</alwaysOn>
+        <updateRate>120</updateRate>
+        <cameraName>top_left_camera</cameraName>
+        <imageTopicName>image_raw</imageTopicName>
+        <cameraInfoTopicName>camera_info</cameraInfoTopicName>
+        <frameName>top_left_camera_optical</frameName>
+        <hackBaseline>0.07</hackBaseline>
+        <distortionK1>0.0</distortionK1>
+        <distortionK2>0.0</distortionK2>
+        <distortionK3>0.0</distortionK3>
+        <distortionT1>0.0</distortionT1>
+        <distortionT2>0.0</distortionT2>
+      </plugin>
+    </sensor>
+  </gazebo>
   <joint name="base_link_to_top_left_camera" type="fixed">
-    <origin xyz="-1.73982644081 0.382407188416 1.25" rpy="4.58485844927e-05 0.226041151401 -0.0962249358456"/>
+    <origin xyz="-1.5 0.12 1.25" rpy="0.0 0.4 0.0"/>
     <parent link="base_link"/>
     <child link="top_left_camera"/>
@@ -85,5 +157,5 @@
   <link name="frontal_laser_mount_link">
     <inertial>
-      <origin xyz="0.0 0.0 0.0" rpy="0.0 0.0 0.0"/>
+      <origin xyz="0.0 0.0 0.0" rpy="0 0 0"/>
       <mass value="0.001"/>
       <inertia ixx="1e-06" ixy="0.0" ixz="0.0" iyy="1e-06" iyz="0.0" izz="1e-06"/>
@@ -97,5 +169,5 @@
   <link name="frontal_laser">
     <inertial>
-      <origin xyz="0.0026 -0.02325 -0.0" rpy="0.0 0.0 0.0"/>
+      <origin xyz="0.0026 -0.02325 -0.0" rpy="0 0 0"/>
       <mass value="1.0"/>
       <inertia ixx="0.00290035300653" ixy="0.0" ixz="0.0" iyy="0.00136918611899" iyz="0.0" izz="0.00297887297512"/>
@@ -121,5 +193,5 @@
   <link name="right_laser">
     <inertial>
-      <origin xyz="0.0 0.0 0.0" rpy="0.0 0.0 0.0"/>
+      <origin xyz="0.0 0.0 0.0" rpy="0 0 0"/>
       <mass value="1.1"/>
       <inertia ixx="0.00307156543804" ixy="0.0" ixz="0.0" iyy="0.00312849041527" iyz="0.0" izz="0.00196432421427"/>
@@ -138,7 +210,38 @@
     </collision>
   </link>
-  <gazebo reference="right_laser"/>
+  <gazebo reference="right_laser"><turnGravityOff>true</turnGravityOff>
+    <sensor name="right_laser" type="ray">
+      <pose>0 0 0 0 0 0</pose>
+      <visualize>false</visualize>
+      <update_rate>50</update_rate>
+      <ray>
+        <scan>
+          <horizontal>
+            <samples>720</samples>
+            <resolution>1</resolution>
+            <min_angle>-2.35619</min_angle>
+            <max_angle>2.35619</max_angle>
+          </horizontal>
+        </scan>
+        <range>
+          <min>0.1</min>
+          <max>30.0</max>
+          <resolution>0.01</resolution>
+        </range>
+        <noise>
+          <type>gaussian</type>
+          <mean>0.0</mean>
+          <stddev>0.001</stddev>
+        </noise>
+      </ray>
+      <plugin filename="libgazebo_ros_laser.so" name="gazebo_ros_laser">
+        <topicName>scan</topicName>
+        <frameName>right_laser</frameName>
+        <robotNamespace>/</robotNamespace>
+      </plugin>
+    </sensor>
+  </gazebo>
   <joint name="base_link_to_right_laser" type="fixed">
-    <origin xyz="-0.0500000007451 -0.699999988079 0.10000000149" rpy="7.91199037381e-09 5.07742774923e-10 -0.802577692221"/>
+    <origin xyz="1.1338140964508057 -2.1695430278778076 0.10000000149011612" rpy="0.0 0.0 -0.630000024243"/>
     <parent link="base_link"/>
     <child link="right_laser"/>
@@ -146,5 +249,5 @@
   <link name="left_laser">
     <inertial>
-      <origin xyz="0.0 0.0 0.0" rpy="0.0 0.0 0.0"/>
+      <origin xyz="0.0 0.0 0.0" rpy="0 0 0"/>
       <mass value="1.1"/>
       <inertia ixx="0.00307156543804" ixy="0.0" ixz="0.0" iyy="0.00312849041527" iyz="0.0" izz="0.00196432421427"/>
@@ -163,7 +266,38 @@
     </collision>
   </link>
-  <gazebo reference="left_laser"/>
+  <gazebo reference="left_laser"><turnGravityOff>true</turnGravityOff>
+    <sensor name="left_laser" type="ray">
+      <pose>0 0 0 0 0 0</pose>
+      <visualize>false</visualize>
+      <update_rate>50</update_rate>
+      <ray>
+        <scan>
+          <horizontal>
+            <samples>720</samples>
+            <resolution>1</resolution>
+            <min_angle>-2.35619</min_angle>
+            <max_angle>2.35619</max_angle>
+          </horizontal>
+        </scan>
+        <range>
+          <min>0.1</min>
+          <max>30.0</max>
+          <resolution>0.01</resolution>
+        </range>
+        <noise>
+          <type>gaussian</type>
+          <mean>0.0</mean>
+          <stddev>0.001</stddev>
+        </noise>
+      </ray>
+      <plugin filename="libgazebo_ros_laser.so" name="gazebo_ros_laser">
+        <topicName>scan</topicName>
+        <frameName>left_laser</frameName>
+        <robotNamespace>/</robotNamespace>
+      </plugin>
+    </sensor>
+  </gazebo>
   <joint name="base_link_to_left_laser" type="fixed">
-    <origin xyz="-0.0500000007451 0.699999988079 0.10000000149" rpy="-1.40600650738e-08 1.04046331119e-08 0.850917484309"/>
+    <origin xyz="-0.05 0.7 0.1" rpy="0.0 -0.0 0.57"/>
     <parent link="base_link"/>
     <child link="left_laser"/>
