Commit message: fix #37 . This was a tricky one: there were some static tf messages in the bag file.

File: interactive_calibration/calibrations/atlascar2/first_guess.urdf.xacro (robot description, xacro)
@@ -84,5 +84,5 @@
   </gazebo>
   <joint name="base_link_to_top_right_camera" type="fixed">
-    <origin xyz="-1.50000011921 -2.5133471489 1.25" rpy="0.0 0.399999989245 0.0"/>
+    <origin xyz="-1.5 -0.12 1.25" rpy="0.0 0.4 0.0"/>
     <parent link="base_link"/>
     <child link="top_right_camera"/>
@@ -151,5 +151,5 @@
   </gazebo>
   <joint name="base_link_to_top_left_camera" type="fixed">
-    <origin xyz="-1.5 0.12 1.25" rpy="0.0 0.4 0.0"/>
+    <origin xyz="1.7934513092041016 0.11999999731779099 1.25" rpy="1.61264849914 -0.0176877887299 0.399629778014"/>
     <parent link="base_link"/>
     <child link="top_left_camera"/>

Commit message: All working now!

File: interactive_calibration/calibrations/atlascar2/first_guess.urdf.xacro (robot description, xacro)
@@ -46,43 +46,7 @@
     <child link="top_right_camera_optical"/>
   </joint>
-  <gazebo reference="top_right_camera_optical"><material>Gazebo/Grey</material>
-    <sensor name="top_right_camera" type="camera">
-      <update_rate>120</update_rate>
-      <camera name="top_right_camera">
-        <pose>0 0 0 0 -1.5707 1.5707</pose>
-        <horizontal_fov>1.0471975512</horizontal_fov>
-        <image>
-          <width>1272</width>
-          <height>1016</height>
-          <format>R8G8B8</format>
-        </image>
-        <clip>
-          <near>0.5</near>
-          <far>300</far>
-        </clip>
-        <noise>
-          <type>gaussian</type>
-          <mean>0.0</mean>
-          <stddev>0.007</stddev>
-        </noise>
-      </camera>
-      <plugin filename="libgazebo_ros_camera.so" name="camera_controller">
-        <alwaysOn>true</alwaysOn>
-        <updateRate>120</updateRate>
-        <cameraName>top_right_camera</cameraName>
-        <imageTopicName>image_raw</imageTopicName>
-        <cameraInfoTopicName>camera_info</cameraInfoTopicName>
-        <frameName>top_right_camera_optical</frameName>
-        <hackBaseline>0.07</hackBaseline>
-        <distortionK1>0.0</distortionK1>
-        <distortionK2>0.0</distortionK2>
-        <distortionK3>0.0</distortionK3>
-        <distortionT1>0.0</distortionT1>
-        <distortionT2>0.0</distortionT2>
-      </plugin>
-    </sensor>
-  </gazebo>
+  <gazebo reference="top_right_camera_optical"/>
   <joint name="base_link_to_top_right_camera" type="fixed">
-    <origin xyz="-1.5 -0.12 1.25" rpy="0.0 0.4 0.0"/>
+    <origin xyz="-1.77280187607 -0.233933746815 1.25" rpy="-6.41765959721e-08 0.236651372034 -0.0570543483677"/>
     <parent link="base_link"/>
     <child link="top_right_camera"/>
@@ -113,43 +77,7 @@
     <child link="top_left_camera_optical"/>
   </joint>
-  <gazebo reference="top_left_camera_optical"><material>Gazebo/Grey</material>
-    <sensor name="top_left_camera" type="camera">
-      <update_rate>120</update_rate>
-      <camera name="top_left_camera">
-        <pose>0 0 0 0 -1.5707 1.5707</pose>
-        <horizontal_fov>1.0471975512</horizontal_fov>
-        <image>
-          <width>1272</width>
-          <height>1016</height>
-          <format>R8G8B8</format>
-        </image>
-        <clip>
-          <near>0.5</near>
-          <far>300</far>
-        </clip>
-        <noise>
-          <type>gaussian</type>
-          <mean>0.0</mean>
-          <stddev>0.007</stddev>
-        </noise>
-      </camera>
-      <plugin filename="libgazebo_ros_camera.so" name="camera_controller">
-        <alwaysOn>true</alwaysOn>
-        <updateRate>120</updateRate>
-        <cameraName>top_left_camera</cameraName>
-        <imageTopicName>image_raw</imageTopicName>
-        <cameraInfoTopicName>camera_info</cameraInfoTopicName>
-        <frameName>top_left_camera_optical</frameName>
-        <hackBaseline>0.07</hackBaseline>
-        <distortionK1>0.0</distortionK1>
-        <distortionK2>0.0</distortionK2>
-        <distortionK3>0.0</distortionK3>
-        <distortionT1>0.0</distortionT1>
-        <distortionT2>0.0</distortionT2>
-      </plugin>
-    </sensor>
-  </gazebo>
+  <gazebo reference="top_left_camera_optical"/>
   <joint name="base_link_to_top_left_camera" type="fixed">
-    <origin xyz="1.7934513092041016 0.11999999731779099 1.25" rpy="1.61264849914 -0.0176877887299 0.399629778014"/>
+    <origin xyz="-1.73982644081 0.382407188416 1.25" rpy="4.58485844927e-05 0.226041151401 -0.0962249358456"/>
     <parent link="base_link"/>
     <child link="top_left_camera"/>
@@ -157,5 +85,5 @@
   <link name="frontal_laser_mount_link">
     <inertial>
-      <origin xyz="0.0 0.0 0.0" rpy="0 0 0"/>
+      <origin xyz="0.0 0.0 0.0" rpy="0.0 0.0 0.0"/>
       <mass value="0.001"/>
       <inertia ixx="1e-06" ixy="0.0" ixz="0.0" iyy="1e-06" iyz="0.0" izz="1e-06"/>
@@ -169,5 +97,5 @@
   <link name="frontal_laser">
     <inertial>
-      <origin xyz="0.0026 -0.02325 -0.0" rpy="0 0 0"/>
+      <origin xyz="0.0026 -0.02325 -0.0" rpy="0.0 0.0 0.0"/>
       <mass value="1.0"/>
       <inertia ixx="0.00290035300653" ixy="0.0" ixz="0.0" iyy="0.00136918611899" iyz="0.0" izz="0.00297887297512"/>
@@ -193,5 +121,5 @@
   <link name="right_laser">
     <inertial>
-      <origin xyz="0.0 0.0 0.0" rpy="0 0 0"/>
+      <origin xyz="0.0 0.0 0.0" rpy="0.0 0.0 0.0"/>
       <mass value="1.1"/>
       <inertia ixx="0.00307156543804" ixy="0.0" ixz="0.0" iyy="0.00312849041527" iyz="0.0" izz="0.00196432421427"/>
@@ -210,38 +138,7 @@
     </collision>
   </link>
-  <gazebo reference="right_laser"><turnGravityOff>true</turnGravityOff>
-    <sensor name="right_laser" type="ray">
-      <pose>0 0 0 0 0 0</pose>
-      <visualize>false</visualize>
-      <update_rate>50</update_rate>
-      <ray>
-        <scan>
-          <horizontal>
-            <samples>720</samples>
-            <resolution>1</resolution>
-            <min_angle>-2.35619</min_angle>
-            <max_angle>2.35619</max_angle>
-          </horizontal>
-        </scan>
-        <range>
-          <min>0.1</min>
-          <max>30.0</max>
-          <resolution>0.01</resolution>
-        </range>
-        <noise>
-          <type>gaussian</type>
-          <mean>0.0</mean>
-          <stddev>0.001</stddev>
-        </noise>
-      </ray>
-      <plugin filename="libgazebo_ros_laser.so" name="gazebo_ros_laser">
-        <topicName>scan</topicName>
-        <frameName>right_laser</frameName>
-        <robotNamespace>/</robotNamespace>
-      </plugin>
-    </sensor>
-  </gazebo>
+  <gazebo reference="right_laser"/>
   <joint name="base_link_to_right_laser" type="fixed">
-    <origin xyz="-0.05 -0.7 0.1" rpy="0.0 0.0 -0.63"/>
+    <origin xyz="-0.0500000007451 -0.699999988079 0.10000000149" rpy="7.91199037381e-09 5.07742774923e-10 -0.802577692221"/>
     <parent link="base_link"/>
     <child link="right_laser"/>
@@ -249,5 +146,5 @@
   <link name="left_laser">
     <inertial>
-      <origin xyz="0.0 0.0 0.0" rpy="0 0 0"/>
+      <origin xyz="0.0 0.0 0.0" rpy="0.0 0.0 0.0"/>
       <mass value="1.1"/>
       <inertia ixx="0.00307156543804" ixy="0.0" ixz="0.0" iyy="0.00312849041527" iyz="0.0" izz="0.00196432421427"/>
@@ -266,38 +163,7 @@
     </collision>
   </link>
-  <gazebo reference="left_laser"><turnGravityOff>true</turnGravityOff>
-    <sensor name="left_laser" type="ray">
-      <pose>0 0 0 0 0 0</pose>
-      <visualize>false</visualize>
-      <update_rate>50</update_rate>
-      <ray>
-        <scan>
-          <horizontal>
-            <samples>720</samples>
-            <resolution>1</resolution>
-            <min_angle>-2.35619</min_angle>
-            <max_angle>2.35619</max_angle>
-          </horizontal>
-        </scan>
-        <range>
-          <min>0.1</min>
-          <max>30.0</max>
-          <resolution>0.01</resolution>
-        </range>
-        <noise>
-          <type>gaussian</type>
-          <mean>0.0</mean>
-          <stddev>0.001</stddev>
-        </noise>
-      </ray>
-      <plugin filename="libgazebo_ros_laser.so" name="gazebo_ros_laser">
-        <topicName>scan</topicName>
-        <frameName>left_laser</frameName>
-        <robotNamespace>/</robotNamespace>
-      </plugin>
-    </sensor>
-  </gazebo>
+  <gazebo reference="left_laser"/>
   <joint name="base_link_to_left_laser" type="fixed">
-    <origin xyz="-0.05 0.7 0.1" rpy="0.0 -0.0 0.57"/>
+    <origin xyz="-0.0500000007451 0.699999988079 0.10000000149" rpy="-1.40600650738e-08 1.04046331119e-08 0.850917484309"/>
     <parent link="base_link"/>
     <child link="left_laser"/>

Commit message: don't know what was changed ...

File: interactive_calibration/calibrations/atlascar2/first_guess.urdf.xacro (robot description, xacro)
@@ -84,5 +84,5 @@
   </gazebo>
   <joint name="base_link_to_top_right_camera" type="fixed">
-    <origin xyz="-1.5 -0.12 1.25" rpy="0.0 0.4 0.0"/>
+    <origin xyz="-1.5 -0.215595543384552 1.25" rpy="2.87639977769e-08 0.231614677419 -0.0695532323982"/>
     <parent link="base_link"/>
     <child link="top_right_camera"/>
@@ -151,5 +151,5 @@
   </gazebo>
   <joint name="base_link_to_top_left_camera" type="fixed">
-    <origin xyz="-1.5 0.12 1.25" rpy="0.0 0.4 0.0"/>
+    <origin xyz="-1.5 0.1799130141735077 1.25" rpy="-7.00049190111e-08 0.234987143739 -0.0603197392008"/>
     <parent link="base_link"/>
     <child link="top_left_camera"/>
@@ -243,5 +243,5 @@
   </gazebo>
   <joint name="base_link_to_right_laser" type="fixed">
-    <origin xyz="1.1338140964508057 -2.1695430278778076 0.10000000149011612" rpy="0.0 0.0 -0.630000024243"/>
+    <origin xyz="-0.05000000074505806 -0.699999988079071 0.10000000149011612" rpy="8.10708019675e-09 7.81548619769e-09 -0.802585229488"/>
     <parent link="base_link"/>
     <child link="right_laser"/>
@@ -299,35 +299,7 @@
   </gazebo>
   <joint name="base_link_to_left_laser" type="fixed">
-    <origin xyz="-0.05 0.7 0.1" rpy="0.0 -0.0 0.57"/>
+    <origin xyz="-0.05000000074505806 0.699999988079071 0.10000000149011612" rpy="-2.78440592625e-09 1.36237645799e-08 0.811567993071"/>
     <parent link="base_link"/>
     <child link="left_laser"/>
   </joint>
-  <sensor name="top_right_camera" update_rate="20.0">
-    <parent link="top_right_camera_optical"/>
-    <origin xyz="0.0 0.0 0.0" rpy="0.0 0.0 0.0"/>
-    <calibration_parent link="base_link"/>
-    <calibration_child link="top_right_camera"/>
-    <topic topic="/top_right_camera/image_color"/>
-  </sensor>
-  <sensor name="top_left_camera" update_rate="20.0">
-    <parent link="top_left_camera_optical"/>
-    <origin xyz="0.0 0.0 0.0" rpy="0.0 0.0 0.0"/>
-    <calibration_parent link="base_link"/>
-    <calibration_child link="top_left_camera"/>
-    <topic topic="/top_right_camera/image_color"/>
-  </sensor>
-  <sensor name="left_laser" update_rate="20.0">
-    <parent link="left_laser"/>
-    <origin xyz="0.0 0.0 0.0" rpy="0.0 0.0 0.0"/>
-    <calibration_parent link="base_link"/>
-    <calibration_child link="left_laser"/>
-    <topic topic="/left_laser/laserscan"/>
-  </sensor>
-  <sensor name="right_laser" update_rate="20.0">
-    <parent link="right_laser"/>
-    <origin xyz="0.0 0.0 0.0" rpy="0.0 0.0 0.0"/>
-    <calibration_parent link="base_link"/>
-    <calibration_child link="right_laser"/>
-    <topic topic="/right_laser/laserscan"/>
-  </sensor>
 </robot>

Commit message: #45 opt working. readme updated

File: interactive_calibration/calibrations/atlascar2/first_guess.urdf.xacro (robot description, xacro)
@@ -84,5 +84,5 @@
   </gazebo>
   <joint name="base_link_to_top_right_camera" type="fixed">
-    <origin xyz="-1.5 -0.215595543384552 1.25" rpy="2.87639977769e-08 0.231614677419 -0.0695532323982"/>
+    <origin xyz="-1.73537778854 -0.222493559122 1.25" rpy="0.00707850991813 0.184877597439 -0.0814686753294"/>
     <parent link="base_link"/>
     <child link="top_right_camera"/>
@@ -151,5 +151,5 @@
   </gazebo>
   <joint name="base_link_to_top_left_camera" type="fixed">
-    <origin xyz="-1.5 0.1799130141735077 1.25" rpy="-7.00049190111e-08 0.234987143739 -0.0603197392008"/>
+    <origin xyz="-1.6680958271 0.206312954426 1.25" rpy="-0.00168771614209 0.207326470221 -0.0632289375909"/>
     <parent link="base_link"/>
     <child link="top_left_camera"/>
@@ -243,5 +243,5 @@
   </gazebo>
   <joint name="base_link_to_right_laser" type="fixed">
-    <origin xyz="-0.05000000074505806 -0.699999988079071 0.10000000149011612" rpy="8.10708019675e-09 7.81548619769e-09 -0.802585229488"/>
+    <origin xyz="-0.0500000007451 -0.699999988079 0.10000000149" rpy="8.72542694465e-09 9.406761646e-09 -0.822308007793"/>
     <parent link="base_link"/>
     <child link="right_laser"/>
@@ -299,5 +299,5 @@
   </gazebo>
   <joint name="base_link_to_left_laser" type="fixed">
-    <origin xyz="-0.05000000074505806 0.699999988079071 0.10000000149011612" rpy="-2.78440592625e-09 1.36237645799e-08 0.811567993071"/>
+    <origin xyz="-0.0500000007451 0.699999988079 0.10000000149" rpy="-2.73615898207e-09 1.28586821716e-08 0.833176939675"/>
     <parent link="base_link"/>
     <child link="left_laser"/>

Commit message: Improving visualization of the optimization procedure using rviz. #50

File: interactive_calibration/calibrations/atlascar2/first_guess.urdf.xacro (robot description, xacro)
@@ -84,5 +84,5 @@
   </gazebo>
   <joint name="base_link_to_top_right_camera" type="fixed">
-    <origin xyz="-1.73537778854 -0.222493559122 1.25" rpy="0.00707850991813 0.184877597439 -0.0814686753294"/>
+    <origin xyz="-1.5 -0.119999997318 1.25" rpy="-1.76654733052e-08 0.0454578709684 -6.59441660169e-09"/>
     <parent link="base_link"/>
     <child link="top_right_camera"/>
@@ -151,5 +151,5 @@
   </gazebo>
   <joint name="base_link_to_top_left_camera" type="fixed">
-    <origin xyz="-1.6680958271 0.206312954426 1.25" rpy="-0.00168771614209 0.207326470221 -0.0632289375909"/>
+    <origin xyz="-1.5 0.119999997318 1.25" rpy="-1.97744116859e-08 0.0317141567665 -5.50452755037e-09"/>
     <parent link="base_link"/>
     <child link="top_left_camera"/>
@@ -243,5 +243,5 @@
   </gazebo>
   <joint name="base_link_to_right_laser" type="fixed">
-    <origin xyz="-0.0500000007451 -0.699999988079 0.10000000149" rpy="8.72542694465e-09 9.406761646e-09 -0.822308007793"/>
+    <origin xyz="-0.05 -0.7 0.1" rpy="0.0 0.0 -0.63"/>
     <parent link="base_link"/>
     <child link="right_laser"/>
@@ -299,5 +299,5 @@
   </gazebo>
   <joint name="base_link_to_left_laser" type="fixed">
-    <origin xyz="-0.0500000007451 0.699999988079 0.10000000149" rpy="-2.73615898207e-09 1.28586821716e-08 0.833176939675"/>
+    <origin xyz="-0.05 0.7 0.1" rpy="0.0 -0.0 0.57"/>
     <parent link="base_link"/>
     <child link="left_laser"/>

Commit message: Close #58 Also tested and refactored collect_and label.

File: interactive_calibration/calibrations/atlascar2/first_guess.urdf.xacro (robot description, xacro)
@@ -84,5 +84,5 @@
   </gazebo>
   <joint name="base_link_to_top_right_camera" type="fixed">
-    <origin xyz="-1.5 -0.119999997318 1.25" rpy="-1.76654733052e-08 0.0454578709684 -6.59441660169e-09"/>
+    <origin xyz="-1.51038885117 -0.119999997318 1.25" rpy="-1.20581738181e-08 0.24062377846 -1.66313963715e-09"/>
     <parent link="base_link"/>
     <child link="top_right_camera"/>
@@ -151,5 +151,5 @@
   </gazebo>
   <joint name="base_link_to_top_left_camera" type="fixed">
-    <origin xyz="-1.5 0.119999997318 1.25" rpy="-1.97744116859e-08 0.0317141567665 -5.50452755037e-09"/>
+    <origin xyz="-1.5 0.119999997318 1.25" rpy="-5.56371389661e-09 0.251846312747 -7.19782432889e-09"/>
     <parent link="base_link"/>
     <child link="top_left_camera"/>
@@ -243,5 +243,5 @@
   </gazebo>
   <joint name="base_link_to_right_laser" type="fixed">
-    <origin xyz="-0.05 -0.7 0.1" rpy="0.0 0.0 -0.63"/>
+    <origin xyz="-0.0500000007451 -0.699999988079 0.10000000149" rpy="2.28357349019e-08 1.20044322881e-08 -0.860756108382"/>
     <parent link="base_link"/>
     <child link="right_laser"/>
@@ -299,5 +299,5 @@
   </gazebo>
   <joint name="base_link_to_left_laser" type="fixed">
-    <origin xyz="-0.05 0.7 0.1" rpy="0.0 -0.0 0.57"/>
+    <origin xyz="-0.0500000007451 0.699999988079 0.10000000149" rpy="-1.45826407349e-08 7.3739377889e-09 0.762926751911"/>
     <parent link="base_link"/>
     <child link="left_laser"/>

Commit message: Close #88. Implemented and tested.

File: interactive_calibration/calibrations/atlascar2/first_guess.urdf.xacro (robot description, xacro)
@@ -2,5 +2,5 @@
 <robot name="atlas">
   <link name="base_link"/>
-  <link name="ground"/>
+  <link name="base_footprint"/>
   <link name="model">
     <visual>
@@ -11,13 +11,13 @@
     </visual>
   </link>
-  <joint name="base_link_to_model" type="fixed">
-    <origin xyz="0.0 0.0 -0.4" rpy="0.0 0.0 1.57079632679"/>
-    <parent link="base_link"/>
+  <joint name="base_link_to_base_footprint" type="fixed">
+    <origin xyz="0.0 0.0 -0.305" rpy="0.0 0.0 0.0"/>
+    <parent link="base_link"/>
+    <child link="base_footprint"/>
+  </joint>
+  <joint name="base_footprint_to_model" type="fixed">
+    <origin xyz="0.0 0.0 0.0" rpy="0.0 0.0 1.57079632679"/>
+    <parent link="base_footprint"/>
     <child link="model"/>
-  </joint>
-  <joint name="base_link_to_ground" type="fixed">
-    <origin xyz="0.0 0.0 -0.4" rpy="0.0 0.0 0.0"/>
-    <parent link="base_link"/>
-    <child link="ground"/>
   </joint>
   <link name="top_right_camera">
@@ -84,5 +84,5 @@
   </gazebo>
   <joint name="base_link_to_top_right_camera" type="fixed">
-    <origin xyz="-1.51038885117 -0.119999997318 1.25" rpy="-1.20581738181e-08 0.24062377846 -1.66313963715e-09"/>
+    <origin xyz="-1.54999995232 -0.219999998808 1.35000002384" rpy="-1.1792504301e-08 0.227291866291 -2.39260131975e-09"/>
     <parent link="base_link"/>
     <child link="top_right_camera"/>
@@ -151,5 +151,5 @@
   </gazebo>
   <joint name="base_link_to_top_left_camera" type="fixed">
-    <origin xyz="-1.5 0.119999997318 1.25" rpy="-5.56371389661e-09 0.251846312747 -7.19782432889e-09"/>
+    <origin xyz="-1.54999995232 0.219999998808 1.35000002384" rpy="-1.10381245545e-08 0.198812341739 -4.69646546231e-09"/>
     <parent link="base_link"/>
     <child link="top_left_camera"/>
@@ -243,5 +243,5 @@
   </gazebo>
   <joint name="base_link_to_right_laser" type="fixed">
-    <origin xyz="-0.0500000007451 -0.699999988079 0.10000000149" rpy="2.28357349019e-08 1.20044322881e-08 -0.860756108382"/>
+    <origin xyz="-0.070000000298 -0.759999990463 0.270000010729" rpy="4.16188557712e-08 -6.35236315078e-09 -0.682818723015"/>
     <parent link="base_link"/>
     <child link="right_laser"/>
@@ -299,7 +299,55 @@
   </gazebo>
   <joint name="base_link_to_left_laser" type="fixed">
-    <origin xyz="-0.0500000007451 0.699999988079 0.10000000149" rpy="-1.45826407349e-08 7.3739377889e-09 0.762926751911"/>
+    <origin xyz="-0.070000000298 0.759999990463 0.270000010729" rpy="-7.55136378913e-08 -5.26812102076e-08 0.944291931471"/>
     <parent link="base_link"/>
     <child link="left_laser"/>
   </joint>
+  <link name="top_center_rgbd_camera_link">
+    <inertial>
+      <origin xyz="0.0 0.0 0.0" rpy="0.0 0.0 0.0"/>
+      <mass value="0.2"/>
+      <inertia ixx="0.00058083" ixy="0.0" ixz="0.0" iyy="3.0833e-05" iyz="0.0" izz="0.00059083"/>
+    </inertial>
+    <visual>
+      <origin xyz="0.0 0.0 0.0" rpy="0.0 0.0 0.0"/>
+      <geometry>
+        <mesh filename="package://atlas2_description/meshes/asus_xtion/asus_xtion_simple.dae"/>
+      </geometry>
+    </visual>
+    <collision>
+      <origin xyz="0.0 0.0 0.0" rpy="0.0 0.0 0.0"/>
+      <geometry>
+        <mesh filename="package://atlas2_description/meshes/asus_xtion/asus_xtion_simple.dae"/>
+      </geometry>
+    </collision>
+  </link>
+  <joint name="top_center_rgbd_camera_depth_joint" type="fixed">
+    <origin xyz="0.0 0.049 0.0" rpy="0.0 0.0 0.0"/>
+    <parent link="top_center_rgbd_camera_link"/>
+    <child link="top_center_rgbd_camera_depth_frame"/>
+  </joint>
+  <link name="top_center_rgbd_camera_depth_frame"/>
+  <joint name="top_center_rgbd_camera_depth_optical_joint" type="fixed">
+    <origin xyz="0.0 0.0 0.0" rpy="-1.57079632679 0.0 -1.57079632679"/>
+    <parent link="top_center_rgbd_camera_depth_frame"/>
+    <child link="top_center_rgbd_camera_depth_optical_frame"/>
+  </joint>
+  <link name="top_center_rgbd_camera_depth_optical_frame"/>
+  <joint name="top_center_rgbd_camera_rgb_joint" type="fixed">
+    <origin xyz="0.0 0.022 0.0" rpy="0.0 0.0 0.0"/>
+    <parent link="top_center_rgbd_camera_link"/>
+    <child link="top_center_rgbd_camera_rgb_frame"/>
+  </joint>
+  <link name="top_center_rgbd_camera_rgb_frame"/>
+  <joint name="top_center_rgbd_camera_rgb_optical_joint" type="fixed">
+    <origin xyz="0.0 0.0 0.0" rpy="-1.57079632679 0.0 -1.57079632679"/>
+    <parent link="top_center_rgbd_camera_rgb_frame"/>
+    <child link="top_center_rgbd_camera_rgb_optical_frame"/>
+  </joint>
+  <link name="top_center_rgbd_camera_rgb_optical_frame"/>
+  <joint name="base_link_to_top_center_rgbd_camera" type="fixed">
+    <origin xyz="-1.51 -0.01 1.27" rpy="0.0 0.4 0.0"/>
+    <parent link="base_link"/>
+    <child link="top_center_rgbd_camera_link"/>
+  </joint>
 </robot>
