Commit message: Graph drawing by Afonso. Visiting dictionaries by order

File: interactive_calibration/calibrations/atlascar2/first_guess.urdf.xacro (robot description, xacro)
@@ -84,5 +84,5 @@
   </gazebo>
   <joint name="base_link_to_top_right_camera" type="fixed">
-    <origin xyz="-1.54999995232 -0.219999998808 1.40112948418" rpy="-1.08223780011e-08 0.164151666864 -6.43161410219e-09"/>
+    <origin xyz="-1.52545705881 -0.234616836053 1.36126320471" rpy="-0.022569779172 0.396104847692 -0.0142500465895"/>
     <parent link="base_link"/>
     <child link="top_right_camera"/>
@@ -151,5 +151,5 @@
   </gazebo>
   <joint name="base_link_to_top_left_camera" type="fixed">
-    <origin xyz="-1.54999995232 0.219999998808 1.38210916519" rpy="-1.49597710582e-08 0.173506001022 -5.12355388858e-09"/>
+    <origin xyz="-1.54999995232 0.219999998808 1.35000002384" rpy="-8.03050052384e-09 0.219301166046 3.19403651722e-09"/>
     <parent link="base_link"/>
     <child link="top_left_camera"/>
@@ -157,5 +157,5 @@
   <link name="frontal_laser_mount_link">
     <inertial>
-      <origin xyz="0.0 0.0 0.0" rpy="0 0 0"/>
+      <origin xyz="0.0 0.0 0.0" rpy="0.0 0.0 0.0"/>
       <mass value="0.001"/>
       <inertia ixx="1e-06" ixy="0.0" ixz="0.0" iyy="1e-06" iyz="0.0" izz="1e-06"/>
@@ -169,5 +169,5 @@
   <link name="frontal_laser">
     <inertial>
-      <origin xyz="0.0026 -0.02325 -0.0" rpy="0 0 0"/>
+      <origin xyz="0.0026 -0.02325 -0.0" rpy="0.0 0.0 0.0"/>
       <mass value="1.0"/>
       <inertia ixx="0.00290035300653" ixy="0.0" ixz="0.0" iyy="0.00136918611899" iyz="0.0" izz="0.00297887297512"/>
@@ -193,5 +193,5 @@
   <link name="right_laser">
     <inertial>
-      <origin xyz="0.0 0.0 0.0" rpy="0 0 0"/>
+      <origin xyz="0.0 0.0 0.0" rpy="0.0 0.0 0.0"/>
       <mass value="1.1"/>
       <inertia ixx="0.00307156543804" ixy="0.0" ixz="0.0" iyy="0.00312849041527" iyz="0.0" izz="0.00196432421427"/>
@@ -243,5 +243,5 @@
   </gazebo>
   <joint name="base_link_to_right_laser" type="fixed">
-    <origin xyz="-0.07 -0.76 0.27" rpy="0.0 0.0 -0.7854"/>
+    <origin xyz="-0.000862088969066 -0.705210390319 0.264663856731" rpy="-0.230924786805 0.192190273954 -0.772049154946"/>
     <parent link="base_link"/>
     <child link="right_laser"/>
@@ -249,5 +249,5 @@
   <link name="left_laser">
     <inertial>
-      <origin xyz="0.0 0.0 0.0" rpy="0 0 0"/>
+      <origin xyz="0.0 0.0 0.0" rpy="0.0 0.0 0.0"/>
       <mass value="1.1"/>
       <inertia ixx="0.00307156543804" ixy="0.0" ixz="0.0" iyy="0.00312849041527" iyz="0.0" izz="0.00196432421427"/>
@@ -299,5 +299,5 @@
   </gazebo>
   <joint name="base_link_to_left_laser" type="fixed">
-    <origin xyz="-0.07 0.76 0.27" rpy="0.0 -0.0 0.7854"/>
+    <origin xyz="-0.117991998792 0.781257987022 0.221049308777" rpy="0.221184457878 0.179632028343 0.918589581792"/>
     <parent link="base_link"/>
     <child link="left_laser"/>
@@ -347,5 +347,5 @@
   <link name="top_center_rgbd_camera_rgb_optical_frame"/>
   <joint name="base_link_to_top_center_rgbd_camera" type="fixed">
-    <origin xyz="-1.51 -0.01 1.338" rpy="0.0 0.207 0.0"/>
+    <origin xyz="-1.51 -0.01 1.338" rpy="-0.0 0.207 -0.0"/>
     <parent link="base_link"/>
     <child link="top_center_rgbd_camera_link"/>

File: interactive_calibration/calibrations/atlascar2/optimized.urdf.xacro (robot description, xacro)
@@ -84,5 +84,5 @@
   </gazebo>
   <joint name="base_link_to_top_right_camera" type="fixed">
-    <origin xyz="-1.53423238886 -0.236720836088 1.31835582197" rpy="-0.0117981741948 0.386468749713 -0.00898751586873"/>
+    <origin xyz="-1.52545705881 -0.234616836053 1.36126320471" rpy="-0.022569779172 0.396104847692 -0.0142500465895"/>
     <parent link="base_link"/>
     <child link="top_right_camera"/>
@@ -151,5 +151,5 @@
   </gazebo>
   <joint name="base_link_to_top_left_camera" type="fixed">
-    <origin xyz="-1.55 0.22 1.35" rpy="2.30612405754e-16 0.399999183858 -1.63927875103e-16"/>
+    <origin xyz="-1.55 0.22 1.35" rpy="-2.16414926544e-16 0.399999183858 -8.97421780096e-17"/>
     <parent link="base_link"/>
     <child link="top_left_camera"/>
@@ -157,5 +157,5 @@
   <link name="frontal_laser_mount_link">
     <inertial>
-      <origin xyz="0.0 0.0 0.0" rpy="0 0 0"/>
+      <origin xyz="0.0 0.0 0.0" rpy="0.0 0.0 0.0"/>
       <mass value="0.001"/>
       <inertia ixx="1e-06" ixy="0.0" ixz="0.0" iyy="1e-06" iyz="0.0" izz="1e-06"/>
@@ -169,5 +169,5 @@
   <link name="frontal_laser">
     <inertial>
-      <origin xyz="0.0026 -0.02325 -0.0" rpy="0 0 0"/>
+      <origin xyz="0.0026 -0.02325 -0.0" rpy="0.0 0.0 0.0"/>
       <mass value="1.0"/>
       <inertia ixx="0.00290035300653" ixy="0.0" ixz="0.0" iyy="0.00136918611899" iyz="0.0" izz="0.00297887297512"/>
@@ -193,5 +193,5 @@
   <link name="right_laser">
     <inertial>
-      <origin xyz="0.0 0.0 0.0" rpy="0 0 0"/>
+      <origin xyz="0.0 0.0 0.0" rpy="0.0 0.0 0.0"/>
       <mass value="1.1"/>
       <inertia ixx="0.00307156543804" ixy="0.0" ixz="0.0" iyy="0.00312849041527" iyz="0.0" izz="0.00196432421427"/>
@@ -243,5 +243,5 @@
   </gazebo>
   <joint name="base_link_to_right_laser" type="fixed">
-    <origin xyz="-0.0121436674251 -0.712532742873 0.260000102267" rpy="-0.0187159454145 0.302001556776 -0.746752860587"/>
+    <origin xyz="-0.000862088969066 -0.705210390319 0.264663856731" rpy="-0.230924786805 0.192190273954 -0.772049154946"/>
     <parent link="base_link"/>
     <child link="right_laser"/>
@@ -249,5 +249,5 @@
   <link name="left_laser">
     <inertial>
-      <origin xyz="0.0 0.0 0.0" rpy="0 0 0"/>
+      <origin xyz="0.0 0.0 0.0" rpy="0.0 0.0 0.0"/>
       <mass value="1.1"/>
       <inertia ixx="0.00307156543804" ixy="0.0" ixz="0.0" iyy="0.00312849041527" iyz="0.0" izz="0.00196432421427"/>
@@ -299,5 +299,5 @@
   </gazebo>
   <joint name="base_link_to_left_laser" type="fixed">
-    <origin xyz="-0.128566476578 0.78830472507 0.260011141723" rpy="0.00013364861577 0.279225582292 0.897002730585"/>
+    <origin xyz="-0.11799199707 0.78125795997 0.265856295369" rpy="0.221184458621 0.17963204854 0.918589541443"/>
     <parent link="base_link"/>
     <child link="left_laser"/>

Commit message: Huge commit, adjusting atlas-core repo to proper naming conventions. Repo now is called atlascar2

File: interactive_calibration/calibrations/atlascar2/first_guess.urdf.xacro (robot description, xacro)
@@ -7,5 +7,5 @@
       <origin xyz="-0.9 0.0 0.0" rpy="0.0 0.0 0.0"/>
       <geometry>
-        <mesh filename="package://atlas2_description/meshes/mitsubishi_miev.dae"/>
+        <mesh filename="package://atlascar2_description/meshes/mitsubishi_miev.dae"/>
       </geometry>
     </visual>
@@ -312,11 +312,11 @@
       <origin xyz="0.0 0.0 0.0" rpy="0.0 0.0 0.0"/>
       <geometry>
-        <mesh filename="package://atlas2_description/meshes/asus_xtion/asus_xtion_simple.dae"/>
-      </geometry>
-    </visual>
-    <collision>
-      <origin xyz="0.0 0.0 0.0" rpy="0.0 0.0 0.0"/>
-      <geometry>
-        <mesh filename="package://atlas2_description/meshes/asus_xtion/asus_xtion_simple.dae"/>
+        <mesh filename="package://atlascar2_description/meshes/asus_xtion/asus_xtion_simple.dae"/>
+      </geometry>
+    </visual>
+    <collision>
+      <origin xyz="0.0 0.0 0.0" rpy="0.0 0.0 0.0"/>
+      <geometry>
+        <mesh filename="package://atlascar2_description/meshes/asus_xtion/asus_xtion_simple.dae"/>
       </geometry>
     </collision>

File: interactive_calibration/calibrations/atlascar2/optimized.urdf.xacro (robot description, xacro)
@@ -7,5 +7,5 @@
       <origin xyz="-0.9 0.0 0.0" rpy="0.0 0.0 0.0"/>
       <geometry>
-        <mesh filename="package://atlas2_description/meshes/mitsubishi_miev.dae"/>
+        <mesh filename="package://atlascar2_description/meshes/mitsubishi_miev.dae"/>
       </geometry>
     </visual>
@@ -312,11 +312,11 @@
       <origin xyz="0.0 0.0 0.0" rpy="0.0 0.0 0.0"/>
       <geometry>
-        <mesh filename="package://atlas2_description/meshes/asus_xtion/asus_xtion_simple.dae"/>
-      </geometry>
-    </visual>
-    <collision>
-      <origin xyz="0.0 0.0 0.0" rpy="0.0 0.0 0.0"/>
-      <geometry>
-        <mesh filename="package://atlas2_description/meshes/asus_xtion/asus_xtion_simple.dae"/>
+        <mesh filename="package://atlascar2_description/meshes/asus_xtion/asus_xtion_simple.dae"/>
+      </geometry>
+    </visual>
+    <collision>
+      <origin xyz="0.0 0.0 0.0" rpy="0.0 0.0 0.0"/>
+      <geometry>
+        <mesh filename="package://atlascar2_description/meshes/asus_xtion/asus_xtion_simple.dae"/>
       </geometry>
     </collision>
