Commit message: #92 implemented. Xacro is saved after optimization. To launch calibration.launch reading this xacro use "read_optimized:=true"

File: interactive_calibration/calibrations/atlascar2/optimized.urdf.xacro (robot description, xacro)
@@ -84,5 +84,5 @@
   </gazebo>
   <joint name="base_link_to_top_right_camera" type="fixed">
-    <origin xyz="-1.54999995232 -0.219999998808 1.40112948418" rpy="-1.08223780011e-08 0.164151666864 -6.43161410219e-09"/>
+    <origin xyz="-1.5291061047 -0.225538555347 1.36850099501" rpy="-0.00925000790269 0.215344433787 -0.00657024505815"/>
     <parent link="base_link"/>
     <child link="top_right_camera"/>
@@ -151,5 +151,5 @@
   </gazebo>
   <joint name="base_link_to_top_left_camera" type="fixed">
-    <origin xyz="-1.54999995232 0.219999998808 1.38210916519" rpy="-1.49597710582e-08 0.173506001022 -5.12355388858e-09"/>
+    <origin xyz="-1.55 0.22 1.35" rpy="1.7239703778e-16 0.198720401856 2.05590041181e-16"/>
     <parent link="base_link"/>
     <child link="top_left_camera"/>
@@ -157,5 +157,5 @@
   <link name="frontal_laser_mount_link">
     <inertial>
-      <origin xyz="0.0 0.0 0.0" rpy="0 0 0"/>
+      <origin xyz="0.0 0.0 0.0" rpy="0.0 0.0 0.0"/>
       <mass value="0.001"/>
       <inertia ixx="1e-06" ixy="0.0" ixz="0.0" iyy="1e-06" iyz="0.0" izz="1e-06"/>
@@ -169,5 +169,5 @@
   <link name="frontal_laser">
     <inertial>
-      <origin xyz="0.0026 -0.02325 -0.0" rpy="0 0 0"/>
+      <origin xyz="0.0026 -0.02325 -0.0" rpy="0.0 0.0 0.0"/>
       <mass value="1.0"/>
       <inertia ixx="0.00290035300653" ixy="0.0" ixz="0.0" iyy="0.00136918611899" iyz="0.0" izz="0.00297887297512"/>
@@ -193,5 +193,5 @@
   <link name="right_laser">
     <inertial>
-      <origin xyz="0.0 0.0 0.0" rpy="0 0 0"/>
+      <origin xyz="0.0 0.0 0.0" rpy="0.0 0.0 0.0"/>
       <mass value="1.1"/>
       <inertia ixx="0.00307156543804" ixy="0.0" ixz="0.0" iyy="0.00312849041527" iyz="0.0" izz="0.00196432421427"/>
@@ -243,5 +243,5 @@
   </gazebo>
   <joint name="base_link_to_right_laser" type="fixed">
-    <origin xyz="-0.07 -0.76 0.27" rpy="0.0 0.0 -0.7854"/>
+    <origin xyz="0.179742917301 -0.69673643837 0.265032392537" rpy="0.0459109423755 0.0368123724128 -0.762021376598"/>
     <parent link="base_link"/>
     <child link="right_laser"/>
@@ -249,5 +249,5 @@
   <link name="left_laser">
     <inertial>
-      <origin xyz="0.0 0.0 0.0" rpy="0 0 0"/>
+      <origin xyz="0.0 0.0 0.0" rpy="0.0 0.0 0.0"/>
       <mass value="1.1"/>
       <inertia ixx="0.00307156543804" ixy="0.0" ixz="0.0" iyy="0.00312849041527" iyz="0.0" izz="0.00196432421427"/>
@@ -299,5 +299,5 @@
   </gazebo>
   <joint name="base_link_to_left_laser" type="fixed">
-    <origin xyz="-0.07 0.76 0.27" rpy="0.0 -0.0 0.7854"/>
+    <origin xyz="0.107754360787 0.841098973506 0.265151192745" rpy="0.0639047713977 -0.0108214584815 0.873585779517"/>
     <parent link="base_link"/>
     <child link="left_laser"/>

Commit message: A lot of stuff. Refarctoring. Reading chessboard parameters from calibration_config.json, rather than command line arguments. Related issues: #60

File: interactive_calibration/calibrations/atlascar2/optimized.urdf.xacro (robot description, xacro)
@@ -84,5 +84,5 @@
   </gazebo>
   <joint name="base_link_to_top_right_camera" type="fixed">
-    <origin xyz="-1.5291061047 -0.225538555347 1.36850099501" rpy="-0.00925000790269 0.215344433787 -0.00657024505815"/>
+    <origin xyz="-1.49884228618 -0.238544097849 1.37837300009" rpy="-0.00819751684561 0.219479998536 -0.00467927025547"/>
     <parent link="base_link"/>
     <child link="top_right_camera"/>
@@ -151,5 +151,5 @@
   </gazebo>
   <joint name="base_link_to_top_left_camera" type="fixed">
-    <origin xyz="-1.55 0.22 1.35" rpy="1.7239703778e-16 0.198720401856 2.05590041181e-16"/>
+    <origin xyz="-1.55 0.22 1.35" rpy="1.75049115904e-16 0.198720401856 1.54943559518e-16"/>
     <parent link="base_link"/>
     <child link="top_left_camera"/>
@@ -243,5 +243,5 @@
   </gazebo>
   <joint name="base_link_to_right_laser" type="fixed">
-    <origin xyz="0.179742917301 -0.69673643837 0.265032392537" rpy="0.0459109423755 0.0368123724128 -0.762021376598"/>
+    <origin xyz="-0.561389488206 -0.775677838173 0.279871683968" rpy="-0.483993663665 0.0875468157422 -0.244101862115"/>
     <parent link="base_link"/>
     <child link="right_laser"/>
@@ -299,5 +299,5 @@
   </gazebo>
   <joint name="base_link_to_left_laser" type="fixed">
-    <origin xyz="0.107754360787 0.841098973506 0.265151192745" rpy="0.0639047713977 -0.0108214584815 0.873585779517"/>
+    <origin xyz="0.0529260416624 1.69699480591 0.279931019861" rpy="0.303682129396 0.155716535888 0.207176080297"/>
     <parent link="base_link"/>
     <child link="left_laser"/>

Commit message: Close #93. New laser beam error computed and validated with images and optimizations.

File: interactive_calibration/calibrations/atlascar2/optimized.urdf.xacro (robot description, xacro)
@@ -84,5 +84,5 @@
   </gazebo>
   <joint name="base_link_to_top_right_camera" type="fixed">
-    <origin xyz="-1.49884228618 -0.238544097849 1.37837300009" rpy="-0.00819751684561 0.219479998536 -0.00467927025547"/>
+    <origin xyz="-1.55 -0.22 1.35" rpy="-0.0 0.227300133871 -0.0"/>
     <parent link="base_link"/>
     <child link="top_right_camera"/>
@@ -151,5 +151,5 @@
   </gazebo>
   <joint name="base_link_to_top_left_camera" type="fixed">
-    <origin xyz="-1.55 0.22 1.35" rpy="1.75049115904e-16 0.198720401856 1.54943559518e-16"/>
+    <origin xyz="-1.55 0.22 1.35" rpy="5.0106362823e-18 0.198720401856 -4.36421700435e-19"/>
     <parent link="base_link"/>
     <child link="top_left_camera"/>
@@ -157,5 +157,5 @@
   <link name="frontal_laser_mount_link">
     <inertial>
-      <origin xyz="0.0 0.0 0.0" rpy="0.0 0.0 0.0"/>
+      <origin xyz="0.0 0.0 0.0" rpy="0 0 0"/>
       <mass value="0.001"/>
       <inertia ixx="1e-06" ixy="0.0" ixz="0.0" iyy="1e-06" iyz="0.0" izz="1e-06"/>
@@ -169,5 +169,5 @@
   <link name="frontal_laser">
     <inertial>
-      <origin xyz="0.0026 -0.02325 -0.0" rpy="0.0 0.0 0.0"/>
+      <origin xyz="0.0026 -0.02325 -0.0" rpy="0 0 0"/>
       <mass value="1.0"/>
       <inertia ixx="0.00290035300653" ixy="0.0" ixz="0.0" iyy="0.00136918611899" iyz="0.0" izz="0.00297887297512"/>
@@ -193,5 +193,5 @@
   <link name="right_laser">
     <inertial>
-      <origin xyz="0.0 0.0 0.0" rpy="0.0 0.0 0.0"/>
+      <origin xyz="0.0 0.0 0.0" rpy="0 0 0"/>
       <mass value="1.1"/>
       <inertia ixx="0.00307156543804" ixy="0.0" ixz="0.0" iyy="0.00312849041527" iyz="0.0" izz="0.00196432421427"/>
@@ -243,5 +243,5 @@
   </gazebo>
   <joint name="base_link_to_right_laser" type="fixed">
-    <origin xyz="-0.561389488206 -0.775677838173 0.279871683968" rpy="-0.483993663665 0.0875468157422 -0.244101862115"/>
+    <origin xyz="0.0132202017686 -0.885333931027 0.273334977076" rpy="0.580334645239 -0.24657385509 -0.688003861727"/>
     <parent link="base_link"/>
     <child link="right_laser"/>
@@ -249,5 +249,5 @@
   <link name="left_laser">
     <inertial>
-      <origin xyz="0.0 0.0 0.0" rpy="0.0 0.0 0.0"/>
+      <origin xyz="0.0 0.0 0.0" rpy="0 0 0"/>
       <mass value="1.1"/>
       <inertia ixx="0.00307156543804" ixy="0.0" ixz="0.0" iyy="0.00312849041527" iyz="0.0" izz="0.00196432421427"/>
@@ -299,5 +299,5 @@
   </gazebo>
   <joint name="base_link_to_left_laser" type="fixed">
-    <origin xyz="0.0529260416624 1.69699480591 0.279931019861" rpy="0.303682129396 0.155716535888 0.207176080297"/>
+    <origin xyz="-0.07 0.76 0.27" rpy="-0.0 0.0 0.944289442264"/>
     <parent link="base_link"/>
     <child link="left_laser"/>
@@ -347,5 +347,5 @@
   <link name="top_center_rgbd_camera_rgb_optical_frame"/>
   <joint name="base_link_to_top_center_rgbd_camera" type="fixed">
-    <origin xyz="-1.51 -0.01 1.338" rpy="0.0 0.207 0.0"/>
+    <origin xyz="-1.51 -0.01 1.338" rpy="-0.0 0.207 -0.0"/>
     <parent link="base_link"/>
     <child link="top_center_rgbd_camera_link"/>

Commit message: Close #105. Implemented.

File: interactive_calibration/calibrations/atlascar2/optimized.urdf.xacro (robot description, xacro)
@@ -84,5 +84,5 @@
   </gazebo>
   <joint name="base_link_to_top_right_camera" type="fixed">
-    <origin xyz="-1.55 -0.22 1.35" rpy="-0.0 0.227300133871 -0.0"/>
+    <origin xyz="-1.55 -0.22 1.35" rpy="-0.0 0.399999183858 -0.0"/>
     <parent link="base_link"/>
     <child link="top_right_camera"/>
@@ -151,5 +151,5 @@
   </gazebo>
   <joint name="base_link_to_top_left_camera" type="fixed">
-    <origin xyz="-1.55 0.22 1.35" rpy="5.0106362823e-18 0.198720401856 -4.36421700435e-19"/>
+    <origin xyz="-1.55 0.22 1.35" rpy="-5.12018340835e-19 0.399999183858 -5.87444891709e-19"/>
     <parent link="base_link"/>
     <child link="top_left_camera"/>
@@ -243,5 +243,5 @@
   </gazebo>
   <joint name="base_link_to_right_laser" type="fixed">
-    <origin xyz="0.0132202017686 -0.885333931027 0.273334977076" rpy="0.580334645239 -0.24657385509 -0.688003861727"/>
+    <origin xyz="-0.0698918431156 -0.760661358765 0.26005" rpy="-0.000621349019053 0.0010885400895 -0.785555100415"/>
     <parent link="base_link"/>
     <child link="right_laser"/>
@@ -299,5 +299,5 @@
   </gazebo>
   <joint name="base_link_to_left_laser" type="fixed">
-    <origin xyz="-0.07 0.76 0.27" rpy="-0.0 0.0 0.944289442264"/>
+    <origin xyz="-0.07 0.76 0.27" rpy="-0.0 0.0 0.785399619817"/>
     <parent link="base_link"/>
     <child link="left_laser"/>

Commit message: #113. Checking if max_delta is within threshold only if max_delta is not None.

File: interactive_calibration/calibrations/atlascar2/optimized.urdf.xacro (robot description, xacro)
@@ -84,5 +84,5 @@
   </gazebo>
   <joint name="base_link_to_top_right_camera" type="fixed">
-    <origin xyz="-1.55 -0.22 1.35" rpy="-0.0 0.399999183858 -0.0"/>
+    <origin xyz="-1.53423238886 -0.236720836088 1.31835582197" rpy="-0.0117981741948 0.386468749713 -0.00898751586873"/>
     <parent link="base_link"/>
     <child link="top_right_camera"/>
@@ -151,5 +151,5 @@
   </gazebo>
   <joint name="base_link_to_top_left_camera" type="fixed">
-    <origin xyz="-1.55 0.22 1.35" rpy="-5.12018340835e-19 0.399999183858 -5.87444891709e-19"/>
+    <origin xyz="-1.55 0.22 1.35" rpy="2.30612405754e-16 0.399999183858 -1.63927875103e-16"/>
     <parent link="base_link"/>
     <child link="top_left_camera"/>
@@ -243,5 +243,5 @@
   </gazebo>
   <joint name="base_link_to_right_laser" type="fixed">
-    <origin xyz="-0.0698918431156 -0.760661358765 0.26005" rpy="-0.000621349019053 0.0010885400895 -0.785555100415"/>
+    <origin xyz="-0.0121436674251 -0.712532742873 0.260000102267" rpy="-0.0187159454145 0.302001556776 -0.746752860587"/>
     <parent link="base_link"/>
     <child link="right_laser"/>
@@ -299,5 +299,5 @@
   </gazebo>
   <joint name="base_link_to_left_laser" type="fixed">
-    <origin xyz="-0.07 0.76 0.27" rpy="-0.0 0.0 0.785399619817"/>
+    <origin xyz="-0.128566476578 0.78830472507 0.260011141723" rpy="0.00013364861577 0.279225582292 0.897002730585"/>
     <parent link="base_link"/>
     <child link="left_laser"/>

Commit message: intrinsics change

File: interactive_calibration/calibrations/atlascar2/optimized.urdf.xacro (robot description, xacro)
@@ -84,5 +84,5 @@
   </gazebo>
   <joint name="base_link_to_top_right_camera" type="fixed">
-    <origin xyz="-1.52545705881 -0.234616836053 1.36126320471" rpy="-0.022569779172 0.396104847692 -0.0142500465895"/>
+    <origin xyz="-1.44941343554 -0.264648436899 1.36662485139" rpy="-0.0230837440638 0.204288550398 -0.00524768479513"/>
     <parent link="base_link"/>
     <child link="top_right_camera"/>
@@ -151,5 +151,5 @@
   </gazebo>
   <joint name="base_link_to_top_left_camera" type="fixed">
-    <origin xyz="-1.55 0.22 1.35" rpy="-2.16414926544e-16 0.399999183858 -8.97421780096e-17"/>
+    <origin xyz="-1.55 0.22 1.35" rpy="-2.26106716838e-17 0.198720401856 -1.50605934828e-17"/>
     <parent link="base_link"/>
     <child link="top_left_camera"/>
@@ -157,5 +157,5 @@
   <link name="frontal_laser_mount_link">
     <inertial>
-      <origin xyz="0.0 0.0 0.0" rpy="0.0 0.0 0.0"/>
+      <origin xyz="0.0 0.0 0.0" rpy="0 0 0"/>
       <mass value="0.001"/>
       <inertia ixx="1e-06" ixy="0.0" ixz="0.0" iyy="1e-06" iyz="0.0" izz="1e-06"/>
@@ -169,5 +169,5 @@
   <link name="frontal_laser">
     <inertial>
-      <origin xyz="0.0026 -0.02325 -0.0" rpy="0.0 0.0 0.0"/>
+      <origin xyz="0.0026 -0.02325 -0.0" rpy="0 0 0"/>
       <mass value="1.0"/>
       <inertia ixx="0.00290035300653" ixy="0.0" ixz="0.0" iyy="0.00136918611899" iyz="0.0" izz="0.00297887297512"/>
@@ -193,5 +193,5 @@
   <link name="right_laser">
     <inertial>
-      <origin xyz="0.0 0.0 0.0" rpy="0.0 0.0 0.0"/>
+      <origin xyz="0.0 0.0 0.0" rpy="0 0 0"/>
       <mass value="1.1"/>
       <inertia ixx="0.00307156543804" ixy="0.0" ixz="0.0" iyy="0.00312849041527" iyz="0.0" izz="0.00196432421427"/>
@@ -243,5 +243,5 @@
   </gazebo>
   <joint name="base_link_to_right_laser" type="fixed">
-    <origin xyz="-0.000862088969066 -0.705210390319 0.264663856731" rpy="-0.230924786805 0.192190273954 -0.772049154946"/>
+    <origin xyz="-0.07 -0.76 0.27" rpy="0.0 0.0 -0.682778722838"/>
     <parent link="base_link"/>
     <child link="right_laser"/>
@@ -249,5 +249,5 @@
   <link name="left_laser">
     <inertial>
-      <origin xyz="0.0 0.0 0.0" rpy="0.0 0.0 0.0"/>
+      <origin xyz="0.0 0.0 0.0" rpy="0 0 0"/>
       <mass value="1.1"/>
       <inertia ixx="0.00307156543804" ixy="0.0" ixz="0.0" iyy="0.00312849041527" iyz="0.0" izz="0.00196432421427"/>
@@ -299,5 +299,5 @@
   </gazebo>
   <joint name="base_link_to_left_laser" type="fixed">
-    <origin xyz="-0.11799199707 0.78125795997 0.265856295369" rpy="0.221184458621 0.17963204854 0.918589541443"/>
+    <origin xyz="-0.07 0.76 0.27" rpy="0.0 -0.0 0.944289442264"/>
     <parent link="base_link"/>
     <child link="left_laser"/>
