Commit message: Add a pattern mesh. Update xacros. Use cross and circles to show detected corners.

File: interactive_calibration/calibrations/ur10e/both_eyes/ur10e.urdf.xacro (robot description, xacro)
@@ -17,2 +17,25 @@
     </joint>
 </robot>
+<robot xmlns:xacro="http://ros.org/wiki/xacro"
+       name="ur10e" >
+  <xacro:include filename="$(find ur_e_description)/urdf/common.gazebo.xacro" />
+  <xacro:include filename="$(find ur_e_description)/urdf/ur10e.urdf.xacro" />
+  <xacro:ur10e_robot prefix="" joint_limited="false"/>
+  <xacro:include filename="$(find ur_e_description)/urdf/astra.urdf.xacro" />
+  <xacro:sensor_astra parent="ee_link" prefix="camera">
+      <!-- NOTE: CHANGE THIS -->
+      <origin xyz="0 0 0" rpy="${pi} 0 0"/>
+      <!-- <origin xyz="0.041311319304504816 -0.06402544453787727 0.044527571211305426" rpy="3.13766148064 -0.00787797070144 0.000110993634886"/> -->
+  </xacro:sensor_astra>
+  <xacro:sensor_astra parent="base_link" prefix="kinect">
+      <!-- NOTE: CHANGE THIS -->
+        <origin xyz="0.9 0.4 0.6" rpy="0 0.57 2.19"/>
+      <!-- <origin xyz="0.041311319304504816 -0.06402544453787727 0.044527571211305426" rpy="3.13766148064 -0.00787797070144 0.000110993634886"/> -->
+  </xacro:sensor_astra>
+  <link name="world" />
+  <joint name="world_joint" type="fixed">
+    <parent link="world" />
+    <child link = "base_link" />
+    <origin xyz="0.0 0.0 0.0" rpy="0.0 0.0 0.0" />
+  </joint>
+</robot>

File: interactive_calibration/calibrations/ur10e/eye_in_hand/ur10e.urdf.xacro (robot description, xacro)
@@ -1,18 +1,19 @@
 <?xml version="1.0"?>
-<robot xmlns:xacro="http://www.ros.org/wiki/xacro" name="ur10e_and_camera">
-    <xacro:include filename="$(find ur_e_description)/urdf/ur10e_joint_limited_robot.urdf.xacro" />
-    <link name="camera_link" />
-    <joint name="camera_joint" type="fixed">
-        <parent link="ee_link"  />
-        <child  link="camera_link"/>
-        <!-- <origin xyz="0 0 0" rpy="3.14159 0 0"/> -->
-        <origin xyz="0.04180196863432179 -0.06175451218256622 0.04753730432804916" rpy="3.13875839937 -0.014541476237 -0.00490489873721"/>
-        <!-- <origin xyz="0.04243085438717736 -0.0617936577879632 0.047406912654841836" rpy="3.1392599224 -0.0144165350185 -0.00496869013782"/> -->
-        <!-- <origin xyz="0.028 -0.06042073982785581 0.04404998419530226" rpy="-3.13882006844 -0.0111143081021 -0.016374601036"/> -->
-        <!-- <origin xyz="-0.0062457294067694916 -0.05731410920995202 0.04361176276990688" rpy="-3.13949475085 -0.0138658614135 -0.00757430945153"/> -->
-        <!-- <origin xyz="-0.008822707453233472 -0.06332039688055228 0.041509902112571245" rpy="-3.14041065678 -0.0142453212306 0.00227888982265"/> -->
-        <!-- <origin xyz="-0.009810813473970764 -0.06283651025908535 0.0410679928911672" rpy="-3.14046952157 -0.0146242521676 0.000841765326346"/> -->
-        <!-- <origin xyz="-0.006197630434814864 -0.05712333621274038 0.04200309311231139" rpy="-3.14146336277 -0.0164354868577 -0.00893770193716"/> -->
-        <!-- <origin xyz="-0.005533759820772154 -0.05820819881411328 0.040155992199870344" rpy="-3.13976600744 -0.0197606039146 -0.00736772190622"/> -->
-    </joint>
+<robot xmlns:xacro="http://ros.org/wiki/xacro"
+       name="ur10e" >
+  <xacro:include filename="$(find ur_e_description)/urdf/common.gazebo.xacro" />
+  <xacro:include filename="$(find ur_e_description)/urdf/ur10e.urdf.xacro" />
+  <xacro:ur10e_robot prefix="" joint_limited="false"/>
+  <xacro:include filename="$(find ur_e_description)/urdf/astra.urdf.xacro" />
+  <xacro:sensor_astra parent="ee_link" prefix="camera">
+      <!-- NOTE: CHANGE THIS -->
+      <origin xyz="0 0 0" rpy="${pi} 0 0"/>
+      <!-- <origin xyz="0.041311319304504816 -0.06402544453787727 0.044527571211305426" rpy="3.13766148064 -0.00787797070144 0.000110993634886"/> -->
+  </xacro:sensor_astra>
+  <link name="world" />
+  <joint name="world_joint" type="fixed">
+    <parent link="world" />
+    <child link = "base_link" />
+    <origin xyz="0.0 0.0 0.0" rpy="0.0 0.0 0.0" />
+  </joint>
 </robot>

File: interactive_calibration/calibrations/ur10e/eye_in_hand_chess/ur10e.urdf.xacro (robot description, xacro)
@@ -1,18 +1,19 @@
 <?xml version="1.0"?>
-<robot xmlns:xacro="http://www.ros.org/wiki/xacro" name="ur10e_and_camera">
-    <xacro:include filename="$(find ur_e_description)/urdf/ur10e_joint_limited_robot.urdf.xacro" />
-    <link name="camera_link" />
-    <joint name="camera_joint" type="fixed">
-        <parent link="ee_link"  />
-        <child  link="camera_link"/>
-        <origin xyz="0 0 0" rpy="3.14159 0 0"/>
-        <!-- <origin xyz="0.04180196863432179 -0.06175451218256622 0.04753730432804916" rpy="3.13875839937 -0.014541476237 -0.00490489873721"/> -->
-        <!-- <origin xyz="0.04243085438717736 -0.0617936577879632 0.047406912654841836" rpy="3.1392599224 -0.0144165350185 -0.00496869013782"/> -->
-        <!-- <origin xyz="0.028 -0.06042073982785581 0.04404998419530226" rpy="-3.13882006844 -0.0111143081021 -0.016374601036"/> -->
-        <!-- <origin xyz="-0.0062457294067694916 -0.05731410920995202 0.04361176276990688" rpy="-3.13949475085 -0.0138658614135 -0.00757430945153"/> -->
-        <!-- <origin xyz="-0.008822707453233472 -0.06332039688055228 0.041509902112571245" rpy="-3.14041065678 -0.0142453212306 0.00227888982265"/> -->
-        <!-- <origin xyz="-0.009810813473970764 -0.06283651025908535 0.0410679928911672" rpy="-3.14046952157 -0.0146242521676 0.000841765326346"/> -->
-        <!-- <origin xyz="-0.006197630434814864 -0.05712333621274038 0.04200309311231139" rpy="-3.14146336277 -0.0164354868577 -0.00893770193716"/> -->
-        <!-- <origin xyz="-0.005533759820772154 -0.05820819881411328 0.040155992199870344" rpy="-3.13976600744 -0.0197606039146 -0.00736772190622"/> -->
-    </joint>
+<robot xmlns:xacro="http://ros.org/wiki/xacro"
+       name="ur10e" >
+  <xacro:include filename="$(find ur_e_description)/urdf/common.gazebo.xacro" />
+  <xacro:include filename="$(find ur_e_description)/urdf/ur10e.urdf.xacro" />
+  <xacro:ur10e_robot prefix="" joint_limited="false"/>
+  <xacro:include filename="$(find ur_e_description)/urdf/astra.urdf.xacro" />
+  <xacro:sensor_astra parent="ee_link" prefix="camera">
+      <!-- NOTE: CHANGE THIS -->
+      <origin xyz="0 0 0" rpy="${pi} 0 0"/>
+      <!-- <origin xyz="0.041311319304504816 -0.06402544453787727 0.044527571211305426" rpy="3.13766148064 -0.00787797070144 0.000110993634886"/> -->
+  </xacro:sensor_astra>
+  <link name="world" />
+  <joint name="world_joint" type="fixed">
+    <parent link="world" />
+    <child link = "base_link" />
+    <origin xyz="0.0 0.0 0.0" rpy="0.0 0.0 0.0" />
+  </joint>
 </robot>

File: interactive_calibration/calibrations/ur10e/eye_to_base/ur10e.urdf.xacro (robot description, xacro)
@@ -1,14 +1,19 @@
 <?xml version="1.0"?>
-<robot xmlns:xacro="http://www.ros.org/wiki/xacro" name="ur10e_and_camera">
-    <xacro:include filename="$(find ur_e_description)/urdf/ur10e_joint_limited_robot.urdf.xacro" />
-    <link name="camera_link" />
-    <joint name="camera_joint" type="fixed">
-        <parent link="base_link"  />
-        <child  link="camera_link"/>
-        <!-- <origin xyz="0.9 0.15 0.5" rpy="0 0.5 2"/> -->
-        <!-- <origin xyz="0.9389990132510372 0.16275628223934924 0.6772718894032261" rpy="0.022279862745 0.563324514996 2.1726142738"/> -->
-        <origin xyz="0.9428549486249146 0.16352956421669793 0.6776344875119994" rpy="0.0255369171865 0.56343124593 2.17569355621"/>
-        <!-- <origin xyz="0.9402073721290084 0.1783001607979796 0.6816250550635298" rpy="0.04493490584157748 0.5742330193173137 2.1978793783108284"/> -->
-        <!-- <origin xyz="0.9489211526634104 0.1792115439633525 0.6842998069879084" rpy="0.0443204555056 0.570345606354 2.19979861613"/> -->
-    </joint>
+<robot xmlns:xacro="http://ros.org/wiki/xacro"
+       name="ur10e" >
+  <xacro:include filename="$(find ur_e_description)/urdf/common.gazebo.xacro" />
+  <xacro:include filename="$(find ur_e_description)/urdf/ur10e.urdf.xacro" />
+  <xacro:ur10e_robot prefix="" joint_limited="false"/>
+  <xacro:include filename="$(find ur_e_description)/urdf/astra.urdf.xacro" />
+  <xacro:sensor_astra parent="ee_link" prefix="camera">
+      <!-- NOTE: CHANGE THIS -->
+      <origin xyz="0 0 0" rpy="${pi} 0 0"/>
+      <!-- <origin xyz="0.041311319304504816 -0.06402544453787727 0.044527571211305426" rpy="3.13766148064 -0.00787797070144 0.000110993634886"/> -->
+  </xacro:sensor_astra>
+  <link name="world" />
+  <joint name="world_joint" type="fixed">
+    <parent link="world" />
+    <child link = "base_link" />
+    <origin xyz="0.0 0.0 0.0" rpy="0.0 0.0 0.0" />
+  </joint>
 </robot>

Commit message: Add several changes to configurations. Add multi-cam error viewer.

File: interactive_calibration/calibrations/ur10e/both_eyes/ur10e.urdf.xacro (robot description, xacro)
@@ -1,20 +1,3 @@
 <?xml version="1.0"?>
-<robot xmlns:xacro="http://www.ros.org/wiki/xacro" name="ur10e_and_camera">
-    <xacro:include filename="$(find ur_e_description)/urdf/ur10e_joint_limited_robot.urdf.xacro" />
-    <link name="astra_link" />
-    <link name="kinect_link" />
-    <joint name="astra_eef_joint" type="fixed">
-        <parent link="ee_link"  />
-        <child  link="astra_link"/>
-        <!-- <origin xyz="0 0 0" rpy="${pi} 0 0"/> -->
-        <origin xyz="-0.010072508540529695 -0.054375082786612516 0.05082669214682842" rpy="-3.14094648692 0.00286920281033 -0.0224607343716"/>
-    </joint>
-    <joint name="kinect_base_joint" type="fixed">
-        <parent link="base_link"  />
-        <child  link="kinect_link"/>
-        <!-- <origin xyz="0.9 0.4 0.6" rpy="0 0.57 2.19"/> -->
-        <origin xyz="0.8131271808015654 0.48037067110684883 0.6644448706526455" rpy="0.0451004185296 0.734284415686 2.35154965264"/>
-    </joint>
-</robot>
 <robot xmlns:xacro="http://ros.org/wiki/xacro"
        name="ur10e" >
@@ -23,5 +6,5 @@
   <xacro:ur10e_robot prefix="" joint_limited="false"/>
   <xacro:include filename="$(find ur_e_description)/urdf/astra.urdf.xacro" />
-  <xacro:sensor_astra parent="ee_link" prefix="camera">
+  <xacro:sensor_astra parent="ee_link" prefix="astra">
       <!-- NOTE: CHANGE THIS -->
       <origin xyz="0 0 0" rpy="${pi} 0 0"/>
@@ -30,5 +13,5 @@
   <xacro:sensor_astra parent="base_link" prefix="kinect">
       <!-- NOTE: CHANGE THIS -->
-        <origin xyz="0.9 0.4 0.6" rpy="0 0.57 2.19"/>
+        <origin xyz="-0.7 0.3 0.6" rpy="-0.3 0.9 -0.5"/>
       <!-- <origin xyz="0.041311319304504816 -0.06402544453787727 0.044527571211305426" rpy="3.13766148064 -0.00787797070144 0.000110993634886"/> -->
   </xacro:sensor_astra>

File: interactive_calibration/calibrations/ur10e/eye_to_base/ur10e.urdf.xacro (robot description, xacro)
@@ -6,7 +6,7 @@
   <xacro:ur10e_robot prefix="" joint_limited="false"/>
   <xacro:include filename="$(find ur_e_description)/urdf/astra.urdf.xacro" />
-  <xacro:sensor_astra parent="ee_link" prefix="camera">
+  <xacro:sensor_astra parent="base_link" prefix="camera">
       <!-- NOTE: CHANGE THIS -->
-      <origin xyz="0 0 0" rpy="${pi} 0 0"/>
+      <origin xyz="-1 0 1" rpy="0 0 0"/>
       <!-- <origin xyz="0.041311319304504816 -0.06402544453787727 0.044527571211305426" rpy="3.13766148064 -0.00787797070144 0.000110993634886"/> -->
   </xacro:sensor_astra>
