Commit message: #617 adding colors, reducing frame rate, removing depth

File: atom_simple_examples/ase_2rgb/ase_2rgb_description/urdf/rgbd_camera.urdf.xacro (robot description, xacro)
@@ -7,5 +7,5 @@
   <xacro:property name="astra_dae_display_scale"   value="0.1" />
   <!-- Parameterised in part by the values in turtlebot_properties.urdf.xacro -->
-  <xacro:macro name="rgbd_camera" params="parent prefix *origin">
+  <xacro:macro name="rgbd_camera" params="parent prefix *origin color:='black'">
     <joint name="${prefix}_joint" type="fixed">
       <xacro:insert_block name="origin" />
@@ -14,12 +14,23 @@
     </joint>
     <link name="${prefix}_link">
-      <material>Gazebo/Red</material>
       <visual>
         <origin xyz="-0.03 -0.06 0" rpy="${pi} 0 ${pi/2}"/>
         <geometry>
+        <xacro:if value="${color == 'red'}">
+          <mesh filename="package://ase_2rgb_description/meshes/rgbd_camera/rgbd_camera_red.dae" scale="1 1 1"/>
+        </xacro:if>
+        <xacro:if value="${color == 'green'}">
+          <mesh filename="package://ase_2rgb_description/meshes/rgbd_camera/rgbd_camera_green.dae" scale="1 1 1"/>
+        </xacro:if>
+        <xacro:if value="${color == 'black'}">
           <mesh filename="package://ase_2rgb_description/meshes/rgbd_camera/rgbd_camera.dae" scale="1 1 1"/>
+        </xacro:if>
+        <xacro:if value="${color != 'red' and color != 'green' and color != 'black'}">
+          <mesh filename="package://ase_2rgb_description/meshes/rgbd_camera/rgbd_camera.dae" scale="1 1 1"/>
+        </xacro:if>
         </geometry>
       <!-- <material>Gazebo/Red</material> -->
       </visual>
+      <material>Gazebo/Red</material>
       <collision>
         <!-- <origin xyz="0.0 0.0 0.0" rpy="0 0 0" /> -->
@@ -66,5 +77,5 @@
     <link name="${prefix}_depth_optical_frame"/>
     <!-- DEPTH Camera sensor-->
-    <gazebo reference="${prefix}_depth_frame">
+    <!-- <gazebo reference="${prefix}_depth_frame">
           <sensor type="depth" name="camera">
               <always_on>true</always_on>
@@ -74,5 +85,4 @@
                   <image>
                       <format>B8G8R8</format>
-                      <!--                      <format>RGB_INT8</format>-->
                       <width>640</width>
                       <height>480</height>
@@ -93,6 +103,5 @@
                   <depthImageCameraInfoTopicName>depth/camera_info</depthImageCameraInfoTopicName>
                   <frameName>${prefix}_depth_optical_frame</frameName>
-                  <baseline>0.1</baseline>
-                  <!-- Apparently this has not effect on the rgb image. Perhaps it is use for the depth camera?-->
+                  <baseline>0.0</baseline>
                   <distortion_k1>0.0</distortion_k1>
                   <distortion_k2>0.0</distortion_k2>
@@ -103,9 +112,9 @@
               </plugin>
           </sensor>
-      </gazebo>
+      </gazebo> -->
       <!-- RGB Camera sensor-->
       <gazebo reference="${prefix}_rgb_frame">
           <sensor type="camera" name="camera">
-              <update_rate>30.0</update_rate>
+              <update_rate>10.0</update_rate>
               <camera>
                   <horizontal_fov>${60.0*pi/180.0}</horizontal_fov>

File: atom_simple_examples/ase_2rgb/ase_2rgb_description/urdf/robot.urdf.xacro (robot description, xacro)
@@ -3,15 +3,16 @@
     <!-- ase_2rgb is a simple robotic system containing two rgb cameras on top of a tripop.  -->
     <xacro:property name="M_PI" value="3.1415926535897931" />
+    <material name="Orange">
+        <color rgba="1.0 0.4 0.0 1.0"/>
+    </material>
     <!-- testing adding a sensor camera -->
     <xacro:include filename="$(find ase_2rgb_description)/urdf/rgbd_camera.urdf.xacro" />
+    <!-- Left Camera -->
+    <xacro:rgbd_camera parent="tripod_left_support" prefix="rgb_left" color="red">
+        <origin xyz="0 0.075 0.015" rpy="0 0 0"/>
+    </xacro:rgbd_camera>
     <!-- Right Camera -->
-    <xacro:rgbd_camera parent="tripod_right_support" prefix="rgb_right">
-        <origin xyz="0 0.05 0.015"
-            rpy="0 0 0" />
-    </xacro:rgbd_camera>
-    <!-- Left Camera -->
-    <xacro:rgbd_camera parent="tripod_left_support" prefix="rgb_left">
-        <origin xyz="0 0.075 0.015"
-            rpy="0 0 0" />
+    <xacro:rgbd_camera parent="tripod_right_support" prefix="rgb_right" color="green">
+        <origin xyz="0 0.05 0.015" rpy="0 0 0"/>
     </xacro:rgbd_camera>
     <material name="grey">
