Commit message: Starting with readme for ase_2rgb

File: atom_simple_examples/ase_2rgb/ase_2rgb_description/urdf/robot.urdf.xacro (robot description, xacro)
@@ -27,5 +27,5 @@
                 <mesh filename="package://ase_2rgb_description/meshes/tripod/tripod.dae" scale="0.04 0.04 0.04" />
             </geometry>
-            <material name="grey" />
+            <material name="grey"/>
         </visual>
         <collision name="tripod_collision">
