Commit message: Renaming ase_2rgb to rgb_rgb_system

File: atom_examples/rgb_rgb_system/rgb_rgb_system_description/urdf/rgbd_camera.urdf.xacro (robot description, xacro)
@@ -18,14 +18,14 @@
         <geometry>
         <xacro:if value="${color == 'red'}">
-          <mesh filename="package://ase_2rgb_description/meshes/rgbd_camera/rgbd_camera_red.dae" scale="1 1 1"/>
+          <mesh filename="package://rgb_rgb_system_description/meshes/rgbd_camera/rgbd_camera_red.dae" scale="1 1 1"/>
         </xacro:if>
         <xacro:if value="${color == 'green'}">
-          <mesh filename="package://ase_2rgb_description/meshes/rgbd_camera/rgbd_camera_green.dae" scale="1 1 1"/>
+          <mesh filename="package://rgb_rgb_system_description/meshes/rgbd_camera/rgbd_camera_green.dae" scale="1 1 1"/>
         </xacro:if>
         <xacro:if value="${color == 'black'}">
-          <mesh filename="package://ase_2rgb_description/meshes/rgbd_camera/rgbd_camera.dae" scale="1 1 1"/>
+          <mesh filename="package://rgb_rgb_system_description/meshes/rgbd_camera/rgbd_camera.dae" scale="1 1 1"/>
         </xacro:if>
         <xacro:if value="${color != 'red' and color != 'green' and color != 'black'}">
-          <mesh filename="package://ase_2rgb_description/meshes/rgbd_camera/rgbd_camera.dae" scale="1 1 1"/>
+          <mesh filename="package://rgb_rgb_system_description/meshes/rgbd_camera/rgbd_camera.dae" scale="1 1 1"/>
         </xacro:if>
         </geometry>

File: atom_examples/rgb_rgb_system/rgb_rgb_system_description/urdf/robot.urdf.xacro (robot description, xacro)
@@ -1,5 +1,5 @@
 <?xml version="1.0"?>
 <robot name="robot" xmlns:xacro="http://ros.org/wiki/xacro">
-    <!-- ase_2rgb is a simple robotic system containing two rgb cameras on top of a tripop.  -->
+    <!-- rgb_rgb_system is a simple robotic system containing two rgb cameras on top of a tripop.  -->
     <xacro:property name="M_PI" value="3.1415926535897931" />
     <material name="Orange">
@@ -7,5 +7,5 @@
     </material>
     <!-- testing adding a sensor camera -->
-    <xacro:include filename="$(find ase_2rgb_description)/urdf/rgbd_camera.urdf.xacro" />
+    <xacro:include filename="$(find rgb_rgb_system_description)/urdf/rgbd_camera.urdf.xacro" />
     <!-- Left Camera -->
     <xacro:rgbd_camera parent="tripod_left_support" prefix="rgb_left" color="red">
@@ -26,5 +26,5 @@
             <origin xyz="0 0 0" rpy="0 0 0" />
             <geometry>
-                <mesh filename="package://ase_2rgb_description/meshes/tripod/tripod.dae" scale="0.04 0.04 0.04" />
+                <mesh filename="package://rgb_rgb_system_description/meshes/tripod/tripod.dae" scale="0.04 0.04 0.04" />
             </geometry>
             <material name="grey"/>
@@ -33,5 +33,5 @@
             <origin xyz="0 0 0" rpy="0 0 0" />
             <geometry>
-                <mesh filename="package://ase_2rgb_description/meshes/tripod/tripod.dae" scale="0.04 0.04 0.04" />
+                <mesh filename="package://rgb_rgb_system_description/meshes/tripod/tripod.dae" scale="0.04 0.04 0.04" />
             </geometry>
         </collision>
