Commit message: Close #625. Better colors in system.

File: atom_examples/rgb_rgb_system/rgb_rgb_system_description/urdf/robot.gazebo.xacro (robot description, xacro)
@@ -2,9 +2,5 @@
 <robot xmlns:xacro="http://ros.org/wiki/xacro">
     <gazebo reference="tripod">
-        <material>Gazebo/Grey</material>
-        <mu1>50.0</mu1>
-        <mu2>50.0</mu2>
-        <kp>1000000.0</kp>
-        <kd>1.0</kd>
+        <material>Gazebo/DarkGrey</material>
         <selfCollide>false</selfCollide>
     </gazebo>

File: atom_examples/rgb_rgb_system/rgb_rgb_system_description/urdf/robot.urdf.xacro (robot description, xacro)
@@ -4,18 +4,19 @@
     <xacro:property name="M_PI" value="3.1415926535897931" />
     <material name="Orange">
-        <color rgba="1.0 0.4 0.0 1.0"/>
+        <color rgba="1.0 0.4 0.0 1.0" />
     </material>
+    <xacro:include filename="$(find rgb_rgb_system_description)/urdf/robot.gazebo.xacro" />
     <!-- testing adding a sensor camera -->
     <xacro:include filename="$(find rgb_rgb_system_description)/urdf/rgbd_camera.urdf.xacro" />
     <!-- Left Camera -->
     <xacro:rgbd_camera parent="tripod_left_support" prefix="rgb_left" color="red">
-        <origin xyz="0 0.075 0.015" rpy="0 0 0"/>
+        <origin xyz="0 0.075 0.015" rpy="0 0 0" />
     </xacro:rgbd_camera>
     <!-- Right Camera -->
     <xacro:rgbd_camera parent="tripod_right_support" prefix="rgb_right" color="green">
-        <origin xyz="0 0.05 0.015" rpy="0 0 0"/>
+        <origin xyz="0 0.05 0.015" rpy="0 0 0" />
     </xacro:rgbd_camera>
-    <material name="grey">
-        <color rgba="0.7 0.7 0.7 1.0" />
+    <material name="tripod_color">
+        <color rgba="0.21 0.21 .21 1" />
     </material>
     <!-- Define links and joints -->
@@ -26,12 +27,14 @@
             <origin xyz="0 0 0" rpy="0 0 0" />
             <geometry>
-                <mesh filename="package://rgb_rgb_system_description/meshes/tripod/tripod.dae" scale="0.04 0.04 0.04" />
+                <mesh filename="package://rgb_rgb_system_description/meshes/tripod/tripod.stl"
+                    scale="0.04 0.04 0.04" />
             </geometry>
-            <material name="grey"/>
+            <material name="tripod_color" />
         </visual>
         <collision name="tripod_collision">
             <origin xyz="0 0 0" rpy="0 0 0" />
             <geometry>
-                <mesh filename="package://rgb_rgb_system_description/meshes/tripod/tripod.dae" scale="0.04 0.04 0.04" />
+                <mesh filename="package://rgb_rgb_system_description/meshes/tripod/tripod.stl"
+                    scale="0.04 0.04 0.04" />
             </geometry>
         </collision>
@@ -42,12 +45,11 @@
         </inertial>
     </link>
-      <!-- parent to tripod -->
+    <!-- parent to tripod -->
     <joint name="world_to_tripod" type="fixed">
         <parent link="world" />
         <child link="tripod" />
-        <!-- <xacro:insert_block name="origin" /> -->
         <origin xyz="0 0 0" rpy="0 0 0" />
     </joint>
-       <link name="tripod_plate">
+    <link name="tripod_plate">
         <visual>
             <origin xyz="0 0 0" rpy="0 0 0" />
@@ -55,5 +57,5 @@
                 <box size="0.04 0.4 0.015" />
             </geometry>
-            <material name="grey" />
+            <material name="tripod_color" />
         </visual>
         <collision name="tripod_collision">
@@ -69,5 +71,5 @@
         </inertial>
     </link>
-       <!-- tripod to tripod plate-->
+    <!-- tripod to tripod plate-->
     <joint name="tripod_to_tripod_plate" type="fixed">
         <parent link="tripod" />
@@ -91,4 +93,3 @@
         <origin xyz="0 -0.18 0.0075" rpy="0 0 0" />
     </joint>
-    <!-- </xacro:macro> -->
 </robot>
