Commit message: #625 changing RGBD camera to Flea AVT camera mesh. Putting everything in meters.

File: atom_examples/rgb_rgb_system/rgb_rgb_system_description/urdf/robot.urdf.xacro (robot description, xacro)
@@ -2,22 +2,30 @@
 <robot name="robot" xmlns:xacro="http://ros.org/wiki/xacro">
     <!-- rgb_rgb_system is a simple robotic system containing two rgb cameras on top of a tripop.  -->
+    <!-- Define  properties -->
     <xacro:property name="M_PI" value="3.1415926535897931" />
     <material name="Orange">
         <color rgba="1.0 0.4 0.0 1.0" />
     </material>
-    <xacro:include filename="$(find rgb_rgb_system_description)/urdf/robot.gazebo.xacro" />
-    <!-- testing adding a sensor camera -->
-    <xacro:include filename="$(find rgb_rgb_system_description)/urdf/rgbd_camera.urdf.xacro" />
-    <!-- Left Camera -->
-    <xacro:rgbd_camera parent="tripod_left_support" prefix="rgb_left" color="red">
-        <origin xyz="0 0.075 0.015" rpy="0 0 0" />
-    </xacro:rgbd_camera>
-    <!-- Right Camera -->
-    <xacro:rgbd_camera parent="tripod_right_support" prefix="rgb_right" color="green">
-        <origin xyz="0 0.05 0.015" rpy="0 0 0" />
-    </xacro:rgbd_camera>
+    <!-- Colors -->
     <material name="tripod_color">
         <color rgba="0.21 0.21 .21 1" />
     </material>
+    <material name="red">
+        <color rgba="0.9 0 0 1" />
+    </material>
+    <material name="green">
+        <color rgba="0 0.9 0 1" />
+    </material>
+    <!-- Includes -->
+    <xacro:include filename="$(find rgb_rgb_system_description)/urdf/robot.gazebo.xacro" />
+    <xacro:include filename="$(find rgb_rgb_system_description)/urdf/rgb_camera.urdf.xacro" />
+    <!-- Left Camera -->
+    <xacro:rgb_camera parent="tripod_left_support" prefix="rgb_left" color="red">
+        <origin xyz="0.015 0 0.012" rpy="0 0 0" />
+    </xacro:rgb_camera>
+    <!-- Right Camera -->
+    <xacro:rgb_camera parent="tripod_right_support" prefix="rgb_right" color="green">
+        <origin xyz="0.015 0 0.012" rpy="0 0 0" />
+    </xacro:rgb_camera>
     <!-- Define links and joints -->
     <link name="world" />
@@ -27,6 +35,5 @@
             <origin xyz="0 0 0" rpy="0 0 0" />
             <geometry>
-                <mesh filename="package://rgb_rgb_system_description/meshes/tripod/tripod.stl"
-                    scale="0.04 0.04 0.04" />
+                <mesh filename="package://rgb_rgb_system_description/meshes/tripod/tripod.stl" scale="1 1 1"/>
             </geometry>
             <material name="tripod_color" />
@@ -35,6 +42,5 @@
             <origin xyz="0 0 0" rpy="0 0 0" />
             <geometry>
-                <mesh filename="package://rgb_rgb_system_description/meshes/tripod/tripod.stl"
-                    scale="0.04 0.04 0.04" />
+                <mesh filename="package://rgb_rgb_system_description/meshes/tripod/tripod.stl" scale="1 1 1"/>
             </geometry>
         </collision>
@@ -75,5 +81,5 @@
         <parent link="tripod" />
         <child link="tripod_plate" />
-        <origin xyz=".01 .03 1.33" rpy="0 0.314 0" />
+        <origin xyz=".01 .03 1.65" rpy="0 0.314 0" />
     </joint>
     <!-- Tripod left support-->
