Commit message: #625 and #626. Setting sensor colors with a xacro argument.

File: atom_examples/rgb_depth_system/rgb_depth_system_description/urdf/rgbd_camera.urdf.xacro (robot description, xacro)
@@ -1,8 +1,12 @@
 <?xml version="1.0"?>
 <robot name="rgbd_camera" xmlns:xacro="http://ros.org/wiki/xacro">
-  <!-- Xacro properties -->
-  <material name="default_camera_color">
-    <color rgba="0.21 0.21 .21 1" />
-  </material>
+	<!-- This is a xacro macro to define an rgbd camera.
+	You can define as arguments the parent coordinate frame, the name of the sensor, the transformation
+	from that parent frame to the camera's root frame, the color to be used in rviz, and the color
+	used in gazebo. Colors should be specified for both rviz and gazebo since these have independent colors.
+	Gazebo colors should be capitalized and from this list:
+		http://wiki.ros.org/simulator_gazebo/Tutorials/ListOfMaterials
+  -->
+  <!-- Start of macro -->
   <xacro:macro name="rgbd_camera" params="parent prefix *origin **color_rgb_rviz **color_depth_rviz color_rgb_gazebo:='DarkGrey' color_depth_gazebo:='DarkGrey'">
     <!-- List of Gazbo materials: http://wiki.ros.org/simulator_gazebo/Tutorials/ListOfMaterials -->

File: atom_examples/rgb_rgb_system/rgb_rgb_system_description/urdf/rgb_camera.urdf.xacro (robot description, xacro)
@@ -1,8 +1,13 @@
 <?xml version="1.0"?>
 <robot name="rgb_camera" xmlns:xacro="http://ros.org/wiki/xacro">
-  <material name="default_camera_color">
-  	<color rgba="0.21 0.21 .21 1" />
-  </material>
-	<xacro:macro name="rgb_camera" params="parent prefix *origin color:='default_camera_color'">
+	<!-- This is a xacro macro to define and rgb camera.
+	You can define as arguments the parent coordinate frame, the name of the sensor, the transformation
+	from that parent frame to the camera's root frame, the color to be used in rviz, and the color
+	used in gazebo. Colors should be specified for both rviz and gazebo since these have independent colors.
+	Gazebo colors should be capitalized and from this list:
+		http://wiki.ros.org/simulator_gazebo/Tutorials/ListOfMaterials
+	-->
+	<!-- Start of macro -->
+	<xacro:macro name="rgb_camera" params="parent prefix *origin **color_rviz color_gazebo">
 		<joint name="${prefix}_joint" type="fixed">
 			<xacro:insert_block name="origin" />
@@ -12,14 +17,18 @@
 		<link name="${prefix}_link">
 			<visual>
-				<origin xyz="0 0 0" rpy="0 0 0"/>
+				<origin xyz="0 0 0" rpy="0 0 0" />
 				<geometry>
-					<mesh filename="package://rgb_rgb_system_description/meshes/rgb_camera/rgb_camera.stl" scale="1 1 1"/>
+					<mesh
+						filename="package://rgb_rgb_system_description/meshes/rgb_camera/rgb_camera.stl"
+						scale="1 1 1" />
 				</geometry>
-				<material name="${color}"/>
+				<xacro:insert_block name="color_rviz" />
 			</visual>
 			<collision>
 				<origin xyz="0.0 0.0 0.0" rpy="0 0 0" />
 				<geometry>
-					<mesh filename="package://rgb_rgb_system_description/meshes/rgb_camera/rgb_camera.stl" scale="1 1 1"/>
+					<mesh
+						filename="package://rgb_rgb_system_description/meshes/rgb_camera/rgb_camera.stl"
+						scale="1 1 1" />
 				</geometry>
 			</collision>
@@ -34,16 +43,5 @@
 		<gazebo reference="${prefix}_link">
 			<selfCollide>false</selfCollide>
-			<xacro:if value="${color == 'red'}">
-				<material>Gazebo/Red</material>
-			</xacro:if>
-			<xacro:if value="${color == 'green'}">
-				<material>Gazebo/Green</material>
-			</xacro:if>
-			<xacro:if value="${color == 'black'}">
-				<material>Gazebo/DarkGrey</material>
-			</xacro:if>
-			<xacro:if value="${color != 'red' and color != 'green' and color != 'black'}">
-				<material>Gazebo/DarkGrey</material>
-			</xacro:if>
+			<material>Gazebo/${color_gazebo}</material>
 		</gazebo>
 		<joint name="${prefix}_optical_joint" type="fixed">

File: atom_examples/rgb_rgb_system/rgb_rgb_system_description/urdf/robot.urdf.xacro (robot description, xacro)
@@ -11,20 +11,24 @@
         <color rgba="0.21 0.21 .21 1" />
     </material>
-    <material name="red">
-        <color rgba="0.9 0 0 1" />
-    </material>
-    <material name="green">
-        <color rgba="0 0.9 0 1" />
-    </material>
     <!-- Includes -->
     <xacro:include filename="$(find rgb_rgb_system_description)/urdf/robot.gazebo.xacro" />
     <xacro:include filename="$(find rgb_rgb_system_description)/urdf/rgb_camera.urdf.xacro" />
     <!-- Left Camera -->
-    <xacro:rgb_camera parent="tripod_left_support" prefix="rgb_left" color="red">
+    <xacro:rgb_camera parent="tripod_left_support" prefix="rgb_left" color_gazebo="Red">
         <origin xyz="0.015 0 0.012" rpy="0 0 0" />
+        <color_rgb_rviz>
+            <material name="red">
+                <color rgba="0.9 0 0 1" />
+            </material>
+        </color_rgb_rviz>
     </xacro:rgb_camera>
     <!-- Right Camera -->
-    <xacro:rgb_camera parent="tripod_right_support" prefix="rgb_right" color="green">
+    <xacro:rgb_camera parent="tripod_right_support" prefix="rgb_right" color_gazebo="Green">
         <origin xyz="0.015 0 0.012" rpy="0 0 0" />
+        <color_rgb_rviz>
+            <material name="green">
+                <color rgba="0 0.9 0 1" />
+            </material>
+        </color_rgb_rviz>
     </xacro:rgb_camera>
     <!-- Define links and joints -->
@@ -35,5 +39,6 @@
             <origin xyz="0 0 0" rpy="0 0 0" />
             <geometry>
-                <mesh filename="package://rgb_rgb_system_description/meshes/tripod/tripod.stl" scale="1 1 1"/>
+                <mesh filename="package://rgb_rgb_system_description/meshes/tripod/tripod.stl"
+                    scale="1 1 1" />
             </geometry>
             <material name="tripod_color" />
@@ -42,5 +47,6 @@
             <origin xyz="0 0 0" rpy="0 0 0" />
             <geometry>
-                <mesh filename="package://rgb_rgb_system_description/meshes/tripod/tripod.stl" scale="1 1 1"/>
+                <mesh filename="package://rgb_rgb_system_description/meshes/tripod/tripod.stl"
+                    scale="1 1 1" />
             </geometry>
         </collision>
