Commit message: Changed fov of camera and placed pattern on top of table

File: atom_examples/rgb_hand_eye_system/rgb_hand_eye_system_description/urdf/rgb_camera.urdf.xacro (robot description, xacro)
@@ -56,5 +56,5 @@
 				<update_rate>10.0</update_rate>
 				<camera>
-					<horizontal_fov>${60.0*pi/180.0}</horizontal_fov>
+					<horizontal_fov>${80.0*pi/180.0}</horizontal_fov>
 					<image>
 						<format>B8G8R8</format>

File: atom_examples/rgb_hand_eye_system/rgb_hand_eye_system_description/urdf/robot.urdf.xacro (robot description, xacro)
@@ -11,5 +11,5 @@
     <xacro:property name="table_height" value="0.795"/>
     <xacro:property name="table_width" value=".9"/>
-    <xacro:property name="table_lenght" value="0.9"/>
+    <xacro:property name="table_lenght" value="1.9"/>
     <xacro:property name="table_tabletop_thickness" value="0.015"/>
     <xacro:property name="table_leg_radius" value="0.02"/>
@@ -67,5 +67,5 @@
         <parent link="tabletop_table" />
         <child link = "base_link"/>
-        <origin xyz="0.0 0.0 0.001" rpy="0.0 0.0 0.0" />
+        <origin xyz="0.0 ${table_lenght/4} 0.001" rpy="0.0 0.0 0.0" />
     </joint>
     <!-- Hand Camera (place hand rgb in the end effector) -->
