Commit message: #686 some more fixes.

File: atom_examples/rgb_hand_eye_system/rgb_hand_eye_system_description/urdf/table.macro.xacro (robot description, xacro)
@@ -26,5 +26,5 @@
         </link>
         <gazebo reference="${name}_${parent}">
-            <material>Gazebo/Grey</material>
+            <material>Gazebo/DarkGrey</material>
             <mu1>1000.0</mu1>
             <mu2>1000.0</mu2>
@@ -75,5 +75,5 @@
         </link>
         <gazebo reference="tabletop_${name}">
-            <material>Gazebo/Grey</material>
+            <material>Gazebo/DarkGrey</material>
             <mu1>50.0</mu1>
             <mu2>50.0</mu2>
