Commit message: Fixed playbag.launch has wrong path to optimized URDF #681

File: atom_examples/rgb_hand_eye_system/rgb_hand_eye_system_calibration/urdf/optimized.urdf.xacro (robot description, xacro)
@@ -496,5 +496,5 @@
   </joint>
   <joint name="rgb_hand_joint" type="fixed">
-    <origin xyz="-0.02006024143466846 -0.000858716864601133 0.06459981075694607" rpy="-1.5162950882882648e-05 0.0009349701051782444 -0.00036697160334501014"/>
+    <origin xyz="-0.06277236389936923 -0.026819473440074244 -0.021320569569813957" rpy="-0.10000000000000024 0.10000000000000028 0.10000000000000024"/>
     <parent link="flange"/>
     <child link="rgb_hand_link"/>

File: atom_examples/rgb_hand_eye_system/rgb_hand_eye_system_calibration/urdf/optimized/optimized_2023_11_19-04_06_08_PM.urdf.xacro (robot description, xacro)
@@ -496,5 +496,5 @@
   </joint>
   <joint name="rgb_hand_joint" type="fixed">
-    <origin xyz="-0.02 0.0 0.065" rpy="0.0 -0.0 0.0"/>
+    <origin xyz="-0.02009392144261138 -0.0006613270878237765 0.0645998786239455" rpy="-1.6886101336922917e-05 0.0009330154291185809 -0.0006036464201587783"/>
     <parent link="flange"/>
     <child link="rgb_hand_link"/>

File: atom_examples/rgb_hand_eye_system/rgb_hand_eye_system_calibration/urdf/optimized/optimized_2023_11_19-04_07_04_PM.urdf.xacro (robot description, xacro)
@@ -496,5 +496,5 @@
   </joint>
   <joint name="rgb_hand_joint" type="fixed">
-    <origin xyz="-0.020099447778044895 -0.0006443776493688325 0.06463790311404494" rpy="-7.208798067884849e-06 0.0009706258078079346 -0.0006333430525854225"/>
+    <origin xyz="-0.0200966335242846 -0.000587052127607229 0.06440374597272519" rpy="-9.417640964575229e-06 0.0007103541380183856 -0.0006530570390561612"/>
     <parent link="flange"/>
     <child link="rgb_hand_link"/>

Commit message: Removing optimized files

File: atom_examples/rgb_hand_eye_system/rgb_hand_eye_system_calibration/urdf/optimized.urdf.xacro (robot description, xacro)
@@ -496,5 +496,5 @@
   </joint>
   <joint name="rgb_hand_joint" type="fixed">
-    <origin xyz="-0.03771855080568588 0.006292799332781859 0.05951314519668275" rpy="0.03157978253310624 -0.009136070447862327 -0.020109593800491963"/>
+    <origin xyz="-0.020154768072671813 0.000903230768571792 0.06438858249503736" rpy="-0.024547665796193486 0.0006110578374771245 -0.0005536269252281365"/>
     <parent link="flange"/>
     <child link="rgb_hand_link"/>

Commit message: Miguelriemoliveira/issue711 (#715)
* #711 adding joint states to dataset

* #711 configure_calibration_pkg handling joints

* #711 saving dataset with joint information

* #711 revolute joint model functional

* #711 joint to transform operational and tested

* #711 returning quat and trans instead of transform

* #711 first successful experiment.

* Removing optimized files

* Create an experiment that shows motor angle bias calibration #703

* Removing stupid print.

File: atom_examples/rgb_hand_eye_system/rgb_hand_eye_system_calibration/urdf/optimized.urdf.xacro (robot description, xacro)
@@ -496,5 +496,5 @@
   </joint>
   <joint name="rgb_hand_joint" type="fixed">
-    <origin xyz="-0.06277236389936923 -0.026819473440074244 -0.021320569569813957" rpy="-0.10000000000000024 0.10000000000000028 0.10000000000000024"/>
+    <origin xyz="-0.020154768072671813 0.000903230768571792 0.06438858249503736" rpy="-0.024547665796193486 0.0006110578374771245 -0.0005536269252281365"/>
     <parent link="flange"/>
     <child link="rgb_hand_link"/>
