Commit message: Advancing #731 and #739

File: atom_examples/eye_in_world_system/eye_in_world_system_calibration/urdf/initial_estimate.urdf.xacro (robot description, xacro)
@@ -14,5 +14,5 @@
     <xacro:property name="table_height" value="0.795"/>
     <xacro:property name="table_width" value=".9"/>
-    <xacro:property name="table_lenght" value="1.9"/>
+    <xacro:property name="table_lenght" value="0.9"/>
     <xacro:property name="table_tabletop_thickness" value="0.015"/>
     <xacro:property name="table_leg_radius" value="0.02"/>

File: atom_examples/eye_in_world_system/eye_in_world_system_description/urdf/rgb_camera.urdf.xacro (robot description, xacro)
@@ -17,5 +17,5 @@
 		<link name="${prefix}_link">
 			<visual>
-				<origin xyz="0 0 0" rpy="0 0 0" />
+				<origin xyz="-0.01 0 0" rpy="0 0 0" />
 				<geometry>
 					<mesh
@@ -26,5 +26,5 @@
 			</visual>
 			<collision>
-				<origin xyz="0.0 0.0 0.0" rpy="0 0 0" />
+				<origin xyz="-0.01 0.0 0.0" rpy="0 0 0" />
 				<geometry>
 					<mesh
@@ -56,5 +56,5 @@
 				<update_rate>10.0</update_rate>
 				<camera>
-					<horizontal_fov>${80.0*pi/180.0}</horizontal_fov>
+					<horizontal_fov>${60.0*pi/180.0}</horizontal_fov>
 					<image>
 						<format>B8G8R8</format>
