Commit message: #731 make ros visualization work with multiple patterns

File: atom_examples/eye_in_world_system/eye_in_world_system_calibration/urdf/optimized/optimized_2023_12_01-04_31_16_PM.urdf.xacro (robot description, xacro)
@@ -555,5 +555,5 @@
   </joint>
   <joint name="rgb_world_joint" type="fixed">
-    <origin xyz="0.0003300090003504614 4.439385181527105e-05 0.030099526391556698" rpy="3.093026387927702e-05 0.0010320398016228462 -0.001026892068148891"/>
+    <origin xyz="0.00022821840053385042 6.737864189111818e-06 0.030028662744143796" rpy="-6.609254869370346e-05 0.000979445272767924 -0.0010028004747610674"/>
     <parent link="tripod_center_support"/>
     <child link="rgb_world_link"/>

File: atom_examples/eye_in_world_system/eye_in_world_system_calibration/urdf/optimized/optimized_2023_12_01-05_52_56_PM.urdf.xacro (robot description, xacro)
@@ -555,5 +555,5 @@
   </joint>
   <joint name="rgb_world_joint" type="fixed">
-    <origin xyz="0.0003300090003504614 4.439385181527105e-05 0.030099526391556698" rpy="3.093026387927702e-05 0.0010320398016228462 -0.001026892068148891"/>
+    <origin xyz="0.00023255307647717462 -9.549273105921314e-06 0.03003460117727573" rpy="-7.85975363293864e-05 0.000990161098644211 -0.0009868678898107789"/>
     <parent link="tripod_center_support"/>
     <child link="rgb_world_link"/>

File: atom_examples/eye_in_world_system/eye_in_world_system_calibration/urdf/optimized/optimized_2023_12_01-05_57_48_PM.urdf.xacro (robot description, xacro)
@@ -555,5 +555,5 @@
   </joint>
   <joint name="rgb_world_joint" type="fixed">
-    <origin xyz="0.0003300090003504614 4.439385181527105e-05 0.030099526391556698" rpy="3.093026387927702e-05 0.0010320398016228462 -0.001026892068148891"/>
+    <origin xyz="0.0002560223303990293 0.00016269270818701175 0.030091872292725287" rpy="0.00018423192122021627 0.0010636507248746147 -0.0011854976024626423"/>
     <parent link="tripod_center_support"/>
     <child link="rgb_world_link"/>

File: atom_examples/eye_in_world_system/eye_in_world_system_calibration/urdf/optimized/optimized_2023_12_01-06_03_42_PM.urdf.xacro (robot description, xacro)
@@ -555,5 +555,5 @@
   </joint>
   <joint name="rgb_world_joint" type="fixed">
-    <origin xyz="0.0003300090003504614 4.439385181527105e-05 0.030099526391556698" rpy="3.093026387927702e-05 0.0010320398016228462 -0.001026892068148891"/>
+    <origin xyz="0.0002632696843608319 0.000161808359603671 0.0301038115185346" rpy="0.0001887138328992879 0.0010767577252159255 -0.0011814116817634062"/>
     <parent link="tripod_center_support"/>
     <child link="rgb_world_link"/>

File: atom_examples/eye_in_world_system/eye_in_world_system_calibration/urdf/optimized/optimized_2023_12_01-06_04_20_PM.urdf.xacro (robot description, xacro)
@@ -555,5 +555,5 @@
   </joint>
   <joint name="rgb_world_joint" type="fixed">
-    <origin xyz="0.0003300090003504614 4.439385181527105e-05 0.030099526391556698" rpy="3.093026387927702e-05 0.0010320398016228462 -0.001026892068148891"/>
+    <origin xyz="0.0002519423445236294 0.0001633092127623563 0.030084644420454172" rpy="0.00018070890144724301 0.00105576358884459 -0.0011882836563493514"/>
     <parent link="tripod_center_support"/>
     <child link="rgb_world_link"/>

File: atom_examples/eye_in_world_system/eye_in_world_system_calibration/urdf/optimized/optimized_2023_12_01-06_04_46_PM.urdf.xacro (robot description, xacro)
@@ -555,5 +555,5 @@
   </joint>
   <joint name="rgb_world_joint" type="fixed">
-    <origin xyz="0.0003300090003504614 4.439385181527105e-05 0.030099526391556698" rpy="3.093026387927702e-05 0.0010320398016228462 -0.001026892068148891"/>
+    <origin xyz="0.00032316276161688153 3.707019936029511e-05 0.030085099653141767" rpy="2.1525438196533998e-05 0.0010171673075574283 -0.0010211457189341906"/>
     <parent link="tripod_center_support"/>
     <child link="rgb_world_link"/>
