Commit message: $741 operational

File: atom_examples/eye_in_world_system/eye_in_world_system_calibration/urdf/optimized/optimized_2023_12_02-09_40_02_AM.urdf.xacro (robot description, xacro)
@@ -555,5 +555,5 @@
   </joint>
   <joint name="rgb_world_joint" type="fixed">
-    <origin xyz="0.00021240475885379683 -9.441426742326197e-06 0.030006557343603333" rpy="-7.587538120222827e-05 0.0009524755246322182 -0.000985795199803372"/>
+    <origin xyz="0.00020896690891106427 -4.1326655694341105e-06 0.03000166736591492" rpy="-7.361472396346798e-05 0.0009472445496182862 -0.0009883279307261587"/>
     <parent link="tripod_center_support"/>
     <child link="rgb_world_link"/>
