Commit message: #775. First functional version.

File: atom_examples/rihbot/rihbot_calibration/urdf/optimized/optimized_2023_12_08-09_47_24_AM.urdf.xacro (robot description, xacro)
@@ -496,5 +496,5 @@
   </joint>
   <joint name="rgb_hand_joint" type="fixed">
-    <origin xyz="-0.06676267790515047 0.08468129188560457 0.09034424510069682" rpy="-0.10000000000000013 -0.1000000000000001 0.10000000000000013"/>
+    <origin xyz="-0.020094574079955862 -0.0007649468871777876 0.0645128290388102" rpy="-2.045967605559065e-05 0.0008250342320148523 -0.0004689990860736754"/>
     <parent link="flange"/>
     <child link="rgb_hand_link"/>

File: atom_examples/rihbot/rihbot_calibration/urdf/optimized/optimized_2023_12_08-09_59_18_AM.urdf.xacro (robot description, xacro)
@@ -496,5 +496,5 @@
   </joint>
   <joint name="rgb_hand_joint" type="fixed">
-    <origin xyz="-0.06676267790515047 0.08468129188560457 0.09034424510069682" rpy="-0.10000000000000013 -0.1000000000000001 0.10000000000000013"/>
+    <origin xyz="-0.02010802419707121 -0.0005866638405162887 0.06443643804075713" rpy="-1.2095805311588843e-05 0.0007430354245569655 -0.0006669807869641449"/>
     <parent link="flange"/>
     <child link="rgb_hand_link"/>

File: atom_examples/rihbot/rihbot_calibration/urdf/optimized/optimized_2023_12_08-10_00_16_AM.urdf.xacro (robot description, xacro)
@@ -496,5 +496,5 @@
   </joint>
   <joint name="rgb_hand_joint" type="fixed">
-    <origin xyz="-0.06676267790515047 0.08468129188560457 0.09034424510069682" rpy="-0.10000000000000013 -0.1000000000000001 0.10000000000000013"/>
+    <origin xyz="-0.020132676605851427 -0.0005692505367896694 0.06466704321699757" rpy="-1.735323179970638e-05 0.0009767068006331227 -0.0007495487400893426"/>
     <parent link="flange"/>
     <child link="rgb_hand_link"/>

File: atom_examples/rihbot/rihbot_calibration/urdf/optimized/optimized_2023_12_08-10_00_49_AM.urdf.xacro (robot description, xacro)
@@ -496,5 +496,5 @@
   </joint>
   <joint name="rgb_hand_joint" type="fixed">
-    <origin xyz="-0.06676267790515047 0.08468129188560457 0.09034424510069682" rpy="-0.10000000000000013 -0.1000000000000001 0.10000000000000013"/>
+    <origin xyz="-0.07102020923736874 0.017428849310824005 0.14922097993419278" rpy="-0.10000000000000024 -0.10000000000000028 -0.10000000000000024"/>
     <parent link="flange"/>
     <child link="rgb_hand_link"/>

File: atom_examples/rihbot/rihbot_calibration/urdf/optimized/optimized_2023_12_08-10_11_38_AM.urdf.xacro (robot description, xacro)
@@ -496,5 +496,5 @@
   </joint>
   <joint name="rgb_hand_joint" type="fixed">
-    <origin xyz="-0.06676267790515047 0.08468129188560457 0.09034424510069682" rpy="-0.10000000000000013 -0.1000000000000001 0.10000000000000013"/>
+    <origin xyz="-0.013325867496910514 -0.050086914255375016 0.1512945941279401" rpy="0.10000000000000024 -0.10000000000000028 0.10000000000000024"/>
     <parent link="flange"/>
     <child link="rgb_hand_link"/>

File: atom_examples/rihbot/rihbot_calibration/urdf/optimized/optimized_2023_12_08-10_11_47_AM.urdf.xacro (robot description, xacro)
@@ -496,5 +496,5 @@
   </joint>
   <joint name="rgb_hand_joint" type="fixed">
-    <origin xyz="-0.06676267790515047 0.08468129188560457 0.09034424510069682" rpy="-0.10000000000000013 -0.1000000000000001 0.10000000000000013"/>
+    <origin xyz="0.05540395921430305 0.05113940542192093 0.02378102199350246" rpy="-0.10000000000000013 -0.1000000000000001 0.10000000000000013"/>
     <parent link="flange"/>
     <child link="rgb_hand_link"/>

File: atom_examples/rihbot/rihbot_calibration/urdf/optimized/optimized_2023_12_08-10_12_13_AM.urdf.xacro (robot description, xacro)
@@ -496,5 +496,5 @@
   </joint>
   <joint name="rgb_hand_joint" type="fixed">
-    <origin xyz="-0.06676267790515047 0.08468129188560457 0.09034424510069682" rpy="-0.10000000000000013 -0.1000000000000001 0.10000000000000013"/>
+    <origin xyz="0.012807816099879129 0.07086572600948837 0.12746355801509096" rpy="0.10000000000000024 0.10000000000000028 -0.10000000000000024"/>
     <parent link="flange"/>
     <child link="rgb_hand_link"/>

File: atom_examples/rihbot/rihbot_calibration/urdf/optimized/optimized_2023_12_08-10_12_50_AM.urdf.xacro (robot description, xacro)
@@ -496,5 +496,5 @@
   </joint>
   <joint name="rgb_hand_joint" type="fixed">
-    <origin xyz="-0.06676267790515047 0.08468129188560457 0.09034424510069682" rpy="-0.10000000000000013 -0.1000000000000001 0.10000000000000013"/>
+    <origin xyz="0.04845382812382561 0.043539709717033165 0.006533196658700169" rpy="0.10000000000000024 -0.10000000000000028 0.10000000000000024"/>
     <parent link="flange"/>
     <child link="rgb_hand_link"/>

File: atom_examples/rihbot/rihbot_calibration/urdf/optimized/optimized_2023_12_08-10_13_36_AM.urdf.xacro (robot description, xacro)
@@ -496,5 +496,5 @@
   </joint>
   <joint name="rgb_hand_joint" type="fixed">
-    <origin xyz="-0.06676267790515047 0.08468129188560457 0.09034424510069682" rpy="-0.10000000000000013 -0.1000000000000001 0.10000000000000013"/>
+    <origin xyz="-0.004981629409367581 -0.04367506658564934 -0.023695755837252586" rpy="0.10000000000000013 -0.1000000000000001 -0.10000000000000013"/>
     <parent link="flange"/>
     <child link="rgb_hand_link"/>

File: atom_examples/rihbot/rihbot_calibration/urdf/optimized/optimized_2023_12_08-10_13_50_AM.urdf.xacro (robot description, xacro)
@@ -496,5 +496,5 @@
   </joint>
   <joint name="rgb_hand_joint" type="fixed">
-    <origin xyz="-0.06676267790515047 0.08468129188560457 0.09034424510069682" rpy="-0.10000000000000013 -0.1000000000000001 0.10000000000000013"/>
+    <origin xyz="0.07010251202541765 0.006980137331230764 0.10781138878320376" rpy="-0.10000000000000013 -0.1000000000000001 0.10000000000000013"/>
     <parent link="flange"/>
     <child link="rgb_hand_link"/>

File: atom_examples/rihbot/rihbot_calibration/urdf/optimized/optimized_2023_12_08-10_16_53_AM.urdf.xacro (robot description, xacro)
@@ -496,5 +496,5 @@
   </joint>
   <joint name="rgb_hand_joint" type="fixed">
-    <origin xyz="-0.06676267790515047 0.08468129188560457 0.09034424510069682" rpy="-0.10000000000000013 -0.1000000000000001 0.10000000000000013"/>
+    <origin xyz="0.01181215093798552 0.08536886880205685 0.10623279389219256" rpy="-0.10000000000000024 0.10000000000000028 0.10000000000000024"/>
     <parent link="flange"/>
     <child link="rgb_hand_link"/>

File: atom_examples/rihbot/rihbot_calibration/urdf/optimized/optimized_2023_12_08-10_24_15_AM.urdf.xacro (robot description, xacro)
@@ -496,5 +496,5 @@
   </joint>
   <joint name="rgb_hand_joint" type="fixed">
-    <origin xyz="-0.06676267790515047 0.08468129188560457 0.09034424510069682" rpy="-0.10000000000000013 -0.1000000000000001 0.10000000000000013"/>
+    <origin xyz="0.017157163213189944 -0.029936121984299114 0.15288158978130476" rpy="0.10000000000000013 -0.1000000000000001 -0.10000000000000013"/>
     <parent link="flange"/>
     <child link="rgb_hand_link"/>

File: atom_examples/rihbot/rihbot_calibration/urdf/optimized/optimized_2023_12_08-10_25_30_AM.urdf.xacro (robot description, xacro)
@@ -496,5 +496,5 @@
   </joint>
   <joint name="rgb_hand_joint" type="fixed">
-    <origin xyz="-0.06676267790515047 0.08468129188560457 0.09034424510069682" rpy="-0.10000000000000013 -0.1000000000000001 0.10000000000000013"/>
+    <origin xyz="0.06558781085441102 -0.03194278469264843 0.1056741335399867" rpy="-0.10000000000000013 -0.1000000000000001 0.10000000000000013"/>
     <parent link="flange"/>
     <child link="rgb_hand_link"/>

File: atom_examples/rihbot/rihbot_calibration/urdf/optimized/optimized_2023_12_08-10_27_36_AM.urdf.xacro (robot description, xacro)
@@ -496,5 +496,5 @@
   </joint>
   <joint name="rgb_hand_joint" type="fixed">
-    <origin xyz="-0.06676267790515047 0.08468129188560457 0.09034424510069682" rpy="-0.10000000000000013 -0.1000000000000001 0.10000000000000013"/>
+    <origin xyz="0.034320743104585036 -0.06438736233739144 0.01111563826304382" rpy="0.10000000000000013 -0.1000000000000001 -0.10000000000000013"/>
     <parent link="flange"/>
     <child link="rgb_hand_link"/>

File: atom_examples/rihbot/rihbot_calibration/urdf/optimized/optimized_2023_12_08-10_32_28_AM.urdf.xacro (robot description, xacro)
@@ -496,5 +496,5 @@
   </joint>
   <joint name="rgb_hand_joint" type="fixed">
-    <origin xyz="-0.06676267790515047 0.08468129188560457 0.09034424510069682" rpy="-0.10000000000000013 -0.1000000000000001 0.10000000000000013"/>
+    <origin xyz="-0.08054928417892335 -0.06104990506993409 0.013944214075464277" rpy="0.10000000000000013 0.1000000000000001 0.10000000000000013"/>
     <parent link="flange"/>
     <child link="rgb_hand_link"/>

File: atom_examples/rihbot/rihbot_calibration/urdf/optimized/optimized_2023_12_08-10_32_49_AM.urdf.xacro (robot description, xacro)
@@ -496,5 +496,5 @@
   </joint>
   <joint name="rgb_hand_joint" type="fixed">
-    <origin xyz="-0.06676267790515047 0.08468129188560457 0.09034424510069682" rpy="-0.10000000000000013 -0.1000000000000001 0.10000000000000013"/>
+    <origin xyz="0.006799175224828705 -0.08016414950321366 0.011562996512759632" rpy="-0.10000000000000013 0.1000000000000001 -0.10000000000000013"/>
     <parent link="flange"/>
     <child link="rgb_hand_link"/>

File: atom_examples/rihbot/rihbot_calibration/urdf/optimized/optimized_2023_12_08-12_04_18_PM.urdf.xacro (robot description, xacro)
@@ -496,5 +496,5 @@
   </joint>
   <joint name="rgb_hand_joint" type="fixed">
-    <origin xyz="-0.06676267790515047 0.08468129188560457 0.09034424510069682" rpy="-0.10000000000000013 -0.1000000000000001 0.10000000000000013"/>
+    <origin xyz="0.032510913868078015 0.03394249178626187 -0.013041727146948998" rpy="0.10000000000000013 0.1000000000000001 0.10000000000000013"/>
     <parent link="flange"/>
     <child link="rgb_hand_link"/>

File: atom_examples/rihbot/rihbot_calibration/urdf/optimized/optimized_2023_12_08-12_04_36_PM.urdf.xacro (robot description, xacro)
@@ -496,5 +496,5 @@
   </joint>
   <joint name="rgb_hand_joint" type="fixed">
-    <origin xyz="-0.06676267790515047 0.08468129188560457 0.09034424510069682" rpy="-0.10000000000000013 -0.1000000000000001 0.10000000000000013"/>
+    <origin xyz="-0.09620390664775706 0.06474992439023503 0.06564179675815293" rpy="0.10000000000000013 -0.1000000000000001 -0.10000000000000013"/>
     <parent link="flange"/>
     <child link="rgb_hand_link"/>

File: atom_examples/rihbot/rihbot_calibration/urdf/optimized/optimized_2023_12_08-12_05_22_PM.urdf.xacro (robot description, xacro)
@@ -496,5 +496,5 @@
   </joint>
   <joint name="rgb_hand_joint" type="fixed">
-    <origin xyz="-0.06676267790515047 0.08468129188560457 0.09034424510069682" rpy="-0.10000000000000013 -0.1000000000000001 0.10000000000000013"/>
+    <origin xyz="-0.037217134543194384 -0.09547294395762777 0.08925875615494763" rpy="0.10000000000000013 -0.1000000000000001 -0.10000000000000013"/>
     <parent link="flange"/>
     <child link="rgb_hand_link"/>

File: atom_examples/rihbot/rihbot_calibration/urdf/optimized/optimized_2023_12_08-12_05_34_PM.urdf.xacro (robot description, xacro)
@@ -496,5 +496,5 @@
   </joint>
   <joint name="rgb_hand_joint" type="fixed">
-    <origin xyz="-0.06676267790515047 0.08468129188560457 0.09034424510069682" rpy="-0.10000000000000013 -0.1000000000000001 0.10000000000000013"/>
+    <origin xyz="-0.0016507010223117367 0.08956161413185809 0.02447814785669878" rpy="-0.10000000000000024 -0.10000000000000028 -0.10000000000000024"/>
     <parent link="flange"/>
     <child link="rgb_hand_link"/>
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