Commit message: Setting calibrate back with correct optimization options.

File: atom_examples/rihbot/rihbot_calibration/urdf/optimized.urdf.xacro (robot description, xacro)
@@ -496,5 +496,5 @@
   </joint>
   <joint name="rgb_hand_joint" type="fixed">
-    <origin xyz="-0.06676267790515047 0.08468129188560457 0.09034424510069682" rpy="-0.10000000000000013 -0.1000000000000001 0.10000000000000013"/>
+    <origin xyz="-0.06604520338605281 -0.08283978769896988 0.03310315346109225" rpy="-0.10000000000000024 -0.10000000000000028 -0.10000000000000024"/>
     <parent link="flange"/>
     <child link="rgb_hand_link"/>

File: atom_examples/rihbot/rihbot_calibration/urdf/optimized_w_pattern.urdf.xacro (robot description, xacro)
@@ -496,5 +496,5 @@
   </joint>
   <joint name="rgb_hand_joint" type="fixed">
-    <origin xyz="-0.06676267790515047 0.08468129188560457 0.09034424510069682" rpy="-0.10000000000000013 -0.1000000000000001 0.10000000000000013"/>
+    <origin xyz="-0.06604520338605281 -0.08283978769896988 0.03310315346109225" rpy="-0.10000000000000024 -0.10000000000000028 -0.10000000000000024"/>
     <parent link="flange"/>
     <child link="rgb_hand_link"/>
