Commit message: Close #796

File: atom_examples/riwbot/riwbot_calibration/urdf/initial_estimate.urdf.xacro (robot description, xacro)
@@ -149,5 +149,5 @@
             <origin xyz="0 0 0" rpy="0 0 0" />
             <geometry>
-                <mesh filename="package://atom_worlds/pattern/models/charuco_200x200_4x4/charuco_200x200_4x4.dae"
+                <mesh filename="package://atom_worlds/pattern/models/charuco_200x200_8x8_20_15_DICT_4x4/model.dae"
                     scale="1 1 1" />
             </geometry>
@@ -157,5 +157,5 @@
             <origin xyz="0 0 0" rpy="0 0 0" />
             <geometry>
-                <mesh filename="package://atom_worlds/pattern/models/charuco_200x200_4x4/charuco_200x200_4x4.dae"
+                <mesh filename="package://atom_worlds/pattern/models/charuco_200x200_8x8_20_15_DICT_4x4/model.dae"
                     scale="1 1 1" />
             </geometry>
