Commit message: Close #800

File: atom_examples/jcpbbot/jcpbbot_calibration/urdf/optimized.urdf.xacro (robot description, xacro)
@@ -400,5 +400,5 @@
   </joint>
   <joint name="shoulder_pan_joint" type="revolute">
-    <origin xyz="0.0 0.0 0.1807" rpy="0.0 0.0 0.0"/>
+    <origin xyz="0.0 0.0 0.1807" rpy="0.0 0.0 0.008890193659224334"/>
     <axis xyz="0.0 0.0 1.0"/>
     <parent link="base_link_inertia"/>
@@ -408,5 +408,5 @@
   </joint>
   <joint name="shoulder_lift_joint" type="revolute">
-    <origin xyz="0.0 0.0 0.0" rpy="1.570796327 0.0 0.0"/>
+    <origin xyz="0.0 0.0 0.0" rpy="1.570796327 0.0 0.008890171935160953"/>
     <axis xyz="0.0 0.0 1.0"/>
     <parent link="shoulder_link"/>
@@ -416,5 +416,5 @@
   </joint>
   <joint name="elbow_joint" type="revolute">
-    <origin xyz="-0.6127 0.0 0.0" rpy="0.0 0.0 0.0"/>
+    <origin xyz="-0.6127 0.0 0.0" rpy="0.0 0.0 0.025686301279139782"/>
     <axis xyz="0.0 0.0 1.0"/>
     <parent link="upper_arm_link"/>
@@ -424,5 +424,5 @@
   </joint>
   <joint name="wrist_1_joint" type="revolute">
-    <origin xyz="-0.57155 0.0 0.17415" rpy="0.0 0.0 0.0"/>
+    <origin xyz="-0.57155 0.0 0.17415" rpy="0.0 0.0 -0.03120098064039958"/>
     <axis xyz="0.0 0.0 1.0"/>
     <parent link="forearm_link"/>
@@ -432,5 +432,5 @@
   </joint>
   <joint name="wrist_2_joint" type="revolute">
-    <origin xyz="0.0 -0.11985 -2.458164590756244e-11" rpy="1.570796327 0.0 0.0"/>
+    <origin xyz="0.0 -0.11985 -2.458164590756244e-11" rpy="1.570796327 0.0 -0.021298137887970636"/>
     <axis xyz="0.0 0.0 1.0"/>
     <parent link="wrist_1_link"/>
@@ -440,5 +440,5 @@
   </joint>
   <joint name="wrist_3_joint" type="revolute">
-    <origin xyz="0.0 0.11655 -2.390480459346185e-11" rpy="1.570796326589793 3.141592653589793 3.141592653589793"/>
+    <origin xyz="0.0 0.11655 -2.390480459346185e-11" rpy="1.570796326589793 3.141592653589793 3.13075084398692"/>
     <axis xyz="0.0 0.0 1.0"/>
     <parent link="wrist_2_link"/>
@@ -496,5 +496,5 @@
   </joint>
   <joint name="rgb_hand_joint" type="fixed">
-    <origin xyz="-0.01990185590294675 -0.0015539059894699035 0.06484572412936336" rpy="0.010604682853474478 0.0011472278262240274 -0.0002151756429437089"/>
+    <origin xyz="-0.021655607917021997 -0.00390675426651832 0.06475692382180025" rpy="0.03044414300186205 0.0013822999375349206 0.0008670472196217079"/>
     <parent link="flange"/>
     <child link="rgb_hand_link"/>

File: atom_examples/jcpbbot/jcpbbot_calibration/urdf/optimized_w_pattern.urdf.xacro (robot description, xacro)
@@ -400,5 +400,5 @@
   </joint>
   <joint name="shoulder_pan_joint" type="revolute">
-    <origin xyz="0.0 0.0 0.1807" rpy="0.0 0.0 0.0"/>
+    <origin xyz="0.0 0.0 0.1807" rpy="0.0 0.0 0.008890193659224334"/>
     <axis xyz="0.0 0.0 1.0"/>
     <parent link="base_link_inertia"/>
@@ -408,5 +408,5 @@
   </joint>
   <joint name="shoulder_lift_joint" type="revolute">
-    <origin xyz="0.0 0.0 0.0" rpy="1.570796327 0.0 0.0"/>
+    <origin xyz="0.0 0.0 0.0" rpy="1.570796327 0.0 0.008890171935160953"/>
     <axis xyz="0.0 0.0 1.0"/>
     <parent link="shoulder_link"/>
@@ -416,5 +416,5 @@
   </joint>
   <joint name="elbow_joint" type="revolute">
-    <origin xyz="-0.6127 0.0 0.0" rpy="0.0 0.0 0.0"/>
+    <origin xyz="-0.6127 0.0 0.0" rpy="0.0 0.0 0.025686301279139782"/>
     <axis xyz="0.0 0.0 1.0"/>
     <parent link="upper_arm_link"/>
@@ -424,5 +424,5 @@
   </joint>
   <joint name="wrist_1_joint" type="revolute">
-    <origin xyz="-0.57155 0.0 0.17415" rpy="0.0 0.0 0.0"/>
+    <origin xyz="-0.57155 0.0 0.17415" rpy="0.0 0.0 -0.03120098064039958"/>
     <axis xyz="0.0 0.0 1.0"/>
     <parent link="forearm_link"/>
@@ -432,5 +432,5 @@
   </joint>
   <joint name="wrist_2_joint" type="revolute">
-    <origin xyz="0.0 -0.11985 -2.458164590756244e-11" rpy="1.570796327 0.0 0.0"/>
+    <origin xyz="0.0 -0.11985 -2.458164590756244e-11" rpy="1.570796327 0.0 -0.021298137887970636"/>
     <axis xyz="0.0 0.0 1.0"/>
     <parent link="wrist_1_link"/>
@@ -440,5 +440,5 @@
   </joint>
   <joint name="wrist_3_joint" type="revolute">
-    <origin xyz="0.0 0.11655 -2.390480459346185e-11" rpy="1.570796326589793 3.141592653589793 3.141592653589793"/>
+    <origin xyz="0.0 0.11655 -2.390480459346185e-11" rpy="1.570796326589793 3.141592653589793 3.13075084398692"/>
     <axis xyz="0.0 0.0 1.0"/>
     <parent link="wrist_2_link"/>
@@ -496,5 +496,5 @@
   </joint>
   <joint name="rgb_hand_joint" type="fixed">
-    <origin xyz="-0.01990185590294675 -0.0015539059894699035 0.06484572412936336" rpy="0.010604682853474478 0.0011472278262240274 -0.0002151756429437089"/>
+    <origin xyz="-0.021655607917021997 -0.00390675426651832 0.06475692382180025" rpy="0.03044414300186205 0.0013822999375349206 0.0008670472196217079"/>
     <parent link="flange"/>
     <child link="rgb_hand_link"/>
@@ -573,5 +573,5 @@
   </link>
   <joint name="world-pattern_link" type="fixed">
-    <origin xyz="-1.0739689399784635 0.29097701455538144 0.8086462226274849" rpy="3.1222672111343126 0.008621355988864494 0.02243043709005299"/>
+    <origin xyz="-1.0770226772570606 0.2931901408646521 0.8003184404186438" rpy="3.1217472174026617 0.03275960050931226 0.029816861385440114"/>
     <parent link="world"/>
     <child link="pattern_link"/>

File: atom_examples/riwmpbot/riwmpbot_calibration/urdf/optimized.urdf.xacro (robot description, xacro)
@@ -403,5 +403,5 @@
   </joint>
   <joint name="shoulder_pan_joint" type="revolute">
-    <origin xyz="-0.0011072022674218484 0.006104470330633574 0.1776131205352634" rpy="-0.024334800436751625 -0.028227058847477848 -0.06020146484737336"/>
+    <origin xyz="0.007821368819945888 0.004461437917977398 0.17456163379972744" rpy="0.006956419073605317 -0.006358233920799441 -0.0007724759947057985"/>
     <axis xyz="0.0 0.0 1.0"/>
     <parent link="base_link_inertia"/>
@@ -411,5 +411,5 @@
   </joint>
   <joint name="shoulder_lift_joint" type="revolute">
-    <origin xyz="0.016431914541455865 -0.015921078340292362 0.010636931179058638" rpy="1.5415716586341253 0.014863657572835746 -0.07258247459143602"/>
+    <origin xyz="-0.009531296053436934 0.0067249256283193285 0.0075457641395848245" rpy="1.5663385979260043 0.004660654849611939 -0.010962503936608999"/>
     <axis xyz="0.0 0.0 1.0"/>
     <parent link="shoulder_link"/>
@@ -419,5 +419,5 @@
   </joint>
   <joint name="elbow_joint" type="revolute">
-    <origin xyz="-0.5996745659350029 -0.00048636814021923297 0.009405942102471837" rpy="-0.014553428819016492 -0.02173367222479105 0.02605134752247605"/>
+    <origin xyz="-0.6102152904073732 0.004328175185936848 0.0062061018415760835" rpy="-0.010057140605404025 -0.004873101280596378 0.0009330003870278563"/>
     <axis xyz="0.0 0.0 1.0"/>
     <parent link="upper_arm_link"/>
@@ -427,5 +427,5 @@
   </joint>
   <joint name="wrist_1_joint" type="revolute">
-    <origin xyz="-0.5652841488249898 0.009018813250154935 0.17706782067685806" rpy="-0.003003155878006817 0.021644677144780536 0.005398823112075103"/>
+    <origin xyz="-0.5704987376211959 0.00011153779929661173 0.19145923932465514" rpy="0.03396777184450894 0.017450246872858784 0.0036295438263922557"/>
     <axis xyz="0.0 0.0 1.0"/>
     <parent link="forearm_link"/>
@@ -435,5 +435,5 @@
   </joint>
   <joint name="wrist_2_joint" type="revolute">
-    <origin xyz="0.0031153126042543534 -0.13407407955813314 -0.01778150734076564" rpy="1.5887420852926646 0.026030532780267963 0.011990836311086397"/>
+    <origin xyz="-0.0017524887429481704 -0.12494427019129475 -0.007826529452888942" rpy="1.5218680988243996 -0.01628060509339201 -0.008227162828881624"/>
     <axis xyz="0.0 0.0 1.0"/>
     <parent link="wrist_1_link"/>
@@ -443,5 +443,5 @@
   </joint>
   <joint name="wrist_3_joint" type="revolute">
-    <origin xyz="-0.013741436377825881 0.10116111685658188 -0.008882501308609786" rpy="1.563230653741768 3.171288905523689 3.159559083662778"/>
+    <origin xyz="-0.0010531673461660613 0.10902818800654597 -0.00782207531345751" rpy="1.604132174646816 3.2263459683256017 3.0950684569871245"/>
     <axis xyz="0.0 0.0 1.0"/>
     <parent link="wrist_2_link"/>
@@ -555,5 +555,5 @@
   </joint>
   <joint name="rgb_world_joint" type="fixed">
-    <origin xyz="-0.01625234687483334 0.007016927088536094 0.04058858883102345" rpy="-0.0033734439638217453 -0.00856908230693528 -0.01718724775946154"/>
+    <origin xyz="-2.2038082383793905e-17 3.0097249768286925e-17 0.030000000000000023" rpy="0.0 -0.0 0.0"/>
     <parent link="tripod_center_support"/>
     <child link="rgb_world_link"/>

File: atom_examples/riwmpbot/riwmpbot_calibration/urdf/optimized_w_pattern.urdf.xacro (robot description, xacro)
@@ -403,5 +403,5 @@
   </joint>
   <joint name="shoulder_pan_joint" type="revolute">
-    <origin xyz="-0.0011072022674218484 0.006104470330633574 0.1776131205352634" rpy="-0.024334800436751625 -0.028227058847477848 -0.06020146484737336"/>
+    <origin xyz="0.007821368819945888 0.004461437917977398 0.17456163379972744" rpy="0.006956419073605317 -0.006358233920799441 -0.0007724759947057985"/>
     <axis xyz="0.0 0.0 1.0"/>
     <parent link="base_link_inertia"/>
@@ -411,5 +411,5 @@
   </joint>
   <joint name="shoulder_lift_joint" type="revolute">
-    <origin xyz="0.016431914541455865 -0.015921078340292362 0.010636931179058638" rpy="1.5415716586341253 0.014863657572835746 -0.07258247459143602"/>
+    <origin xyz="-0.009531296053436934 0.0067249256283193285 0.0075457641395848245" rpy="1.5663385979260043 0.004660654849611939 -0.010962503936608999"/>
     <axis xyz="0.0 0.0 1.0"/>
     <parent link="shoulder_link"/>
@@ -419,5 +419,5 @@
   </joint>
   <joint name="elbow_joint" type="revolute">
-    <origin xyz="-0.5996745659350029 -0.00048636814021923297 0.009405942102471837" rpy="-0.014553428819016492 -0.02173367222479105 0.02605134752247605"/>
+    <origin xyz="-0.6102152904073732 0.004328175185936848 0.0062061018415760835" rpy="-0.010057140605404025 -0.004873101280596378 0.0009330003870278563"/>
     <axis xyz="0.0 0.0 1.0"/>
     <parent link="upper_arm_link"/>
@@ -427,5 +427,5 @@
   </joint>
   <joint name="wrist_1_joint" type="revolute">
-    <origin xyz="-0.5652841488249898 0.009018813250154935 0.17706782067685806" rpy="-0.003003155878006817 0.021644677144780536 0.005398823112075103"/>
+    <origin xyz="-0.5704987376211959 0.00011153779929661173 0.19145923932465514" rpy="0.03396777184450894 0.017450246872858784 0.0036295438263922557"/>
     <axis xyz="0.0 0.0 1.0"/>
     <parent link="forearm_link"/>
@@ -435,5 +435,5 @@
   </joint>
   <joint name="wrist_2_joint" type="revolute">
-    <origin xyz="0.0031153126042543534 -0.13407407955813314 -0.01778150734076564" rpy="1.5887420852926646 0.026030532780267963 0.011990836311086397"/>
+    <origin xyz="-0.0017524887429481704 -0.12494427019129475 -0.007826529452888942" rpy="1.5218680988243996 -0.01628060509339201 -0.008227162828881624"/>
     <axis xyz="0.0 0.0 1.0"/>
     <parent link="wrist_1_link"/>
@@ -443,5 +443,5 @@
   </joint>
   <joint name="wrist_3_joint" type="revolute">
-    <origin xyz="-0.013741436377825881 0.10116111685658188 -0.008882501308609786" rpy="1.563230653741768 3.171288905523689 3.159559083662778"/>
+    <origin xyz="-0.0010531673461660613 0.10902818800654597 -0.00782207531345751" rpy="1.604132174646816 3.2263459683256017 3.0950684569871245"/>
     <axis xyz="0.0 0.0 1.0"/>
     <parent link="wrist_2_link"/>
@@ -555,5 +555,5 @@
   </joint>
   <joint name="rgb_world_joint" type="fixed">
-    <origin xyz="-0.01625234687483334 0.007016927088536094 0.04058858883102345" rpy="-0.0033734439638217453 -0.00856908230693528 -0.01718724775946154"/>
+    <origin xyz="-2.2038082383793905e-17 3.0097249768286925e-17 0.030000000000000023" rpy="0.0 -0.0 0.0"/>
     <parent link="tripod_center_support"/>
     <child link="rgb_world_link"/>
@@ -694,17 +694,17 @@
     <child link="charuco_200x120_3x6"/>
   </joint>
-  <link name="charuco_200x120_3x6">
+  <link name="charuco_200x200_8x8">
     <origin xyz="0 0 0" rpy="0 0 0"/>
-    <visual name="upper_arm_pattern_visual">
+    <visual name="hand_pattern_visual">
       <origin xyz="0 0 0" rpy="0 0 0"/>
       <geometry>
-        <mesh filename="package://atom_worlds/pattern/models/charuco_200x120_3x6_30_22_DICT_7X7/model.dae"/>
-      </geometry>
-    </visual>
-  </link>
-  <joint name="upper_arm_link-charuco_200x120_3x6" type="fixed">
-    <origin xyz="-0.24724257841518812 0.027060264928568997 0.09275845601095882" rpy="0.17982634684246238 -0.07152623039388409 3.114638642012699"/>
-    <parent link="upper_arm_link"/>
-    <child link="charuco_200x120_3x6"/>
+        <mesh filename="package://atom_worlds/pattern/models/charuco_200x200_8x8_20_15_DICT_4x4/model.dae"/>
+      </geometry>
+    </visual>
+  </link>
+  <joint name="flange-charuco_200x200_8x8" type="fixed">
+    <origin xyz="0.06284689449174259 -0.06169188719256874 -0.0021115299484201298" rpy="0.0549892021296988 0.009459459824831469 -0.03629135780865045"/>
+    <parent link="flange"/>
+    <child link="charuco_200x200_8x8"/>
   </joint>
 </robot>
