Commit message: #804 adding spjbot

File: atom_examples/jcpbbot/jcpbbot_calibration/urdf/optimized_w_pattern.urdf.xacro (robot description, xacro)
@@ -400,5 +400,5 @@
   </joint>
   <joint name="shoulder_pan_joint" type="revolute">
-    <origin xyz="0.0 0.0 0.1807" rpy="0.0 0.0 0.008890193659224334"/>
+    <origin xyz="0.0 0.0 0.1807" rpy="0.0 0.0 0.00014031039604744884"/>
     <axis xyz="0.0 0.0 1.0"/>
     <parent link="base_link_inertia"/>
@@ -408,5 +408,5 @@
   </joint>
   <joint name="shoulder_lift_joint" type="revolute">
-    <origin xyz="0.0 0.0 0.0" rpy="1.570796327 0.0 0.008890171935160953"/>
+    <origin xyz="0.0 0.0 0.0" rpy="1.570796327 0.0 -0.0009261595168105932"/>
     <axis xyz="0.0 0.0 1.0"/>
     <parent link="shoulder_link"/>
@@ -416,5 +416,5 @@
   </joint>
   <joint name="elbow_joint" type="revolute">
-    <origin xyz="-0.6127 0.0 0.0" rpy="0.0 0.0 0.025686301279139782"/>
+    <origin xyz="-0.6127 0.0 0.0" rpy="0.0 0.0 -0.00010839958495199559"/>
     <axis xyz="0.0 0.0 1.0"/>
     <parent link="upper_arm_link"/>
@@ -424,5 +424,5 @@
   </joint>
   <joint name="wrist_1_joint" type="revolute">
-    <origin xyz="-0.57155 0.0 0.17415" rpy="0.0 0.0 -0.03120098064039958"/>
+    <origin xyz="-0.57155 0.0 0.17415" rpy="0.0 0.0 -0.00029681911014016964"/>
     <axis xyz="0.0 0.0 1.0"/>
     <parent link="forearm_link"/>
@@ -432,5 +432,5 @@
   </joint>
   <joint name="wrist_2_joint" type="revolute">
-    <origin xyz="0.0 -0.11985 -2.458164590756244e-11" rpy="1.570796327 0.0 -0.021298137887970636"/>
+    <origin xyz="0.0 -0.11985 -2.458164590756244e-11" rpy="1.570796327 0.0 -0.000302218444609945"/>
     <axis xyz="0.0 0.0 1.0"/>
     <parent link="wrist_1_link"/>
@@ -440,5 +440,5 @@
   </joint>
   <joint name="wrist_3_joint" type="revolute">
-    <origin xyz="0.0 0.11655 -2.390480459346185e-11" rpy="1.570796326589793 3.141592653589793 3.13075084398692"/>
+    <origin xyz="0.0 0.11655 -2.390480459346185e-11" rpy="1.570796326589793 3.141592653589793 3.1661151174607403"/>
     <axis xyz="0.0 0.0 1.0"/>
     <parent link="wrist_2_link"/>
@@ -496,5 +496,5 @@
   </joint>
   <joint name="rgb_hand_joint" type="fixed">
-    <origin xyz="-0.021655607917021997 -0.00390675426651832 0.06475692382180025" rpy="0.03044414300186205 0.0013822999375349206 0.0008670472196217079"/>
+    <origin xyz="-0.019982951884471575 -0.001961981172213678 0.06491048040896849" rpy="0.025530448434516823 0.0005159001432154428 -0.00020622759433453703"/>
     <parent link="flange"/>
     <child link="rgb_hand_link"/>
@@ -573,5 +573,5 @@
   </link>
   <joint name="world-pattern_link" type="fixed">
-    <origin xyz="-1.0770226772570606 0.2931901408646521 0.8003184404186438" rpy="3.1217472174026617 0.03275960050931226 0.029816861385440114"/>
+    <origin xyz="-1.0735925587747162 0.29069768954733965 0.8086384083085831" rpy="3.121567682705762 0.005247331692640813 0.022879484524049337"/>
     <parent link="world"/>
     <child link="pattern_link"/>
