Commit message: Close #824

File: atom_examples/riwmpbot/riwmpbot_calibration/urdf/optimized/optimized_2024_01_11-05_11_26_PM.urdf.xacro (robot description, xacro)
@@ -403,5 +403,5 @@
   </joint>
   <joint name="shoulder_pan_joint" type="revolute">
-    <origin xyz="0.0 0.0 0.1807" rpy="0.0 0.0 -0.08207204208585493"/>
+    <origin xyz="0.0 0.0 0.1807" rpy="0.0 0.0 -0.08201689992593077"/>
     <axis xyz="0.0 0.0 1.0"/>
     <parent link="base_link_inertia"/>
@@ -411,5 +411,5 @@
   </joint>
   <joint name="shoulder_lift_joint" type="revolute">
-    <origin xyz="0.0 0.0 0.0" rpy="1.570796327 0.0 0.05436123631567176"/>
+    <origin xyz="0.0 0.0 0.0" rpy="1.570796327 0.0 0.054295445866449514"/>
     <axis xyz="0.0 0.0 1.0"/>
     <parent link="shoulder_link"/>
@@ -419,5 +419,5 @@
   </joint>
   <joint name="elbow_joint" type="revolute">
-    <origin xyz="-0.6127 0.0 0.0" rpy="0.0 0.0 0.004078404020126384"/>
+    <origin xyz="-0.6127 0.0 0.0" rpy="0.0 0.0 0.004071350423621178"/>
     <axis xyz="0.0 0.0 1.0"/>
     <parent link="upper_arm_link"/>
@@ -427,5 +427,5 @@
   </joint>
   <joint name="wrist_1_joint" type="revolute">
-    <origin xyz="-0.57155 0.0 0.17415" rpy="0.0 0.0 0.001249152402600338"/>
+    <origin xyz="-0.57155 0.0 0.17415" rpy="0.0 0.0 0.001249043537771606"/>
     <axis xyz="0.0 0.0 1.0"/>
     <parent link="forearm_link"/>
@@ -435,5 +435,5 @@
   </joint>
   <joint name="wrist_2_joint" type="revolute">
-    <origin xyz="0.0 -0.11985 -2.458164590756244e-11" rpy="1.570796327 0.0 -0.0031671515977441554"/>
+    <origin xyz="0.0 -0.11985 -2.458164590756244e-11" rpy="1.570796327 0.0 -0.0025378026514718045"/>
     <axis xyz="0.0 0.0 1.0"/>
     <parent link="wrist_1_link"/>
@@ -443,5 +443,5 @@
   </joint>
   <joint name="wrist_3_joint" type="revolute">
-    <origin xyz="0.0 0.11655 -2.390480459346185e-11" rpy="1.570796326589793 3.141592653589793 3.131730950999273"/>
+    <origin xyz="0.0 0.11655 -2.390480459346185e-11" rpy="1.570796326589793 3.141592653589793 3.13143449152036"/>
     <axis xyz="0.0 0.0 1.0"/>
     <parent link="wrist_2_link"/>
@@ -555,5 +555,5 @@
   </joint>
   <joint name="rgb_world_joint" type="fixed">
-    <origin xyz="-0.02804793754764452 0.02875482141608135 -0.010685232209137863" rpy="0.07960990590367759 -0.009056331952273752 -0.059898132857513435"/>
+    <origin xyz="-0.0278241996218845 0.0287777554785989 -0.010541692705009223" rpy="0.07968130596450307 -0.008926821311892909 -0.059921863057529196"/>
     <parent link="tripod_center_support"/>
     <child link="rgb_world_link"/>

File: atom_examples/riwmpbot/riwmpbot_calibration/urdf/optimized/optimized_2024_01_11-05_11_53_PM.urdf.xacro (robot description, xacro)
@@ -403,5 +403,5 @@
   </joint>
   <joint name="shoulder_pan_joint" type="revolute">
-    <origin xyz="0.0 0.0 0.1807" rpy="0.0 0.0 -0.08207204208585493"/>
+    <origin xyz="0.0 0.0 0.1807" rpy="0.0 0.0 -0.05625165425337494"/>
     <axis xyz="0.0 0.0 1.0"/>
     <parent link="base_link_inertia"/>
@@ -411,5 +411,5 @@
   </joint>
   <joint name="shoulder_lift_joint" type="revolute">
-    <origin xyz="0.0 0.0 0.0" rpy="1.570796327 0.0 0.05436123631567176"/>
+    <origin xyz="0.0 0.0 0.0" rpy="1.570796327 0.0 0.001523594063923136"/>
     <axis xyz="0.0 0.0 1.0"/>
     <parent link="shoulder_link"/>
@@ -419,5 +419,5 @@
   </joint>
   <joint name="elbow_joint" type="revolute">
-    <origin xyz="-0.6127 0.0 0.0" rpy="0.0 0.0 0.004078404020126384"/>
+    <origin xyz="-0.6127 0.0 0.0" rpy="0.0 0.0 -0.0003168872004018331"/>
     <axis xyz="0.0 0.0 1.0"/>
     <parent link="upper_arm_link"/>
@@ -427,5 +427,5 @@
   </joint>
   <joint name="wrist_1_joint" type="revolute">
-    <origin xyz="-0.57155 0.0 0.17415" rpy="0.0 0.0 0.001249152402600338"/>
+    <origin xyz="-0.57155 0.0 0.17415" rpy="0.0 0.0 -0.0005063622910966569"/>
     <axis xyz="0.0 0.0 1.0"/>
     <parent link="forearm_link"/>
@@ -435,5 +435,5 @@
   </joint>
   <joint name="wrist_2_joint" type="revolute">
-    <origin xyz="0.0 -0.11985 -2.458164590756244e-11" rpy="1.570796327 0.0 -0.0031671515977441554"/>
+    <origin xyz="0.0 -0.11985 -2.458164590756244e-11" rpy="1.570796327 0.0 -0.0005243698082626411"/>
     <axis xyz="0.0 0.0 1.0"/>
     <parent link="wrist_1_link"/>
@@ -443,5 +443,5 @@
   </joint>
   <joint name="wrist_3_joint" type="revolute">
-    <origin xyz="0.0 0.11655 -2.390480459346185e-11" rpy="1.570796326589793 3.141592653589793 3.131730950999273"/>
+    <origin xyz="0.0 0.11655 -2.390480459346185e-11" rpy="1.570796326589793 3.141592653589793 3.145851420705217"/>
     <axis xyz="0.0 0.0 1.0"/>
     <parent link="wrist_2_link"/>
@@ -555,5 +555,5 @@
   </joint>
   <joint name="rgb_world_joint" type="fixed">
-    <origin xyz="-0.02804793754764452 0.02875482141608135 -0.010685232209137863" rpy="0.07960990590367759 -0.009056331952273752 -0.059898132857513435"/>
+    <origin xyz="-0.01852046309669971 0.04355794030949294 0.022928976216741517" rpy="0.018774531776997533 0.00033413141586237784 -0.05369666833386372"/>
     <parent link="tripod_center_support"/>
     <child link="rgb_world_link"/>

File: atom_examples/riwmpbot/riwmpbot_calibration/urdf/optimized/optimized_2024_01_11-05_15_12_PM.urdf.xacro (robot description, xacro)
@@ -403,5 +403,5 @@
   </joint>
   <joint name="shoulder_pan_joint" type="revolute">
-    <origin xyz="0.0 0.0 0.1807" rpy="0.0 0.0 -0.08207204208585493"/>
+    <origin xyz="0.0 0.0 0.1807" rpy="0.0 0.0 -0.05776965030841434"/>
     <axis xyz="0.0 0.0 1.0"/>
     <parent link="base_link_inertia"/>
@@ -411,5 +411,5 @@
   </joint>
   <joint name="shoulder_lift_joint" type="revolute">
-    <origin xyz="0.0 0.0 0.0" rpy="1.570796327 0.0 0.05436123631567176"/>
+    <origin xyz="0.0 0.0 0.0" rpy="1.570796327 0.0 -5.659871149584597e-05"/>
     <axis xyz="0.0 0.0 1.0"/>
     <parent link="shoulder_link"/>
@@ -419,5 +419,5 @@
   </joint>
   <joint name="elbow_joint" type="revolute">
-    <origin xyz="-0.6127 0.0 0.0" rpy="0.0 0.0 0.004078404020126384"/>
+    <origin xyz="-0.6127 0.0 0.0" rpy="0.0 0.0 -4.2263208679146634e-05"/>
     <axis xyz="0.0 0.0 1.0"/>
     <parent link="upper_arm_link"/>
@@ -427,5 +427,5 @@
   </joint>
   <joint name="wrist_1_joint" type="revolute">
-    <origin xyz="-0.57155 0.0 0.17415" rpy="0.0 0.0 0.001249152402600338"/>
+    <origin xyz="-0.57155 0.0 0.17415" rpy="0.0 0.0 6.929046592161943e-06"/>
     <axis xyz="0.0 0.0 1.0"/>
     <parent link="forearm_link"/>
@@ -435,5 +435,5 @@
   </joint>
   <joint name="wrist_2_joint" type="revolute">
-    <origin xyz="0.0 -0.11985 -2.458164590756244e-11" rpy="1.570796327 0.0 -0.0031671515977441554"/>
+    <origin xyz="0.0 -0.11985 -2.458164590756244e-11" rpy="1.570796327 0.0 -0.0003960192397898969"/>
     <axis xyz="0.0 0.0 1.0"/>
     <parent link="wrist_1_link"/>
@@ -443,5 +443,5 @@
   </joint>
   <joint name="wrist_3_joint" type="revolute">
-    <origin xyz="0.0 0.11655 -2.390480459346185e-11" rpy="1.570796326589793 3.141592653589793 3.131730950999273"/>
+    <origin xyz="0.0 0.11655 -2.390480459346185e-11" rpy="1.570796326589793 3.141592653589793 3.1354885886874353"/>
     <axis xyz="0.0 0.0 1.0"/>
     <parent link="wrist_2_link"/>
@@ -555,5 +555,5 @@
   </joint>
   <joint name="rgb_world_joint" type="fixed">
-    <origin xyz="-0.02804793754764452 0.02875482141608135 -0.010685232209137863" rpy="0.07960990590367759 -0.009056331952273752 -0.059898132857513435"/>
+    <origin xyz="-0.018824022470692075 0.04569474543337988 0.023766732947070403" rpy="0.018065337851757183 0.0009183727921052177 -0.05553702603545949"/>
     <parent link="tripod_center_support"/>
     <child link="rgb_world_link"/>

File: atom_examples/riwmpbot/riwmpbot_calibration/urdf/optimized/optimized_2024_01_11-05_15_37_PM.urdf.xacro (robot description, xacro)
@@ -403,5 +403,5 @@
   </joint>
   <joint name="shoulder_pan_joint" type="revolute">
-    <origin xyz="0.0 0.0 0.1807" rpy="0.0 0.0 -0.08207204208585493"/>
+    <origin xyz="0.0 0.0 0.1807" rpy="0.0 0.0 -0.055824784805964034"/>
     <axis xyz="0.0 0.0 1.0"/>
     <parent link="base_link_inertia"/>
@@ -411,5 +411,5 @@
   </joint>
   <joint name="shoulder_lift_joint" type="revolute">
-    <origin xyz="0.0 0.0 0.0" rpy="1.570796327 0.0 0.05436123631567176"/>
+    <origin xyz="0.0 0.0 0.0" rpy="1.570796327 0.0 0.0004191340405698486"/>
     <axis xyz="0.0 0.0 1.0"/>
     <parent link="shoulder_link"/>
@@ -419,5 +419,5 @@
   </joint>
   <joint name="elbow_joint" type="revolute">
-    <origin xyz="-0.6127 0.0 0.0" rpy="0.0 0.0 0.004078404020126384"/>
+    <origin xyz="-0.6127 0.0 0.0" rpy="0.0 0.0 -0.00012199234274091296"/>
     <axis xyz="0.0 0.0 1.0"/>
     <parent link="upper_arm_link"/>
@@ -427,5 +427,5 @@
   </joint>
   <joint name="wrist_1_joint" type="revolute">
-    <origin xyz="-0.57155 0.0 0.17415" rpy="0.0 0.0 0.001249152402600338"/>
+    <origin xyz="-0.57155 0.0 0.17415" rpy="0.0 0.0 0.0003049186915297218"/>
     <axis xyz="0.0 0.0 1.0"/>
     <parent link="forearm_link"/>
@@ -435,5 +435,5 @@
   </joint>
   <joint name="wrist_2_joint" type="revolute">
-    <origin xyz="0.0 -0.11985 -2.458164590756244e-11" rpy="1.570796327 0.0 -0.0031671515977441554"/>
+    <origin xyz="0.0 -0.11985 -2.458164590756244e-11" rpy="1.570796327 0.0 -0.00028458414088896374"/>
     <axis xyz="0.0 0.0 1.0"/>
     <parent link="wrist_1_link"/>
@@ -443,5 +443,5 @@
   </joint>
   <joint name="wrist_3_joint" type="revolute">
-    <origin xyz="0.0 0.11655 -2.390480459346185e-11" rpy="1.570796326589793 3.141592653589793 3.131730950999273"/>
+    <origin xyz="0.0 0.11655 -2.390480459346185e-11" rpy="1.570796326589793 3.141592653589793 3.145431949637309"/>
     <axis xyz="0.0 0.0 1.0"/>
     <parent link="wrist_2_link"/>
@@ -555,5 +555,5 @@
   </joint>
   <joint name="rgb_world_joint" type="fixed">
-    <origin xyz="-0.02804793754764452 0.02875482141608135 -0.010685232209137863" rpy="0.07960990590367759 -0.009056331952273752 -0.059898132857513435"/>
+    <origin xyz="-0.018316541647082324 0.0438544120262841 0.023722283773137804" rpy="0.017774018014233776 0.0008023816599838934 -0.05345578161134431"/>
     <parent link="tripod_center_support"/>
     <child link="rgb_world_link"/>

File: atom_examples/riwmpbot/riwmpbot_calibration/urdf/optimized/optimized_2024_01_11-05_20_31_PM.urdf.xacro (robot description, xacro)
@@ -403,5 +403,5 @@
   </joint>
   <joint name="shoulder_pan_joint" type="revolute">
-    <origin xyz="0.0 0.0 0.1807" rpy="0.0 0.0 -0.08207204208585493"/>
+    <origin xyz="0.0 0.0 0.1807" rpy="0.0 0.0 -0.07539656561108604"/>
     <axis xyz="0.0 0.0 1.0"/>
     <parent link="base_link_inertia"/>
@@ -411,5 +411,5 @@
   </joint>
   <joint name="shoulder_lift_joint" type="revolute">
-    <origin xyz="0.0 0.0 0.0" rpy="1.570796327 0.0 0.05436123631567176"/>
+    <origin xyz="0.0 0.0 0.0" rpy="1.570796327 0.0 0.0429353399369651"/>
     <axis xyz="0.0 0.0 1.0"/>
     <parent link="shoulder_link"/>
@@ -419,5 +419,5 @@
   </joint>
   <joint name="elbow_joint" type="revolute">
-    <origin xyz="-0.6127 0.0 0.0" rpy="0.0 0.0 0.004078404020126384"/>
+    <origin xyz="-0.6127 0.0 0.0" rpy="0.0 0.0 0.000334279950863777"/>
     <axis xyz="0.0 0.0 1.0"/>
     <parent link="upper_arm_link"/>
@@ -427,5 +427,5 @@
   </joint>
   <joint name="wrist_1_joint" type="revolute">
-    <origin xyz="-0.57155 0.0 0.17415" rpy="0.0 0.0 0.001249152402600338"/>
+    <origin xyz="-0.57155 0.0 0.17415" rpy="0.0 0.0 -0.007349029915744015"/>
     <axis xyz="0.0 0.0 1.0"/>
     <parent link="forearm_link"/>
@@ -435,5 +435,5 @@
   </joint>
   <joint name="wrist_2_joint" type="revolute">
-    <origin xyz="0.0 -0.11985 -2.458164590756244e-11" rpy="1.570796327 0.0 -0.0031671515977441554"/>
+    <origin xyz="0.0 -0.11985 -2.458164590756244e-11" rpy="1.570796327 0.0 -0.002317302945072222"/>
     <axis xyz="0.0 0.0 1.0"/>
     <parent link="wrist_1_link"/>
@@ -443,5 +443,5 @@
   </joint>
   <joint name="wrist_3_joint" type="revolute">
-    <origin xyz="0.0 0.11655 -2.390480459346185e-11" rpy="1.570796326589793 3.141592653589793 3.131730950999273"/>
+    <origin xyz="0.0 0.11655 -2.390480459346185e-11" rpy="1.570796326589793 3.141592653589793 3.141085006480729"/>
     <axis xyz="0.0 0.0 1.0"/>
     <parent link="wrist_2_link"/>
@@ -555,5 +555,5 @@
   </joint>
   <joint name="rgb_world_joint" type="fixed">
-    <origin xyz="-0.02804793754764452 0.02875482141608135 -0.010685232209137863" rpy="0.07960990590367759 -0.009056331952273752 -0.059898132857513435"/>
+    <origin xyz="-0.02399444226746137 0.029973311766144685 -0.0033393634601115714" rpy="0.06243562243480677 -0.007104716239631031 -0.05889872193683924"/>
     <parent link="tripod_center_support"/>
     <child link="rgb_world_link"/>

File: atom_examples/riwmpbot/riwmpbot_calibration/urdf/optimized_w_pattern.urdf.xacro (robot description, xacro)
@@ -403,5 +403,5 @@
   </joint>
   <joint name="shoulder_pan_joint" type="revolute">
-    <origin xyz="0.0 0.0 0.1807" rpy="0.0 0.0 -0.05625165425337494"/>
+    <origin xyz="0.0 0.0 0.1807" rpy="0.0 0.0 -0.08207204208585493"/>
     <axis xyz="0.0 0.0 1.0"/>
     <parent link="base_link_inertia"/>
@@ -411,5 +411,5 @@
   </joint>
   <joint name="shoulder_lift_joint" type="revolute">
-    <origin xyz="0.0 0.0 0.0" rpy="1.570796327 0.0 0.001523594063923136"/>
+    <origin xyz="0.0 0.0 0.0" rpy="1.570796327 0.0 0.05436123631567176"/>
     <axis xyz="0.0 0.0 1.0"/>
     <parent link="shoulder_link"/>
@@ -419,5 +419,5 @@
   </joint>
   <joint name="elbow_joint" type="revolute">
-    <origin xyz="-0.6127 0.0 0.0" rpy="0.0 0.0 -0.0003168872004018331"/>
+    <origin xyz="-0.6127 0.0 0.0" rpy="0.0 0.0 0.004078404020126384"/>
     <axis xyz="0.0 0.0 1.0"/>
     <parent link="upper_arm_link"/>
@@ -427,5 +427,5 @@
   </joint>
   <joint name="wrist_1_joint" type="revolute">
-    <origin xyz="-0.57155 0.0 0.17415" rpy="0.0 0.0 -0.0005063622910966569"/>
+    <origin xyz="-0.57155 0.0 0.17415" rpy="0.0 0.0 0.001249152402600338"/>
     <axis xyz="0.0 0.0 1.0"/>
     <parent link="forearm_link"/>
@@ -435,5 +435,5 @@
   </joint>
   <joint name="wrist_2_joint" type="revolute">
-    <origin xyz="0.0 -0.11985 -2.458164590756244e-11" rpy="1.570796327 0.0 -0.0005243698082626411"/>
+    <origin xyz="0.0 -0.11985 -2.458164590756244e-11" rpy="1.570796327 0.0 -0.0031671515977441554"/>
     <axis xyz="0.0 0.0 1.0"/>
     <parent link="wrist_1_link"/>
@@ -443,5 +443,5 @@
   </joint>
   <joint name="wrist_3_joint" type="revolute">
-    <origin xyz="0.0 0.11655 -2.390480459346185e-11" rpy="1.570796326589793 3.141592653589793 3.145851420705217"/>
+    <origin xyz="0.0 0.11655 -2.390480459346185e-11" rpy="1.570796326589793 3.141592653589793 3.131730950999273"/>
     <axis xyz="0.0 0.0 1.0"/>
     <parent link="wrist_2_link"/>
@@ -555,5 +555,5 @@
   </joint>
   <joint name="rgb_world_joint" type="fixed">
-    <origin xyz="-0.01852046309669971 0.04355794030949294 0.022928976216741517" rpy="0.018774531776997533 0.00033413141586237784 -0.05369666833386372"/>
+    <origin xyz="-0.02804793754764452 0.02875482141608135 -0.010685232209137863" rpy="0.07960990590367759 -0.009056331952273752 -0.059898132857513435"/>
     <parent link="tripod_center_support"/>
     <child link="rgb_world_link"/>
@@ -694,18 +694,4 @@
     <child link="charuco_200x120_3x6"/>
   </joint>
-  <link name="charuco_170x100_3x6">
-    <origin xyz="0 0 0" rpy="0 0 0"/>
-    <visual name="forearm_pattern_visual">
-      <origin xyz="0 0 0" rpy="0 0 0"/>
-      <geometry>
-        <mesh filename="package://atom_worlds/pattern/models/charuco_170x100_3x6_25_18_DICT_6X6/model.dae"/>
-      </geometry>
-    </visual>
-  </link>
-  <joint name="forearm_link-charuco_170x100_3x6" type="fixed">
-    <origin xyz="-0.19991939172654224 0.019908773347669356 -0.029667247195872347" rpy="-8.580415694149842e-05 -0.0027796983125768456 3.140571696094266"/>
-    <parent link="forearm_link"/>
-    <child link="charuco_170x100_3x6"/>
-  </joint>
   <link name="charuco_200x200_8x8">
     <origin xyz="0 0 0" rpy="0 0 0"/>
@@ -718,21 +704,7 @@
   </link>
   <joint name="flange-charuco_200x200_8x8" type="fixed">
-    <origin xyz="0.060207072669968005 -0.059545882239939146 0.0009528583981800399" rpy="-0.005252217162090667 0.0006430595110670217 0.0005278650964964551"/>
+    <origin xyz="0.06042907727439765 -0.05970960104276578 0.0005633484812680199" rpy="0.0036482304087431037 0.002681590952068309 -0.0007273360247412384"/>
     <parent link="flange"/>
     <child link="charuco_200x200_8x8"/>
   </joint>
-  <link name="charuco_200x120_3x6">
-    <origin xyz="0 0 0" rpy="0 0 0"/>
-    <visual name="upper_arm_pattern_visual">
-      <origin xyz="0 0 0" rpy="0 0 0"/>
-      <geometry>
-        <mesh filename="package://atom_worlds/pattern/models/charuco_200x120_3x6_30_22_DICT_7X7/model.dae"/>
-      </geometry>
-    </visual>
-  </link>
-  <joint name="upper_arm_link-charuco_200x120_3x6" type="fixed">
-    <origin xyz="-0.24018329232428023 0.030002889981482102 0.09056138171280471" rpy="0.0008115095891808838 -0.00022301930081180068 3.139962337622029"/>
-    <parent link="upper_arm_link"/>
-    <child link="charuco_200x120_3x6"/>
-  </joint>
 </robot>
