Commit message: Close #815

File: atom_examples/riwmpbot/riwmpbot_calibration/urdf/initial_estimate.urdf.xacro (robot description, xacro)
@@ -144,6 +144,6 @@
         </color_rgb_rviz>
     </xacro:rgb_camera>
-    <!-- charuco 200x200_4x4 link-->
-    <link name="charuco_200x200_4x4">
+    <!-- charuco 200x200_8x8 link-->
+    <link name="charuco_200x200_8x8">
         <visual>
             <origin xyz="0 0 0" rpy="0 0 0" />
@@ -153,5 +153,5 @@
             </geometry>
         </visual>
-        <collision name="charuco_200x200_4x4_collision">
+        <collision name="charuco_200x200_8x8_collision">
             <origin xyz="0 0 0" rpy="0 0 0" />
             <geometry>
@@ -167,7 +167,7 @@
     </link>
     <!-- tripod plate to tripod center support -->
-    <joint name="flange_to_charuco_200x200_4x4" type="fixed">
+    <joint name="flange_to_charuco_200x200_8x8" type="fixed">
         <parent link="flange" />
-        <child link="charuco_200x200_4x4"/>
+        <child link="charuco_200x200_8x8"/>
         <origin xyz="0.06 -0.06 0" rpy="0 0 0" />
     </joint>

File: atom_examples/riwmpbot/riwmpbot_calibration/urdf/optimized/optimized_2024_01_06-06_09_47_PM.urdf.xacro (robot description, xacro)
@@ -622,5 +622,5 @@
     </sensor>
   </gazebo>
-  <link name="charuco_200x200_4x4">
+  <link name="charuco_200x200_8x8">
     <inertial>
       <origin xyz="0.0 0.0 0.0" rpy="0.0 0.0 0.0"/>
@@ -634,5 +634,5 @@
       </geometry>
     </visual>
-    <collision name="charuco_200x200_4x4_collision">
+    <collision name="charuco_200x200_8x8_collision">
       <origin xyz="0.0 0.0 0.0" rpy="0.0 0.0 0.0"/>
       <geometry>
@@ -641,8 +641,8 @@
     </collision>
   </link>
-  <joint name="flange_to_charuco_200x200_4x4" type="fixed">
+  <joint name="flange_to_charuco_200x200_8x8" type="fixed">
     <origin xyz="0.06 -0.06 0.0" rpy="0.0 0.0 0.0"/>
     <parent link="flange"/>
-    <child link="charuco_200x200_4x4"/>
+    <child link="charuco_200x200_8x8"/>
   </joint>
   <link name="charuco_170x100_3x6">

File: atom_examples/riwmpbot/riwmpbot_calibration/urdf/optimized/optimized_2024_01_06-06_19_31_PM.urdf.xacro (robot description, xacro)
@@ -622,5 +622,5 @@
     </sensor>
   </gazebo>
-  <link name="charuco_200x200_4x4">
+  <link name="charuco_200x200_8x8">
     <inertial>
       <origin xyz="0.0 0.0 0.0" rpy="0.0 0.0 0.0"/>
@@ -634,5 +634,5 @@
       </geometry>
     </visual>
-    <collision name="charuco_200x200_4x4_collision">
+    <collision name="charuco_200x200_8x8_collision">
       <origin xyz="0.0 0.0 0.0" rpy="0.0 0.0 0.0"/>
       <geometry>
@@ -641,8 +641,8 @@
     </collision>
   </link>
-  <joint name="flange_to_charuco_200x200_4x4" type="fixed">
+  <joint name="flange_to_charuco_200x200_8x8" type="fixed">
     <origin xyz="0.06 -0.06 0.0" rpy="0.0 0.0 0.0"/>
     <parent link="flange"/>
-    <child link="charuco_200x200_4x4"/>
+    <child link="charuco_200x200_8x8"/>
   </joint>
   <link name="charuco_170x100_3x6">

File: atom_examples/riwmpbot/riwmpbot_calibration/urdf/optimized/optimized_2024_01_06-06_29_12_PM.urdf.xacro (robot description, xacro)
@@ -622,5 +622,5 @@
     </sensor>
   </gazebo>
-  <link name="charuco_200x200_4x4">
+  <link name="charuco_200x200_8x8">
     <inertial>
       <origin xyz="0.0 0.0 0.0" rpy="0.0 0.0 0.0"/>
@@ -634,5 +634,5 @@
       </geometry>
     </visual>
-    <collision name="charuco_200x200_4x4_collision">
+    <collision name="charuco_200x200_8x8_collision">
       <origin xyz="0.0 0.0 0.0" rpy="0.0 0.0 0.0"/>
       <geometry>
@@ -641,8 +641,8 @@
     </collision>
   </link>
-  <joint name="flange_to_charuco_200x200_4x4" type="fixed">
+  <joint name="flange_to_charuco_200x200_8x8" type="fixed">
     <origin xyz="0.06 -0.06 0.0" rpy="0.0 0.0 0.0"/>
     <parent link="flange"/>
-    <child link="charuco_200x200_4x4"/>
+    <child link="charuco_200x200_8x8"/>
   </joint>
   <link name="charuco_170x100_3x6">

File: atom_examples/riwmpbot/riwmpbot_calibration/urdf/optimized/optimized_2024_01_06-06_34_29_PM.urdf.xacro (robot description, xacro)
@@ -403,5 +403,5 @@
   </joint>
   <joint name="shoulder_pan_joint" type="revolute">
-    <origin xyz="0.030013588573195266 0.05686696227252827 0.1635094773256277" rpy="0.05702852003551948 0.09205097399777515 0.05210776731467597"/>
+    <origin xyz="0.00024422376785000196 0.00013036195489719884 0.1812143296649731" rpy="-0.0005934056130731003 -0.00024722274587935726 0.005601691224054914"/>
     <axis xyz="0.0 0.0 1.0"/>
     <parent link="base_link_inertia"/>
@@ -411,5 +411,5 @@
   </joint>
   <joint name="shoulder_lift_joint" type="revolute">
-    <origin xyz="2.0976375909276394e-06 -0.00046264991059465766 -0.016123245770184376" rpy="1.5716681713317302 0.05447586190727257 -0.009630583279776584"/>
+    <origin xyz="-0.00011717272253161418 0.00021600724855901999 0.0005097604016397806" rpy="1.5739013839224691 0.004451822615207797 -0.01927691121593465"/>
     <axis xyz="0.0 0.0 1.0"/>
     <parent link="shoulder_link"/>
@@ -419,5 +419,5 @@
   </joint>
   <joint name="elbow_joint" type="revolute">
-    <origin xyz="-0.6122954982521817 -0.005729943615135425 0.0006184984139877967" rpy="0.00011930474567768142 -0.0007059121669211998 -0.005423710553731192"/>
+    <origin xyz="-0.6121110056897291 0.009173802880366127 -0.0001828252231203098" rpy="-0.0005967709703862414 -0.0006783112732437526 0.005211744478394779"/>
     <axis xyz="0.0 0.0 1.0"/>
     <parent link="upper_arm_link"/>
@@ -427,5 +427,5 @@
   </joint>
   <joint name="wrist_1_joint" type="revolute">
-    <origin xyz="-0.571211894006938 -0.00850449190647048 0.17324964690287908" rpy="-0.00020369853628720362 -0.0004703033563587233 0.009884308896398939"/>
+    <origin xyz="-0.5710410747161365 -0.005042934244336245 0.1737803583328213" rpy="-0.009512958957014386 0.002731661668813146 -0.00895497938033842"/>
     <axis xyz="0.0 0.0 1.0"/>
     <parent link="forearm_link"/>
@@ -435,5 +435,5 @@
   </joint>
   <joint name="wrist_2_joint" type="revolute">
-    <origin xyz="0.0005758340866357628 -0.1198737073402209 -0.0009731294050206196" rpy="1.5707379597204476 0.005352130258525568 0.0003898441178316597"/>
+    <origin xyz="-0.0031237413818445527 -0.11797686731189387 -0.0007884643429365136" rpy="1.5710837063006033 -0.008097364504885173 -0.0010247604414818578"/>
     <axis xyz="0.0 0.0 1.0"/>
     <parent link="wrist_1_link"/>
@@ -443,5 +443,5 @@
   </joint>
   <joint name="wrist_3_joint" type="revolute">
-    <origin xyz="0.00019304377429973438 0.11687495721172371 6.640346168519403e-05" rpy="1.5700101538005655 3.142121934838785 3.1364306908615047"/>
+    <origin xyz="0.00040774849156171975 0.11704761717978333 -0.0017145561909262695" rpy="1.5579416274425038 3.140638839916929 3.170316915425923"/>
     <axis xyz="0.0 0.0 1.0"/>
     <parent link="wrist_2_link"/>
@@ -555,5 +555,5 @@
   </joint>
   <joint name="rgb_world_joint" type="fixed">
-    <origin xyz="0.014151350146913986 0.014497285934665066 0.08255401423915493" rpy="-0.11612192145829489 0.06648091025609308 0.07181956490236753"/>
+    <origin xyz="-4.4332017122705513e-16 -2.3617318500109856e-16 0.030000000000000106" rpy="4.391519488174491e-16 -2.0777236658116091e-16 -3.703499248994207e-16"/>
     <parent link="tripod_center_support"/>
     <child link="rgb_world_link"/>

File: atom_examples/riwmpbot/riwmpbot_calibration/urdf/optimized/optimized_2024_01_09-12_06_40_PM.urdf.xacro (robot description, xacro)
@@ -403,5 +403,5 @@
   </joint>
   <joint name="shoulder_pan_joint" type="revolute">
-    <origin xyz="0.030013588573195266 0.05686696227252827 0.1635094773256277" rpy="0.05702852003551948 0.09205097399777515 0.05210776731467597"/>
+    <origin xyz="0.0 0.0 0.1807" rpy="0.0 0.0 0.012076744034826033"/>
     <axis xyz="0.0 0.0 1.0"/>
     <parent link="base_link_inertia"/>
@@ -411,5 +411,5 @@
   </joint>
   <joint name="shoulder_lift_joint" type="revolute">
-    <origin xyz="2.0976375909276394e-06 -0.00046264991059465766 -0.016123245770184376" rpy="1.5716681713317302 0.05447586190727257 -0.009630583279776584"/>
+    <origin xyz="0.0 0.0 0.0" rpy="1.570796327 0.0 0.004911877847328692"/>
     <axis xyz="0.0 0.0 1.0"/>
     <parent link="shoulder_link"/>
@@ -419,5 +419,5 @@
   </joint>
   <joint name="elbow_joint" type="revolute">
-    <origin xyz="-0.6122954982521817 -0.005729943615135425 0.0006184984139877967" rpy="0.00011930474567768142 -0.0007059121669211998 -0.005423710553731192"/>
+    <origin xyz="-0.6127 0.0 0.0" rpy="0.0 0.0 -0.0008491953796697204"/>
     <axis xyz="0.0 0.0 1.0"/>
     <parent link="upper_arm_link"/>
@@ -427,5 +427,5 @@
   </joint>
   <joint name="wrist_1_joint" type="revolute">
-    <origin xyz="-0.571211894006938 -0.00850449190647048 0.17324964690287908" rpy="-0.00020369853628720362 -0.0004703033563587233 0.009884308896398939"/>
+    <origin xyz="-0.57155 0.0 0.17415" rpy="0.0 0.0 -0.000767961357501709"/>
     <axis xyz="0.0 0.0 1.0"/>
     <parent link="forearm_link"/>
@@ -435,5 +435,5 @@
   </joint>
   <joint name="wrist_2_joint" type="revolute">
-    <origin xyz="0.0005758340866357628 -0.1198737073402209 -0.0009731294050206196" rpy="1.5707379597204476 0.005352130258525568 0.0003898441178316597"/>
+    <origin xyz="0.0 -0.11985 -2.458164590756244e-11" rpy="1.570796327 0.0 -0.00011766774487074417"/>
     <axis xyz="0.0 0.0 1.0"/>
     <parent link="wrist_1_link"/>
@@ -443,5 +443,5 @@
   </joint>
   <joint name="wrist_3_joint" type="revolute">
-    <origin xyz="0.00019304377429973438 0.11687495721172371 6.640346168519403e-05" rpy="1.5700101538005655 3.142121934838785 3.1364306908615047"/>
+    <origin xyz="0.0 0.11655 -2.390480459346185e-11" rpy="1.570796326589793 3.141592653589793 3.0967987524622913"/>
     <axis xyz="0.0 0.0 1.0"/>
     <parent link="wrist_2_link"/>
@@ -555,5 +555,5 @@
   </joint>
   <joint name="rgb_world_joint" type="fixed">
-    <origin xyz="0.014151350146913986 0.014497285934665066 0.08255401423915493" rpy="-0.11612192145829489 0.06648091025609308 0.07181956490236753"/>
+    <origin xyz="-0.005808658073823805 -0.011809027207634474 0.027179032469690192" rpy="0.0022250970542084234 0.046702672451380406 0.05467002375672697"/>
     <parent link="tripod_center_support"/>
     <child link="rgb_world_link"/>

File: atom_examples/riwmpbot/riwmpbot_calibration/urdf/optimized/optimized_2024_01_09-12_09_56_PM.urdf.xacro (robot description, xacro)
@@ -403,5 +403,5 @@
   </joint>
   <joint name="shoulder_pan_joint" type="revolute">
-    <origin xyz="0.030013588573195266 0.05686696227252827 0.1635094773256277" rpy="0.05702852003551948 0.09205097399777515 0.05210776731467597"/>
+    <origin xyz="0.0 0.0 0.1807" rpy="0.0 0.0 -0.0004010320695844992"/>
     <axis xyz="0.0 0.0 1.0"/>
     <parent link="base_link_inertia"/>
@@ -411,5 +411,5 @@
   </joint>
   <joint name="shoulder_lift_joint" type="revolute">
-    <origin xyz="2.0976375909276394e-06 -0.00046264991059465766 -0.016123245770184376" rpy="1.5716681713317302 0.05447586190727257 -0.009630583279776584"/>
+    <origin xyz="0.0 0.0 0.0" rpy="1.570796327 0.0 -0.00023184340814435444"/>
     <axis xyz="0.0 0.0 1.0"/>
     <parent link="shoulder_link"/>
@@ -419,5 +419,5 @@
   </joint>
   <joint name="elbow_joint" type="revolute">
-    <origin xyz="-0.6122954982521817 -0.005729943615135425 0.0006184984139877967" rpy="0.00011930474567768142 -0.0007059121669211998 -0.005423710553731192"/>
+    <origin xyz="-0.6127 0.0 0.0" rpy="0.0 0.0 0.0002801345355589936"/>
     <axis xyz="0.0 0.0 1.0"/>
     <parent link="upper_arm_link"/>
@@ -427,5 +427,5 @@
   </joint>
   <joint name="wrist_1_joint" type="revolute">
-    <origin xyz="-0.571211894006938 -0.00850449190647048 0.17324964690287908" rpy="-0.00020369853628720362 -0.0004703033563587233 0.009884308896398939"/>
+    <origin xyz="-0.57155 0.0 0.17415" rpy="0.0 0.0 -9.070024266779476e-05"/>
     <axis xyz="0.0 0.0 1.0"/>
     <parent link="forearm_link"/>
@@ -435,5 +435,5 @@
   </joint>
   <joint name="wrist_2_joint" type="revolute">
-    <origin xyz="0.0005758340866357628 -0.1198737073402209 -0.0009731294050206196" rpy="1.5707379597204476 0.005352130258525568 0.0003898441178316597"/>
+    <origin xyz="0.0 -0.11985 -2.458164590756244e-11" rpy="1.570796327 0.0 3.8259965082873196e-05"/>
     <axis xyz="0.0 0.0 1.0"/>
     <parent link="wrist_1_link"/>
@@ -443,5 +443,5 @@
   </joint>
   <joint name="wrist_3_joint" type="revolute">
-    <origin xyz="0.00019304377429973438 0.11687495721172371 6.640346168519403e-05" rpy="1.5700101538005655 3.142121934838785 3.1364306908615047"/>
+    <origin xyz="0.0 0.11655 -2.390480459346185e-11" rpy="1.570796326589793 3.141592653589793 3.1318701213327738"/>
     <axis xyz="0.0 0.0 1.0"/>
     <parent link="wrist_2_link"/>
@@ -555,5 +555,5 @@
   </joint>
   <joint name="rgb_world_joint" type="fixed">
-    <origin xyz="0.014151350146913986 0.014497285934665066 0.08255401423915493" rpy="-0.11612192145829489 0.06648091025609308 0.07181956490236753"/>
+    <origin xyz="5.894251768888878e-05 0.00022973835237531957 0.029917572365194087" rpy="3.0884984257724895e-05 0.0004951649187620921 -0.0006679800411015755"/>
     <parent link="tripod_center_support"/>
     <child link="rgb_world_link"/>

File: atom_examples/riwmpbot/riwmpbot_calibration/urdf/optimized/optimized_2024_01_09-12_16_10_PM.urdf.xacro (robot description, xacro)
@@ -403,5 +403,5 @@
   </joint>
   <joint name="shoulder_pan_joint" type="revolute">
-    <origin xyz="0.030013588573195266 0.05686696227252827 0.1635094773256277" rpy="0.05702852003551948 0.09205097399777515 0.05210776731467597"/>
+    <origin xyz="0.0 0.0 0.1807" rpy="0.0 0.0 -0.004407596928497583"/>
     <axis xyz="0.0 0.0 1.0"/>
     <parent link="base_link_inertia"/>
@@ -411,5 +411,5 @@
   </joint>
   <joint name="shoulder_lift_joint" type="revolute">
-    <origin xyz="2.0976375909276394e-06 -0.00046264991059465766 -0.016123245770184376" rpy="1.5716681713317302 0.05447586190727257 -0.009630583279776584"/>
+    <origin xyz="0.0 0.0 0.0" rpy="1.570796327 0.0 0.024400887175286705"/>
     <axis xyz="0.0 0.0 1.0"/>
     <parent link="shoulder_link"/>
@@ -419,5 +419,5 @@
   </joint>
   <joint name="elbow_joint" type="revolute">
-    <origin xyz="-0.6122954982521817 -0.005729943615135425 0.0006184984139877967" rpy="0.00011930474567768142 -0.0007059121669211998 -0.005423710553731192"/>
+    <origin xyz="-0.6127 0.0 0.0" rpy="0.0 0.0 -0.02686442540407979"/>
     <axis xyz="0.0 0.0 1.0"/>
     <parent link="upper_arm_link"/>
@@ -427,5 +427,5 @@
   </joint>
   <joint name="wrist_1_joint" type="revolute">
-    <origin xyz="-0.571211894006938 -0.00850449190647048 0.17324964690287908" rpy="-0.00020369853628720362 -0.0004703033563587233 0.009884308896398939"/>
+    <origin xyz="-0.57155 0.0 0.17415" rpy="0.0 0.0 0.04988600887799914"/>
     <axis xyz="0.0 0.0 1.0"/>
     <parent link="forearm_link"/>
@@ -435,5 +435,5 @@
   </joint>
   <joint name="wrist_2_joint" type="revolute">
-    <origin xyz="0.0005758340866357628 -0.1198737073402209 -0.0009731294050206196" rpy="1.5707379597204476 0.005352130258525568 0.0003898441178316597"/>
+    <origin xyz="0.0 -0.11985 -2.458164590756244e-11" rpy="1.570796327 0.0 0.00153508224062201"/>
     <axis xyz="0.0 0.0 1.0"/>
     <parent link="wrist_1_link"/>
@@ -443,5 +443,5 @@
   </joint>
   <joint name="wrist_3_joint" type="revolute">
-    <origin xyz="0.00019304377429973438 0.11687495721172371 6.640346168519403e-05" rpy="1.5700101538005655 3.142121934838785 3.1364306908615047"/>
+    <origin xyz="0.0 0.11655 -2.390480459346185e-11" rpy="1.570796326589793 3.141592653589793 3.0848372994307423"/>
     <axis xyz="0.0 0.0 1.0"/>
     <parent link="wrist_2_link"/>
@@ -555,5 +555,5 @@
   </joint>
   <joint name="rgb_world_joint" type="fixed">
-    <origin xyz="0.014151350146913986 0.014497285934665066 0.08255401423915493" rpy="-0.11612192145829489 0.06648091025609308 0.07181956490236753"/>
+    <origin xyz="0.006727059356489782 -0.0029517498912495724 0.030302518179022013" rpy="0.009609671594261845 -0.0005302612340337872 -0.002566826195569769"/>
     <parent link="tripod_center_support"/>
     <child link="rgb_world_link"/>

File: atom_examples/riwmpbot/riwmpbot_calibration/urdf/optimized_w_pattern.urdf.xacro (robot description, xacro)
@@ -403,5 +403,5 @@
   </joint>
   <joint name="shoulder_pan_joint" type="revolute">
-    <origin xyz="0.00010344046978209419 0.00046598326215834717 0.181258110135952" rpy="-0.0005231680686939936 -0.0001358324499671006 0.005077478546179187"/>
+    <origin xyz="0.0 0.0 0.1807" rpy="0.0 0.0 -0.0004010320695844992"/>
     <axis xyz="0.0 0.0 1.0"/>
     <parent link="base_link_inertia"/>
@@ -411,5 +411,5 @@
   </joint>
   <joint name="shoulder_lift_joint" type="revolute">
-    <origin xyz="-4.243898212575611e-05 3.0499867732174428e-05 0.0005574493960652489" rpy="1.5714015763860585 0.005230369459552412 -0.019162490089765713"/>
+    <origin xyz="0.0 0.0 0.0" rpy="1.570796327 0.0 -0.00023184340814435444"/>
     <axis xyz="0.0 0.0 1.0"/>
     <parent link="shoulder_link"/>
@@ -419,5 +419,5 @@
   </joint>
   <joint name="elbow_joint" type="revolute">
-    <origin xyz="-0.6120607313531528 0.009191813827082614 3.839286194396276e-05" rpy="-0.0001793129218587502 -0.000603818417143185 0.0030418710937143998"/>
+    <origin xyz="-0.6127 0.0 0.0" rpy="0.0 0.0 0.0002801345355589936"/>
     <axis xyz="0.0 0.0 1.0"/>
     <parent link="upper_arm_link"/>
@@ -427,5 +427,5 @@
   </joint>
   <joint name="wrist_1_joint" type="revolute">
-    <origin xyz="-0.5710651694620934 -0.006931277314576469 0.1738342544494194" rpy="7.695515136454388e-05 -0.00014551388364625724 -0.021417987999603923"/>
+    <origin xyz="-0.57155 0.0 0.17415" rpy="0.0 0.0 -9.070024266779476e-05"/>
     <axis xyz="0.0 0.0 1.0"/>
     <parent link="forearm_link"/>
@@ -435,5 +435,5 @@
   </joint>
   <joint name="wrist_2_joint" type="revolute">
-    <origin xyz="-0.00198563175106734 -0.11976740282204376 -0.0002675326371526897" rpy="1.5706504149948477 -0.016544210769609453 -0.003283559980458237"/>
+    <origin xyz="0.0 -0.11985 -2.458164590756244e-11" rpy="1.570796327 0.0 3.8259965082873196e-05"/>
     <axis xyz="0.0 0.0 1.0"/>
     <parent link="wrist_1_link"/>
@@ -443,5 +443,5 @@
   </joint>
   <joint name="wrist_3_joint" type="revolute">
-    <origin xyz="0.0008822072226631115 0.11686641816431564 -2.687987868929874e-05" rpy="1.5707879559190074 3.1355655091133166 3.1622193000532604"/>
+    <origin xyz="0.0 0.11655 -2.390480459346185e-11" rpy="1.570796326589793 3.141592653589793 3.1318701213327738"/>
     <axis xyz="0.0 0.0 1.0"/>
     <parent link="wrist_2_link"/>
@@ -555,5 +555,5 @@
   </joint>
   <joint name="rgb_world_joint" type="fixed">
-    <origin xyz="4.33572667713854e-16 1.603094455713604e-16 0.029999999999999905" rpy="-3.27021676846164e-16 -1.538215921728581e-16 2.7357838773931337e-16"/>
+    <origin xyz="5.892761652769493e-05 0.00022973835237531957 0.029917572365194087" rpy="3.0884984257724895e-05 0.0004951649187620921 -0.0006679800411015755"/>
     <parent link="tripod_center_support"/>
     <child link="rgb_world_link"/>
@@ -622,5 +622,5 @@
     </sensor>
   </gazebo>
-  <link name="charuco_200x200_4x4">
+  <link name="charuco_200x200_8x8">
     <inertial>
       <origin xyz="0.0 0.0 0.0" rpy="0.0 0.0 0.0"/>
@@ -634,5 +634,5 @@
       </geometry>
     </visual>
-    <collision name="charuco_200x200_4x4_collision">
+    <collision name="charuco_200x200_8x8_collision">
       <origin xyz="0.0 0.0 0.0" rpy="0.0 0.0 0.0"/>
       <geometry>
@@ -641,8 +641,8 @@
     </collision>
   </link>
-  <joint name="flange_to_charuco_200x200_4x4" type="fixed">
+  <joint name="flange_to_charuco_200x200_8x8" type="fixed">
     <origin xyz="0.06 -0.06 0.0" rpy="0.0 0.0 0.0"/>
     <parent link="flange"/>
-    <child link="charuco_200x200_4x4"/>
+    <child link="charuco_200x200_8x8"/>
   </joint>
   <link name="charuco_170x100_3x6">
@@ -704,5 +704,5 @@
   </link>
   <joint name="forearm_link-charuco_170x100_3x6" type="fixed">
-    <origin xyz="-0.20001992107713848 0.017544481502449968 -0.030208017365889808" rpy="-0.0002061234142036553 -0.0014701550138355006 -3.130785474359424"/>
+    <origin xyz="-0.20008580568177226 0.019919799457434204 -0.029854775295023537" rpy="-0.00036195646247965687 -0.0026743352686167533 3.140320321522196"/>
     <parent link="forearm_link"/>
     <child link="charuco_170x100_3x6"/>
@@ -718,5 +718,5 @@
   </link>
   <joint name="flange-charuco_200x200_8x8" type="fixed">
-    <origin xyz="0.059510160433123196 -0.05975327545308545 0.00020757901290140604" rpy="0.006761553091396381 2.972160527080662e-05 -0.00030985026839631285"/>
+    <origin xyz="0.06002712502628293 -0.059781613938339466 0.0002716311990354525" rpy="0.00727690753486573 0.0014890423579220797 -0.00027463328142973405"/>
     <parent link="flange"/>
     <child link="charuco_200x200_8x8"/>
@@ -732,5 +732,5 @@
   </link>
   <joint name="upper_arm_link-charuco_200x120_3x6" type="fixed">
-    <origin xyz="-0.2393934938599728 0.03366517679733379 0.09014514616049173" rpy="0.0002998413455321967 0.0012451394875890567 3.1257550667715552"/>
+    <origin xyz="-0.24010307356598123 0.029948558008097037 0.09023355977097662" rpy="0.0007155347212871894 -0.0002605057086586673 3.140345994543496"/>
     <parent link="upper_arm_link"/>
     <child link="charuco_200x120_3x6"/>
