Commit message: Close #820. Also deleted several urdf/optimized folders in atom examples.

File: atom_examples/riwmpbot/riwmpbot_calibration/urdf/optimized.urdf.xacro (robot description, xacro)
@@ -403,5 +403,5 @@
   </joint>
   <joint name="shoulder_pan_joint" type="revolute">
-    <origin xyz="0.0 0.0 0.1807" rpy="0.0 0.0 -0.08207204208585493"/>
+    <origin xyz="0.0 0.0 0.1807" rpy="0.0 0.0 -0.04301026383664127"/>
     <axis xyz="0.0 0.0 1.0"/>
     <parent link="base_link_inertia"/>
@@ -411,5 +411,5 @@
   </joint>
   <joint name="shoulder_lift_joint" type="revolute">
-    <origin xyz="0.0 0.0 0.0" rpy="1.570796327 0.0 0.05436123631567176"/>
+    <origin xyz="0.0 0.0 0.0" rpy="1.570796327 0.0 0.003839909252167141"/>
     <axis xyz="0.0 0.0 1.0"/>
     <parent link="shoulder_link"/>
@@ -419,5 +419,5 @@
   </joint>
   <joint name="elbow_joint" type="revolute">
-    <origin xyz="-0.6127 0.0 0.0" rpy="0.0 0.0 0.004078404020126384"/>
+    <origin xyz="-0.6127 0.0 0.0" rpy="0.0 0.0 0.0002082846020888875"/>
     <axis xyz="0.0 0.0 1.0"/>
     <parent link="upper_arm_link"/>
@@ -427,5 +427,5 @@
   </joint>
   <joint name="wrist_1_joint" type="revolute">
-    <origin xyz="-0.57155 0.0 0.17415" rpy="0.0 0.0 0.001249152402600338"/>
+    <origin xyz="-0.57155 0.0 0.17415" rpy="0.0 0.0 9.012209423031764e-05"/>
     <axis xyz="0.0 0.0 1.0"/>
     <parent link="forearm_link"/>
@@ -435,5 +435,5 @@
   </joint>
   <joint name="wrist_2_joint" type="revolute">
-    <origin xyz="0.0 -0.11985 -2.458164590756244e-11" rpy="1.570796327 0.0 -0.0031671515977441554"/>
+    <origin xyz="0.0 -0.11985 -2.458164590756244e-11" rpy="1.570796327 0.0 -0.0005085943213929098"/>
     <axis xyz="0.0 0.0 1.0"/>
     <parent link="wrist_1_link"/>
@@ -443,5 +443,5 @@
   </joint>
   <joint name="wrist_3_joint" type="revolute">
-    <origin xyz="0.0 0.11655 -2.390480459346185e-11" rpy="1.570796326589793 3.141592653589793 3.131730950999273"/>
+    <origin xyz="0.0 0.11655 -2.390480459346185e-11" rpy="1.570796326589793 3.141592653589793 3.1273477612817056"/>
     <axis xyz="0.0 0.0 1.0"/>
     <parent link="wrist_2_link"/>
@@ -555,5 +555,5 @@
   </joint>
   <joint name="rgb_world_joint" type="fixed">
-    <origin xyz="-0.02804793754764452 0.02875482141608135 -0.010685232209137863" rpy="0.07960990590367759 -0.009056331952273752 -0.059898132857513435"/>
+    <origin xyz="-0.01424371390973975 0.03119637180293375 0.023111965994740306" rpy="0.01733924703690017 3.200465589616032e-05 -0.040101527183436694"/>
     <parent link="tripod_center_support"/>
     <child link="rgb_world_link"/>

File: atom_examples/riwmpbot/riwmpbot_calibration/urdf/optimized_w_pattern.urdf.xacro (robot description, xacro)
@@ -403,5 +403,5 @@
   </joint>
   <joint name="shoulder_pan_joint" type="revolute">
-    <origin xyz="0.0 0.0 0.1807" rpy="0.0 0.0 -0.08207204208585493"/>
+    <origin xyz="0.0 0.0 0.1807" rpy="0.0 0.0 -0.04301026383664127"/>
     <axis xyz="0.0 0.0 1.0"/>
     <parent link="base_link_inertia"/>
@@ -411,5 +411,5 @@
   </joint>
   <joint name="shoulder_lift_joint" type="revolute">
-    <origin xyz="0.0 0.0 0.0" rpy="1.570796327 0.0 0.05436123631567176"/>
+    <origin xyz="0.0 0.0 0.0" rpy="1.570796327 0.0 0.003839909252167141"/>
     <axis xyz="0.0 0.0 1.0"/>
     <parent link="shoulder_link"/>
@@ -419,5 +419,5 @@
   </joint>
   <joint name="elbow_joint" type="revolute">
-    <origin xyz="-0.6127 0.0 0.0" rpy="0.0 0.0 0.004078404020126384"/>
+    <origin xyz="-0.6127 0.0 0.0" rpy="0.0 0.0 0.0002082846020888875"/>
     <axis xyz="0.0 0.0 1.0"/>
     <parent link="upper_arm_link"/>
@@ -427,5 +427,5 @@
   </joint>
   <joint name="wrist_1_joint" type="revolute">
-    <origin xyz="-0.57155 0.0 0.17415" rpy="0.0 0.0 0.001249152402600338"/>
+    <origin xyz="-0.57155 0.0 0.17415" rpy="0.0 0.0 9.012209423031764e-05"/>
     <axis xyz="0.0 0.0 1.0"/>
     <parent link="forearm_link"/>
@@ -435,5 +435,5 @@
   </joint>
   <joint name="wrist_2_joint" type="revolute">
-    <origin xyz="0.0 -0.11985 -2.458164590756244e-11" rpy="1.570796327 0.0 -0.0031671515977441554"/>
+    <origin xyz="0.0 -0.11985 -2.458164590756244e-11" rpy="1.570796327 0.0 -0.0005085943213929098"/>
     <axis xyz="0.0 0.0 1.0"/>
     <parent link="wrist_1_link"/>
@@ -443,5 +443,5 @@
   </joint>
   <joint name="wrist_3_joint" type="revolute">
-    <origin xyz="0.0 0.11655 -2.390480459346185e-11" rpy="1.570796326589793 3.141592653589793 3.131730950999273"/>
+    <origin xyz="0.0 0.11655 -2.390480459346185e-11" rpy="1.570796326589793 3.141592653589793 3.1273477612817056"/>
     <axis xyz="0.0 0.0 1.0"/>
     <parent link="wrist_2_link"/>
@@ -555,5 +555,5 @@
   </joint>
   <joint name="rgb_world_joint" type="fixed">
-    <origin xyz="-0.02804793754764452 0.02875482141608135 -0.010685232209137863" rpy="0.07960990590367759 -0.009056331952273752 -0.059898132857513435"/>
+    <origin xyz="-0.01424371390973975 0.03119637180293375 0.023111965994740306" rpy="0.01733924703690017 3.200465589616032e-05 -0.040101527183436694"/>
     <parent link="tripod_center_support"/>
     <child link="rgb_world_link"/>
@@ -704,5 +704,5 @@
   </link>
   <joint name="flange-charuco_200x200_8x8" type="fixed">
-    <origin xyz="0.06042907727439765 -0.05970960104276578 0.0005633484812680199" rpy="0.0036482304087431037 0.002681590952068309 -0.0007273360247412384"/>
+    <origin xyz="0.06013804387081968 -0.05970861845038463 -7.986535573664649e-05" rpy="0.01296741455882643 0.001080329541757302 -6.464771519985488e-05"/>
     <parent link="flange"/>
     <child link="charuco_200x200_8x8"/>

Commit message: #821 new calibration

File: atom_examples/riwmpbot/riwmpbot_calibration/urdf/optimized.urdf.xacro (robot description, xacro)
@@ -403,5 +403,5 @@
   </joint>
   <joint name="shoulder_pan_joint" type="revolute">
-    <origin xyz="0.0 0.0 0.1807" rpy="0.0 0.0 -0.04301026383664127"/>
+    <origin xyz="0.0 0.0 0.1807" rpy="0.0 0.0 0.038166999186922436"/>
     <axis xyz="0.0 0.0 1.0"/>
     <parent link="base_link_inertia"/>
@@ -411,5 +411,5 @@
   </joint>
   <joint name="shoulder_lift_joint" type="revolute">
-    <origin xyz="0.0 0.0 0.0" rpy="1.570796327 0.0 0.003839909252167141"/>
+    <origin xyz="0.0 0.0 0.0" rpy="1.570796327 0.0 0.0002410801554328166"/>
     <axis xyz="0.0 0.0 1.0"/>
     <parent link="shoulder_link"/>
@@ -419,5 +419,5 @@
   </joint>
   <joint name="elbow_joint" type="revolute">
-    <origin xyz="-0.6127 0.0 0.0" rpy="0.0 0.0 0.0002082846020888875"/>
+    <origin xyz="-0.6127 0.0 0.0" rpy="0.0 0.0 -0.00014109124769039037"/>
     <axis xyz="0.0 0.0 1.0"/>
     <parent link="upper_arm_link"/>
@@ -427,5 +427,5 @@
   </joint>
   <joint name="wrist_1_joint" type="revolute">
-    <origin xyz="-0.57155 0.0 0.17415" rpy="0.0 0.0 9.012209423031764e-05"/>
+    <origin xyz="-0.57155 0.0 0.17415" rpy="0.0 0.0 0.0003550199178989447"/>
     <axis xyz="0.0 0.0 1.0"/>
     <parent link="forearm_link"/>
@@ -435,5 +435,5 @@
   </joint>
   <joint name="wrist_2_joint" type="revolute">
-    <origin xyz="0.0 -0.11985 -2.458164590756244e-11" rpy="1.570796327 0.0 -0.0005085943213929098"/>
+    <origin xyz="0.0 -0.11985 -2.458164590756244e-11" rpy="1.570796327 0.0 -0.0002689963824359225"/>
     <axis xyz="0.0 0.0 1.0"/>
     <parent link="wrist_1_link"/>
@@ -443,5 +443,5 @@
   </joint>
   <joint name="wrist_3_joint" type="revolute">
-    <origin xyz="0.0 0.11655 -2.390480459346185e-11" rpy="1.570796326589793 3.141592653589793 3.1273477612817056"/>
+    <origin xyz="0.0 0.11655 -2.390480459346185e-11" rpy="1.570796326589793 3.141592653589793 3.690243256024751"/>
     <axis xyz="0.0 0.0 1.0"/>
     <parent link="wrist_2_link"/>
@@ -555,5 +555,5 @@
   </joint>
   <joint name="rgb_world_joint" type="fixed">
-    <origin xyz="-0.01424371390973975 0.03119637180293375 0.023111965994740306" rpy="0.01733924703690017 3.200465589616032e-05 -0.040101527183436694"/>
+    <origin xyz="0.014254098736259803 -0.029596611953133758 0.03441572458900362" rpy="-0.011422006499824446 0.0005894249803577792 0.035864080268757585"/>
     <parent link="tripod_center_support"/>
     <child link="rgb_world_link"/>

File: atom_examples/riwmpbot/riwmpbot_calibration/urdf/optimized_w_pattern.urdf.xacro (robot description, xacro)
@@ -403,5 +403,5 @@
   </joint>
   <joint name="shoulder_pan_joint" type="revolute">
-    <origin xyz="0.0 0.0 0.1807" rpy="0.0 0.0 -0.04301026383664127"/>
+    <origin xyz="0.0 0.0 0.1807" rpy="0.0 0.0 0.038166999186922436"/>
     <axis xyz="0.0 0.0 1.0"/>
     <parent link="base_link_inertia"/>
@@ -411,5 +411,5 @@
   </joint>
   <joint name="shoulder_lift_joint" type="revolute">
-    <origin xyz="0.0 0.0 0.0" rpy="1.570796327 0.0 0.003839909252167141"/>
+    <origin xyz="0.0 0.0 0.0" rpy="1.570796327 0.0 0.0002410801554328166"/>
     <axis xyz="0.0 0.0 1.0"/>
     <parent link="shoulder_link"/>
@@ -419,5 +419,5 @@
   </joint>
   <joint name="elbow_joint" type="revolute">
-    <origin xyz="-0.6127 0.0 0.0" rpy="0.0 0.0 0.0002082846020888875"/>
+    <origin xyz="-0.6127 0.0 0.0" rpy="0.0 0.0 -0.00014109124769039037"/>
     <axis xyz="0.0 0.0 1.0"/>
     <parent link="upper_arm_link"/>
@@ -427,5 +427,5 @@
   </joint>
   <joint name="wrist_1_joint" type="revolute">
-    <origin xyz="-0.57155 0.0 0.17415" rpy="0.0 0.0 9.012209423031764e-05"/>
+    <origin xyz="-0.57155 0.0 0.17415" rpy="0.0 0.0 0.0003550199178989447"/>
     <axis xyz="0.0 0.0 1.0"/>
     <parent link="forearm_link"/>
@@ -435,5 +435,5 @@
   </joint>
   <joint name="wrist_2_joint" type="revolute">
-    <origin xyz="0.0 -0.11985 -2.458164590756244e-11" rpy="1.570796327 0.0 -0.0005085943213929098"/>
+    <origin xyz="0.0 -0.11985 -2.458164590756244e-11" rpy="1.570796327 0.0 -0.0002689963824359225"/>
     <axis xyz="0.0 0.0 1.0"/>
     <parent link="wrist_1_link"/>
@@ -443,5 +443,5 @@
   </joint>
   <joint name="wrist_3_joint" type="revolute">
-    <origin xyz="0.0 0.11655 -2.390480459346185e-11" rpy="1.570796326589793 3.141592653589793 3.1273477612817056"/>
+    <origin xyz="0.0 0.11655 -2.390480459346185e-11" rpy="1.570796326589793 3.141592653589793 3.690243256024751"/>
     <axis xyz="0.0 0.0 1.0"/>
     <parent link="wrist_2_link"/>
@@ -555,5 +555,5 @@
   </joint>
   <joint name="rgb_world_joint" type="fixed">
-    <origin xyz="-0.01424371390973975 0.03119637180293375 0.023111965994740306" rpy="0.01733924703690017 3.200465589616032e-05 -0.040101527183436694"/>
+    <origin xyz="0.014254098736259803 -0.029596611953133758 0.03441572458900362" rpy="-0.011422006499824446 0.0005894249803577792 0.035864080268757585"/>
     <parent link="tripod_center_support"/>
     <child link="rgb_world_link"/>
@@ -694,4 +694,18 @@
     <child link="charuco_200x120_3x6"/>
   </joint>
+  <link name="charuco_170x100_3x6">
+    <origin xyz="0 0 0" rpy="0 0 0"/>
+    <visual name="forearm_pattern_visual">
+      <origin xyz="0 0 0" rpy="0 0 0"/>
+      <geometry>
+        <mesh filename="package://atom_worlds/pattern/models/charuco_170x100_3x6_25_18_DICT_6X6/model.dae"/>
+      </geometry>
+    </visual>
+  </link>
+  <joint name="forearm_link-charuco_170x100_3x6" type="fixed">
+    <origin xyz="-0.19996677202099444 0.019940200710195966 -0.029753981827784964" rpy="-0.0006066104009218485 -0.0024571496901093547 3.140422851894435"/>
+    <parent link="forearm_link"/>
+    <child link="charuco_170x100_3x6"/>
+  </joint>
   <link name="charuco_200x200_8x8">
     <origin xyz="0 0 0" rpy="0 0 0"/>
@@ -704,7 +718,21 @@
   </link>
   <joint name="flange-charuco_200x200_8x8" type="fixed">
-    <origin xyz="0.06013804387081968 -0.05970861845038463 -7.986535573664649e-05" rpy="0.01296741455882643 0.001080329541757302 -6.464771519985488e-05"/>
+    <origin xyz="0.060064632848067616 -0.05054174158147217 0.031735088702376804" rpy="-0.5496360181832282 0.000789818353599876 -0.0009559281276057386"/>
     <parent link="flange"/>
     <child link="charuco_200x200_8x8"/>
   </joint>
+  <link name="charuco_200x120_3x6">
+    <origin xyz="0 0 0" rpy="0 0 0"/>
+    <visual name="upper_arm_pattern_visual">
+      <origin xyz="0 0 0" rpy="0 0 0"/>
+      <geometry>
+        <mesh filename="package://atom_worlds/pattern/models/charuco_200x120_3x6_30_22_DICT_7X7/model.dae"/>
+      </geometry>
+    </visual>
+  </link>
+  <joint name="upper_arm_link-charuco_200x120_3x6" type="fixed">
+    <origin xyz="-0.24026296567067007 0.0299454157226812 0.09031747894862198" rpy="0.0007937379615085811 -0.0002364599986537006 3.140187367391834"/>
+    <parent link="upper_arm_link"/>
+    <child link="charuco_200x120_3x6"/>
+  </joint>
 </robot>

Commit message: Saving yaml with command line args (Close #831)

File: atom_examples/riwmpbot/riwmpbot_calibration/urdf/optimized.urdf.xacro (robot description, xacro)
@@ -403,5 +403,5 @@
   </joint>
   <joint name="shoulder_pan_joint" type="revolute">
-    <origin xyz="0.0 0.0 0.1807" rpy="0.0 0.0 0.038166999186922436"/>
+    <origin xyz="0.0 0.0 0.1807" rpy="0.0 0.0 0.5"/>
     <axis xyz="0.0 0.0 1.0"/>
     <parent link="base_link_inertia"/>
@@ -411,5 +411,5 @@
   </joint>
   <joint name="shoulder_lift_joint" type="revolute">
-    <origin xyz="0.0 0.0 0.0" rpy="1.570796327 0.0 0.0002410801554328166"/>
+    <origin xyz="0.0 0.0 0.0" rpy="1.570796327 0.0 0.0"/>
     <axis xyz="0.0 0.0 1.0"/>
     <parent link="shoulder_link"/>
@@ -419,5 +419,5 @@
   </joint>
   <joint name="elbow_joint" type="revolute">
-    <origin xyz="-0.6127 0.0 0.0" rpy="0.0 0.0 -0.00014109124769039037"/>
+    <origin xyz="-0.6127 0.0 0.0" rpy="0.0 0.0 0.0"/>
     <axis xyz="0.0 0.0 1.0"/>
     <parent link="upper_arm_link"/>
@@ -427,5 +427,5 @@
   </joint>
   <joint name="wrist_1_joint" type="revolute">
-    <origin xyz="-0.57155 0.0 0.17415" rpy="0.0 0.0 0.0003550199178989447"/>
+    <origin xyz="-0.57155 0.0 0.17415" rpy="0.0 0.0 0.0"/>
     <axis xyz="0.0 0.0 1.0"/>
     <parent link="forearm_link"/>
@@ -435,5 +435,5 @@
   </joint>
   <joint name="wrist_2_joint" type="revolute">
-    <origin xyz="0.0 -0.11985 -2.458164590756244e-11" rpy="1.570796327 0.0 -0.0002689963824359225"/>
+    <origin xyz="0.0 -0.11985 -2.458164590756244e-11" rpy="1.570796327 0.0 0.0"/>
     <axis xyz="0.0 0.0 1.0"/>
     <parent link="wrist_1_link"/>
@@ -443,5 +443,5 @@
   </joint>
   <joint name="wrist_3_joint" type="revolute">
-    <origin xyz="0.0 0.11655 -2.390480459346185e-11" rpy="1.570796326589793 3.141592653589793 3.690243256024751"/>
+    <origin xyz="0.0 0.11655 -2.390480459346185e-11" rpy="1.570796326589793 3.141592653589793 3.141592653589793"/>
     <axis xyz="0.0 0.0 1.0"/>
     <parent link="wrist_2_link"/>
@@ -555,5 +555,5 @@
   </joint>
   <joint name="rgb_world_joint" type="fixed">
-    <origin xyz="0.014254098736259803 -0.029596611953133758 0.03441572458900362" rpy="-0.011422006499824446 0.0005894249803577792 0.035864080268757585"/>
+    <origin xyz="-0.082828372041667 0.05472190577167546 0.017959492799592403" rpy="0.0 -0.0 0.0"/>
     <parent link="tripod_center_support"/>
     <child link="rgb_world_link"/>

File: atom_examples/riwmpbot/riwmpbot_calibration/urdf/optimized_w_pattern.urdf.xacro (robot description, xacro)
@@ -403,5 +403,5 @@
   </joint>
   <joint name="shoulder_pan_joint" type="revolute">
-    <origin xyz="0.0 0.0 0.1807" rpy="0.0 0.0 0.038166999186922436"/>
+    <origin xyz="0.0 0.0 0.1807" rpy="0.0 0.0 0.5"/>
     <axis xyz="0.0 0.0 1.0"/>
     <parent link="base_link_inertia"/>
@@ -411,5 +411,5 @@
   </joint>
   <joint name="shoulder_lift_joint" type="revolute">
-    <origin xyz="0.0 0.0 0.0" rpy="1.570796327 0.0 0.0002410801554328166"/>
+    <origin xyz="0.0 0.0 0.0" rpy="1.570796327 0.0 0.0"/>
     <axis xyz="0.0 0.0 1.0"/>
     <parent link="shoulder_link"/>
@@ -419,5 +419,5 @@
   </joint>
   <joint name="elbow_joint" type="revolute">
-    <origin xyz="-0.6127 0.0 0.0" rpy="0.0 0.0 -0.00014109124769039037"/>
+    <origin xyz="-0.6127 0.0 0.0" rpy="0.0 0.0 0.0"/>
     <axis xyz="0.0 0.0 1.0"/>
     <parent link="upper_arm_link"/>
@@ -427,5 +427,5 @@
   </joint>
   <joint name="wrist_1_joint" type="revolute">
-    <origin xyz="-0.57155 0.0 0.17415" rpy="0.0 0.0 0.0003550199178989447"/>
+    <origin xyz="-0.57155 0.0 0.17415" rpy="0.0 0.0 0.0"/>
     <axis xyz="0.0 0.0 1.0"/>
     <parent link="forearm_link"/>
@@ -435,5 +435,5 @@
   </joint>
   <joint name="wrist_2_joint" type="revolute">
-    <origin xyz="0.0 -0.11985 -2.458164590756244e-11" rpy="1.570796327 0.0 -0.0002689963824359225"/>
+    <origin xyz="0.0 -0.11985 -2.458164590756244e-11" rpy="1.570796327 0.0 0.0"/>
     <axis xyz="0.0 0.0 1.0"/>
     <parent link="wrist_1_link"/>
@@ -443,5 +443,5 @@
   </joint>
   <joint name="wrist_3_joint" type="revolute">
-    <origin xyz="0.0 0.11655 -2.390480459346185e-11" rpy="1.570796326589793 3.141592653589793 3.690243256024751"/>
+    <origin xyz="0.0 0.11655 -2.390480459346185e-11" rpy="1.570796326589793 3.141592653589793 3.141592653589793"/>
     <axis xyz="0.0 0.0 1.0"/>
     <parent link="wrist_2_link"/>
@@ -555,5 +555,5 @@
   </joint>
   <joint name="rgb_world_joint" type="fixed">
-    <origin xyz="0.014254098736259803 -0.029596611953133758 0.03441572458900362" rpy="-0.011422006499824446 0.0005894249803577792 0.035864080268757585"/>
+    <origin xyz="-0.082828372041667 0.05472190577167546 0.017959492799592403" rpy="0.0 -0.0 0.0"/>
     <parent link="tripod_center_support"/>
     <child link="rgb_world_link"/>
@@ -694,18 +694,4 @@
     <child link="charuco_200x120_3x6"/>
   </joint>
-  <link name="charuco_170x100_3x6">
-    <origin xyz="0 0 0" rpy="0 0 0"/>
-    <visual name="forearm_pattern_visual">
-      <origin xyz="0 0 0" rpy="0 0 0"/>
-      <geometry>
-        <mesh filename="package://atom_worlds/pattern/models/charuco_170x100_3x6_25_18_DICT_6X6/model.dae"/>
-      </geometry>
-    </visual>
-  </link>
-  <joint name="forearm_link-charuco_170x100_3x6" type="fixed">
-    <origin xyz="-0.19996677202099444 0.019940200710195966 -0.029753981827784964" rpy="-0.0006066104009218485 -0.0024571496901093547 3.140422851894435"/>
-    <parent link="forearm_link"/>
-    <child link="charuco_170x100_3x6"/>
-  </joint>
   <link name="charuco_200x200_8x8">
     <origin xyz="0 0 0" rpy="0 0 0"/>
@@ -718,21 +704,7 @@
   </link>
   <joint name="flange-charuco_200x200_8x8" type="fixed">
-    <origin xyz="0.060064632848067616 -0.05054174158147217 0.031735088702376804" rpy="-0.5496360181832282 0.000789818353599876 -0.0009559281276057386"/>
+    <origin xyz="0.059192651234109564 -0.05901301787209429 -0.00025930332406831624" rpy="-0.0028885781540415973 0.006681756014590649 -0.00024896564602461203"/>
     <parent link="flange"/>
     <child link="charuco_200x200_8x8"/>
   </joint>
-  <link name="charuco_200x120_3x6">
-    <origin xyz="0 0 0" rpy="0 0 0"/>
-    <visual name="upper_arm_pattern_visual">
-      <origin xyz="0 0 0" rpy="0 0 0"/>
-      <geometry>
-        <mesh filename="package://atom_worlds/pattern/models/charuco_200x120_3x6_30_22_DICT_7X7/model.dae"/>
-      </geometry>
-    </visual>
-  </link>
-  <joint name="upper_arm_link-charuco_200x120_3x6" type="fixed">
-    <origin xyz="-0.24026296567067007 0.0299454157226812 0.09031747894862198" rpy="0.0007937379615085811 -0.0002364599986537006 3.140187367391834"/>
-    <parent link="upper_arm_link"/>
-    <child link="charuco_200x120_3x6"/>
-  </joint>
 </robot>
