Commit message: #829 on the way ...

File: atom_examples/riwmpbot/riwmpbot_calibration/urdf/optimized.urdf.xacro (robot description, xacro)
@@ -411,5 +411,5 @@
   </joint>
   <joint name="shoulder_lift_joint" type="revolute">
-    <origin xyz="0.0 0.0 0.0" rpy="1.570796327 0.0 0.0"/>
+    <origin xyz="0.0 0.0 0.0" rpy="1.570796327 0.0 0.5"/>
     <axis xyz="0.0 0.0 1.0"/>
     <parent link="shoulder_link"/>
@@ -419,5 +419,5 @@
   </joint>
   <joint name="elbow_joint" type="revolute">
-    <origin xyz="-0.6127 0.0 0.0" rpy="0.0 0.0 0.0"/>
+    <origin xyz="-0.6127 0.0 0.0" rpy="0.0 0.0 0.5"/>
     <axis xyz="0.0 0.0 1.0"/>
     <parent link="upper_arm_link"/>
@@ -427,5 +427,5 @@
   </joint>
   <joint name="wrist_1_joint" type="revolute">
-    <origin xyz="-0.57155 0.0 0.17415" rpy="0.0 0.0 0.0"/>
+    <origin xyz="-0.57155 0.0 0.17415" rpy="0.0 0.0 0.5"/>
     <axis xyz="0.0 0.0 1.0"/>
     <parent link="forearm_link"/>
@@ -435,5 +435,5 @@
   </joint>
   <joint name="wrist_2_joint" type="revolute">
-    <origin xyz="0.0 -0.11985 -2.458164590756244e-11" rpy="1.570796327 0.0 0.0"/>
+    <origin xyz="0.0 -0.11985 -2.458164590756244e-11" rpy="1.570796327 0.0 0.5"/>
     <axis xyz="0.0 0.0 1.0"/>
     <parent link="wrist_1_link"/>
@@ -443,5 +443,5 @@
   </joint>
   <joint name="wrist_3_joint" type="revolute">
-    <origin xyz="0.0 0.11655 -2.390480459346185e-11" rpy="1.570796326589793 3.141592653589793 3.141592653589793"/>
+    <origin xyz="0.0 0.11655 -2.390480459346185e-11" rpy="1.570796326589793 3.141592653589793 3.641592653589793"/>
     <axis xyz="0.0 0.0 1.0"/>
     <parent link="wrist_2_link"/>
@@ -555,5 +555,5 @@
   </joint>
   <joint name="rgb_world_joint" type="fixed">
-    <origin xyz="-0.082828372041667 0.05472190577167546 0.017959492799592403" rpy="0.0 -0.0 0.0"/>
+    <origin xyz="-0.414141860208335 0.2736095288583773 -0.030202536002037976" rpy="0.5000000000000001 0.5 -0.5000000000000001"/>
     <parent link="tripod_center_support"/>
     <child link="rgb_world_link"/>

File: atom_examples/riwmpbot/riwmpbot_calibration/urdf/optimized_w_pattern.urdf.xacro (robot description, xacro)
@@ -411,5 +411,5 @@
   </joint>
   <joint name="shoulder_lift_joint" type="revolute">
-    <origin xyz="0.0 0.0 0.0" rpy="1.570796327 0.0 0.0"/>
+    <origin xyz="0.0 0.0 0.0" rpy="1.570796327 0.0 0.5"/>
     <axis xyz="0.0 0.0 1.0"/>
     <parent link="shoulder_link"/>
@@ -419,5 +419,5 @@
   </joint>
   <joint name="elbow_joint" type="revolute">
-    <origin xyz="-0.6127 0.0 0.0" rpy="0.0 0.0 0.0"/>
+    <origin xyz="-0.6127 0.0 0.0" rpy="0.0 0.0 0.5"/>
     <axis xyz="0.0 0.0 1.0"/>
     <parent link="upper_arm_link"/>
@@ -427,5 +427,5 @@
   </joint>
   <joint name="wrist_1_joint" type="revolute">
-    <origin xyz="-0.57155 0.0 0.17415" rpy="0.0 0.0 0.0"/>
+    <origin xyz="-0.57155 0.0 0.17415" rpy="0.0 0.0 0.5"/>
     <axis xyz="0.0 0.0 1.0"/>
     <parent link="forearm_link"/>
@@ -435,5 +435,5 @@
   </joint>
   <joint name="wrist_2_joint" type="revolute">
-    <origin xyz="0.0 -0.11985 -2.458164590756244e-11" rpy="1.570796327 0.0 0.0"/>
+    <origin xyz="0.0 -0.11985 -2.458164590756244e-11" rpy="1.570796327 0.0 0.5"/>
     <axis xyz="0.0 0.0 1.0"/>
     <parent link="wrist_1_link"/>
@@ -443,5 +443,5 @@
   </joint>
   <joint name="wrist_3_joint" type="revolute">
-    <origin xyz="0.0 0.11655 -2.390480459346185e-11" rpy="1.570796326589793 3.141592653589793 3.141592653589793"/>
+    <origin xyz="0.0 0.11655 -2.390480459346185e-11" rpy="1.570796326589793 3.141592653589793 3.641592653589793"/>
     <axis xyz="0.0 0.0 1.0"/>
     <parent link="wrist_2_link"/>
@@ -555,5 +555,5 @@
   </joint>
   <joint name="rgb_world_joint" type="fixed">
-    <origin xyz="-0.082828372041667 0.05472190577167546 0.017959492799592403" rpy="0.0 -0.0 0.0"/>
+    <origin xyz="-0.414141860208335 0.2736095288583773 -0.030202536002037976" rpy="0.5000000000000001 0.5 -0.5000000000000001"/>
     <parent link="tripod_center_support"/>
     <child link="rgb_world_link"/>

Commit message: #829 fixing path related bug in  saveAtomDataset

File: atom_examples/riwmpbot/riwmpbot_calibration/urdf/optimized.urdf.xacro (robot description, xacro)
@@ -403,5 +403,5 @@
   </joint>
   <joint name="shoulder_pan_joint" type="revolute">
-    <origin xyz="0.0 0.0 0.1807" rpy="0.0 0.0 0.5"/>
+    <origin xyz="0.0 0.0 0.1807" rpy="0.0 0.0 0.01"/>
     <axis xyz="0.0 0.0 1.0"/>
     <parent link="base_link_inertia"/>
@@ -411,5 +411,5 @@
   </joint>
   <joint name="shoulder_lift_joint" type="revolute">
-    <origin xyz="0.0 0.0 0.0" rpy="1.570796327 0.0 0.5"/>
+    <origin xyz="0.0 0.0 0.0" rpy="1.570796327 0.0 0.01"/>
     <axis xyz="0.0 0.0 1.0"/>
     <parent link="shoulder_link"/>
@@ -419,5 +419,5 @@
   </joint>
   <joint name="elbow_joint" type="revolute">
-    <origin xyz="-0.6127 0.0 0.0" rpy="0.0 0.0 0.5"/>
+    <origin xyz="-0.6127 0.0 0.0" rpy="0.0 0.0 0.01"/>
     <axis xyz="0.0 0.0 1.0"/>
     <parent link="upper_arm_link"/>
@@ -427,5 +427,5 @@
   </joint>
   <joint name="wrist_1_joint" type="revolute">
-    <origin xyz="-0.57155 0.0 0.17415" rpy="0.0 0.0 0.5"/>
+    <origin xyz="-0.57155 0.0 0.17415" rpy="0.0 0.0 0.01"/>
     <axis xyz="0.0 0.0 1.0"/>
     <parent link="forearm_link"/>
@@ -435,5 +435,5 @@
   </joint>
   <joint name="wrist_2_joint" type="revolute">
-    <origin xyz="0.0 -0.11985 -2.458164590756244e-11" rpy="1.570796327 0.0 0.5"/>
+    <origin xyz="0.0 -0.11985 -2.458164590756244e-11" rpy="1.570796327 0.0 0.01"/>
     <axis xyz="0.0 0.0 1.0"/>
     <parent link="wrist_1_link"/>
@@ -443,5 +443,5 @@
   </joint>
   <joint name="wrist_3_joint" type="revolute">
-    <origin xyz="0.0 0.11655 -2.390480459346185e-11" rpy="1.570796326589793 3.141592653589793 3.641592653589793"/>
+    <origin xyz="0.0 0.11655 -2.390480459346185e-11" rpy="1.570796326589793 3.141592653589793 3.151592653589793"/>
     <axis xyz="0.0 0.0 1.0"/>
     <parent link="wrist_2_link"/>
@@ -555,5 +555,5 @@
   </joint>
   <joint name="rgb_world_joint" type="fixed">
-    <origin xyz="-0.414141860208335 0.2736095288583773 -0.030202536002037976" rpy="0.5000000000000001 0.5 -0.5000000000000001"/>
+    <origin xyz="-0.0082828372041667 0.0054721905771675464 0.028795949279959238" rpy="0.00999999999999406 0.009999999999994 -0.00999999999999406"/>
     <parent link="tripod_center_support"/>
     <child link="rgb_world_link"/>

File: atom_examples/riwmpbot/riwmpbot_calibration/urdf/optimized_w_pattern.urdf.xacro (robot description, xacro)
@@ -403,5 +403,5 @@
   </joint>
   <joint name="shoulder_pan_joint" type="revolute">
-    <origin xyz="0.0 0.0 0.1807" rpy="0.0 0.0 0.5"/>
+    <origin xyz="0.0 0.0 0.1807" rpy="0.0 0.0 0.01"/>
     <axis xyz="0.0 0.0 1.0"/>
     <parent link="base_link_inertia"/>
@@ -411,5 +411,5 @@
   </joint>
   <joint name="shoulder_lift_joint" type="revolute">
-    <origin xyz="0.0 0.0 0.0" rpy="1.570796327 0.0 0.5"/>
+    <origin xyz="0.0 0.0 0.0" rpy="1.570796327 0.0 0.01"/>
     <axis xyz="0.0 0.0 1.0"/>
     <parent link="shoulder_link"/>
@@ -419,5 +419,5 @@
   </joint>
   <joint name="elbow_joint" type="revolute">
-    <origin xyz="-0.6127 0.0 0.0" rpy="0.0 0.0 0.5"/>
+    <origin xyz="-0.6127 0.0 0.0" rpy="0.0 0.0 0.01"/>
     <axis xyz="0.0 0.0 1.0"/>
     <parent link="upper_arm_link"/>
@@ -427,5 +427,5 @@
   </joint>
   <joint name="wrist_1_joint" type="revolute">
-    <origin xyz="-0.57155 0.0 0.17415" rpy="0.0 0.0 0.5"/>
+    <origin xyz="-0.57155 0.0 0.17415" rpy="0.0 0.0 0.01"/>
     <axis xyz="0.0 0.0 1.0"/>
     <parent link="forearm_link"/>
@@ -435,5 +435,5 @@
   </joint>
   <joint name="wrist_2_joint" type="revolute">
-    <origin xyz="0.0 -0.11985 -2.458164590756244e-11" rpy="1.570796327 0.0 0.5"/>
+    <origin xyz="0.0 -0.11985 -2.458164590756244e-11" rpy="1.570796327 0.0 0.01"/>
     <axis xyz="0.0 0.0 1.0"/>
     <parent link="wrist_1_link"/>
@@ -443,5 +443,5 @@
   </joint>
   <joint name="wrist_3_joint" type="revolute">
-    <origin xyz="0.0 0.11655 -2.390480459346185e-11" rpy="1.570796326589793 3.141592653589793 3.641592653589793"/>
+    <origin xyz="0.0 0.11655 -2.390480459346185e-11" rpy="1.570796326589793 3.141592653589793 3.151592653589793"/>
     <axis xyz="0.0 0.0 1.0"/>
     <parent link="wrist_2_link"/>
@@ -555,5 +555,5 @@
   </joint>
   <joint name="rgb_world_joint" type="fixed">
-    <origin xyz="-0.414141860208335 0.2736095288583773 -0.030202536002037976" rpy="0.5000000000000001 0.5 -0.5000000000000001"/>
+    <origin xyz="-0.0082828372041667 0.0054721905771675464 0.028795949279959238" rpy="0.00999999999999406 0.009999999999994 -0.00999999999999406"/>
     <parent link="tripod_center_support"/>
     <child link="rgb_world_link"/>
@@ -704,5 +704,5 @@
   </link>
   <joint name="flange-charuco_200x200_8x8" type="fixed">
-    <origin xyz="0.059192651234109564 -0.05901301787209429 -0.00025930332406831624" rpy="-0.0028885781540415973 0.006681756014590649 -0.00024896564602461203"/>
+    <origin xyz="0.05917124724289985 -0.05901082259689297 -0.0002946986181739941" rpy="-0.005259297838487501 0.0010016490675282493 0.0002558599283795088"/>
     <parent link="flange"/>
     <child link="charuco_200x200_8x8"/>

Commit message: #829 Improving riwmpbot readme

File: atom_examples/riwmpbot/riwmpbot_calibration/urdf/optimized.urdf.xacro (robot description, xacro)
@@ -403,5 +403,5 @@
   </joint>
   <joint name="shoulder_pan_joint" type="revolute">
-    <origin xyz="0.0 0.0 0.1807" rpy="0.0 0.0 0.01"/>
+    <origin xyz="0.0 0.0 0.1807" rpy="0.0 0.0 0.03634655935070443"/>
     <axis xyz="0.0 0.0 1.0"/>
     <parent link="base_link_inertia"/>
@@ -411,5 +411,5 @@
   </joint>
   <joint name="shoulder_lift_joint" type="revolute">
-    <origin xyz="0.0 0.0 0.0" rpy="1.570796327 0.0 0.01"/>
+    <origin xyz="0.0 0.0 0.0" rpy="1.570796327 0.0 -0.0023131534458055852"/>
     <axis xyz="0.0 0.0 1.0"/>
     <parent link="shoulder_link"/>
@@ -419,5 +419,5 @@
   </joint>
   <joint name="elbow_joint" type="revolute">
-    <origin xyz="-0.6127 0.0 0.0" rpy="0.0 0.0 0.01"/>
+    <origin xyz="-0.6127 0.0 0.0" rpy="0.0 0.0 -0.0005715973521791428"/>
     <axis xyz="0.0 0.0 1.0"/>
     <parent link="upper_arm_link"/>
@@ -427,5 +427,5 @@
   </joint>
   <joint name="wrist_1_joint" type="revolute">
-    <origin xyz="-0.57155 0.0 0.17415" rpy="0.0 0.0 0.01"/>
+    <origin xyz="-0.57155 0.0 0.17415" rpy="0.0 0.0 0.0006760042247028275"/>
     <axis xyz="0.0 0.0 1.0"/>
     <parent link="forearm_link"/>
@@ -435,5 +435,5 @@
   </joint>
   <joint name="wrist_2_joint" type="revolute">
-    <origin xyz="0.0 -0.11985 -2.458164590756244e-11" rpy="1.570796327 0.0 0.01"/>
+    <origin xyz="0.0 -0.11985 -2.458164590756244e-11" rpy="1.570796327 0.0 -7.078490365845218e-05"/>
     <axis xyz="0.0 0.0 1.0"/>
     <parent link="wrist_1_link"/>
@@ -443,5 +443,5 @@
   </joint>
   <joint name="wrist_3_joint" type="revolute">
-    <origin xyz="0.0 0.11655 -2.390480459346185e-11" rpy="1.570796326589793 3.141592653589793 3.151592653589793"/>
+    <origin xyz="0.0 0.11655 -2.390480459346185e-11" rpy="1.570796326589793 3.141592653589793 3.124803289385984"/>
     <axis xyz="0.0 0.0 1.0"/>
     <parent link="wrist_2_link"/>
@@ -555,5 +555,5 @@
   </joint>
   <joint name="rgb_world_joint" type="fixed">
-    <origin xyz="-0.0082828372041667 0.0054721905771675464 0.028795949279959238" rpy="0.00999999999999406 0.009999999999994 -0.00999999999999406"/>
+    <origin xyz="0.013394030071812666 -0.026310892081452705 0.03577688783114847" rpy="-0.013565370501995258 0.0010644695313850908 0.033183886003169655"/>
     <parent link="tripod_center_support"/>
     <child link="rgb_world_link"/>

File: atom_examples/riwmpbot/riwmpbot_calibration/urdf/optimized_w_pattern.urdf.xacro (robot description, xacro)
@@ -403,5 +403,5 @@
   </joint>
   <joint name="shoulder_pan_joint" type="revolute">
-    <origin xyz="0.0 0.0 0.1807" rpy="0.0 0.0 0.01"/>
+    <origin xyz="0.0 0.0 0.1807" rpy="0.0 0.0 0.03634655935070443"/>
     <axis xyz="0.0 0.0 1.0"/>
     <parent link="base_link_inertia"/>
@@ -411,5 +411,5 @@
   </joint>
   <joint name="shoulder_lift_joint" type="revolute">
-    <origin xyz="0.0 0.0 0.0" rpy="1.570796327 0.0 0.01"/>
+    <origin xyz="0.0 0.0 0.0" rpy="1.570796327 0.0 -0.0023131534458055852"/>
     <axis xyz="0.0 0.0 1.0"/>
     <parent link="shoulder_link"/>
@@ -419,5 +419,5 @@
   </joint>
   <joint name="elbow_joint" type="revolute">
-    <origin xyz="-0.6127 0.0 0.0" rpy="0.0 0.0 0.01"/>
+    <origin xyz="-0.6127 0.0 0.0" rpy="0.0 0.0 -0.0005715973521791428"/>
     <axis xyz="0.0 0.0 1.0"/>
     <parent link="upper_arm_link"/>
@@ -427,5 +427,5 @@
   </joint>
   <joint name="wrist_1_joint" type="revolute">
-    <origin xyz="-0.57155 0.0 0.17415" rpy="0.0 0.0 0.01"/>
+    <origin xyz="-0.57155 0.0 0.17415" rpy="0.0 0.0 0.0006760042247028275"/>
     <axis xyz="0.0 0.0 1.0"/>
     <parent link="forearm_link"/>
@@ -435,5 +435,5 @@
   </joint>
   <joint name="wrist_2_joint" type="revolute">
-    <origin xyz="0.0 -0.11985 -2.458164590756244e-11" rpy="1.570796327 0.0 0.01"/>
+    <origin xyz="0.0 -0.11985 -2.458164590756244e-11" rpy="1.570796327 0.0 -7.078490365845218e-05"/>
     <axis xyz="0.0 0.0 1.0"/>
     <parent link="wrist_1_link"/>
@@ -443,5 +443,5 @@
   </joint>
   <joint name="wrist_3_joint" type="revolute">
-    <origin xyz="0.0 0.11655 -2.390480459346185e-11" rpy="1.570796326589793 3.141592653589793 3.151592653589793"/>
+    <origin xyz="0.0 0.11655 -2.390480459346185e-11" rpy="1.570796326589793 3.141592653589793 3.124803289385984"/>
     <axis xyz="0.0 0.0 1.0"/>
     <parent link="wrist_2_link"/>
@@ -555,5 +555,5 @@
   </joint>
   <joint name="rgb_world_joint" type="fixed">
-    <origin xyz="-0.0082828372041667 0.0054721905771675464 0.028795949279959238" rpy="0.00999999999999406 0.009999999999994 -0.00999999999999406"/>
+    <origin xyz="0.013394030071812666 -0.026310892081452705 0.03577688783114847" rpy="-0.013565370501995258 0.0010644695313850908 0.033183886003169655"/>
     <parent link="tripod_center_support"/>
     <child link="rgb_world_link"/>
@@ -694,4 +694,18 @@
     <child link="charuco_200x120_3x6"/>
   </joint>
+  <link name="charuco_170x100_3x6">
+    <origin xyz="0 0 0" rpy="0 0 0"/>
+    <visual name="forearm_pattern_visual">
+      <origin xyz="0 0 0" rpy="0 0 0"/>
+      <geometry>
+        <mesh filename="package://atom_worlds/pattern/models/charuco_170x100_3x6_25_18_DICT_6X6/model.dae"/>
+      </geometry>
+    </visual>
+  </link>
+  <joint name="forearm_link-charuco_170x100_3x6" type="fixed">
+    <origin xyz="-0.20003820858777968 0.02003969873103348 -0.030065457658919482" rpy="-0.0003544588477039648 -0.0016851197539375835 3.1404797081519056"/>
+    <parent link="forearm_link"/>
+    <child link="charuco_170x100_3x6"/>
+  </joint>
   <link name="charuco_200x200_8x8">
     <origin xyz="0 0 0" rpy="0 0 0"/>
@@ -704,7 +718,21 @@
   </link>
   <joint name="flange-charuco_200x200_8x8" type="fixed">
-    <origin xyz="0.05917124724289985 -0.05901082259689297 -0.0002946986181739941" rpy="-0.005259297838487501 0.0010016490675282493 0.0002558599283795088"/>
+    <origin xyz="0.05996674983679648 -0.05967044649362541 -0.000311555003907855" rpy="0.01601689702333116 0.001249372397008772 -0.0006768858846253315"/>
     <parent link="flange"/>
     <child link="charuco_200x200_8x8"/>
   </joint>
+  <link name="charuco_200x120_3x6">
+    <origin xyz="0 0 0" rpy="0 0 0"/>
+    <visual name="upper_arm_pattern_visual">
+      <origin xyz="0 0 0" rpy="0 0 0"/>
+      <geometry>
+        <mesh filename="package://atom_worlds/pattern/models/charuco_200x120_3x6_30_22_DICT_7X7/model.dae"/>
+      </geometry>
+    </visual>
+  </link>
+  <joint name="upper_arm_link-charuco_200x120_3x6" type="fixed">
+    <origin xyz="-0.240555983627542 0.029648592086992248 0.09012527467553003" rpy="0.00029099773474286305 0.0009833268437052449 3.140441884224232"/>
+    <parent link="upper_arm_link"/>
+    <child link="charuco_200x120_3x6"/>
+  </joint>
 </robot>

Commit message: Some changes ...

File: atom_examples/riwmpbot/riwmpbot_calibration/urdf/optimized.urdf.xacro (robot description, xacro)
@@ -403,5 +403,5 @@
   </joint>
   <joint name="shoulder_pan_joint" type="revolute">
-    <origin xyz="0.0 0.0 0.1807" rpy="0.0 0.0 0.03634655935070443"/>
+    <origin xyz="0.0 0.0 0.1807" rpy="0.0 0.0 0.0"/>
     <axis xyz="0.0 0.0 1.0"/>
     <parent link="base_link_inertia"/>
@@ -411,5 +411,5 @@
   </joint>
   <joint name="shoulder_lift_joint" type="revolute">
-    <origin xyz="0.0 0.0 0.0" rpy="1.570796327 0.0 -0.0023131534458055852"/>
+    <origin xyz="0.0 0.0 0.0" rpy="1.570796327 0.0 0.0"/>
     <axis xyz="0.0 0.0 1.0"/>
     <parent link="shoulder_link"/>
@@ -419,5 +419,5 @@
   </joint>
   <joint name="elbow_joint" type="revolute">
-    <origin xyz="-0.6127 0.0 0.0" rpy="0.0 0.0 -0.0005715973521791428"/>
+    <origin xyz="-0.6127 0.0 0.0" rpy="0.0 0.0 0.0"/>
     <axis xyz="0.0 0.0 1.0"/>
     <parent link="upper_arm_link"/>
@@ -427,5 +427,5 @@
   </joint>
   <joint name="wrist_1_joint" type="revolute">
-    <origin xyz="-0.57155 0.0 0.17415" rpy="0.0 0.0 0.0006760042247028275"/>
+    <origin xyz="-0.57155 0.0 0.17415" rpy="0.0 0.0 0.0"/>
     <axis xyz="0.0 0.0 1.0"/>
     <parent link="forearm_link"/>
@@ -435,5 +435,5 @@
   </joint>
   <joint name="wrist_2_joint" type="revolute">
-    <origin xyz="0.0 -0.11985 -2.458164590756244e-11" rpy="1.570796327 0.0 -7.078490365845218e-05"/>
+    <origin xyz="0.0 -0.11985 -2.458164590756244e-11" rpy="1.570796327 0.0 0.0"/>
     <axis xyz="0.0 0.0 1.0"/>
     <parent link="wrist_1_link"/>
@@ -443,5 +443,5 @@
   </joint>
   <joint name="wrist_3_joint" type="revolute">
-    <origin xyz="0.0 0.11655 -2.390480459346185e-11" rpy="1.570796326589793 3.141592653589793 3.124803289385984"/>
+    <origin xyz="0.0 0.11655 -2.390480459346185e-11" rpy="1.570796326589793 3.141592653589793 3.141592653589793"/>
     <axis xyz="0.0 0.0 1.0"/>
     <parent link="wrist_2_link"/>
@@ -555,5 +555,5 @@
   </joint>
   <joint name="rgb_world_joint" type="fixed">
-    <origin xyz="0.013394030071812666 -0.026310892081452705 0.03577688783114847" rpy="-0.013565370501995258 0.0010644695313850908 0.033183886003169655"/>
+    <origin xyz="0.0001936539500976023 -0.00016191314933734286 0.029838542958375673" rpy="0.0001650933494972848 0.0003522326651783465 -0.0003120672703493318"/>
     <parent link="tripod_center_support"/>
     <child link="rgb_world_link"/>

File: atom_examples/riwmpbot/riwmpbot_calibration/urdf/optimized_w_pattern.urdf.xacro (robot description, xacro)
@@ -403,5 +403,5 @@
   </joint>
   <joint name="shoulder_pan_joint" type="revolute">
-    <origin xyz="0.0 0.0 0.1807" rpy="0.0 0.0 0.03634655935070443"/>
+    <origin xyz="0.0 0.0 0.1807" rpy="0.0 0.0 0.0"/>
     <axis xyz="0.0 0.0 1.0"/>
     <parent link="base_link_inertia"/>
@@ -411,5 +411,5 @@
   </joint>
   <joint name="shoulder_lift_joint" type="revolute">
-    <origin xyz="0.0 0.0 0.0" rpy="1.570796327 0.0 -0.0023131534458055852"/>
+    <origin xyz="0.0 0.0 0.0" rpy="1.570796327 0.0 0.0"/>
     <axis xyz="0.0 0.0 1.0"/>
     <parent link="shoulder_link"/>
@@ -419,5 +419,5 @@
   </joint>
   <joint name="elbow_joint" type="revolute">
-    <origin xyz="-0.6127 0.0 0.0" rpy="0.0 0.0 -0.0005715973521791428"/>
+    <origin xyz="-0.6127 0.0 0.0" rpy="0.0 0.0 0.0"/>
     <axis xyz="0.0 0.0 1.0"/>
     <parent link="upper_arm_link"/>
@@ -427,5 +427,5 @@
   </joint>
   <joint name="wrist_1_joint" type="revolute">
-    <origin xyz="-0.57155 0.0 0.17415" rpy="0.0 0.0 0.0006760042247028275"/>
+    <origin xyz="-0.57155 0.0 0.17415" rpy="0.0 0.0 0.0"/>
     <axis xyz="0.0 0.0 1.0"/>
     <parent link="forearm_link"/>
@@ -435,5 +435,5 @@
   </joint>
   <joint name="wrist_2_joint" type="revolute">
-    <origin xyz="0.0 -0.11985 -2.458164590756244e-11" rpy="1.570796327 0.0 -7.078490365845218e-05"/>
+    <origin xyz="0.0 -0.11985 -2.458164590756244e-11" rpy="1.570796327 0.0 0.0"/>
     <axis xyz="0.0 0.0 1.0"/>
     <parent link="wrist_1_link"/>
@@ -443,5 +443,5 @@
   </joint>
   <joint name="wrist_3_joint" type="revolute">
-    <origin xyz="0.0 0.11655 -2.390480459346185e-11" rpy="1.570796326589793 3.141592653589793 3.124803289385984"/>
+    <origin xyz="0.0 0.11655 -2.390480459346185e-11" rpy="1.570796326589793 3.141592653589793 3.141592653589793"/>
     <axis xyz="0.0 0.0 1.0"/>
     <parent link="wrist_2_link"/>
@@ -555,5 +555,5 @@
   </joint>
   <joint name="rgb_world_joint" type="fixed">
-    <origin xyz="0.013394030071812666 -0.026310892081452705 0.03577688783114847" rpy="-0.013565370501995258 0.0010644695313850908 0.033183886003169655"/>
+    <origin xyz="0.0001936539500976023 -0.00016191314933734286 0.029838542958375673" rpy="0.0001650933494972848 0.0003522326651783465 -0.0003120672703493318"/>
     <parent link="tripod_center_support"/>
     <child link="rgb_world_link"/>
@@ -704,5 +704,5 @@
   </link>
   <joint name="forearm_link-charuco_170x100_3x6" type="fixed">
-    <origin xyz="-0.20003820858777968 0.02003969873103348 -0.030065457658919482" rpy="-0.0003544588477039648 -0.0016851197539375835 3.1404797081519056"/>
+    <origin xyz="-0.20003582318367094 0.019887174654697356 -0.029787617867588132" rpy="-0.0005609789112673702 -0.0028280828893094186 3.1403772001109416"/>
     <parent link="forearm_link"/>
     <child link="charuco_170x100_3x6"/>
@@ -718,5 +718,5 @@
   </link>
   <joint name="flange-charuco_200x200_8x8" type="fixed">
-    <origin xyz="0.05996674983679648 -0.05967044649362541 -0.000311555003907855" rpy="0.01601689702333116 0.001249372397008772 -0.0006768858846253315"/>
+    <origin xyz="0.060134596703514884 -0.05970062714560451 0.0007050628705367494" rpy="-0.0010141889176716477 0.0013578865818770053 -0.00012542545331538986"/>
     <parent link="flange"/>
     <child link="charuco_200x200_8x8"/>
@@ -732,5 +732,5 @@
   </link>
   <joint name="upper_arm_link-charuco_200x120_3x6" type="fixed">
-    <origin xyz="-0.240555983627542 0.029648592086992248 0.09012527467553003" rpy="0.00029099773474286305 0.0009833268437052449 3.140441884224232"/>
+    <origin xyz="-0.24019155126625746 0.02993734965722452 0.09026801721299614" rpy="0.0010219364358067206 -0.000267508570479523 3.140221331384571"/>
     <parent link="upper_arm_link"/>
     <child link="charuco_200x120_3x6"/>
