Commit message: #849 implemented

File: atom_examples/riwmpbot/riwmpbot_calibration/urdf/optimized.urdf.xacro (robot description, xacro)
@@ -1,7 +1,4 @@
 <?xml version="1.0" ?>
 <robot name="riwmpbot" version="1.0">
-  <material name="tripod_color">
-    <color rgba="0.21 0.21 0.21 1.0"/>
-  </material>
   <material name="Yellow">
     <color rgba="1.0 1.0 0.0 1.0"/>
@@ -403,5 +400,5 @@
   </joint>
   <joint name="shoulder_pan_joint" type="revolute">
-    <origin xyz="0.0 0.0 0.1807" rpy="0.0 0.0 0.0"/>
+    <origin xyz="0.0 0.0 0.1807" rpy="0.0 0.0 0.01975145569862588"/>
     <axis xyz="0.0 0.0 1.0"/>
     <parent link="base_link_inertia"/>
@@ -411,5 +408,5 @@
   </joint>
   <joint name="shoulder_lift_joint" type="revolute">
-    <origin xyz="0.0 0.0 0.0" rpy="1.570796327 0.0 0.0"/>
+    <origin xyz="0.0 0.0 0.0" rpy="1.570796327 0.0 0.05792003874793546"/>
     <axis xyz="0.0 0.0 1.0"/>
     <parent link="shoulder_link"/>
@@ -419,5 +416,5 @@
   </joint>
   <joint name="elbow_joint" type="revolute">
-    <origin xyz="-0.6127 0.0 0.0" rpy="0.0 0.0 0.0"/>
+    <origin xyz="-0.6127 0.0 0.0" rpy="0.0 0.0 0.1000000149011612"/>
     <axis xyz="0.0 0.0 1.0"/>
     <parent link="upper_arm_link"/>
@@ -427,5 +424,5 @@
   </joint>
   <joint name="wrist_1_joint" type="revolute">
-    <origin xyz="-0.57155 0.0 0.17415" rpy="0.0 0.0 0.0"/>
+    <origin xyz="-0.57155 0.0 0.17415" rpy="0.0 0.0 0.1"/>
     <axis xyz="0.0 0.0 1.0"/>
     <parent link="forearm_link"/>
@@ -435,5 +432,5 @@
   </joint>
   <joint name="wrist_2_joint" type="revolute">
-    <origin xyz="0.0 -0.11985 -2.458164590756244e-11" rpy="1.570796327 0.0 0.0"/>
+    <origin xyz="0.0 -0.11985 -2.458164590756244e-11" rpy="1.570796327 0.0 0.1"/>
     <axis xyz="0.0 0.0 1.0"/>
     <parent link="wrist_1_link"/>
@@ -443,5 +440,5 @@
   </joint>
   <joint name="wrist_3_joint" type="revolute">
-    <origin xyz="0.0 0.11655 -2.390480459346185e-11" rpy="1.570796326589793 3.141592653589793 3.141592653589793"/>
+    <origin xyz="0.0 0.11655 -2.390480459346185e-11" rpy="1.570796326589793 3.141592653589793 3.241592653589793"/>
     <axis xyz="0.0 0.0 1.0"/>
     <parent link="wrist_2_link"/>
@@ -509,5 +506,7 @@
         <mesh filename="package://riwmpbot_description/meshes/tripod/tripod.stl" scale="1.0 1.0 1.0"/>
       </geometry>
-      <material name="tripod_color"/>
+      <material name="tripod_color">
+        <color rgba="0.21 0.21 0.21 1.0"/>
+      </material>
     </visual>
     <collision name="tripod_collision">
@@ -534,5 +533,7 @@
         <box size="0.04 0.4 0.015"/>
       </geometry>
-      <material name="tripod_color"/>
+      <material name="tripod_color">
+        <color rgba="0.21 0.21 0.21 1.0"/>
+      </material>
     </visual>
     <collision name="tripod_collision">
@@ -555,5 +556,5 @@
   </joint>
   <joint name="rgb_world_joint" type="fixed">
-    <origin xyz="0.0001936539500976023 -0.00016191314933734286 0.029838542958375673" rpy="0.0001650933494972848 0.0003522326651783465 -0.0003120672703493318"/>
+    <origin xyz="0.00845867852242976 -0.018804586436127927 0.03272963808730215" rpy="-0.005846135346919141 0.0006280903221295673 0.022082037670039148"/>
     <parent link="tripod_center_support"/>
     <child link="rgb_world_link"/>

File: atom_examples/riwmpbot/riwmpbot_calibration/urdf/optimized_w_pattern.urdf.xacro (robot description, xacro)
@@ -1,7 +1,4 @@
 <?xml version="1.0" ?>
 <robot name="riwmpbot" version="1.0">
-  <material name="tripod_color">
-    <color rgba="0.21 0.21 0.21 1.0"/>
-  </material>
   <material name="Yellow">
     <color rgba="1.0 1.0 0.0 1.0"/>
@@ -403,5 +400,5 @@
   </joint>
   <joint name="shoulder_pan_joint" type="revolute">
-    <origin xyz="0.0 0.0 0.1807" rpy="0.0 0.0 0.0"/>
+    <origin xyz="0.0 0.0 0.1807" rpy="0.0 0.0 0.01975145569862588"/>
     <axis xyz="0.0 0.0 1.0"/>
     <parent link="base_link_inertia"/>
@@ -411,5 +408,5 @@
   </joint>
   <joint name="shoulder_lift_joint" type="revolute">
-    <origin xyz="0.0 0.0 0.0" rpy="1.570796327 0.0 0.0"/>
+    <origin xyz="0.0 0.0 0.0" rpy="1.570796327 0.0 0.05792003874793546"/>
     <axis xyz="0.0 0.0 1.0"/>
     <parent link="shoulder_link"/>
@@ -419,5 +416,5 @@
   </joint>
   <joint name="elbow_joint" type="revolute">
-    <origin xyz="-0.6127 0.0 0.0" rpy="0.0 0.0 0.0"/>
+    <origin xyz="-0.6127 0.0 0.0" rpy="0.0 0.0 0.1000000149011612"/>
     <axis xyz="0.0 0.0 1.0"/>
     <parent link="upper_arm_link"/>
@@ -427,5 +424,5 @@
   </joint>
   <joint name="wrist_1_joint" type="revolute">
-    <origin xyz="-0.57155 0.0 0.17415" rpy="0.0 0.0 0.0"/>
+    <origin xyz="-0.57155 0.0 0.17415" rpy="0.0 0.0 0.1"/>
     <axis xyz="0.0 0.0 1.0"/>
     <parent link="forearm_link"/>
@@ -435,5 +432,5 @@
   </joint>
   <joint name="wrist_2_joint" type="revolute">
-    <origin xyz="0.0 -0.11985 -2.458164590756244e-11" rpy="1.570796327 0.0 0.0"/>
+    <origin xyz="0.0 -0.11985 -2.458164590756244e-11" rpy="1.570796327 0.0 0.1"/>
     <axis xyz="0.0 0.0 1.0"/>
     <parent link="wrist_1_link"/>
@@ -443,5 +440,5 @@
   </joint>
   <joint name="wrist_3_joint" type="revolute">
-    <origin xyz="0.0 0.11655 -2.390480459346185e-11" rpy="1.570796326589793 3.141592653589793 3.141592653589793"/>
+    <origin xyz="0.0 0.11655 -2.390480459346185e-11" rpy="1.570796326589793 3.141592653589793 3.241592653589793"/>
     <axis xyz="0.0 0.0 1.0"/>
     <parent link="wrist_2_link"/>
@@ -509,5 +506,7 @@
         <mesh filename="package://riwmpbot_description/meshes/tripod/tripod.stl" scale="1.0 1.0 1.0"/>
       </geometry>
-      <material name="tripod_color"/>
+      <material name="tripod_color">
+        <color rgba="0.21 0.21 0.21 1.0"/>
+      </material>
     </visual>
     <collision name="tripod_collision">
@@ -534,5 +533,7 @@
         <box size="0.04 0.4 0.015"/>
       </geometry>
-      <material name="tripod_color"/>
+      <material name="tripod_color">
+        <color rgba="0.21 0.21 0.21 1.0"/>
+      </material>
     </visual>
     <collision name="tripod_collision">
@@ -555,5 +556,5 @@
   </joint>
   <joint name="rgb_world_joint" type="fixed">
-    <origin xyz="0.0001936539500976023 -0.00016191314933734286 0.029838542958375673" rpy="0.0001650933494972848 0.0003522326651783465 -0.0003120672703493318"/>
+    <origin xyz="0.00845867852242976 -0.018804586436127927 0.03272963808730215" rpy="-0.005846135346919141 0.0006280903221295673 0.022082037670039148"/>
     <parent link="tripod_center_support"/>
     <child link="rgb_world_link"/>
@@ -694,32 +695,4 @@
     <child link="charuco_200x120_3x6"/>
   </joint>
-  <link name="charuco_170x100_3x6">
-    <origin xyz="0 0 0" rpy="0 0 0"/>
-    <visual name="forearm_pattern_visual">
-      <origin xyz="0 0 0" rpy="0 0 0"/>
-      <geometry>
-        <mesh filename="package://atom_worlds/pattern/models/charuco_170x100_3x6_25_18_DICT_6X6/model.dae"/>
-      </geometry>
-    </visual>
-  </link>
-  <joint name="forearm_link-charuco_170x100_3x6" type="fixed">
-    <origin xyz="-0.20003582318367094 0.019887174654697356 -0.029787617867588132" rpy="-0.0005609789112673702 -0.0028280828893094186 3.1403772001109416"/>
-    <parent link="forearm_link"/>
-    <child link="charuco_170x100_3x6"/>
-  </joint>
-  <link name="charuco_200x200_8x8">
-    <origin xyz="0 0 0" rpy="0 0 0"/>
-    <visual name="hand_pattern_visual">
-      <origin xyz="0 0 0" rpy="0 0 0"/>
-      <geometry>
-        <mesh filename="package://atom_worlds/pattern/models/charuco_200x200_8x8_20_15_DICT_4x4/model.dae"/>
-      </geometry>
-    </visual>
-  </link>
-  <joint name="flange-charuco_200x200_8x8" type="fixed">
-    <origin xyz="0.060134596703514884 -0.05970062714560451 0.0007050628705367494" rpy="-0.0010141889176716477 0.0013578865818770053 -0.00012542545331538986"/>
-    <parent link="flange"/>
-    <child link="charuco_200x200_8x8"/>
-  </joint>
   <link name="charuco_200x120_3x6">
     <origin xyz="0 0 0" rpy="0 0 0"/>
@@ -732,5 +705,5 @@
   </link>
   <joint name="upper_arm_link-charuco_200x120_3x6" type="fixed">
-    <origin xyz="-0.24019155126625746 0.02993734965722452 0.09026801721299614" rpy="0.0010219364358067206 -0.000267508570479523 3.140221331384571"/>
+    <origin xyz="-0.23847704330245673 0.04398775918561481 0.09009886105268892" rpy="0.0038944889255176215 -0.001053401234966295 3.083018460864498"/>
     <parent link="upper_arm_link"/>
     <child link="charuco_200x120_3x6"/>

Commit message: #979 not sure this is not breaking something ...

File: atom_examples/riwmpbot/riwmpbot_calibration/urdf/optimized.urdf.xacro (robot description, xacro)
@@ -400,5 +400,5 @@
   </joint>
   <joint name="shoulder_pan_joint" type="revolute">
-    <origin xyz="0.0 0.0 0.1807" rpy="0.0 0.0 0.01975145569862588"/>
+    <origin xyz="0.01 0.01 0.1907" rpy="0.01 0.01 -0.010592558477970875"/>
     <axis xyz="0.0 0.0 1.0"/>
     <parent link="base_link_inertia"/>
@@ -408,5 +408,5 @@
   </joint>
   <joint name="shoulder_lift_joint" type="revolute">
-    <origin xyz="0.0 0.0 0.0" rpy="1.570796327 0.0 0.05792003874793546"/>
+    <origin xyz="0.01 0.01 0.01" rpy="1.580796327 0.01 0.00944167160288373"/>
     <axis xyz="0.0 0.0 1.0"/>
     <parent link="shoulder_link"/>
@@ -416,5 +416,5 @@
   </joint>
   <joint name="elbow_joint" type="revolute">
-    <origin xyz="-0.6127 0.0 0.0" rpy="0.0 0.0 0.1000000149011612"/>
+    <origin xyz="-0.6027 0.01 0.01" rpy="0.01 0.01 0.014434684315030902"/>
     <axis xyz="0.0 0.0 1.0"/>
     <parent link="upper_arm_link"/>
@@ -424,5 +424,5 @@
   </joint>
   <joint name="wrist_1_joint" type="revolute">
-    <origin xyz="-0.57155 0.0 0.17415" rpy="0.0 0.0 0.1"/>
+    <origin xyz="-0.56155 0.01 0.18415" rpy="0.01 0.01 -0.08163482372003837"/>
     <axis xyz="0.0 0.0 1.0"/>
     <parent link="forearm_link"/>
@@ -432,5 +432,5 @@
   </joint>
   <joint name="wrist_2_joint" type="revolute">
-    <origin xyz="0.0 -0.11985 -2.458164590756244e-11" rpy="1.570796327 0.0 0.1"/>
+    <origin xyz="0.01 -0.10985 0.009999999975418354" rpy="1.580796327 0.01 0.003446624604334964"/>
     <axis xyz="0.0 0.0 1.0"/>
     <parent link="wrist_1_link"/>
@@ -440,5 +440,5 @@
   </joint>
   <joint name="wrist_3_joint" type="revolute">
-    <origin xyz="0.0 0.11655 -2.390480459346185e-11" rpy="1.570796326589793 3.141592653589793 3.241592653589793"/>
+    <origin xyz="0.01 0.12655 0.009999999976095195" rpy="1.580796326589793 3.151592653589793 2.9732490752583485"/>
     <axis xyz="0.0 0.0 1.0"/>
     <parent link="wrist_2_link"/>
@@ -556,5 +556,5 @@
   </joint>
   <joint name="rgb_world_joint" type="fixed">
-    <origin xyz="0.00845867852242976 -0.018804586436127927 0.03272963808730215" rpy="-0.005846135346919141 0.0006280903221295673 0.022082037670039148"/>
+    <origin xyz="0.022296483486666293 -0.008751527534067098 0.06409294918539783" rpy="-0.010598941974837519 0.023653515563518888 0.041152533629886794"/>
     <parent link="tripod_center_support"/>
     <child link="rgb_world_link"/>

File: atom_examples/riwmpbot/riwmpbot_calibration/urdf/optimized_w_pattern.urdf.xacro (robot description, xacro)
@@ -400,5 +400,5 @@
   </joint>
   <joint name="shoulder_pan_joint" type="revolute">
-    <origin xyz="0.0 0.0 0.1807" rpy="0.0 0.0 0.01975145569862588"/>
+    <origin xyz="0.01 0.01 0.1907" rpy="0.01 0.01 -0.010592558477970875"/>
     <axis xyz="0.0 0.0 1.0"/>
     <parent link="base_link_inertia"/>
@@ -408,5 +408,5 @@
   </joint>
   <joint name="shoulder_lift_joint" type="revolute">
-    <origin xyz="0.0 0.0 0.0" rpy="1.570796327 0.0 0.05792003874793546"/>
+    <origin xyz="0.01 0.01 0.01" rpy="1.580796327 0.01 0.00944167160288373"/>
     <axis xyz="0.0 0.0 1.0"/>
     <parent link="shoulder_link"/>
@@ -416,5 +416,5 @@
   </joint>
   <joint name="elbow_joint" type="revolute">
-    <origin xyz="-0.6127 0.0 0.0" rpy="0.0 0.0 0.1000000149011612"/>
+    <origin xyz="-0.6027 0.01 0.01" rpy="0.01 0.01 0.014434684315030902"/>
     <axis xyz="0.0 0.0 1.0"/>
     <parent link="upper_arm_link"/>
@@ -424,5 +424,5 @@
   </joint>
   <joint name="wrist_1_joint" type="revolute">
-    <origin xyz="-0.57155 0.0 0.17415" rpy="0.0 0.0 0.1"/>
+    <origin xyz="-0.56155 0.01 0.18415" rpy="0.01 0.01 -0.08163482372003837"/>
     <axis xyz="0.0 0.0 1.0"/>
     <parent link="forearm_link"/>
@@ -432,5 +432,5 @@
   </joint>
   <joint name="wrist_2_joint" type="revolute">
-    <origin xyz="0.0 -0.11985 -2.458164590756244e-11" rpy="1.570796327 0.0 0.1"/>
+    <origin xyz="0.01 -0.10985 0.009999999975418354" rpy="1.580796327 0.01 0.003446624604334964"/>
     <axis xyz="0.0 0.0 1.0"/>
     <parent link="wrist_1_link"/>
@@ -440,5 +440,5 @@
   </joint>
   <joint name="wrist_3_joint" type="revolute">
-    <origin xyz="0.0 0.11655 -2.390480459346185e-11" rpy="1.570796326589793 3.141592653589793 3.241592653589793"/>
+    <origin xyz="0.01 0.12655 0.009999999976095195" rpy="1.580796326589793 3.151592653589793 2.9732490752583485"/>
     <axis xyz="0.0 0.0 1.0"/>
     <parent link="wrist_2_link"/>
@@ -556,5 +556,5 @@
   </joint>
   <joint name="rgb_world_joint" type="fixed">
-    <origin xyz="0.00845867852242976 -0.018804586436127927 0.03272963808730215" rpy="-0.005846135346919141 0.0006280903221295673 0.022082037670039148"/>
+    <origin xyz="0.022296483486666293 -0.008751527534067098 0.06409294918539783" rpy="-0.010598941974837519 0.023653515563518888 0.041152533629886794"/>
     <parent link="tripod_center_support"/>
     <child link="rgb_world_link"/>
@@ -695,4 +695,18 @@
     <child link="charuco_200x120_3x6"/>
   </joint>
+  <link name="charuco_200x200_8x8">
+    <origin xyz="0 0 0" rpy="0 0 0"/>
+    <visual name="hand_pattern_visual">
+      <origin xyz="0 0 0" rpy="0 0 0"/>
+      <geometry>
+        <mesh filename="package://atom_worlds/pattern/models/charuco_200x200_8x8_20_15_DICT_4x4/model.dae"/>
+      </geometry>
+    </visual>
+  </link>
+  <joint name="flange-charuco_200x200_8x8" type="fixed">
+    <origin xyz="0.050332518643287874 -0.05473769774536921 -0.008068461355240385" rpy="0.1279252290303904 -0.04225486679693917 0.02535454892339298"/>
+    <parent link="flange"/>
+    <child link="charuco_200x200_8x8"/>
+  </joint>
   <link name="charuco_200x120_3x6">
     <origin xyz="0 0 0" rpy="0 0 0"/>
@@ -705,5 +719,5 @@
   </link>
   <joint name="upper_arm_link-charuco_200x120_3x6" type="fixed">
-    <origin xyz="-0.23847704330245673 0.04398775918561481 0.09009886105268892" rpy="0.0038944889255176215 -0.001053401234966295 3.083018460864498"/>
+    <origin xyz="-0.23693903442687866 0.032489229890061186 0.09361493114969863" rpy="0.036837020859623315 0.02179716755024598 -3.1293625047103806"/>
     <parent link="upper_arm_link"/>
     <child link="charuco_200x120_3x6"/>

Commit message: Clsoe #980

File: atom_examples/riwmpbot/riwmpbot_calibration/urdf/optimized.urdf.xacro (robot description, xacro)
@@ -400,5 +400,5 @@
   </joint>
   <joint name="shoulder_pan_joint" type="revolute">
-    <origin xyz="0.01 0.01 0.1907" rpy="0.01 0.01 -0.010592558477970875"/>
+    <origin xyz="0.0 0.0 0.1807" rpy="0.0 0.0 0.0"/>
     <axis xyz="0.0 0.0 1.0"/>
     <parent link="base_link_inertia"/>
@@ -408,5 +408,5 @@
   </joint>
   <joint name="shoulder_lift_joint" type="revolute">
-    <origin xyz="0.01 0.01 0.01" rpy="1.580796327 0.01 0.00944167160288373"/>
+    <origin xyz="0.0 0.0 0.0" rpy="1.570796327 0.0 0.0"/>
     <axis xyz="0.0 0.0 1.0"/>
     <parent link="shoulder_link"/>
@@ -416,5 +416,5 @@
   </joint>
   <joint name="elbow_joint" type="revolute">
-    <origin xyz="-0.6027 0.01 0.01" rpy="0.01 0.01 0.014434684315030902"/>
+    <origin xyz="-0.6127 0.0 0.0" rpy="0.0 0.0 0.0"/>
     <axis xyz="0.0 0.0 1.0"/>
     <parent link="upper_arm_link"/>
@@ -424,5 +424,5 @@
   </joint>
   <joint name="wrist_1_joint" type="revolute">
-    <origin xyz="-0.56155 0.01 0.18415" rpy="0.01 0.01 -0.08163482372003837"/>
+    <origin xyz="-0.57155 0.0 0.17415" rpy="0.0 0.0 0.0"/>
     <axis xyz="0.0 0.0 1.0"/>
     <parent link="forearm_link"/>
@@ -432,5 +432,5 @@
   </joint>
   <joint name="wrist_2_joint" type="revolute">
-    <origin xyz="0.01 -0.10985 0.009999999975418354" rpy="1.580796327 0.01 0.003446624604334964"/>
+    <origin xyz="0.0 -0.11985 -2.458164590756244e-11" rpy="1.570796327 0.0 0.0"/>
     <axis xyz="0.0 0.0 1.0"/>
     <parent link="wrist_1_link"/>
@@ -440,5 +440,5 @@
   </joint>
   <joint name="wrist_3_joint" type="revolute">
-    <origin xyz="0.01 0.12655 0.009999999976095195" rpy="1.580796326589793 3.151592653589793 2.9732490752583485"/>
+    <origin xyz="0.0 0.11655 -2.390480459346185e-11" rpy="1.570796326589793 3.141592653589793 3.141592653589793"/>
     <axis xyz="0.0 0.0 1.0"/>
     <parent link="wrist_2_link"/>
@@ -556,5 +556,5 @@
   </joint>
   <joint name="rgb_world_joint" type="fixed">
-    <origin xyz="0.022296483486666293 -0.008751527534067098 0.06409294918539783" rpy="-0.010598941974837519 0.023653515563518888 0.041152533629886794"/>
+    <origin xyz="0.025716081273418394 -0.014141121777331733 0.07070233827966066" rpy="-0.016854646101008588 0.026221422548421313 0.05308311591115321"/>
     <parent link="tripod_center_support"/>
     <child link="rgb_world_link"/>

File: atom_examples/riwmpbot/riwmpbot_calibration/urdf/optimized_w_pattern.urdf.xacro (robot description, xacro)
@@ -400,5 +400,5 @@
   </joint>
   <joint name="shoulder_pan_joint" type="revolute">
-    <origin xyz="0.01 0.01 0.1907" rpy="0.01 0.01 -0.010592558477970875"/>
+    <origin xyz="0.0 0.0 0.1807" rpy="0.0 0.0 0.0"/>
     <axis xyz="0.0 0.0 1.0"/>
     <parent link="base_link_inertia"/>
@@ -408,5 +408,5 @@
   </joint>
   <joint name="shoulder_lift_joint" type="revolute">
-    <origin xyz="0.01 0.01 0.01" rpy="1.580796327 0.01 0.00944167160288373"/>
+    <origin xyz="0.0 0.0 0.0" rpy="1.570796327 0.0 0.0"/>
     <axis xyz="0.0 0.0 1.0"/>
     <parent link="shoulder_link"/>
@@ -416,5 +416,5 @@
   </joint>
   <joint name="elbow_joint" type="revolute">
-    <origin xyz="-0.6027 0.01 0.01" rpy="0.01 0.01 0.014434684315030902"/>
+    <origin xyz="-0.6127 0.0 0.0" rpy="0.0 0.0 0.0"/>
     <axis xyz="0.0 0.0 1.0"/>
     <parent link="upper_arm_link"/>
@@ -424,5 +424,5 @@
   </joint>
   <joint name="wrist_1_joint" type="revolute">
-    <origin xyz="-0.56155 0.01 0.18415" rpy="0.01 0.01 -0.08163482372003837"/>
+    <origin xyz="-0.57155 0.0 0.17415" rpy="0.0 0.0 0.0"/>
     <axis xyz="0.0 0.0 1.0"/>
     <parent link="forearm_link"/>
@@ -432,5 +432,5 @@
   </joint>
   <joint name="wrist_2_joint" type="revolute">
-    <origin xyz="0.01 -0.10985 0.009999999975418354" rpy="1.580796327 0.01 0.003446624604334964"/>
+    <origin xyz="0.0 -0.11985 -2.458164590756244e-11" rpy="1.570796327 0.0 0.0"/>
     <axis xyz="0.0 0.0 1.0"/>
     <parent link="wrist_1_link"/>
@@ -440,5 +440,5 @@
   </joint>
   <joint name="wrist_3_joint" type="revolute">
-    <origin xyz="0.01 0.12655 0.009999999976095195" rpy="1.580796326589793 3.151592653589793 2.9732490752583485"/>
+    <origin xyz="0.0 0.11655 -2.390480459346185e-11" rpy="1.570796326589793 3.141592653589793 3.141592653589793"/>
     <axis xyz="0.0 0.0 1.0"/>
     <parent link="wrist_2_link"/>
@@ -556,5 +556,5 @@
   </joint>
   <joint name="rgb_world_joint" type="fixed">
-    <origin xyz="0.022296483486666293 -0.008751527534067098 0.06409294918539783" rpy="-0.010598941974837519 0.023653515563518888 0.041152533629886794"/>
+    <origin xyz="0.025716081273418394 -0.014141121777331733 0.07070233827966066" rpy="-0.016854646101008588 0.026221422548421313 0.05308311591115321"/>
     <parent link="tripod_center_support"/>
     <child link="rgb_world_link"/>
@@ -695,4 +695,18 @@
     <child link="charuco_200x120_3x6"/>
   </joint>
+  <link name="charuco_170x100_3x6">
+    <origin xyz="0 0 0" rpy="0 0 0"/>
+    <visual name="forearm_pattern_visual">
+      <origin xyz="0 0 0" rpy="0 0 0"/>
+      <geometry>
+        <mesh filename="package://atom_worlds/pattern/models/charuco_170x100_3x6_25_18_DICT_6X6/model.dae"/>
+      </geometry>
+    </visual>
+  </link>
+  <joint name="forearm_link-charuco_170x100_3x6" type="fixed">
+    <origin xyz="-0.20341016483746766 0.026991408060476767 -0.024993282175946045" rpy="0.013754746149187633 -0.02642361277150804 3.123602880801382"/>
+    <parent link="forearm_link"/>
+    <child link="charuco_170x100_3x6"/>
+  </joint>
   <link name="charuco_200x200_8x8">
     <origin xyz="0 0 0" rpy="0 0 0"/>
@@ -705,5 +719,5 @@
   </link>
   <joint name="flange-charuco_200x200_8x8" type="fixed">
-    <origin xyz="0.050332518643287874 -0.05473769774536921 -0.008068461355240385" rpy="0.1279252290303904 -0.04225486679693917 0.02535454892339298"/>
+    <origin xyz="0.05527130904158837 -0.06702237686678414 -0.0002576381629635623" rpy="-0.03618929553684075 -0.019723133672620276 -0.049702790337666475"/>
     <parent link="flange"/>
     <child link="charuco_200x200_8x8"/>
@@ -719,5 +733,5 @@
   </link>
   <joint name="upper_arm_link-charuco_200x120_3x6" type="fixed">
-    <origin xyz="-0.23693903442687866 0.032489229890061186 0.09361493114969863" rpy="0.036837020859623315 0.02179716755024598 -3.1293625047103806"/>
+    <origin xyz="-0.23960446118082143 0.03511273854903906 0.0924623863997716" rpy="0.02889586028611301 0.021978940040478217 -3.1317682824231388"/>
     <parent link="upper_arm_link"/>
     <child link="charuco_200x120_3x6"/>
