Commit message: riwmpbot_real #846

File: atom_examples/riwmpbot/riwmpbot_description/urdf/robot.urdf.xacro (robot description, xacro)
@@ -8,7 +8,4 @@
     <!--  args are used with $(arg arg_name), properties are used as ${property_name}-->
     <xacro:property name="M_PI" value="3.1415926535897931" />
-    <material name="tripod_color">
-        <color rgba="0.21 0.21 .21 1" />
-    </material>
     <!-- Tables properties-->
     <xacro:property name="table_height" value="0.795"/>
@@ -80,5 +77,7 @@
                     scale="1 1 1" />
             </geometry>
-            <material name="tripod_color" />
+            <material name="tripod_color">
+                <color rgba="0.21 0.21 .21 1" />
+            </material>
         </visual>
         <collision name="tripod_collision">
@@ -107,5 +106,7 @@
                 <box size="0.04 0.4 0.015" />
             </geometry>
-            <material name="tripod_color" />
+            <material name="tripod_color">
+                <color rgba="0.21 0.21 .21 1" />
+            </material>
         </visual>
         <collision name="tripod_collision">
