Commit message: Close #857

File: atom_examples/riwmpbot/riwmpbot_real_calibration/urdf/optimized.urdf.xacro (robot description, xacro)
@@ -232,5 +232,5 @@
   </joint>
   <joint name="shoulder_pan_joint" type="revolute">
-    <origin xyz="0.0 0.0 0.1807" rpy="0.0 0.0 0.0822535575194899"/>
+    <origin xyz="0.0 0.0 0.1807" rpy="0.0 0.0 0.07674188501164143"/>
     <axis xyz="0.0 0.0 1.0"/>
     <parent link="base_link_inertia"/>
@@ -240,5 +240,5 @@
   </joint>
   <joint name="shoulder_lift_joint" type="revolute">
-    <origin xyz="0.0 0.0 0.0" rpy="1.570796327 0.0 -0.003077477915289702"/>
+    <origin xyz="0.0 0.0 0.0" rpy="1.570796327 0.0 0.03186955739531561"/>
     <axis xyz="0.0 0.0 1.0"/>
     <parent link="shoulder_link"/>
@@ -248,5 +248,5 @@
   </joint>
   <joint name="elbow_joint" type="revolute">
-    <origin xyz="-0.6127 0.0 0.0" rpy="0.0 0.0 0.0019060893780688103"/>
+    <origin xyz="-0.6127 0.0 0.0" rpy="0.0 0.0 0.001576827651516932"/>
     <axis xyz="0.0 0.0 1.0"/>
     <parent link="upper_arm_link"/>
@@ -256,5 +256,5 @@
   </joint>
   <joint name="wrist_1_joint" type="revolute">
-    <origin xyz="-0.57155 0.0 0.17415" rpy="0.0 0.0 -0.0196407938674062"/>
+    <origin xyz="-0.57155 0.0 0.17415" rpy="0.0 0.0 -0.011303978157411944"/>
     <axis xyz="0.0 0.0 1.0"/>
     <parent link="forearm_link"/>
@@ -264,5 +264,5 @@
   </joint>
   <joint name="wrist_2_joint" type="revolute">
-    <origin xyz="0.0 -0.11985 -2.458164590756244e-11" rpy="1.570796327 0.0 -0.005612778984260009"/>
+    <origin xyz="0.0 -0.11985 -2.458164590756244e-11" rpy="1.570796327 0.0 -0.002380656087006292"/>
     <axis xyz="0.0 0.0 1.0"/>
     <parent link="wrist_1_link"/>
@@ -272,5 +272,5 @@
   </joint>
   <joint name="wrist_3_joint" type="revolute">
-    <origin xyz="0.0 0.11655 -2.390480459346185e-11" rpy="1.570796326589793 3.141592653589793 3.246983445260619"/>
+    <origin xyz="0.0 0.11655 -2.390480459346185e-11" rpy="1.570796326589793 3.141592653589793 3.2323974286067454"/>
     <axis xyz="0.0 0.0 1.0"/>
     <parent link="wrist_2_link"/>
@@ -328,5 +328,5 @@
   </joint>
   <joint name="rgb_world_joint" type="fixed">
-    <origin xyz="0.8931029691791313 0.38392855381454083 0.8020176114575999" rpy="-0.002604594734949345 0.19851701840569935 3.0990262706245266"/>
+    <origin xyz="0.8951212301869304 0.3937247041762815 0.7840209137014122" rpy="0.037490854275979126 0.1969284950477124 3.0944840129391333"/>
     <parent link="world"/>
     <child link="rgb_world_link"/>

File: atom_examples/riwmpbot/riwmpbot_real_calibration/urdf/optimized_w_pattern.urdf.xacro (robot description, xacro)
@@ -232,5 +232,5 @@
   </joint>
   <joint name="shoulder_pan_joint" type="revolute">
-    <origin xyz="0.0 0.0 0.1807" rpy="0.0 0.0 0.0822535575194899"/>
+    <origin xyz="0.0 0.0 0.1807" rpy="0.0 0.0 0.07674188501164143"/>
     <axis xyz="0.0 0.0 1.0"/>
     <parent link="base_link_inertia"/>
@@ -240,5 +240,5 @@
   </joint>
   <joint name="shoulder_lift_joint" type="revolute">
-    <origin xyz="0.0 0.0 0.0" rpy="1.570796327 0.0 -0.003077477915289702"/>
+    <origin xyz="0.0 0.0 0.0" rpy="1.570796327 0.0 0.03186955739531561"/>
     <axis xyz="0.0 0.0 1.0"/>
     <parent link="shoulder_link"/>
@@ -248,5 +248,5 @@
   </joint>
   <joint name="elbow_joint" type="revolute">
-    <origin xyz="-0.6127 0.0 0.0" rpy="0.0 0.0 0.0019060893780688103"/>
+    <origin xyz="-0.6127 0.0 0.0" rpy="0.0 0.0 0.001576827651516932"/>
     <axis xyz="0.0 0.0 1.0"/>
     <parent link="upper_arm_link"/>
@@ -256,5 +256,5 @@
   </joint>
   <joint name="wrist_1_joint" type="revolute">
-    <origin xyz="-0.57155 0.0 0.17415" rpy="0.0 0.0 -0.0196407938674062"/>
+    <origin xyz="-0.57155 0.0 0.17415" rpy="0.0 0.0 -0.011303978157411944"/>
     <axis xyz="0.0 0.0 1.0"/>
     <parent link="forearm_link"/>
@@ -264,5 +264,5 @@
   </joint>
   <joint name="wrist_2_joint" type="revolute">
-    <origin xyz="0.0 -0.11985 -2.458164590756244e-11" rpy="1.570796327 0.0 -0.005612778984260009"/>
+    <origin xyz="0.0 -0.11985 -2.458164590756244e-11" rpy="1.570796327 0.0 -0.002380656087006292"/>
     <axis xyz="0.0 0.0 1.0"/>
     <parent link="wrist_1_link"/>
@@ -272,5 +272,5 @@
   </joint>
   <joint name="wrist_3_joint" type="revolute">
-    <origin xyz="0.0 0.11655 -2.390480459346185e-11" rpy="1.570796326589793 3.141592653589793 3.246983445260619"/>
+    <origin xyz="0.0 0.11655 -2.390480459346185e-11" rpy="1.570796326589793 3.141592653589793 3.2323974286067454"/>
     <axis xyz="0.0 0.0 1.0"/>
     <parent link="wrist_2_link"/>
@@ -328,5 +328,5 @@
   </joint>
   <joint name="rgb_world_joint" type="fixed">
-    <origin xyz="0.8931029691791313 0.38392855381454083 0.8020176114575999" rpy="-0.002604594734949345 0.19851701840569935 3.0990262706245266"/>
+    <origin xyz="0.8951212301869304 0.3937247041762815 0.7840209137014122" rpy="0.037490854275979126 0.1969284950477124 3.0944840129391333"/>
     <parent link="world"/>
     <child link="rgb_world_link"/>
@@ -477,5 +477,5 @@
   </link>
   <joint name="forearm_link-charuco_170x100_3x6" type="fixed">
-    <origin xyz="-0.23056521535284497 0.02747537749464569 -0.03985315741468601" rpy="0.14249884319887532 0.007164390109794233 3.110841435202628"/>
+    <origin xyz="-0.22966736710237823 0.026105100098055254 -0.04512410891294524" rpy="0.15871386790872472 0.005642000937622307 3.114305564264507"/>
     <parent link="forearm_link"/>
     <child link="charuco_170x100_3x6"/>
@@ -491,5 +491,5 @@
   </link>
   <joint name="flange-charuco_200x200_8x8" type="fixed">
-    <origin xyz="0.2886496045601343 -0.009590828795216744 -0.09221767192167213" rpy="-3.0178107994617207 -1.5068585496336824 1.4594440711983472"/>
+    <origin xyz="0.28955203126849505 -0.00937358897679858 -0.08860266131624434" rpy="-3.0219825477134528 -1.5256196387167134 1.4675909306433417"/>
     <parent link="flange"/>
     <child link="charuco_200x200_8x8"/>
@@ -505,5 +505,5 @@
   </link>
   <joint name="upper_arm_link-charuco_200x120_3x6" type="fixed">
-    <origin xyz="-0.2529807018710277 0.03336967152319507 0.07769663968516914" rpy="0.23244669846873295 -0.006432718302185027 -3.138286006883133"/>
+    <origin xyz="-0.25346715294220046 0.03461940931950556 0.08090259818003159" rpy="0.22523871749433652 0.0012112585337772158 -3.134170290667222"/>
     <parent link="upper_arm_link"/>
     <child link="charuco_200x120_3x6"/>

Commit message: #866 implemented and working

File: atom_examples/riwmpbot/riwmpbot_real_calibration/urdf/optimized.urdf.xacro (robot description, xacro)
@@ -232,5 +232,5 @@
   </joint>
   <joint name="shoulder_pan_joint" type="revolute">
-    <origin xyz="0.0 0.0 0.1807" rpy="0.0 0.0 0.07674188501164143"/>
+    <origin xyz="0.0 0.0 0.1807" rpy="0.0 0.0 0.08247610195389375"/>
     <axis xyz="0.0 0.0 1.0"/>
     <parent link="base_link_inertia"/>
@@ -240,5 +240,5 @@
   </joint>
   <joint name="shoulder_lift_joint" type="revolute">
-    <origin xyz="0.0 0.0 0.0" rpy="1.570796327 0.0 0.03186955739531561"/>
+    <origin xyz="0.0 0.0 0.0" rpy="1.570796327 0.0 0.00384052180304222"/>
     <axis xyz="0.0 0.0 1.0"/>
     <parent link="shoulder_link"/>
@@ -248,5 +248,5 @@
   </joint>
   <joint name="elbow_joint" type="revolute">
-    <origin xyz="-0.6127 0.0 0.0" rpy="0.0 0.0 0.001576827651516932"/>
+    <origin xyz="-0.6127 0.0 0.0" rpy="0.0 0.0 0.0021025736190257885"/>
     <axis xyz="0.0 0.0 1.0"/>
     <parent link="upper_arm_link"/>
@@ -256,5 +256,5 @@
   </joint>
   <joint name="wrist_1_joint" type="revolute">
-    <origin xyz="-0.57155 0.0 0.17415" rpy="0.0 0.0 -0.011303978157411944"/>
+    <origin xyz="-0.57155 0.0 0.17415" rpy="0.0 0.0 -0.011638934121678272"/>
     <axis xyz="0.0 0.0 1.0"/>
     <parent link="forearm_link"/>
@@ -264,5 +264,5 @@
   </joint>
   <joint name="wrist_2_joint" type="revolute">
-    <origin xyz="0.0 -0.11985 -2.458164590756244e-11" rpy="1.570796327 0.0 -0.002380656087006292"/>
+    <origin xyz="0.0 -0.11985 -2.458164590756244e-11" rpy="1.570796327 0.0 0.000817516768077408"/>
     <axis xyz="0.0 0.0 1.0"/>
     <parent link="wrist_1_link"/>
@@ -272,5 +272,5 @@
   </joint>
   <joint name="wrist_3_joint" type="revolute">
-    <origin xyz="0.0 0.11655 -2.390480459346185e-11" rpy="1.570796326589793 3.141592653589793 3.2323974286067454"/>
+    <origin xyz="0.0 0.11655 -2.390480459346185e-11" rpy="1.570796326589793 3.141592653589793 3.040682888934066"/>
     <axis xyz="0.0 0.0 1.0"/>
     <parent link="wrist_2_link"/>
@@ -328,5 +328,5 @@
   </joint>
   <joint name="rgb_world_joint" type="fixed">
-    <origin xyz="0.8951212301869304 0.3937247041762815 0.7840209137014122" rpy="0.037490854275979126 0.1969284950477124 3.0944840129391333"/>
+    <origin xyz="0.8972664603191516 0.38546506644465894 0.7890661252208409" rpy="0.006699252263354212 0.19001137670858192 3.097424746424984"/>
     <parent link="world"/>
     <child link="rgb_world_link"/>

File: atom_examples/riwmpbot/riwmpbot_real_calibration/urdf/optimized_w_pattern.urdf.xacro (robot description, xacro)
@@ -232,5 +232,5 @@
   </joint>
   <joint name="shoulder_pan_joint" type="revolute">
-    <origin xyz="0.0 0.0 0.1807" rpy="0.0 0.0 0.07674188501164143"/>
+    <origin xyz="0.0 0.0 0.1807" rpy="0.0 0.0 0.08247610195389375"/>
     <axis xyz="0.0 0.0 1.0"/>
     <parent link="base_link_inertia"/>
@@ -240,5 +240,5 @@
   </joint>
   <joint name="shoulder_lift_joint" type="revolute">
-    <origin xyz="0.0 0.0 0.0" rpy="1.570796327 0.0 0.03186955739531561"/>
+    <origin xyz="0.0 0.0 0.0" rpy="1.570796327 0.0 0.00384052180304222"/>
     <axis xyz="0.0 0.0 1.0"/>
     <parent link="shoulder_link"/>
@@ -248,5 +248,5 @@
   </joint>
   <joint name="elbow_joint" type="revolute">
-    <origin xyz="-0.6127 0.0 0.0" rpy="0.0 0.0 0.001576827651516932"/>
+    <origin xyz="-0.6127 0.0 0.0" rpy="0.0 0.0 0.0021025736190257885"/>
     <axis xyz="0.0 0.0 1.0"/>
     <parent link="upper_arm_link"/>
@@ -256,5 +256,5 @@
   </joint>
   <joint name="wrist_1_joint" type="revolute">
-    <origin xyz="-0.57155 0.0 0.17415" rpy="0.0 0.0 -0.011303978157411944"/>
+    <origin xyz="-0.57155 0.0 0.17415" rpy="0.0 0.0 -0.011638934121678272"/>
     <axis xyz="0.0 0.0 1.0"/>
     <parent link="forearm_link"/>
@@ -264,5 +264,5 @@
   </joint>
   <joint name="wrist_2_joint" type="revolute">
-    <origin xyz="0.0 -0.11985 -2.458164590756244e-11" rpy="1.570796327 0.0 -0.002380656087006292"/>
+    <origin xyz="0.0 -0.11985 -2.458164590756244e-11" rpy="1.570796327 0.0 0.000817516768077408"/>
     <axis xyz="0.0 0.0 1.0"/>
     <parent link="wrist_1_link"/>
@@ -272,5 +272,5 @@
   </joint>
   <joint name="wrist_3_joint" type="revolute">
-    <origin xyz="0.0 0.11655 -2.390480459346185e-11" rpy="1.570796326589793 3.141592653589793 3.2323974286067454"/>
+    <origin xyz="0.0 0.11655 -2.390480459346185e-11" rpy="1.570796326589793 3.141592653589793 3.040682888934066"/>
     <axis xyz="0.0 0.0 1.0"/>
     <parent link="wrist_2_link"/>
@@ -328,5 +328,5 @@
   </joint>
   <joint name="rgb_world_joint" type="fixed">
-    <origin xyz="0.8951212301869304 0.3937247041762815 0.7840209137014122" rpy="0.037490854275979126 0.1969284950477124 3.0944840129391333"/>
+    <origin xyz="0.8972664603191516 0.38546506644465894 0.7890661252208409" rpy="0.006699252263354212 0.19001137670858192 3.097424746424984"/>
     <parent link="world"/>
     <child link="rgb_world_link"/>
@@ -477,5 +477,5 @@
   </link>
   <joint name="forearm_link-charuco_170x100_3x6" type="fixed">
-    <origin xyz="-0.22966736710237823 0.026105100098055254 -0.04512410891294524" rpy="0.15871386790872472 0.005642000937622307 3.114305564264507"/>
+    <origin xyz="-0.23030947470677612 0.025210805053674967 -0.04174991167465683" rpy="0.1353812095591838 0.01980013496555183 3.1105799226323128"/>
     <parent link="forearm_link"/>
     <child link="charuco_170x100_3x6"/>
@@ -491,5 +491,5 @@
   </link>
   <joint name="flange-charuco_200x200_8x8" type="fixed">
-    <origin xyz="0.28955203126849505 -0.00937358897679858 -0.08860266131624434" rpy="-3.0219825477134528 -1.5256196387167134 1.4675909306433417"/>
+    <origin xyz="0.28965456812260126 0.007407915025531259 -0.08703857822070203" rpy="0.040428928763401824 -1.4260207807947143 -1.5991767846382356"/>
     <parent link="flange"/>
     <child link="charuco_200x200_8x8"/>
@@ -505,5 +505,5 @@
   </link>
   <joint name="upper_arm_link-charuco_200x120_3x6" type="fixed">
-    <origin xyz="-0.25346715294220046 0.03461940931950556 0.08090259818003159" rpy="0.22523871749433652 0.0012112585337772158 -3.134170290667222"/>
+    <origin xyz="-0.25082800139087297 0.03383564570676676 0.08218412165297458" rpy="0.20773107808394004 -0.007553680282443692 -3.1397727918595697"/>
     <parent link="upper_arm_link"/>
     <child link="charuco_200x120_3x6"/>

Commit message: Experimenting with #860

File: atom_examples/riwmpbot/riwmpbot_real_calibration/urdf/optimized.urdf.xacro (robot description, xacro)
@@ -232,5 +232,5 @@
   </joint>
   <joint name="shoulder_pan_joint" type="revolute">
-    <origin xyz="0.0 0.0 0.1807" rpy="0.0 0.0 0.08247610195389375"/>
+    <origin xyz="0.0 0.0 0.1807" rpy="0.0 0.0 0.06848837454606206"/>
     <axis xyz="0.0 0.0 1.0"/>
     <parent link="base_link_inertia"/>
@@ -240,5 +240,5 @@
   </joint>
   <joint name="shoulder_lift_joint" type="revolute">
-    <origin xyz="0.0 0.0 0.0" rpy="1.570796327 0.0 0.00384052180304222"/>
+    <origin xyz="0.0 0.0 0.0" rpy="1.570796327 0.0 0.011814835200384313"/>
     <axis xyz="0.0 0.0 1.0"/>
     <parent link="shoulder_link"/>
@@ -248,5 +248,5 @@
   </joint>
   <joint name="elbow_joint" type="revolute">
-    <origin xyz="-0.6127 0.0 0.0" rpy="0.0 0.0 0.0021025736190257885"/>
+    <origin xyz="-0.6127 0.0 0.0" rpy="0.0 0.0 -0.003229602699436045"/>
     <axis xyz="0.0 0.0 1.0"/>
     <parent link="upper_arm_link"/>
@@ -256,5 +256,5 @@
   </joint>
   <joint name="wrist_1_joint" type="revolute">
-    <origin xyz="-0.57155 0.0 0.17415" rpy="0.0 0.0 -0.011638934121678272"/>
+    <origin xyz="-0.57155 0.0 0.17415" rpy="0.0 0.0 -0.0032761411013731002"/>
     <axis xyz="0.0 0.0 1.0"/>
     <parent link="forearm_link"/>
@@ -264,5 +264,5 @@
   </joint>
   <joint name="wrist_2_joint" type="revolute">
-    <origin xyz="0.0 -0.11985 -2.458164590756244e-11" rpy="1.570796327 0.0 0.000817516768077408"/>
+    <origin xyz="0.0 -0.11985 -2.458164590756244e-11" rpy="1.570796327 0.0 0.0027982324082962743"/>
     <axis xyz="0.0 0.0 1.0"/>
     <parent link="wrist_1_link"/>
@@ -272,5 +272,5 @@
   </joint>
   <joint name="wrist_3_joint" type="revolute">
-    <origin xyz="0.0 0.11655 -2.390480459346185e-11" rpy="1.570796326589793 3.141592653589793 3.040682888934066"/>
+    <origin xyz="0.0 0.11655 -2.390480459346185e-11" rpy="1.570796326589793 3.141592653589793 2.973454438310112"/>
     <axis xyz="0.0 0.0 1.0"/>
     <parent link="wrist_2_link"/>
@@ -328,5 +328,5 @@
   </joint>
   <joint name="rgb_world_joint" type="fixed">
-    <origin xyz="0.8972664603191516 0.38546506644465894 0.7890661252208409" rpy="0.006699252263354212 0.19001137670858192 3.097424746424984"/>
+    <origin xyz="0.9021379781351333 0.38095822950567626 0.7833526678103171" rpy="0.014966413136018054 0.18528211848316328 3.088214539170947"/>
     <parent link="world"/>
     <child link="rgb_world_link"/>

File: atom_examples/riwmpbot/riwmpbot_real_calibration/urdf/optimized_w_pattern.urdf.xacro (robot description, xacro)
@@ -232,5 +232,5 @@
   </joint>
   <joint name="shoulder_pan_joint" type="revolute">
-    <origin xyz="0.0 0.0 0.1807" rpy="0.0 0.0 0.08247610195389375"/>
+    <origin xyz="0.0 0.0 0.1807" rpy="0.0 0.0 0.06848837454606206"/>
     <axis xyz="0.0 0.0 1.0"/>
     <parent link="base_link_inertia"/>
@@ -240,5 +240,5 @@
   </joint>
   <joint name="shoulder_lift_joint" type="revolute">
-    <origin xyz="0.0 0.0 0.0" rpy="1.570796327 0.0 0.00384052180304222"/>
+    <origin xyz="0.0 0.0 0.0" rpy="1.570796327 0.0 0.011814835200384313"/>
     <axis xyz="0.0 0.0 1.0"/>
     <parent link="shoulder_link"/>
@@ -248,5 +248,5 @@
   </joint>
   <joint name="elbow_joint" type="revolute">
-    <origin xyz="-0.6127 0.0 0.0" rpy="0.0 0.0 0.0021025736190257885"/>
+    <origin xyz="-0.6127 0.0 0.0" rpy="0.0 0.0 -0.003229602699436045"/>
     <axis xyz="0.0 0.0 1.0"/>
     <parent link="upper_arm_link"/>
@@ -256,5 +256,5 @@
   </joint>
   <joint name="wrist_1_joint" type="revolute">
-    <origin xyz="-0.57155 0.0 0.17415" rpy="0.0 0.0 -0.011638934121678272"/>
+    <origin xyz="-0.57155 0.0 0.17415" rpy="0.0 0.0 -0.0032761411013731002"/>
     <axis xyz="0.0 0.0 1.0"/>
     <parent link="forearm_link"/>
@@ -264,5 +264,5 @@
   </joint>
   <joint name="wrist_2_joint" type="revolute">
-    <origin xyz="0.0 -0.11985 -2.458164590756244e-11" rpy="1.570796327 0.0 0.000817516768077408"/>
+    <origin xyz="0.0 -0.11985 -2.458164590756244e-11" rpy="1.570796327 0.0 0.0027982324082962743"/>
     <axis xyz="0.0 0.0 1.0"/>
     <parent link="wrist_1_link"/>
@@ -272,5 +272,5 @@
   </joint>
   <joint name="wrist_3_joint" type="revolute">
-    <origin xyz="0.0 0.11655 -2.390480459346185e-11" rpy="1.570796326589793 3.141592653589793 3.040682888934066"/>
+    <origin xyz="0.0 0.11655 -2.390480459346185e-11" rpy="1.570796326589793 3.141592653589793 2.973454438310112"/>
     <axis xyz="0.0 0.0 1.0"/>
     <parent link="wrist_2_link"/>
@@ -328,5 +328,5 @@
   </joint>
   <joint name="rgb_world_joint" type="fixed">
-    <origin xyz="0.8972664603191516 0.38546506644465894 0.7890661252208409" rpy="0.006699252263354212 0.19001137670858192 3.097424746424984"/>
+    <origin xyz="0.9021379781351333 0.38095822950567626 0.7833526678103171" rpy="0.014966413136018054 0.18528211848316328 3.088214539170947"/>
     <parent link="world"/>
     <child link="rgb_world_link"/>
@@ -477,5 +477,5 @@
   </link>
   <joint name="forearm_link-charuco_170x100_3x6" type="fixed">
-    <origin xyz="-0.23030947470677612 0.025210805053674967 -0.04174991167465683" rpy="0.1353812095591838 0.01980013496555183 3.1105799226323128"/>
+    <origin xyz="-0.23109462446549722 0.025706559880365132 -0.040633966157589005" rpy="0.1351470404273847 0.01071248050696558 3.1141077061624918"/>
     <parent link="forearm_link"/>
     <child link="charuco_170x100_3x6"/>
@@ -491,5 +491,5 @@
   </link>
   <joint name="flange-charuco_200x200_8x8" type="fixed">
-    <origin xyz="0.28965456812260126 0.007407915025531259 -0.08703857822070203" rpy="0.040428928763401824 -1.4260207807947143 -1.5991767846382356"/>
+    <origin xyz="0.28940004303144296 0.011881558302268787 -0.08451163577354652" rpy="0.051068679126574486 -1.370247976848198 -1.6171851349548847"/>
     <parent link="flange"/>
     <child link="charuco_200x200_8x8"/>
@@ -505,5 +505,5 @@
   </link>
   <joint name="upper_arm_link-charuco_200x120_3x6" type="fixed">
-    <origin xyz="-0.25082800139087297 0.03383564570676676 0.08218412165297458" rpy="0.20773107808394004 -0.007553680282443692 -3.1397727918595697"/>
+    <origin xyz="-0.25283165508403355 0.03419449186892774 0.08431092908305873" rpy="0.20698495147970403 -0.006320871714294667 3.1414110319318524"/>
     <parent link="upper_arm_link"/>
     <child link="charuco_200x120_3x6"/>
