Commit message: #860 Several corrections in scripts.

File: atom_examples/riwmpbot/riwmpbot_real_calibration/urdf/optimized.urdf.xacro (robot description, xacro)
@@ -232,5 +232,5 @@
   </joint>
   <joint name="shoulder_pan_joint" type="revolute">
-    <origin xyz="0.0 0.0 0.1807" rpy="0.0 0.0 0.06848837454606206"/>
+    <origin xyz="0.0 0.0 0.1807" rpy="0.0 0.0 0.06401148706013562"/>
     <axis xyz="0.0 0.0 1.0"/>
     <parent link="base_link_inertia"/>
@@ -240,5 +240,5 @@
   </joint>
   <joint name="shoulder_lift_joint" type="revolute">
-    <origin xyz="0.0 0.0 0.0" rpy="1.570796327 0.0 0.011814835200384313"/>
+    <origin xyz="0.0 0.0 0.0" rpy="1.570796327 0.0 0.009910204783218489"/>
     <axis xyz="0.0 0.0 1.0"/>
     <parent link="shoulder_link"/>
@@ -248,5 +248,5 @@
   </joint>
   <joint name="elbow_joint" type="revolute">
-    <origin xyz="-0.6127 0.0 0.0" rpy="0.0 0.0 -0.003229602699436045"/>
+    <origin xyz="-0.6127 0.0 0.0" rpy="0.0 0.0 -0.002139318459194392"/>
     <axis xyz="0.0 0.0 1.0"/>
     <parent link="upper_arm_link"/>
@@ -256,5 +256,5 @@
   </joint>
   <joint name="wrist_1_joint" type="revolute">
-    <origin xyz="-0.57155 0.0 0.17415" rpy="0.0 0.0 -0.0032761411013731002"/>
+    <origin xyz="-0.57155 0.0 0.17415" rpy="0.0 0.0 -0.011633411894526994"/>
     <axis xyz="0.0 0.0 1.0"/>
     <parent link="forearm_link"/>
@@ -264,5 +264,5 @@
   </joint>
   <joint name="wrist_2_joint" type="revolute">
-    <origin xyz="0.0 -0.11985 -2.458164590756244e-11" rpy="1.570796327 0.0 0.0027982324082962743"/>
+    <origin xyz="0.0 -0.11985 -2.458164590756244e-11" rpy="1.570796327 0.0 0.00235299412437361"/>
     <axis xyz="0.0 0.0 1.0"/>
     <parent link="wrist_1_link"/>
@@ -272,5 +272,5 @@
   </joint>
   <joint name="wrist_3_joint" type="revolute">
-    <origin xyz="0.0 0.11655 -2.390480459346185e-11" rpy="1.570796326589793 3.141592653589793 2.973454438310112"/>
+    <origin xyz="0.0 0.11655 -2.390480459346185e-11" rpy="1.570796326589793 3.141592653589793 2.971795491526189"/>
     <axis xyz="0.0 0.0 1.0"/>
     <parent link="wrist_2_link"/>
@@ -328,5 +328,5 @@
   </joint>
   <joint name="rgb_world_joint" type="fixed">
-    <origin xyz="0.9021379781351333 0.38095822950567626 0.7833526678103171" rpy="0.014966413136018054 0.18528211848316328 3.088214539170947"/>
+    <origin xyz="0.9040307558583056 0.37340685909697446 0.7863156345009282" rpy="0.011250318836873024 0.18824459381100403 3.0808278801572553"/>
     <parent link="world"/>
     <child link="rgb_world_link"/>

File: atom_examples/riwmpbot/riwmpbot_real_calibration/urdf/optimized_w_pattern.urdf.xacro (robot description, xacro)
@@ -232,5 +232,5 @@
   </joint>
   <joint name="shoulder_pan_joint" type="revolute">
-    <origin xyz="0.0 0.0 0.1807" rpy="0.0 0.0 0.06848837454606206"/>
+    <origin xyz="0.0 0.0 0.1807" rpy="0.0 0.0 0.06401148706013562"/>
     <axis xyz="0.0 0.0 1.0"/>
     <parent link="base_link_inertia"/>
@@ -240,5 +240,5 @@
   </joint>
   <joint name="shoulder_lift_joint" type="revolute">
-    <origin xyz="0.0 0.0 0.0" rpy="1.570796327 0.0 0.011814835200384313"/>
+    <origin xyz="0.0 0.0 0.0" rpy="1.570796327 0.0 0.009910204783218489"/>
     <axis xyz="0.0 0.0 1.0"/>
     <parent link="shoulder_link"/>
@@ -248,5 +248,5 @@
   </joint>
   <joint name="elbow_joint" type="revolute">
-    <origin xyz="-0.6127 0.0 0.0" rpy="0.0 0.0 -0.003229602699436045"/>
+    <origin xyz="-0.6127 0.0 0.0" rpy="0.0 0.0 -0.002139318459194392"/>
     <axis xyz="0.0 0.0 1.0"/>
     <parent link="upper_arm_link"/>
@@ -256,5 +256,5 @@
   </joint>
   <joint name="wrist_1_joint" type="revolute">
-    <origin xyz="-0.57155 0.0 0.17415" rpy="0.0 0.0 -0.0032761411013731002"/>
+    <origin xyz="-0.57155 0.0 0.17415" rpy="0.0 0.0 -0.011633411894526994"/>
     <axis xyz="0.0 0.0 1.0"/>
     <parent link="forearm_link"/>
@@ -264,5 +264,5 @@
   </joint>
   <joint name="wrist_2_joint" type="revolute">
-    <origin xyz="0.0 -0.11985 -2.458164590756244e-11" rpy="1.570796327 0.0 0.0027982324082962743"/>
+    <origin xyz="0.0 -0.11985 -2.458164590756244e-11" rpy="1.570796327 0.0 0.00235299412437361"/>
     <axis xyz="0.0 0.0 1.0"/>
     <parent link="wrist_1_link"/>
@@ -272,5 +272,5 @@
   </joint>
   <joint name="wrist_3_joint" type="revolute">
-    <origin xyz="0.0 0.11655 -2.390480459346185e-11" rpy="1.570796326589793 3.141592653589793 2.973454438310112"/>
+    <origin xyz="0.0 0.11655 -2.390480459346185e-11" rpy="1.570796326589793 3.141592653589793 2.971795491526189"/>
     <axis xyz="0.0 0.0 1.0"/>
     <parent link="wrist_2_link"/>
@@ -328,5 +328,5 @@
   </joint>
   <joint name="rgb_world_joint" type="fixed">
-    <origin xyz="0.9021379781351333 0.38095822950567626 0.7833526678103171" rpy="0.014966413136018054 0.18528211848316328 3.088214539170947"/>
+    <origin xyz="0.9040307558583056 0.37340685909697446 0.7863156345009282" rpy="0.011250318836873024 0.18824459381100403 3.0808278801572553"/>
     <parent link="world"/>
     <child link="rgb_world_link"/>
@@ -467,18 +467,4 @@
     <child link="charuco_200x120_3x6"/>
   </joint>
-  <link name="charuco_170x100_3x6">
-    <origin xyz="0 0 0" rpy="0 0 0"/>
-    <visual name="forearm_pattern_visual">
-      <origin xyz="0 0 0" rpy="0 0 0"/>
-      <geometry>
-        <mesh filename="package://atom_worlds/pattern/models/charuco_170x100_3x6_25_18_DICT_6X6/model.dae"/>
-      </geometry>
-    </visual>
-  </link>
-  <joint name="forearm_link-charuco_170x100_3x6" type="fixed">
-    <origin xyz="-0.23109462446549722 0.025706559880365132 -0.040633966157589005" rpy="0.1351470404273847 0.01071248050696558 3.1141077061624918"/>
-    <parent link="forearm_link"/>
-    <child link="charuco_170x100_3x6"/>
-  </joint>
   <link name="charuco_200x200_8x8">
     <origin xyz="0 0 0" rpy="0 0 0"/>
@@ -491,21 +477,7 @@
   </link>
   <joint name="flange-charuco_200x200_8x8" type="fixed">
-    <origin xyz="0.28940004303144296 0.011881558302268787 -0.08451163577354652" rpy="0.051068679126574486 -1.370247976848198 -1.6171851349548847"/>
+    <origin xyz="0.29025985756421346 0.013223176403322864 -0.08712675178453624" rpy="0.02985713217726388 -1.365031616760473 -1.5927739084396466"/>
     <parent link="flange"/>
     <child link="charuco_200x200_8x8"/>
   </joint>
-  <link name="charuco_200x120_3x6">
-    <origin xyz="0 0 0" rpy="0 0 0"/>
-    <visual name="upper_arm_pattern_visual">
-      <origin xyz="0 0 0" rpy="0 0 0"/>
-      <geometry>
-        <mesh filename="package://atom_worlds/pattern/models/charuco_200x120_3x6_30_22_DICT_7X7/model.dae"/>
-      </geometry>
-    </visual>
-  </link>
-  <joint name="upper_arm_link-charuco_200x120_3x6" type="fixed">
-    <origin xyz="-0.25283165508403355 0.03419449186892774 0.08431092908305873" rpy="0.20698495147970403 -0.006320871714294667 3.1414110319318524"/>
-    <parent link="upper_arm_link"/>
-    <child link="charuco_200x120_3x6"/>
-  </joint>
 </robot>

Commit message: Minor changes

File: atom_examples/riwmpbot/riwmpbot_real_calibration/urdf/optimized.urdf.xacro (robot description, xacro)
@@ -232,5 +232,5 @@
   </joint>
   <joint name="shoulder_pan_joint" type="revolute">
-    <origin xyz="0.0 0.0 0.1807" rpy="0.0 0.0 0.06401148706013562"/>
+    <origin xyz="0.0 0.0 0.1807" rpy="0.0 0.0 0.06054631110770013"/>
     <axis xyz="0.0 0.0 1.0"/>
     <parent link="base_link_inertia"/>
@@ -240,5 +240,5 @@
   </joint>
   <joint name="shoulder_lift_joint" type="revolute">
-    <origin xyz="0.0 0.0 0.0" rpy="1.570796327 0.0 0.009910204783218489"/>
+    <origin xyz="0.0 0.0 0.0" rpy="1.570796327 0.0 0.00843600239413617"/>
     <axis xyz="0.0 0.0 1.0"/>
     <parent link="shoulder_link"/>
@@ -248,5 +248,5 @@
   </joint>
   <joint name="elbow_joint" type="revolute">
-    <origin xyz="-0.6127 0.0 0.0" rpy="0.0 0.0 -0.002139318459194392"/>
+    <origin xyz="-0.6127 0.0 0.0" rpy="0.0 0.0 0.0034924794019561226"/>
     <axis xyz="0.0 0.0 1.0"/>
     <parent link="upper_arm_link"/>
@@ -256,5 +256,5 @@
   </joint>
   <joint name="wrist_1_joint" type="revolute">
-    <origin xyz="-0.57155 0.0 0.17415" rpy="0.0 0.0 -0.011633411894526994"/>
+    <origin xyz="-0.57155 0.0 0.17415" rpy="0.0 0.0 -0.0038882384676595"/>
     <axis xyz="0.0 0.0 1.0"/>
     <parent link="forearm_link"/>
@@ -264,5 +264,5 @@
   </joint>
   <joint name="wrist_2_joint" type="revolute">
-    <origin xyz="0.0 -0.11985 -2.458164590756244e-11" rpy="1.570796327 0.0 0.00235299412437361"/>
+    <origin xyz="0.0 -0.11985 -2.458164590756244e-11" rpy="1.570796327 0.0 0.0011432279000107165"/>
     <axis xyz="0.0 0.0 1.0"/>
     <parent link="wrist_1_link"/>
@@ -272,5 +272,5 @@
   </joint>
   <joint name="wrist_3_joint" type="revolute">
-    <origin xyz="0.0 0.11655 -2.390480459346185e-11" rpy="1.570796326589793 3.141592653589793 2.971795491526189"/>
+    <origin xyz="0.0 0.11655 -2.390480459346185e-11" rpy="1.570796326589793 3.141592653589793 3.0555958845900384"/>
     <axis xyz="0.0 0.0 1.0"/>
     <parent link="wrist_2_link"/>
@@ -328,5 +328,5 @@
   </joint>
   <joint name="rgb_world_joint" type="fixed">
-    <origin xyz="0.9040307558583056 0.37340685909697446 0.7863156345009282" rpy="0.011250318836873024 0.18824459381100403 3.0808278801572553"/>
+    <origin xyz="0.9037432096416733 0.37228473224250047 0.7818112606308044" rpy="0.012699362404344034 0.18629151269149116 3.080059426410463"/>
     <parent link="world"/>
     <child link="rgb_world_link"/>
@@ -415,5 +415,5 @@
   </link>
   <joint name="flange_to_charuco_200x200_8x8" type="fixed">
-    <origin xyz="0.29 0.0 -0.1" rpy="-1.5707963267948966 -1.5707963267948966 0.0"/>
+    <origin xyz="0.28943924319848274 0.004388912856234545 -0.08400990383902193" rpy="0.12446009135288653 -1.4490551595331114 -1.7025546842710928"/>
     <parent link="flange"/>
     <child link="charuco_200x200_8x8"/>

File: atom_examples/riwmpbot/riwmpbot_real_calibration/urdf/optimized_w_pattern.urdf.xacro (robot description, xacro)
@@ -232,5 +232,5 @@
   </joint>
   <joint name="shoulder_pan_joint" type="revolute">
-    <origin xyz="0.0 0.0 0.1807" rpy="0.0 0.0 0.06401148706013562"/>
+    <origin xyz="0.0 0.0 0.1807" rpy="0.0 0.0 0.06054631110770013"/>
     <axis xyz="0.0 0.0 1.0"/>
     <parent link="base_link_inertia"/>
@@ -240,5 +240,5 @@
   </joint>
   <joint name="shoulder_lift_joint" type="revolute">
-    <origin xyz="0.0 0.0 0.0" rpy="1.570796327 0.0 0.009910204783218489"/>
+    <origin xyz="0.0 0.0 0.0" rpy="1.570796327 0.0 0.00843600239413617"/>
     <axis xyz="0.0 0.0 1.0"/>
     <parent link="shoulder_link"/>
@@ -248,5 +248,5 @@
   </joint>
   <joint name="elbow_joint" type="revolute">
-    <origin xyz="-0.6127 0.0 0.0" rpy="0.0 0.0 -0.002139318459194392"/>
+    <origin xyz="-0.6127 0.0 0.0" rpy="0.0 0.0 0.0034924794019561226"/>
     <axis xyz="0.0 0.0 1.0"/>
     <parent link="upper_arm_link"/>
@@ -256,5 +256,5 @@
   </joint>
   <joint name="wrist_1_joint" type="revolute">
-    <origin xyz="-0.57155 0.0 0.17415" rpy="0.0 0.0 -0.011633411894526994"/>
+    <origin xyz="-0.57155 0.0 0.17415" rpy="0.0 0.0 -0.0038882384676595"/>
     <axis xyz="0.0 0.0 1.0"/>
     <parent link="forearm_link"/>
@@ -264,5 +264,5 @@
   </joint>
   <joint name="wrist_2_joint" type="revolute">
-    <origin xyz="0.0 -0.11985 -2.458164590756244e-11" rpy="1.570796327 0.0 0.00235299412437361"/>
+    <origin xyz="0.0 -0.11985 -2.458164590756244e-11" rpy="1.570796327 0.0 0.0011432279000107165"/>
     <axis xyz="0.0 0.0 1.0"/>
     <parent link="wrist_1_link"/>
@@ -272,5 +272,5 @@
   </joint>
   <joint name="wrist_3_joint" type="revolute">
-    <origin xyz="0.0 0.11655 -2.390480459346185e-11" rpy="1.570796326589793 3.141592653589793 2.971795491526189"/>
+    <origin xyz="0.0 0.11655 -2.390480459346185e-11" rpy="1.570796326589793 3.141592653589793 3.0555958845900384"/>
     <axis xyz="0.0 0.0 1.0"/>
     <parent link="wrist_2_link"/>
@@ -328,5 +328,5 @@
   </joint>
   <joint name="rgb_world_joint" type="fixed">
-    <origin xyz="0.9040307558583056 0.37340685909697446 0.7863156345009282" rpy="0.011250318836873024 0.18824459381100403 3.0808278801572553"/>
+    <origin xyz="0.9037432096416733 0.37228473224250047 0.7818112606308044" rpy="0.012699362404344034 0.18629151269149116 3.080059426410463"/>
     <parent link="world"/>
     <child link="rgb_world_link"/>
@@ -415,5 +415,5 @@
   </link>
   <joint name="flange_to_charuco_200x200_8x8" type="fixed">
-    <origin xyz="0.29 0.0 -0.1" rpy="-1.5707963267948966 -1.5707963267948966 0.0"/>
+    <origin xyz="0.28943924319848274 0.004388912856234545 -0.08400990383902193" rpy="0.12446009135288653 -1.4490551595331114 -1.7025546842710928"/>
     <parent link="flange"/>
     <child link="charuco_200x200_8x8"/>
@@ -467,5 +467,5 @@
     <child link="charuco_200x120_3x6"/>
   </joint>
-  <link name="charuco_200x200_8x8">
+  <link name="charuco_200x200_8x8_manuel">
     <origin xyz="0 0 0" rpy="0 0 0"/>
     <visual name="hand_pattern_visual">
@@ -476,8 +476,8 @@
     </visual>
   </link>
-  <joint name="flange-charuco_200x200_8x8" type="fixed">
-    <origin xyz="0.29025985756421346 0.013223176403322864 -0.08712675178453624" rpy="0.02985713217726388 -1.365031616760473 -1.5927739084396466"/>
+  <joint name="flange-charuco_200x200_8x8_manuel" type="fixed">
+    <origin xyz="0.28943924319848274 0.004388912856234545 -0.08400990383902193" rpy="0.12446009135288653 -1.4490551595331114 -1.7025546842710928"/>
     <parent link="flange"/>
-    <child link="charuco_200x200_8x8"/>
+    <child link="charuco_200x200_8x8_manuel"/>
   </joint>
 </robot>

Commit message: #876 created new atom_batch_execution package.

File: atom_examples/riwmpbot/riwmpbot_real_calibration/urdf/optimized.urdf.xacro (robot description, xacro)
@@ -232,5 +232,5 @@
   </joint>
   <joint name="shoulder_pan_joint" type="revolute">
-    <origin xyz="0.0 0.0 0.1807" rpy="0.0 0.0 0.06054631110770013"/>
+    <origin xyz="-0.04243023342119992 0.02872124469384848 0.15881936808135252" rpy="-0.0195933334702188 0.06875369076132443 0.06701992747872942"/>
     <axis xyz="0.0 0.0 1.0"/>
     <parent link="base_link_inertia"/>
@@ -240,5 +240,5 @@
   </joint>
   <joint name="shoulder_lift_joint" type="revolute">
-    <origin xyz="0.0 0.0 0.0" rpy="1.570796327 0.0 0.00843600239413617"/>
+    <origin xyz="0.010361832007509522 -0.030445093549602564 -0.006119436359917189" rpy="1.507620465725977 0.019577206221855943 0.007077945616583159"/>
     <axis xyz="0.0 0.0 1.0"/>
     <parent link="shoulder_link"/>
@@ -248,5 +248,5 @@
   </joint>
   <joint name="elbow_joint" type="revolute">
-    <origin xyz="-0.6127 0.0 0.0" rpy="0.0 0.0 0.0034924794019561226"/>
+    <origin xyz="-0.6097368987036205 -0.010345563613577132 0.032198066941223444" rpy="-0.00869850791158205 0.06138931491000319 -0.038609913009545506"/>
     <axis xyz="0.0 0.0 1.0"/>
     <parent link="upper_arm_link"/>
@@ -256,5 +256,5 @@
   </joint>
   <joint name="wrist_1_joint" type="revolute">
-    <origin xyz="-0.57155 0.0 0.17415" rpy="0.0 0.0 -0.0038882384676595"/>
+    <origin xyz="-0.57155 0.0 0.17415" rpy="0.0 0.0 0.0"/>
     <axis xyz="0.0 0.0 1.0"/>
     <parent link="forearm_link"/>
@@ -264,5 +264,5 @@
   </joint>
   <joint name="wrist_2_joint" type="revolute">
-    <origin xyz="0.0 -0.11985 -2.458164590756244e-11" rpy="1.570796327 0.0 0.0011432279000107165"/>
+    <origin xyz="0.0 -0.11985 -2.458164590756244e-11" rpy="1.570796327 0.0 0.0"/>
     <axis xyz="0.0 0.0 1.0"/>
     <parent link="wrist_1_link"/>
@@ -272,5 +272,5 @@
   </joint>
   <joint name="wrist_3_joint" type="revolute">
-    <origin xyz="0.0 0.11655 -2.390480459346185e-11" rpy="1.570796326589793 3.141592653589793 3.0555958845900384"/>
+    <origin xyz="0.0 0.11655 -2.390480459346185e-11" rpy="1.570796326589793 3.141592653589793 3.141592653589793"/>
     <axis xyz="0.0 0.0 1.0"/>
     <parent link="wrist_2_link"/>
@@ -328,5 +328,5 @@
   </joint>
   <joint name="rgb_world_joint" type="fixed">
-    <origin xyz="0.9037432096416733 0.37228473224250047 0.7818112606308044" rpy="0.012699362404344034 0.18629151269149116 3.080059426410463"/>
+    <origin xyz="0.8802099649376963 0.378721262741837 0.8063964574154846" rpy="0.00826593348904808 0.24524521496388046 3.1352715273508194"/>
     <parent link="world"/>
     <child link="rgb_world_link"/>
@@ -415,5 +415,5 @@
   </link>
   <joint name="flange_to_charuco_200x200_8x8" type="fixed">
-    <origin xyz="0.28943924319848274 0.004388912856234545 -0.08400990383902193" rpy="0.12446009135288653 -1.4490551595331114 -1.7025546842710928"/>
+    <origin xyz="0.29 0.0 -0.1" rpy="-1.5707963267948966 -1.5707963267948966 0.0"/>
     <parent link="flange"/>
     <child link="charuco_200x200_8x8"/>

File: atom_examples/riwmpbot/riwmpbot_real_calibration/urdf/optimized_w_pattern.urdf.xacro (robot description, xacro)
@@ -232,5 +232,5 @@
   </joint>
   <joint name="shoulder_pan_joint" type="revolute">
-    <origin xyz="0.0 0.0 0.1807" rpy="0.0 0.0 0.06054631110770013"/>
+    <origin xyz="-0.04243023342119992 0.02872124469384848 0.15881936808135252" rpy="-0.0195933334702188 0.06875369076132443 0.06701992747872942"/>
     <axis xyz="0.0 0.0 1.0"/>
     <parent link="base_link_inertia"/>
@@ -240,5 +240,5 @@
   </joint>
   <joint name="shoulder_lift_joint" type="revolute">
-    <origin xyz="0.0 0.0 0.0" rpy="1.570796327 0.0 0.00843600239413617"/>
+    <origin xyz="0.010361832007509522 -0.030445093549602564 -0.006119436359917189" rpy="1.507620465725977 0.019577206221855943 0.007077945616583159"/>
     <axis xyz="0.0 0.0 1.0"/>
     <parent link="shoulder_link"/>
@@ -248,5 +248,5 @@
   </joint>
   <joint name="elbow_joint" type="revolute">
-    <origin xyz="-0.6127 0.0 0.0" rpy="0.0 0.0 0.0034924794019561226"/>
+    <origin xyz="-0.6097368987036205 -0.010345563613577132 0.032198066941223444" rpy="-0.00869850791158205 0.06138931491000319 -0.038609913009545506"/>
     <axis xyz="0.0 0.0 1.0"/>
     <parent link="upper_arm_link"/>
@@ -256,5 +256,5 @@
   </joint>
   <joint name="wrist_1_joint" type="revolute">
-    <origin xyz="-0.57155 0.0 0.17415" rpy="0.0 0.0 -0.0038882384676595"/>
+    <origin xyz="-0.57155 0.0 0.17415" rpy="0.0 0.0 0.0"/>
     <axis xyz="0.0 0.0 1.0"/>
     <parent link="forearm_link"/>
@@ -264,5 +264,5 @@
   </joint>
   <joint name="wrist_2_joint" type="revolute">
-    <origin xyz="0.0 -0.11985 -2.458164590756244e-11" rpy="1.570796327 0.0 0.0011432279000107165"/>
+    <origin xyz="0.0 -0.11985 -2.458164590756244e-11" rpy="1.570796327 0.0 0.0"/>
     <axis xyz="0.0 0.0 1.0"/>
     <parent link="wrist_1_link"/>
@@ -272,5 +272,5 @@
   </joint>
   <joint name="wrist_3_joint" type="revolute">
-    <origin xyz="0.0 0.11655 -2.390480459346185e-11" rpy="1.570796326589793 3.141592653589793 3.0555958845900384"/>
+    <origin xyz="0.0 0.11655 -2.390480459346185e-11" rpy="1.570796326589793 3.141592653589793 3.141592653589793"/>
     <axis xyz="0.0 0.0 1.0"/>
     <parent link="wrist_2_link"/>
@@ -328,5 +328,5 @@
   </joint>
   <joint name="rgb_world_joint" type="fixed">
-    <origin xyz="0.9037432096416733 0.37228473224250047 0.7818112606308044" rpy="0.012699362404344034 0.18629151269149116 3.080059426410463"/>
+    <origin xyz="0.8802099649376963 0.378721262741837 0.8063964574154846" rpy="0.00826593348904808 0.24524521496388046 3.1352715273508194"/>
     <parent link="world"/>
     <child link="rgb_world_link"/>
@@ -415,5 +415,5 @@
   </link>
   <joint name="flange_to_charuco_200x200_8x8" type="fixed">
-    <origin xyz="0.28943924319848274 0.004388912856234545 -0.08400990383902193" rpy="0.12446009135288653 -1.4490551595331114 -1.7025546842710928"/>
+    <origin xyz="0.29 0.0 -0.1" rpy="-1.5707963267948966 -1.5707963267948966 0.0"/>
     <parent link="flange"/>
     <child link="charuco_200x200_8x8"/>
@@ -467,17 +467,17 @@
     <child link="charuco_200x120_3x6"/>
   </joint>
-  <link name="charuco_200x200_8x8_manuel">
+  <link name="charuco_170x100_3x6">
     <origin xyz="0 0 0" rpy="0 0 0"/>
-    <visual name="hand_pattern_visual">
+    <visual name="forearm_pattern_visual">
       <origin xyz="0 0 0" rpy="0 0 0"/>
       <geometry>
-        <mesh filename="package://atom_worlds/pattern/models/charuco_200x200_8x8_20_15_DICT_4x4/model.dae"/>
-      </geometry>
-    </visual>
-  </link>
-  <joint name="flange-charuco_200x200_8x8_manuel" type="fixed">
-    <origin xyz="0.28943924319848274 0.004388912856234545 -0.08400990383902193" rpy="0.12446009135288653 -1.4490551595331114 -1.7025546842710928"/>
-    <parent link="flange"/>
-    <child link="charuco_200x200_8x8_manuel"/>
+        <mesh filename="package://atom_worlds/pattern/models/charuco_170x100_3x6_25_18_DICT_6X6/model.dae"/>
+      </geometry>
+    </visual>
+  </link>
+  <joint name="forearm_link-charuco_170x100_3x6" type="fixed">
+    <origin xyz="-0.23099342029169603 0.012255504822925839 -0.061598102548465386" rpy="0.14073687230426346 -0.015878044834702135 -3.1137421085335695"/>
+    <parent link="forearm_link"/>
+    <child link="charuco_170x100_3x6"/>
   </joint>
 </robot>
