Commit message: #854

File: atom_examples/mrjbot/mrjbot_calibration/urdf/optimized.urdf.xacro (robot description, xacro)
@@ -400,5 +400,5 @@
   </joint>
   <joint name="shoulder_pan_joint" type="revolute">
-    <origin xyz="0.0 0.0 0.1807" rpy="0.0 0.0 0.0013568124129685489"/>
+    <origin xyz="0.0 0.0 0.1807" rpy="0.0 0.0 -0.0058076144738942945"/>
     <axis xyz="0.0 0.0 1.0"/>
     <parent link="base_link_inertia"/>
@@ -408,5 +408,5 @@
   </joint>
   <joint name="shoulder_lift_joint" type="revolute">
-    <origin xyz="0.0 0.0 0.0" rpy="1.570796327 0.0 -0.0367671582048375"/>
+    <origin xyz="0.0 0.0 0.0" rpy="1.570796327 0.0 -0.00013482689797681706"/>
     <axis xyz="0.0 0.0 1.0"/>
     <parent link="shoulder_link"/>
@@ -416,5 +416,5 @@
   </joint>
   <joint name="elbow_joint" type="revolute">
-    <origin xyz="-0.6127 0.0 0.0" rpy="0.0 0.0 0.03050308661669396"/>
+    <origin xyz="-0.6127 0.0 0.0" rpy="0.0 0.0 -0.0005352064535000297"/>
     <axis xyz="0.0 0.0 1.0"/>
     <parent link="upper_arm_link"/>
@@ -424,5 +424,5 @@
   </joint>
   <joint name="wrist_1_joint" type="revolute">
-    <origin xyz="-0.57155 0.0 0.17415" rpy="0.0 0.0 -0.04998223281159626"/>
+    <origin xyz="-0.57155 0.0 0.17415" rpy="0.0 0.0 -0.00011013451914100814"/>
     <axis xyz="0.0 0.0 1.0"/>
     <parent link="forearm_link"/>
@@ -432,5 +432,5 @@
   </joint>
   <joint name="wrist_2_joint" type="revolute">
-    <origin xyz="0.0 -0.11985 -2.458164590756244e-11" rpy="1.570796327 0.0 -0.010239526293651985"/>
+    <origin xyz="0.0 -0.11985 -2.458164590756244e-11" rpy="1.570796327 0.0 -0.0005642817927798282"/>
     <axis xyz="0.0 0.0 1.0"/>
     <parent link="wrist_1_link"/>
@@ -440,5 +440,5 @@
   </joint>
   <joint name="wrist_3_joint" type="revolute">
-    <origin xyz="0.0 0.11655 -2.390480459346185e-11" rpy="1.570796326589793 3.141592653589793 3.223174766552955"/>
+    <origin xyz="0.0 0.11655 -2.390480459346185e-11" rpy="1.570796326589793 3.141592653589793 3.1545844528569202"/>
     <axis xyz="0.0 0.0 1.0"/>
     <parent link="wrist_2_link"/>
@@ -496,5 +496,5 @@
   </joint>
   <joint name="rgb_hand_joint" type="fixed">
-    <origin xyz="-0.019989702829571635 0.002822546796168539 0.06465687328387897" rpy="-0.05148356002025044 0.00022778897199553032 -6.211217675559517e-06"/>
+    <origin xyz="-0.01998450459954139 0.00042366327864966585 0.06495783245819241" rpy="-0.012895716899611562 0.0005084406397419439 -8.388590465424347e-05"/>
     <parent link="flange"/>
     <child link="rgb_hand_link"/>

File: atom_examples/mrjbot/mrjbot_calibration/urdf/optimized_w_pattern.urdf.xacro (robot description, xacro)
@@ -400,5 +400,5 @@
   </joint>
   <joint name="shoulder_pan_joint" type="revolute">
-    <origin xyz="0.0 0.0 0.1807" rpy="0.0 0.0 0.0013568124129685489"/>
+    <origin xyz="0.0 0.0 0.1807" rpy="0.0 0.0 -0.0058076144738942945"/>
     <axis xyz="0.0 0.0 1.0"/>
     <parent link="base_link_inertia"/>
@@ -408,5 +408,5 @@
   </joint>
   <joint name="shoulder_lift_joint" type="revolute">
-    <origin xyz="0.0 0.0 0.0" rpy="1.570796327 0.0 -0.0367671582048375"/>
+    <origin xyz="0.0 0.0 0.0" rpy="1.570796327 0.0 -0.00013482689797681706"/>
     <axis xyz="0.0 0.0 1.0"/>
     <parent link="shoulder_link"/>
@@ -416,5 +416,5 @@
   </joint>
   <joint name="elbow_joint" type="revolute">
-    <origin xyz="-0.6127 0.0 0.0" rpy="0.0 0.0 0.03050308661669396"/>
+    <origin xyz="-0.6127 0.0 0.0" rpy="0.0 0.0 -0.0005352064535000297"/>
     <axis xyz="0.0 0.0 1.0"/>
     <parent link="upper_arm_link"/>
@@ -424,5 +424,5 @@
   </joint>
   <joint name="wrist_1_joint" type="revolute">
-    <origin xyz="-0.57155 0.0 0.17415" rpy="0.0 0.0 -0.04998223281159626"/>
+    <origin xyz="-0.57155 0.0 0.17415" rpy="0.0 0.0 -0.00011013451914100814"/>
     <axis xyz="0.0 0.0 1.0"/>
     <parent link="forearm_link"/>
@@ -432,5 +432,5 @@
   </joint>
   <joint name="wrist_2_joint" type="revolute">
-    <origin xyz="0.0 -0.11985 -2.458164590756244e-11" rpy="1.570796327 0.0 -0.010239526293651985"/>
+    <origin xyz="0.0 -0.11985 -2.458164590756244e-11" rpy="1.570796327 0.0 -0.0005642817927798282"/>
     <axis xyz="0.0 0.0 1.0"/>
     <parent link="wrist_1_link"/>
@@ -440,5 +440,5 @@
   </joint>
   <joint name="wrist_3_joint" type="revolute">
-    <origin xyz="0.0 0.11655 -2.390480459346185e-11" rpy="1.570796326589793 3.141592653589793 3.223174766552955"/>
+    <origin xyz="0.0 0.11655 -2.390480459346185e-11" rpy="1.570796326589793 3.141592653589793 3.1545844528569202"/>
     <axis xyz="0.0 0.0 1.0"/>
     <parent link="wrist_2_link"/>
@@ -496,5 +496,5 @@
   </joint>
   <joint name="rgb_hand_joint" type="fixed">
-    <origin xyz="-0.019989702829571635 0.002822546796168539 0.06465687328387897" rpy="-0.05148356002025044 0.00022778897199553032 -6.211217675559517e-06"/>
+    <origin xyz="-0.01998450459954139 0.00042366327864966585 0.06495783245819241" rpy="-0.012895716899611562 0.0005084406397419439 -8.388590465424347e-05"/>
     <parent link="flange"/>
     <child link="rgb_hand_link"/>
@@ -573,5 +573,5 @@
   </link>
   <joint name="world-pattern_link" type="fixed">
-    <origin xyz="-1.0713854011719626 0.2892365420722536 0.8091858310174166" rpy="3.1219400543506337 0.004029172412454752 0.013928690109818691"/>
+    <origin xyz="-1.0718264978338097 0.2894132134132596 0.8085917289566622" rpy="3.1215260167136463 0.0057932095358872795 0.01693882272884173"/>
     <parent link="world"/>
     <child link="pattern_link"/>
