Commit message: MWE of #950
New minimal dataset, issue persists

File: atom_examples/rrbot/rrbot_calibration/urdf/optimized.urdf.xacro (robot description, xacro)
@@ -12,5 +12,5 @@
   </gazebo>
   <joint name="rgb_left_joint" type="fixed">
-    <origin xyz="0.01499999999999957 -3.2057426077360894e-16 0.012000000000000375" rpy="-3.0805097672264623e-16 4.385950745910349e-16 2.603825111285602e-17"/>
+    <origin xyz="0.015000000000000102 1.0529035217929657e-18 0.01199999999999993" rpy="0.0 -0.0 0.0"/>
     <parent link="tripod_left_support"/>
     <child link="rgb_left_link"/>
@@ -80,5 +80,5 @@
   </gazebo>
   <joint name="rgb_right_joint" type="fixed">
-    <origin xyz="0.014896101514833615 -0.00010643945277278731 0.011919487541689396" rpy="-9.733722284792457e-05 -8.500523015444027e-05 7.164825060903521e-05"/>
+    <origin xyz="0.014934704018840839 1.4987356524735855e-05 0.012006008392206915" rpy="-2.935288573546465e-05 -4.82107800907422e-06 9.485646754006965e-06"/>
     <parent link="tripod_right_support"/>
     <child link="rgb_right_link"/>

File: atom_examples/softbot/softbot_calibration/urdf/optimized.urdf.xacro (robot description, xacro)
@@ -374,5 +374,5 @@
   </joint>
   <joint name="lidar3d_base_mount_joint" type="fixed">
-    <origin xyz="0.026070094492783986 0.08090068489378434 -0.05268234388155041" rpy="-0.1408262861752613 -0.12753878610701955 0.06246451120781566"/>
+    <origin xyz="0.0028254144209154215 -0.013395193512239738 0.004850313222099985" rpy="0.014503735363548332 0.0014857154949072043 -0.0005824514027874011"/>
     <parent link="lidar3d_plate_link"/>
     <child link="lidar3d_base_link"/>
@@ -494,5 +494,5 @@
   </gazebo>
   <joint name="front_left_camera_rgb_joint" type="fixed">
-    <origin xyz="0.0 -0.045 0.0" rpy="0.0 -0.0 0.0"/>
+    <origin xyz="-4.027602181686306e-16 -0.04500000000000013 3.981386551795197e-16" rpy="3.536179784170619e-16 -4.4169569843523917e-16 -4.2956954775829523e-16"/>
     <parent link="front_left_camera_link"/>
     <child link="front_left_camera_rgb_frame"/>
@@ -587,5 +587,5 @@
   </gazebo>
   <joint name="front_right_camera_rgb_joint" type="fixed">
-    <origin xyz="0.08129789885837509 0.012677215992655845 -0.007999399761853444" rpy="-0.07776858741095248 0.17377759615848334 0.0612649482614982"/>
+    <origin xyz="0.008443559681907525 -0.043294643774964815 -0.0018107834871628117" rpy="-3.7070187953149723e-05 0.0011010415412782812 0.00019369508561694696"/>
     <parent link="front_right_camera_link"/>
     <child link="front_right_camera_rgb_frame"/>

File: atom_examples/softbot/softbot_calibration/urdf/optimized_w_pattern.urdf.xacro (robot description, xacro)
@@ -374,5 +374,5 @@
   </joint>
   <joint name="lidar3d_base_mount_joint" type="fixed">
-    <origin xyz="0.026070094492783986 0.08090068489378434 -0.05268234388155041" rpy="-0.1408262861752613 -0.12753878610701955 0.06246451120781566"/>
+    <origin xyz="0.0028254144209154215 -0.013395193512239738 0.004850313222099985" rpy="0.014503735363548332 0.0014857154949072043 -0.0005824514027874011"/>
     <parent link="lidar3d_plate_link"/>
     <child link="lidar3d_base_link"/>
@@ -494,5 +494,5 @@
   </gazebo>
   <joint name="front_left_camera_rgb_joint" type="fixed">
-    <origin xyz="0.0 -0.045 0.0" rpy="0.0 -0.0 0.0"/>
+    <origin xyz="-4.027602181686306e-16 -0.04500000000000013 3.981386551795197e-16" rpy="3.536179784170619e-16 -4.4169569843523917e-16 -4.2956954775829523e-16"/>
     <parent link="front_left_camera_link"/>
     <child link="front_left_camera_rgb_frame"/>
@@ -587,5 +587,5 @@
   </gazebo>
   <joint name="front_right_camera_rgb_joint" type="fixed">
-    <origin xyz="0.08129789885837509 0.012677215992655845 -0.007999399761853444" rpy="-0.07776858741095248 0.17377759615848334 0.0612649482614982"/>
+    <origin xyz="0.008443559681907525 -0.043294643774964815 -0.0018107834871628117" rpy="-3.7070187953149723e-05 0.0011010415412782812 0.00019369508561694696"/>
     <parent link="front_right_camera_link"/>
     <child link="front_right_camera_rgb_frame"/>
@@ -656,5 +656,5 @@
   </link>
   <joint name="world-pattern_link" type="fixed">
-    <origin xyz="1.2614922173941845 0.5264182580609444 0.628486864545439" rpy="-1.575754145238051 -0.48969892004844584 -1.589852144614163"/>
+    <origin xyz="1.2685783052563422 0.5283358637135223 0.5983424343829683" rpy="-1.5740466856396542 -0.7494681775648704 -1.5918306448375452"/>
     <parent link="world"/>
     <child link="pattern_link"/>
