Commit message: bug fix with controller movement on softbot

File: atom_examples/softbot/softbot_calibration/urdf/optimized.urdf.xacro (robot description, xacro)
@@ -374,5 +374,5 @@
   </joint>
   <joint name="lidar3d_base_mount_joint" type="fixed">
-    <origin xyz="-0.0015142375046177249 -0.0022052142273190152 -0.000283564068925264" rpy="-0.007757658250765604 0.0009838709879697281 -0.014847674947914611"/>
+    <origin xyz="0.017463735313789735 0.07897433824844577 -0.1400037282305365" rpy="-0.20376686400067778 -0.11053008665683066 -0.13108335720725953"/>
     <parent link="lidar3d_plate_link"/>
     <child link="lidar3d_base_link"/>
@@ -494,5 +494,5 @@
   </gazebo>
   <joint name="front_left_camera_rgb_joint" type="fixed">
-    <origin xyz="-4.399872653456163e-16 -0.04499999999999956 3.1045954087761856e-16" rpy="-4.440829884921592e-16 4.4301780635402403e-16 4.438903032319087e-16"/>
+    <origin xyz="-4.440892098256497e-16 -0.04500000000000039 -2.8358888819958457e-16" rpy="-4.4408920984991584e-16 4.4000580436205306e-16 -4.186665822382241e-16"/>
     <parent link="front_left_camera_link"/>
     <child link="front_left_camera_rgb_frame"/>
@@ -587,5 +587,5 @@
   </gazebo>
   <joint name="front_right_camera_rgb_joint" type="fixed">
-    <origin xyz="0.002030911322794242 -0.03938584552044518 -1.2175099096372358e-05" rpy="-0.005222638857532736 0.001007139992505166 -0.0037596367537089353"/>
+    <origin xyz="0.09243180469369233 -0.3473751152266134 0.04711695023964141" rpy="-0.18196626526519744 -0.024961233149158223 0.19858171654705145"/>
     <parent link="front_right_camera_link"/>
     <child link="front_right_camera_rgb_frame"/>

File: atom_examples/softbot/softbot_calibration/urdf/optimized_w_pattern.urdf.xacro (robot description, xacro)
@@ -374,5 +374,5 @@
   </joint>
   <joint name="lidar3d_base_mount_joint" type="fixed">
-    <origin xyz="-0.0015142375046177249 -0.0022052142273190152 -0.000283564068925264" rpy="-0.007757658250765604 0.0009838709879697281 -0.014847674947914611"/>
+    <origin xyz="0.017463735313789735 0.07897433824844577 -0.1400037282305365" rpy="-0.20376686400067778 -0.11053008665683066 -0.13108335720725953"/>
     <parent link="lidar3d_plate_link"/>
     <child link="lidar3d_base_link"/>
@@ -494,5 +494,5 @@
   </gazebo>
   <joint name="front_left_camera_rgb_joint" type="fixed">
-    <origin xyz="-4.399872653456163e-16 -0.04499999999999956 3.1045954087761856e-16" rpy="-4.440829884921592e-16 4.4301780635402403e-16 4.438903032319087e-16"/>
+    <origin xyz="-4.440892098256497e-16 -0.04500000000000039 -2.8358888819958457e-16" rpy="-4.4408920984991584e-16 4.4000580436205306e-16 -4.186665822382241e-16"/>
     <parent link="front_left_camera_link"/>
     <child link="front_left_camera_rgb_frame"/>
@@ -587,5 +587,5 @@
   </gazebo>
   <joint name="front_right_camera_rgb_joint" type="fixed">
-    <origin xyz="0.002030911322794242 -0.03938584552044518 -1.2175099096372358e-05" rpy="-0.005222638857532736 0.001007139992505166 -0.0037596367537089353"/>
+    <origin xyz="0.09243180469369233 -0.3473751152266134 0.04711695023964141" rpy="-0.18196626526519744 -0.024961233149158223 0.19858171654705145"/>
     <parent link="front_right_camera_link"/>
     <child link="front_right_camera_rgb_frame"/>
@@ -656,5 +656,5 @@
   </link>
   <joint name="world-pattern_link" type="fixed">
-    <origin xyz="1.273180549764564 0.5275071795462576 0.9180241714021727" rpy="-1.57238029953394 -0.7458089302748174 -1.6092354412755343"/>
+    <origin xyz="1.3322546011433598 0.4210347386754081 0.8744491472651467" rpy="-1.3907955156192924 -0.7379453471528676 -1.9435532968678002"/>
     <parent link="world"/>
     <child link="pattern_link"/>

Commit message: pushing test prints #929

File: atom_examples/softbot/softbot_calibration/urdf/optimized.urdf.xacro (robot description, xacro)
@@ -374,5 +374,5 @@
   </joint>
   <joint name="lidar3d_base_mount_joint" type="fixed">
-    <origin xyz="0.017463735313789735 0.07897433824844577 -0.1400037282305365" rpy="-0.20376686400067778 -0.11053008665683066 -0.13108335720725953"/>
+    <origin xyz="0.677678848709759 -0.28984759629015294 -0.6758252354982285" rpy="0.0 -0.0 0.0"/>
     <parent link="lidar3d_plate_link"/>
     <child link="lidar3d_base_link"/>
@@ -494,5 +494,5 @@
   </gazebo>
   <joint name="front_left_camera_rgb_joint" type="fixed">
-    <origin xyz="-4.440892098256497e-16 -0.04500000000000039 -2.8358888819958457e-16" rpy="-4.4408920984991584e-16 4.4000580436205306e-16 -4.186665822382241e-16"/>
+    <origin xyz="0.0 -0.045 0.0" rpy="0.0 -0.0 0.0"/>
     <parent link="front_left_camera_link"/>
     <child link="front_left_camera_rgb_frame"/>
@@ -587,5 +587,5 @@
   </gazebo>
   <joint name="front_right_camera_rgb_joint" type="fixed">
-    <origin xyz="0.09243180469369233 -0.3473751152266134 0.04711695023964141" rpy="-0.18196626526519744 -0.024961233149158223 0.19858171654705145"/>
+    <origin xyz="0.5958415120769323 0.7271358414701619 -0.22085998914026986" rpy="0.0 -0.0 0.0"/>
     <parent link="front_right_camera_link"/>
     <child link="front_right_camera_rgb_frame"/>

File: atom_examples/softbot/softbot_calibration/urdf/optimized_w_pattern.urdf.xacro (robot description, xacro)
@@ -374,5 +374,5 @@
   </joint>
   <joint name="lidar3d_base_mount_joint" type="fixed">
-    <origin xyz="0.017463735313789735 0.07897433824844577 -0.1400037282305365" rpy="-0.20376686400067778 -0.11053008665683066 -0.13108335720725953"/>
+    <origin xyz="0.677678848709759 -0.28984759629015294 -0.6758252354982285" rpy="0.0 -0.0 0.0"/>
     <parent link="lidar3d_plate_link"/>
     <child link="lidar3d_base_link"/>
@@ -494,5 +494,5 @@
   </gazebo>
   <joint name="front_left_camera_rgb_joint" type="fixed">
-    <origin xyz="-4.440892098256497e-16 -0.04500000000000039 -2.8358888819958457e-16" rpy="-4.4408920984991584e-16 4.4000580436205306e-16 -4.186665822382241e-16"/>
+    <origin xyz="0.0 -0.045 0.0" rpy="0.0 -0.0 0.0"/>
     <parent link="front_left_camera_link"/>
     <child link="front_left_camera_rgb_frame"/>
@@ -587,5 +587,5 @@
   </gazebo>
   <joint name="front_right_camera_rgb_joint" type="fixed">
-    <origin xyz="0.09243180469369233 -0.3473751152266134 0.04711695023964141" rpy="-0.18196626526519744 -0.024961233149158223 0.19858171654705145"/>
+    <origin xyz="0.5958415120769323 0.7271358414701619 -0.22085998914026986" rpy="0.0 -0.0 0.0"/>
     <parent link="front_right_camera_link"/>
     <child link="front_right_camera_rgb_frame"/>
@@ -656,5 +656,5 @@
   </link>
   <joint name="world-pattern_link" type="fixed">
-    <origin xyz="1.3322546011433598 0.4210347386754081 0.8744491472651467" rpy="-1.3907955156192924 -0.7379453471528676 -1.9435532968678002"/>
+    <origin xyz="1.2614922173941845 0.5264182580609444 0.628486864545439" rpy="-1.575754145238051 -0.48969892004844584 -1.589852144614163"/>
     <parent link="world"/>
     <child link="pattern_link"/>

Commit message: Making changes.

File: atom_examples/softbot/softbot_calibration/urdf/optimized.urdf.xacro (robot description, xacro)
@@ -374,5 +374,5 @@
   </joint>
   <joint name="lidar3d_base_mount_joint" type="fixed">
-    <origin xyz="0.677678848709759 -0.28984759629015294 -0.6758252354982285" rpy="0.0 -0.0 0.0"/>
+    <origin xyz="0.0 0.0 0.0" rpy="0.1999999999999997 0.19999999999999976 0.1999999999999997"/>
     <parent link="lidar3d_plate_link"/>
     <child link="lidar3d_base_link"/>
@@ -587,5 +587,5 @@
   </gazebo>
   <joint name="front_right_camera_rgb_joint" type="fixed">
-    <origin xyz="0.5958415120769323 0.7271358414701619 -0.22085998914026986" rpy="0.0 -0.0 0.0"/>
+    <origin xyz="0.0 -0.045 0.0" rpy="-0.1999999999999998 -0.19999999999999976 -0.1999999999999998"/>
     <parent link="front_right_camera_link"/>
     <child link="front_right_camera_rgb_frame"/>

File: atom_examples/softbot/softbot_calibration/urdf/optimized_w_pattern.urdf.xacro (robot description, xacro)
@@ -374,5 +374,5 @@
   </joint>
   <joint name="lidar3d_base_mount_joint" type="fixed">
-    <origin xyz="0.677678848709759 -0.28984759629015294 -0.6758252354982285" rpy="0.0 -0.0 0.0"/>
+    <origin xyz="0.0 0.0 0.0" rpy="0.1999999999999997 0.19999999999999976 0.1999999999999997"/>
     <parent link="lidar3d_plate_link"/>
     <child link="lidar3d_base_link"/>
@@ -587,5 +587,5 @@
   </gazebo>
   <joint name="front_right_camera_rgb_joint" type="fixed">
-    <origin xyz="0.5958415120769323 0.7271358414701619 -0.22085998914026986" rpy="0.0 -0.0 0.0"/>
+    <origin xyz="0.0 -0.045 0.0" rpy="-0.1999999999999998 -0.19999999999999976 -0.1999999999999998"/>
     <parent link="front_right_camera_link"/>
     <child link="front_right_camera_rgb_frame"/>
@@ -656,5 +656,5 @@
   </link>
   <joint name="world-pattern_link" type="fixed">
-    <origin xyz="1.2614922173941845 0.5264182580609444 0.628486864545439" rpy="-1.575754145238051 -0.48969892004844584 -1.589852144614163"/>
+    <origin xyz="1.2757788804507506 0.5301311241542276 0.9188773423440849" rpy="-1.569108802477336 -0.7474694626503291 -1.593046298472195"/>
     <parent link="world"/>
     <child link="pattern_link"/>

Commit message: added a function computeNoise() to reduce repeated code in addNoiseToTF()

File: atom_examples/softbot/softbot_calibration/urdf/optimized.urdf.xacro (robot description, xacro)
@@ -374,5 +374,5 @@
   </joint>
   <joint name="lidar3d_base_mount_joint" type="fixed">
-    <origin xyz="0.0 0.0 0.0" rpy="0.1999999999999997 0.19999999999999976 0.1999999999999997"/>
+    <origin xyz="0.0 0.0 0.0" rpy="-2.1405550590122413 -0.8086221225642877 1.9401428561414575"/>
     <parent link="lidar3d_plate_link"/>
     <child link="lidar3d_base_link"/>
@@ -587,5 +587,5 @@
   </gazebo>
   <joint name="front_right_camera_rgb_joint" type="fixed">
-    <origin xyz="0.0 -0.045 0.0" rpy="-0.1999999999999998 -0.19999999999999976 -0.1999999999999998"/>
+    <origin xyz="0.0 -0.045 0.0" rpy="-2.542801302217737 0.611445320927222 -1.4697945968590278"/>
     <parent link="front_right_camera_link"/>
     <child link="front_right_camera_rgb_frame"/>

File: atom_examples/softbot/softbot_calibration/urdf/optimized_w_pattern.urdf.xacro (robot description, xacro)
@@ -374,5 +374,5 @@
   </joint>
   <joint name="lidar3d_base_mount_joint" type="fixed">
-    <origin xyz="0.0 0.0 0.0" rpy="0.1999999999999997 0.19999999999999976 0.1999999999999997"/>
+    <origin xyz="0.0 0.0 0.0" rpy="-2.1405550590122413 -0.8086221225642877 1.9401428561414575"/>
     <parent link="lidar3d_plate_link"/>
     <child link="lidar3d_base_link"/>
@@ -587,5 +587,5 @@
   </gazebo>
   <joint name="front_right_camera_rgb_joint" type="fixed">
-    <origin xyz="0.0 -0.045 0.0" rpy="-0.1999999999999998 -0.19999999999999976 -0.1999999999999998"/>
+    <origin xyz="0.0 -0.045 0.0" rpy="-2.542801302217737 0.611445320927222 -1.4697945968590278"/>
     <parent link="front_right_camera_link"/>
     <child link="front_right_camera_rgb_frame"/>
@@ -656,5 +656,5 @@
   </link>
   <joint name="world-pattern_link" type="fixed">
-    <origin xyz="1.2757788804507506 0.5301311241542276 0.9188773423440849" rpy="-1.569108802477336 -0.7474694626503291 -1.593046298472195"/>
+    <origin xyz="1.2614922173941845 0.5264182580609444 0.628486864545439" rpy="-1.575754145238051 -0.48969892004844584 -1.589852144614163"/>
     <parent link="world"/>
     <child link="pattern_link"/>

Commit message: somehow good?

File: atom_examples/softbot/softbot_calibration/urdf/optimized.urdf.xacro (robot description, xacro)
@@ -374,5 +374,5 @@
   </joint>
   <joint name="lidar3d_base_mount_joint" type="fixed">
-    <origin xyz="0.0028254144209154215 -0.013395193512239738 0.004850313222099985" rpy="0.014503735363548332 0.0014857154949072043 -0.0005824514027874011"/>
+    <origin xyz="0.004584426271837506 -0.027961679593396724 -0.004792219565041315" rpy="-0.0004742907483454052 -0.0016456838288880277 0.002537469692258793"/>
     <parent link="lidar3d_plate_link"/>
     <child link="lidar3d_base_link"/>
@@ -494,5 +494,5 @@
   </gazebo>
   <joint name="front_left_camera_rgb_joint" type="fixed">
-    <origin xyz="-4.027602181686306e-16 -0.04500000000000013 3.981386551795197e-16" rpy="3.536179784170619e-16 -4.4169569843523917e-16 -4.2956954775829523e-16"/>
+    <origin xyz="4.4011615097286576e-16 -0.04499999999999962 -2.1711566348555953e-16" rpy="3.489631507473564e-16 9.622932523192844e-17 -7.218146406389889e-17"/>
     <parent link="front_left_camera_link"/>
     <child link="front_left_camera_rgb_frame"/>
@@ -587,5 +587,5 @@
   </gazebo>
   <joint name="front_right_camera_rgb_joint" type="fixed">
-    <origin xyz="0.008443559681907525 -0.043294643774964815 -0.0018107834871628117" rpy="-3.7070187953149723e-05 0.0011010415412782812 0.00019369508561694696"/>
+    <origin xyz="0.009362024554976343 -0.04318447448867149 -0.003351463118968243" rpy="0.00022975616965910704 0.00010438305192130979 0.00018246201032929391"/>
     <parent link="front_right_camera_link"/>
     <child link="front_right_camera_rgb_frame"/>

File: atom_examples/softbot/softbot_calibration/urdf/optimized_w_pattern.urdf.xacro (robot description, xacro)
@@ -374,5 +374,5 @@
   </joint>
   <joint name="lidar3d_base_mount_joint" type="fixed">
-    <origin xyz="0.0028254144209154215 -0.013395193512239738 0.004850313222099985" rpy="0.014503735363548332 0.0014857154949072043 -0.0005824514027874011"/>
+    <origin xyz="0.004584426271837506 -0.027961679593396724 -0.004792219565041315" rpy="-0.0004742907483454052 -0.0016456838288880277 0.002537469692258793"/>
     <parent link="lidar3d_plate_link"/>
     <child link="lidar3d_base_link"/>
@@ -494,5 +494,5 @@
   </gazebo>
   <joint name="front_left_camera_rgb_joint" type="fixed">
-    <origin xyz="-4.027602181686306e-16 -0.04500000000000013 3.981386551795197e-16" rpy="3.536179784170619e-16 -4.4169569843523917e-16 -4.2956954775829523e-16"/>
+    <origin xyz="4.4011615097286576e-16 -0.04499999999999962 -2.1711566348555953e-16" rpy="3.489631507473564e-16 9.622932523192844e-17 -7.218146406389889e-17"/>
     <parent link="front_left_camera_link"/>
     <child link="front_left_camera_rgb_frame"/>
@@ -587,5 +587,5 @@
   </gazebo>
   <joint name="front_right_camera_rgb_joint" type="fixed">
-    <origin xyz="0.008443559681907525 -0.043294643774964815 -0.0018107834871628117" rpy="-3.7070187953149723e-05 0.0011010415412782812 0.00019369508561694696"/>
+    <origin xyz="0.009362024554976343 -0.04318447448867149 -0.003351463118968243" rpy="0.00022975616965910704 0.00010438305192130979 0.00018246201032929391"/>
     <parent link="front_right_camera_link"/>
     <child link="front_right_camera_rgb_frame"/>
@@ -656,5 +656,5 @@
   </link>
   <joint name="world-pattern_link" type="fixed">
-    <origin xyz="1.2685783052563422 0.5283358637135223 0.5983424343829683" rpy="-1.5740466856396542 -0.7494681775648704 -1.5918306448375452"/>
+    <origin xyz="1.268544757688894 0.5280755194426742 0.5985660367150162" rpy="-1.5692498330443023 -0.7484180052846267 -1.5918128787375028"/>
     <parent link="world"/>
     <child link="pattern_link"/>

Commit message: Big merge from bruno's branch, more info below
This is a big merge from the work I was doing during my MsC thesis.
Amongst others, these are the changes : - Added rrbot and softbot batch
examples- Fixed multiple small bugs associated with batch execution. I
will test this thoroughly now when running the batches for Zau. I think
I was the last one using batch executions so my fixes still make sense.-
Added the plotting script for the batch execution.- Added a few utility
functions such as
"stripAutomaticSuffixes","mutually_inclusive_conditions","parse_list_of_transformations","deleteCollectionFromDataset".-
Change the name of function "addNoiseToJointParameters" to
"addBiasToJointParameter" to better reflect function behavior.- Reworked
how noise works with rotations. Now it uses a uniform function instead
of choice. Now all noises use a main "computeNoise" function.- Added the
functionality to add noise to specific transformations in the calibrate
script.

File: atom_examples/softbot/softbot_calibration/urdf/optimized.urdf.xacro (robot description, xacro)
@@ -374,5 +374,5 @@
   </joint>
   <joint name="lidar3d_base_mount_joint" type="fixed">
-    <origin xyz="-0.0015142375046177249 -0.0022052142273190152 -0.000283564068925264" rpy="-0.007757658250765604 0.0009838709879697281 -0.014847674947914611"/>
+    <origin xyz="0.026070094492783986 0.08090068489378434 -0.05268234388155041" rpy="-0.1408262861752613 -0.12753878610701955 0.06246451120781566"/>
     <parent link="lidar3d_plate_link"/>
     <child link="lidar3d_base_link"/>
@@ -494,5 +494,5 @@
   </gazebo>
   <joint name="front_left_camera_rgb_joint" type="fixed">
-    <origin xyz="-4.399872653456163e-16 -0.04499999999999956 3.1045954087761856e-16" rpy="-4.440829884921592e-16 4.4301780635402403e-16 4.438903032319087e-16"/>
+    <origin xyz="0.0 -0.045 0.0" rpy="0.0 -0.0 0.0"/>
     <parent link="front_left_camera_link"/>
     <child link="front_left_camera_rgb_frame"/>
@@ -587,5 +587,5 @@
   </gazebo>
   <joint name="front_right_camera_rgb_joint" type="fixed">
-    <origin xyz="0.002030911322794242 -0.03938584552044518 -1.2175099096372358e-05" rpy="-0.005222638857532736 0.001007139992505166 -0.0037596367537089353"/>
+    <origin xyz="0.08129789885837509 0.012677215992655845 -0.007999399761853444" rpy="-0.07776858741095248 0.17377759615848334 0.0612649482614982"/>
     <parent link="front_right_camera_link"/>
     <child link="front_right_camera_rgb_frame"/>

File: atom_examples/softbot/softbot_calibration/urdf/optimized_w_pattern.urdf.xacro (robot description, xacro)
@@ -374,5 +374,5 @@
   </joint>
   <joint name="lidar3d_base_mount_joint" type="fixed">
-    <origin xyz="-0.0015142375046177249 -0.0022052142273190152 -0.000283564068925264" rpy="-0.007757658250765604 0.0009838709879697281 -0.014847674947914611"/>
+    <origin xyz="0.026070094492783986 0.08090068489378434 -0.05268234388155041" rpy="-0.1408262861752613 -0.12753878610701955 0.06246451120781566"/>
     <parent link="lidar3d_plate_link"/>
     <child link="lidar3d_base_link"/>
@@ -494,5 +494,5 @@
   </gazebo>
   <joint name="front_left_camera_rgb_joint" type="fixed">
-    <origin xyz="-4.399872653456163e-16 -0.04499999999999956 3.1045954087761856e-16" rpy="-4.440829884921592e-16 4.4301780635402403e-16 4.438903032319087e-16"/>
+    <origin xyz="0.0 -0.045 0.0" rpy="0.0 -0.0 0.0"/>
     <parent link="front_left_camera_link"/>
     <child link="front_left_camera_rgb_frame"/>
@@ -587,5 +587,5 @@
   </gazebo>
   <joint name="front_right_camera_rgb_joint" type="fixed">
-    <origin xyz="0.002030911322794242 -0.03938584552044518 -1.2175099096372358e-05" rpy="-0.005222638857532736 0.001007139992505166 -0.0037596367537089353"/>
+    <origin xyz="0.08129789885837509 0.012677215992655845 -0.007999399761853444" rpy="-0.07776858741095248 0.17377759615848334 0.0612649482614982"/>
     <parent link="front_right_camera_link"/>
     <child link="front_right_camera_rgb_frame"/>
@@ -656,5 +656,5 @@
   </link>
   <joint name="world-pattern_link" type="fixed">
-    <origin xyz="1.273180549764564 0.5275071795462576 0.9180241714021727" rpy="-1.57238029953394 -0.7458089302748174 -1.6092354412755343"/>
+    <origin xyz="1.2614922173941845 0.5264182580609444 0.628486864545439" rpy="-1.575754145238051 -0.48969892004844584 -1.589852144614163"/>
     <parent link="world"/>
     <child link="pattern_link"/>
